Commit message: Add parallel gripper and "null" end effector types
- Update kits with these options.

File: urdf/hebi.xacro (robot description, xacro)
@@ -26,3 +26,4 @@
   <xacro:include filename="./link.xacro"/>
   <xacro:include filename="./bracket.xacro"/>
+  <xacro:include filename="./end_effector.xacro"/>
 </robot>

File: urdf/kits/A-2084-01-parallel-gripper.xacro (robot description, xacro)
@@ -18,5 +18,5 @@
   <xacro:link name="elbow_wrist1" child="HEBI/wrist1" extension="0.325" twist="0"/>
   <xacro:actuator name="HEBI/wrist1" child="end_effector" type="X5_1"/>
-  <!-- placeholder end link at end of arm -->
-  <xacro:null_end_effector name="end_effector"/>
+  <!-- parallel gripper end effector -->
+  <xacro:gripper name="end_effector" type="parallel"/>
 </robot>

File: urdf/kits/A-2085-04-parallel-gripper.xacro (robot description, xacro)
@@ -18,5 +18,5 @@
   <xacro:link name="elbow_wrist1" child="HEBI/wrist1" extension="0.325" twist="${pi}"/>
   <xacro:actuator name="HEBI/wrist1" child="end_effector" type="X5_1"/>
-  <!-- placeholder end link at end of arm -->
-  <xacro:null_end_effector name="end_effector"/>
+  <!-- parallel gripper end effector -->
+  <xacro:gripper name="end_effector" type="parallel"/>
 </robot>

File: urdf/kits/A-2085-05-parallel-gripper.xacro (robot description, xacro)
@@ -20,5 +20,5 @@
   <xacro:bracket name="wrist1_wrist2" child="HEBI/wrist2" type="X5LightRight"/>
   <xacro:actuator name="HEBI/wrist2" child="end_effector" type="X5_1"/>
-  <!-- placeholder end link at end of arm -->
-  <xacro:null_end_effector name="end_effector"/>
+  <!-- parallel gripper end effector -->
+  <xacro:gripper name="end_effector" type="parallel"/>
 </robot>

File: urdf/kits/A-2085-06-parallel-gripper.xacro (robot description, xacro)
@@ -1,5 +1,5 @@
 <?xml version="1.0"?>
-<!-- HEBI A-2085-05 5-DoF Robot Arm Kit -->
-<robot xmlns:xacro="http://www.ros.org/wiki/xacro" name="A-2085-05">
+<!-- HEBI A-2085-06 6-DoF Robot Arm Kit -->
+<robot xmlns:xacro="http://www.ros.org/wiki/xacro" name="A-2085-06">
   <xacro:include filename="$(find hebi_description)/urdf/hebi.xacro"/>
   <!-- world -->
@@ -17,8 +17,10 @@
   <xacro:actuator name="HEBI/elbow" child="elbow_wrist1" type="X8_9" limits="${[-3,3]}"/>
   <xacro:link name="elbow_wrist1" child="HEBI/wrist1" extension="0.325" twist="${pi}"/>
-  <xacro:actuator name="HEBI/wrist1" child="wrist1_wrist2" type="X5_1" limits="${[-2 * pi,2 * pi]}"/>
+  <xacro:actuator name="HEBI/wrist1" child="wrist1_wrist2" type="X5_1" limits="${[-2 * pi, 2 * pi]}"/>
   <xacro:bracket name="wrist1_wrist2" child="HEBI/wrist2" type="X5LightRight"/>
-  <xacro:actuator name="HEBI/wrist2" child="end_effector" type="X5_1"/>
-  <!-- placeholder end link at end of arm -->
-  <xacro:null_end_effector name="end_effector"/>
+  <xacro:actuator name="HEBI/wrist2" child="wrist2_wrist3" type="X5_1" limits="${[-1.5 * pi, 1.5 * pi]}"/>
+  <xacro:bracket name="wrist2_wrist3" child="HEBI/wrist3" type="X5LightRight"/>
+  <xacro:actuator name="HEBI/wrist3" child="end_effector" type="X5_1"/>
+  <!-- parallel gripper end effector -->
+  <xacro:gripper name="end_effector" type="parallel"/>
 </robot>

File: urdf/kits/A-2085-06.xacro (robot description, xacro)
@@ -22,6 +22,5 @@
   <xacro:bracket name="wrist2_wrist3" child="HEBI/wrist3" type="X5LightRight"/>
   <xacro:actuator name="HEBI/wrist3" child="end_effector" type="X5_1"/>
-  <!-- end link -->
-  <link name="end_effector/INPUT_INTERFACE">
-  </link>
+  <!-- placeholder end link at end of arm -->
+  <xacro:null_end_effector name="end_effector"/>
 </robot>
