Commit message: Add mimic joints to ensure the end effector properly moves together.

File: urdf/end_effector.xacro (robot description, xacro)
@@ -4,25 +4,4 @@
   <xacro:macro name="null_end_effector" params="name">
     <link name="${name}/INPUT_INTERFACE"/>
-  </xacro:macro>
-  <xacro:macro name="parallel_gripper_inner_subassembly" params="name prefix">
-    <link name="${name}/${prefix}_inner_linkage">
-      <visual>
-        <origin xyz="-0.0115 -0.004 -0.004" rpy="0 0 0" />
-        <geometry>
-          <mesh filename="package://hebi_description/meshes/PM-2359-02.stl" scale="0.001 0.001 0.001"/>
-        </geometry>
-        <xacro:black_material/>
-      </visual>
-    </link>
-    <joint name="${name}/center_hub_${prefix}_inner_linkage" type="continuous">
-      <xacro:if value="${prefix == 'l'}">
-        <origin xyz="0 0.005 0.023" rpy="0 0 0" />
-      </xacro:if>
-      <xacro:if value="${prefix == 'r'}">
-        <origin xyz="0 -0.005 0.023" rpy="0 0 ${pi}" />
-      </xacro:if>
-      <parent link="${name}/center_hub"/>
-      <child link="${name}/${prefix}_inner_linkage"/>
-    </joint>
   </xacro:macro>
   <xacro:macro name="parallel_gripper_outer_subassembly" params="name prefix">
@@ -66,4 +45,5 @@
       <xacro:if value="${prefix == 'r'}">
         <origin xyz="0 -0.0125 .0115" rpy="0 0 ${pi}" />
+        <mimic joint="${name}/input_l_finger" multiplier="1.0" offset="0" />
       </xacro:if>
       <parent link="${name}/INPUT_INTERFACE"/>
@@ -80,4 +60,27 @@
       <parent link="${name}/${prefix}_outer_linkage"/>
       <child link="${name}/${prefix}_gripper"/>
+      <mimic joint="${name}/input_l_finger" multiplier="-1.0" offset="${pi/2}" />
+    </joint>
+  </xacro:macro>
+  <xacro:macro name="parallel_gripper_inner_subassembly" params="name prefix">
+    <link name="${name}/${prefix}_inner_linkage">
+      <visual>
+        <origin xyz="-0.0115 -0.004 -0.004" rpy="0 0 0" />
+        <geometry>
+          <mesh filename="package://hebi_description/meshes/PM-2359-02.stl" scale="0.001 0.001 0.001"/>
+        </geometry>
+        <xacro:black_material/>
+      </visual>
+    </link>
+    <joint name="${name}/center_hub_${prefix}_inner_linkage" type="continuous">
+      <xacro:if value="${prefix == 'l'}">
+        <origin xyz="0 0.005 0.023" rpy="0 0 0" />
+      </xacro:if>
+      <xacro:if value="${prefix == 'r'}">
+        <origin xyz="0 -0.005 0.023" rpy="0 0 ${pi}" />
+      </xacro:if>
+      <parent link="${name}/center_hub"/>
+      <child link="${name}/${prefix}_inner_linkage"/>
+      <mimic joint="${name}/input_l_finger" multiplier="1.0" offset="-1.145" />
     </joint>
   </xacro:macro>
@@ -109,10 +112,10 @@
       <child link="${name}/center_hub"/>
     </joint>
+    <!-- Tree branches for fingers, outer linkages, and grippers -->
+    <xacro:parallel_gripper_outer_subassembly name="${name}" prefix="l"/>
+    <xacro:parallel_gripper_outer_subassembly name="${name}" prefix="r"/>
     <!-- Tree branches for inner linkages -->
     <xacro:parallel_gripper_inner_subassembly name="${name}" prefix="l"/>
     <xacro:parallel_gripper_inner_subassembly name="${name}" prefix="r"/>
-    <!-- Tree branches for fingers, outer linkages, and grippers -->
-    <xacro:parallel_gripper_outer_subassembly name="${name}" prefix="l"/>
-    <xacro:parallel_gripper_outer_subassembly name="${name}" prefix="r"/>
   </xacro:macro>
 </robot>

Commit message: Addresses PR Feedback

File: urdf/end_effector.xacro (robot description, xacro)
@@ -97,5 +97,7 @@
     </joint>
   </xacro:macro>
-  <xacro:macro name="gripper" params="name type">
+  <xacro:macro name="gripper" params="name type:=Custom mass:=0.001 com_trans:='0 0 0.0005' output_trans:='0 0 0'">
+    <xacro:property name="com_trans_list" value="${com_trans.split(' ')}"/>
+    <xacro:property name="len" value="${sqrt( pow(float(com_trans_list[0]), 2) + pow(float(com_trans_list[1]), 2) + pow(float(com_trans_list[2]), 2) )}"/>
     <xacro:if value="${type == 'Custom'}">
       <link name="${name}/INPUT_INTERFACE">
@@ -113,10 +115,10 @@
         </visual>
         <inertial>
-        <origin xyz="0 0 0" rpy="0 0 0"/>
-          <mass value="0.001"/>
+          <origin xyz="${com_trans}" rpy="0 0 0"/>
+          <mass value="${mass}"/>
           <inertia
-            ixx="0.001" ixy="0.0" ixz="0.0"
-            iyy="0.001" iyz="0.0"
-            izz="0.001"/>
+            ixx="${mass*len*len*2.0/5.0}" ixy="0.0" ixz="0.0"
+            iyy="${mass*len*len*2.0/5.0}" iyz="0.0"
+            izz="${mass*len*len*2.0/5.0}"/>
         </inertial>
       </link>

File: urdf/kits/a-2084-01-parallel-gripper.xacro (robot description, xacro)
@@ -1,6 +1,6 @@
 <?xml version='1.0' encoding='UTF-8'?>
-<robot xmlns:xacro="http://www.ros.org/wiki/xacro" version="1.2.0" name="a-2085-04">
+<robot xmlns:xacro="http://www.ros.org/wiki/xacro" version="1.2.0" name="a-2084-01-parallel-gripper">
   <xacro:include filename="$(find hebi_description)/urdf/hebi.xacro"/>
-  <!-- HEBI a-2085-04 Style Arm Kit -->
+  <!-- HEBI a-2084-01-parallel-gripper Style Arm Kit -->
   <link name="world"/>
   <joint name="world_joint" type="fixed">
@@ -12,8 +12,8 @@
   <xacro:bracket type="X5HeavyRightOutside" name="shoulder_bracket" child="Arm/shoulder"/>
   <xacro:actuator type="X5_9" name="Arm/shoulder" child="shoulder_elbow"/>
-  <xacro:link type="X5" extension="0.325" twist="${pi}" name="shoulder_elbow" child="Arm/elbow"/>
+  <xacro:link type="X5" extension="0.325" twist="${pi/2}" name="shoulder_elbow" child="Arm/elbow"/>
   <xacro:actuator type="X5_4" name="Arm/elbow" child="elbow_wrist1"/>
-  <xacro:link type="X5" extension="0.325" twist="${pi}" name="elbow_wrist1" child="Arm/wrist1"/>
+  <xacro:link type="X5" extension="0.325" twist="0" name="elbow_wrist1" child="Arm/wrist1"/>
   <xacro:actuator type="X5_1" name="Arm/wrist1" child="end_effector"/>
-  <xacro:gripper type="Custom" name="end_effector"/>
+  <xacro:gripper type="X5Parallel" name="end_effector"/>
 </robot>

File: urdf/kits/a-2084-01.xacro (robot description, xacro)
@@ -1,4 +1,4 @@
 <?xml version='1.0' encoding='UTF-8'?>
-<robot xmlns:xacro="http://www.ros.org/wiki/xacro" version="1.1.0" name="a-2084-01">
+<robot xmlns:xacro="http://www.ros.org/wiki/xacro" version="1.2.0" name="a-2084-01">
   <xacro:include filename="$(find hebi_description)/urdf/hebi.xacro"/>
   <!-- HEBI a-2084-01 Style Arm Kit -->
@@ -7,13 +7,13 @@
     <origin xyz="0 0 0" rpy="0 0 0"/>
     <parent link="world"/>
-    <child link="HEBI/base/INPUT_INTERFACE"/>
+    <child link="Arm/base/INPUT_INTERFACE"/>
   </joint>
-  <xacro:actuator type="X5_4" name="HEBI/base" child="shoulder_bracket"/>
-  <xacro:bracket type="X5HeavyRightOutside" name="shoulder_bracket" child="HEBI/shoulder"/>
-  <xacro:actuator type="X5_9" name="HEBI/shoulder" child="shoulder_elbow"/>
-  <xacro:link type="X5" extension="0.325" twist="${pi/2}" name="shoulder_elbow" child="HEBI/elbow"/>
-  <xacro:actuator type="X5_4" name="HEBI/elbow" child="elbow_wrist1"/>
-  <xacro:link type="X5" extension="0.325" twist="0" name="elbow_wrist1" child="HEBI/wrist1"/>
-  <xacro:actuator type="X5_1" name="HEBI/wrist1" child="end_effector"/>
-  <xacro:null_end_effector name="end_effector"/>
+  <xacro:actuator type="X5_4" name="Arm/base" child="shoulder_bracket"/>
+  <xacro:bracket type="X5HeavyRightOutside" name="shoulder_bracket" child="Arm/shoulder"/>
+  <xacro:actuator type="X5_9" name="Arm/shoulder" child="shoulder_elbow"/>
+  <xacro:link type="X5" extension="0.325" twist="${pi/2}" name="shoulder_elbow" child="Arm/elbow"/>
+  <xacro:actuator type="X5_4" name="Arm/elbow" child="elbow_wrist1"/>
+  <xacro:link type="X5" extension="0.325" twist="0" name="elbow_wrist1" child="Arm/wrist1"/>
+  <xacro:actuator type="X5_1" name="Arm/wrist1" child="end_effector"/>
+  <xacro:gripper type="Custom" name="end_effector"/>
 </robot>

File: urdf/kits/a-2085-04-parallel-gripper.xacro (robot description, xacro)
@@ -1,6 +1,6 @@
 <?xml version='1.0' encoding='UTF-8'?>
-<robot xmlns:xacro="http://www.ros.org/wiki/xacro" version="1.2.0" name="a-2085-04">
+<robot xmlns:xacro="http://www.ros.org/wiki/xacro" version="1.2.0" name="a-2085-04-parallel-gripper">
   <xacro:include filename="$(find hebi_description)/urdf/hebi.xacro"/>
-  <!-- HEBI a-2085-04 Style Arm Kit -->
+  <!-- HEBI a-2085-04-parallel-gripper Style Arm Kit -->
   <link name="world"/>
   <joint name="world_joint" type="fixed">
@@ -16,4 +16,4 @@
   <xacro:link type="X5" extension="0.325" twist="${pi}" name="elbow_wrist1" child="Arm/wrist1"/>
   <xacro:actuator type="X5_1" name="Arm/wrist1" child="end_effector"/>
-  <xacro:gripper type="Custom" name="end_effector"/>
+  <xacro:gripper type="X5Parallel" name="end_effector"/>
 </robot>

File: urdf/kits/a-2085-05-parallel-gripper.xacro (robot description, xacro)
@@ -1,6 +1,6 @@
 <?xml version='1.0' encoding='UTF-8'?>
-<robot xmlns:xacro="http://www.ros.org/wiki/xacro" version="1.2.0" name="a-2085-06">
+<robot xmlns:xacro="http://www.ros.org/wiki/xacro" version="1.2.0" name="a-2085-05-parallel-gripper">
   <xacro:include filename="$(find hebi_description)/urdf/hebi.xacro"/>
-  <!-- HEBI a-2085-06 Style Arm Kit -->
+  <!-- HEBI a-2085-05-parallel-gripper Style Arm Kit -->
   <link name="world"/>
   <joint name="world_joint" type="fixed">
@@ -17,7 +17,5 @@
   <xacro:actuator type="X5_1" name="Arm/wrist1" child="wrist2_bracket"/>
   <xacro:bracket type="X5LightRight" name="wrist2_bracket" child="Arm/wrist2"/>
-  <xacro:actuator type="X5_1" name="Arm/wrist2" child="wrist3_bracket"/>
-  <xacro:bracket type="X5LightRight" name="wrist3_bracket" child="Arm/wrist3"/>
-  <xacro:actuator type="X5_1" name="Arm/wrist3" child="end_effector"/>
-  <xacro:gripper type="Custom" name="end_effector"/>
+  <xacro:actuator type="X5_1" name="Arm/wrist2" child="end_effector"/>
+  <xacro:gripper type="X5Parallel" name="end_effector"/>
 </robot>

File: urdf/kits/a-2085-05.xacro (robot description, xacro)
@@ -1,4 +1,4 @@
 <?xml version='1.0' encoding='UTF-8'?>
-<robot xmlns:xacro="http://www.ros.org/wiki/xacro" version="1.1.0" name="a-2085-05">
+<robot xmlns:xacro="http://www.ros.org/wiki/xacro" version="1.2.0" name="a-2085-05">
   <xacro:include filename="$(find hebi_description)/urdf/hebi.xacro"/>
   <!-- HEBI a-2085-05 Style Arm Kit -->
@@ -7,15 +7,15 @@
     <origin xyz="0 0 0" rpy="0 0 0"/>
     <parent link="world"/>
-    <child link="HEBI/base/INPUT_INTERFACE"/>
+    <child link="Arm/base/INPUT_INTERFACE"/>
   </joint>
-  <xacro:actuator type="X8_9" name="HEBI/base" child="shoulder_bracket"/>
-  <xacro:bracket type="X5HeavyRightOutside" name="shoulder_bracket" child="HEBI/shoulder"/>
-  <xacro:actuator type="X8_16" name="HEBI/shoulder" child="shoulder_elbow"/>
-  <xacro:link type="X5" extension="0.325" twist="${pi}" name="shoulder_elbow" child="HEBI/elbow"/>
-  <xacro:actuator type="X8_9" name="HEBI/elbow" child="elbow_wrist1"/>
-  <xacro:link type="X5" extension="0.325" twist="${pi}" name="elbow_wrist1" child="HEBI/wrist1"/>
-  <xacro:actuator type="X5_1" name="HEBI/wrist1" child="wrist2_bracket"/>
-  <xacro:bracket type="X5LightRight" name="wrist2_bracket" child="HEBI/wrist2"/>
-  <xacro:actuator type="X5_1" name="HEBI/wrist2" child="end_effector"/>
-  <xacro:null_end_effector name="end_effector"/>
+  <xacro:actuator type="X8_9" name="Arm/base" child="shoulder_bracket"/>
+  <xacro:bracket type="X5HeavyRightOutside" name="shoulder_bracket" child="Arm/shoulder"/>
+  <xacro:actuator type="X8_16" name="Arm/shoulder" child="shoulder_elbow"/>
+  <xacro:link type="X5" extension="0.325" twist="${pi}" name="shoulder_elbow" child="Arm/elbow"/>
+  <xacro:actuator type="X8_9" name="Arm/elbow" child="elbow_wrist1"/>
+  <xacro:link type="X5" extension="0.325" twist="${pi}" name="elbow_wrist1" child="Arm/wrist1"/>
+  <xacro:actuator type="X5_1" name="Arm/wrist1" child="wrist2_bracket"/>
+  <xacro:bracket type="X5LightRight" name="wrist2_bracket" child="Arm/wrist2"/>
+  <xacro:actuator type="X5_1" name="Arm/wrist2" child="end_effector"/>
+  <xacro:gripper type="Custom" name="end_effector"/>
 </robot>

File: urdf/kits/a-2085-06-parallel-gripper.xacro (robot description, xacro)
@@ -1,6 +1,6 @@
 <?xml version='1.0' encoding='UTF-8'?>
-<robot xmlns:xacro="http://www.ros.org/wiki/xacro" version="1.2.0" name="a-2085-06">
+<robot xmlns:xacro="http://www.ros.org/wiki/xacro" version="1.2.0" name="a-2085-06-parallel-gripper">
   <xacro:include filename="$(find hebi_description)/urdf/hebi.xacro"/>
-  <!-- HEBI a-2085-06 Style Arm Kit -->
+  <!-- HEBI a-2085-06-parallel-gripper Style Arm Kit -->
   <link name="world"/>
   <joint name="world_joint" type="fixed">
@@ -20,4 +20,4 @@
   <xacro:bracket type="X5LightRight" name="wrist3_bracket" child="Arm/wrist3"/>
   <xacro:actuator type="X5_1" name="Arm/wrist3" child="end_effector"/>
-  <xacro:gripper type="Custom" name="end_effector"/>
+  <xacro:gripper type="X5Parallel" name="end_effector"/>
 </robot>
