Commit message: Adds physically modeled gripper to simulation.
Still some glitches with high transient accelerations,
pinion needs physics parameter tuning.

File: urdf/end_effector.xacro (robot description, xacro)
@@ -1,22 +1,21 @@
 <?xml version="1.0"?>
 <robot xmlns:xacro="http://www.ros.org/wiki/xacro">
-  <!-- TODO: add collision and inertial elements -->
   <xacro:macro name="null_end_effector" params="name">
     <link name="${name}/INPUT_INTERFACE">
       <collision>
         <origin xyz="0 0 0.0005" rpy="0 0 0"/>
-	<geometry>
-          <box size="0.001 0.001 0.001" rpy="0 0 0"/>
-	</geometry>
+          <geometry>
+            <box size="0.001 0.001 0.001" rpy="0 0 0"/>
+          </geometry>
       </collision>
       <visual>
         <origin xyz="0 0 0.0005" rpy="0 0 0"/>
-	<geometry>
-          <box size="0.001 0.001 0.001" rpy="0 0 0"/>
-	</geometry>
+          <geometry>
+            <box size="0.001 0.001 0.001" rpy="0 0 0"/>
+          </geometry>
       </visual>
       <inertial>
         <origin xyz="0 0 0.0005" rpy="0 0 0"/>
-	<mass value="0.001"/>
+          <mass value="0.001"/>
         <inertia
           ixx="0.001" ixy="0.0" ixz="0.0"
@@ -35,5 +34,24 @@
         <xacro:silver_material/>
       </visual>
-    </link>
+      <collision>
+        <origin xyz="-0.006 -0.0055 -0.0045" rpy="${pi/2} 0 ${pi/2}" />
+        <geometry>
+          <mesh filename="package://hebi_description/meshes/PM-2221-01.stl" scale="0.001 0.001 0.001"/>
+        </geometry>
+      </collision>
+      <inertial>
+        <origin xyz="0 0.015 0" rpy="${0.5*pi} 0 ${0.0*pi}"/>
+        <mass value="0.022"/>
+        <!-- h = 0.007 w = 0.011 d = 0.03 -->
+        <inertia
+          ixx="${1/12 * 0.022 * (0.007*0.007 + 0.03*0.03)}" ixy="0.0" ixz="0.0"
+          iyy="${1/12 * 0.022 * (0.011*0.011 + 0.03*0.03)}" iyz="0.0"
+          izz="${1/12 * 0.022 * (0.011*0.011 + 0.007*0.007)}"/>
+      </inertial>
+      <self_collide>true</self_collide>
+    </link>
+    <gazebo reference="${name}/${prefix}_finger">
+      <xacro:gazebo_silver_material/>
+    </gazebo>
     <link name="${name}/${prefix}_outer_linkage">
       <visual>
@@ -44,8 +62,20 @@
         <xacro:black_material/>
       </visual>
-    </link>
+      <inertial>
+        <origin xyz="0 0.015 0.007" rpy="0 0 0"/>
+        <mass value="0.010"/>
+        <!-- h = 0.03 w = 0.025 d = 0.03 -->
+        <inertia
+          ixx="${1/12 * 0.010 * (0.03*0.03 + 0.03*0.03)}" ixy="0.0" ixz="0.0"
+          iyy="${1/12 * 0.010 * (0.023*0.023 + 0.03*0.03)}" iyz="0.0"
+          izz="${1/12 * 0.010 * (0.023*0.023 + 0.03*0.03)}"/>
+      </inertial>
+    </link>
+    <gazebo reference="${name}/${prefix}_outer_linkage">
+      <xacro:gazebo_black_material/>
+    </gazebo>
     <link name="${name}/${prefix}_gripper">
       <visual>
-        <origin xyz="-0.006 -0.004 0.0115" rpy="0 ${pi/2} 0" />
+        <origin xyz="-0.006 -0.0115 -0.0036" rpy="${0.5*pi} ${0.0*pi} ${0.5*pi}" />
         <geometry>
           <mesh filename="package://hebi_description/meshes/PM-2360-02.stl" scale="0.001 0.001 0.001"/>
@@ -54,22 +84,70 @@
       </visual>
       <collision>
-        <origin xyz="-0.006 -0.004 0.0115" rpy="0 ${pi/2} 0" />
+        <origin xyz="-0.006 -0.0115 -0.0036" rpy="${0.5*pi} ${0.0*pi} ${0.5*pi}" />
         <geometry>
           <mesh filename="package://hebi_description/meshes/PM-2360-02.stl" scale="0.001 0.001 0.001"/>
         </geometry>
       </collision>
-    </link>
+      <inertial>
+        <origin xyz="0 -0.005 0.02" rpy="0 0 0"/>
+        <mass value="0.014"/>
+        <inertia
+          ixx="${1/12 * 0.014 * ( 0.01*0.01 + 0.05*0.05 )}" ixy="0.0" ixz="0.0"
+          iyy="${1/12 * 0.014 * ( 0.01*0.01 + 0.05*0.05 )}" iyz="0.0"
+          izz="${1/12 * 0.014 * ( 0.01*0.01 + 0.01*0.01 )}"/>
+      </inertial>
+    </link>
+    <gazebo reference="${name}/${prefix}_gripper">
+      <xacro:gazebo_black_material/>
+    </gazebo>
+    <link name="${name}/${prefix}_gripper_bend">
+      <visual>
+        <origin xyz="0 0 0" rpy="0 ${0.5*pi} 0"/>
+        <geometry>
+          <cylinder length="0.02" radius=".002" />
+        </geometry>
+        <xacro:silver_material/>
+      </visual>
+      <inertial>
+        <origin xyz="0 0 0" rpy="0 ${0.5*pi} 0"/>
+        <mass value="0.001"/>
+        <!-- Approximated as slender rod -->
+        <inertia
+          ixx="${1/12 * 0.001 * (3*pow(0.002, 2) + 0.02*0.02)}" ixy="0.0" ixz="0.0"
+          iyy="${1/12 * 0.001 * (3*pow(0.002, 2) + 0.02*0.02)}" iyz="0.0"
+          izz="${1/2  * 0.001 * pow(0.002, 2)}"/>
+      </inertial>
+    </link>
+    <gazebo reference="${name}/${prefix}_gripper_bend">
+      <xacro:gazebo_silver_material/>
+    </gazebo>
+    <joint name="${name}/${prefix}_gripper_finger_${prefix}_gripper_bend" type="fixed">
+      <origin xyz="0.0 -0.0075 0.0165" rpy="0 0 0" />
+      <parent link="${name}/${prefix}_gripper"/>
+      <child link="${name}/${prefix}_gripper_bend"/>
+    </joint>
+    <gazebo reference="${name}/${prefix}_gripper_finger_${prefix}_gripper_bend">
+      <disableFixedJointLumping>true</disableFixedJointLumping>
+      <preserveFixedJoint>true</preserveFixedJoint>
+    </gazebo>
     <joint name="${name}/input_${prefix}_finger" type="revolute">
       <xacro:if value="${prefix == 'l'}">
-        <origin xyz="0 0.0125 .0115" rpy="0 0 0" />
+        <origin xyz="0 0.01265 .0115" rpy="0 0 0" />
       </xacro:if>
       <xacro:if value="${prefix == 'r'}">
-        <origin xyz="0 -0.0125 .0115" rpy="0 0 ${pi}" />
+        <origin xyz="0 -0.01265 .0115" rpy="0 0 ${pi}" />
         <mimic joint="${name}/input_l_finger" multiplier="1.0" offset="0" />
       </xacro:if>
       <parent link="${name}/INPUT_INTERFACE"/>
       <child link="${name}/${prefix}_finger"/>
-      <limit effort="1000" velocity="1000" lower="0" upper="1.1675"/>
-    </joint>
+      <limit effort="1000" velocity="1000" lower="0" upper="${0.37*pi}"/>
+    </joint>
+    <gazebo reference="${name}/input_${prefix}_finger">
+      <physics>
+        <ode>
+          <implicit_spring_damper>true</implicit_spring_damper>
+        </ode>
+      </physics>
+    </gazebo>
     <joint name="${name}/${prefix}_finger_${prefix}_outer_linkage" type="fixed">
       <origin xyz="0 0.015 0" rpy="0 0 0" />
@@ -77,13 +155,10 @@
       <child link="${name}/${prefix}_outer_linkage"/>
     </joint>
-    <gazebo reference="${name}/${prefix}_finger_${prefix}_outer_linkage">
-      <disableFixedJointLumping>true</disableFixedJointLumping>
-      <preserveFixedJoint>true</preserveFixedJoint>
-    </gazebo>
-    <joint name="${name}/${prefix}_outer_linkage_${prefix}_gripper" type="continuous">
-      <origin xyz="0 0.025 0.018" rpy="0 0 0" />
+    <joint name="${name}/${prefix}_outer_linkage_${prefix}_gripper" type="revolute">
+      <origin xyz="0 0.025 0.018" rpy="${0.0*pi} 0 0" />
       <parent link="${name}/${prefix}_outer_linkage"/>
       <child link="${name}/${prefix}_gripper"/>
       <mimic joint="${name}/input_l_finger" multiplier="-1.0" offset="${pi/2}" />
+      <limit effort="1000" velocity="1000" lower="${-pi/2}" upper="0"/>
     </joint>
   </xacro:macro>
@@ -97,11 +172,23 @@
         <xacro:black_material/>
       </visual>
-    </link>
+      <inertial>
+        <origin xyz="0 0 0.0215" rpy="${pi/2} 0 0"/>
+        <mass value="0.010"/>
+        <!-- h = 0.05, w = 0.02 d = 0.005 -->
+        <inertia
+          ixx="${1/12 * 0.010 * (0.05*0.05 + 0.005*0.005)}" ixy="0.0" ixz="0.0"
+          iyy="${1/12 * 0.010 * (0.02*0.02 + 0.005*0.005)}" iyz="0.0"
+          izz="${1/12 * 0.010 * (0.02*0.02 + 0.05*0.05)}"/>
+      </inertial>
+    </link>
+    <gazebo reference="${name}/${prefix}_inner_linkage">
+      <xacro:gazebo_black_material/>
+    </gazebo>
     <joint name="${name}/center_hub_${prefix}_inner_linkage" type="continuous">
       <xacro:if value="${prefix == 'l'}">
-        <origin xyz="0 0.005 0.023" rpy="0 0 0" />
+        <origin xyz="0 0.005 0.023" rpy="${-0.36*pi} 0 0" />
       </xacro:if>
       <xacro:if value="${prefix == 'r'}">
-        <origin xyz="0 -0.005 0.023" rpy="0 0 ${pi}" />
+        <origin xyz="0 -0.005 0.023" rpy="${-0.36*pi} 0 ${pi}" />
       </xacro:if>
       <parent link="${name}/center_hub"/>
@@ -110,41 +197,175 @@
     </joint>
   </xacro:macro>
-  <!-- NOTE: only "parallel" is currently supported for type -->
-  <xacro:macro name="gripper" params="name type">
-    <!-- The base body of the gripper -->
-    <link name="${name}/INPUT_INTERFACE">
-      <visual>
-        <origin xyz="0 0 0.00375" />
-          <geometry>
-          <cylinder length="0.0075" radius=".0225" />
-        </geometry>
-        <xacro:black_material/>
-      </visual>
-    </link>
-    <!-- Tree branch for center hub -->
-    <link name="${name}/center_hub">
-      <visual>
-        <origin xyz="-0.0225 0.0225 0" rpy="${pi/2} 0 0" />
-        <geometry>
-          <mesh filename="package://hebi_description/meshes/PM-2357-02.stl" scale="0.001 0.001 0.001"/>
-        </geometry>
-        <xacro:black_material/>
-      </visual>
-    </link>
-    <joint name="${name}/input_center_hub" type="fixed">
-      <origin xyz="0 0 0.0045" rpy="0 0 0" />
-      <parent link="${name}/INPUT_INTERFACE"/>
-      <child link="${name}/center_hub"/>
-    </joint>
-    <gazebo reference="${name}/input_center_hub">
-      <disableFixedJointLumping>true</disableFixedJointLumping>
-      <preserveFixedJoint>true</preserveFixedJoint>
-    </gazebo>
-    <!-- Tree branches for fingers, outer linkages, and grippers -->
-    <xacro:parallel_gripper_outer_subassembly name="${name}" prefix="l"/>
-    <xacro:parallel_gripper_outer_subassembly name="${name}" prefix="r"/>
-    <!-- Tree branches for inner linkages -->
-    <xacro:parallel_gripper_inner_subassembly name="${name}" prefix="l"/>
-    <xacro:parallel_gripper_inner_subassembly name="${name}" prefix="r"/>
+  <xacro:macro name="gripper" params="name type:=Custom mass:=0.001 com_trans:='0 0 0.0005' output_trans:='0 0 0'">
+    <xacro:property name="com_trans_list" value="${com_trans.split(' ')}"/>
+    <xacro:property name="len" value="${sqrt( pow(float(com_trans_list[0]), 2) + pow(float(com_trans_list[1]), 2) + pow(float(com_trans_list[2]), 2) )}"/>
+    <xacro:if value="${type == 'Custom'}">
+      <link name="${name}/INPUT_INTERFACE">
+        <collision>
+          <origin xyz="0 0 0.0005" rpy="0 0 0"/>
+          <geometry>
+            <box size="0.001 0.001 0.001" rpy="0 0 0"/>
+          </geometry>
+        </collision>
+        <visual>
+          <origin xyz="0 0 0.0005" rpy="0 0 0"/>
+          <geometry>
+            <box size="0.001 0.001 0.001" rpy="0 0 0"/>
+          </geometry>
+        </visual>
+        <inertial>
+          <origin xyz="${com_trans}" rpy="0 0 0"/>
+          <mass value="${mass}"/>
+          <inertia
+            ixx="${2.0/5.0 * mass * pow(len, 2)}" ixy="0.0" ixz="0.0"
+            iyy="${2.0/5.0 * mass * pow(len, 2)}" iyz="0.0"
+            izz="${2.0/5.0 * mass * pow(len, 2)}"/>
+        </inertial>
+      </link>
+    </xacro:if>
+    <xacro:if value="${type.endswith('Parallel')}">
+      <!-- The base body of the gripper -->
+      <link name="${name}/INPUT_INTERFACE">
+        <visual>
+          <origin xyz="0 0 0.00375" />
+            <geometry>
+            <cylinder length="0.0075" radius=".0225" />
+          </geometry>
+          <xacro:black_material/>
+        </visual>
+        <inertial>
+          <origin xyz="0 0 0" rpy="0 0 0"/>
+          <mass value="0.072"/>
+          <!-- Approximated as solid cylinder -->
+          <inertia
+            ixx="${1.0/12.0 * 0.072 * (3*pow(0.0225, 2) + pow(0.0075, 2))}" ixy="0.0" ixz="0.0"
+            iyy="${1.0/12.0 * 0.072 * (3*pow(0.0225, 2) + pow(0.0075, 2))}" iyz="0.0"
+            izz="${1.0/2.0  * 0.072 * pow(0.0225, 2)}"/>
+        </inertial>
+      </link>
+      <gazebo reference="${name}/INPUT_INTERFACE">
+        <xacro:gazebo_black_material/>
+      </gazebo>
+      <!-- Tree branch for center hub -->
+      <link name="${name}/center_hub">
+        <visual>
+          <origin xyz="-0.0225 0.0225 0" rpy="${pi/2} 0 0" />
+          <geometry>
+            <mesh filename="package://hebi_description/meshes/PM-2357-02.stl" scale="0.001 0.001 0.001"/>
+          </geometry>
+          <xacro:black_material/>
+        </visual>
+        <inertial>
+          <origin xyz="0 0 0" rpy="0 0 0"/>
+          <mass value="0.010"/>
+          <!-- Approximated as hollow sphere -->
+          <inertia
+            ixx="${0.66*0.010*pow(0.0225, 2)}" ixy="0.0" ixz="0.0"
+            iyy="${0.66*0.010*pow(0.0225, 2)}" iyz="0.0"
+            izz="${0.66*0.010*pow(0.0225, 2)}"/>
+        </inertial>
+      </link>
+      <gazebo reference="${name}/center_hub">
+        <xacro:gazebo_black_material/>
+      </gazebo>
+      <joint name="${name}/input_center_hub" type="fixed">
+        <origin xyz="0 0 0.0045" rpy="0 0 0" />
+        <parent link="${name}/INPUT_INTERFACE"/>
+        <child link="${name}/center_hub"/>
+      </joint>
+      <link name="${name}/center_pinion">
+        <visual>
+          <origin xyz="-0.0145 -0.008 0.0038" rpy="${0.5*pi} ${0.0*pi} ${0.5*pi}" />
+          <geometry>
+            <mesh filename="package://hebi_description/meshes/PM-2291-01.stl" scale="0.001 0.001 0.001"/>
+          </geometry>
+          <xacro:silver_material/>
+        </visual>
+        <collision>
+          <origin xyz="-0.0145 -0.008 0.004" rpy="${0.5*pi} ${0.0*pi} ${0.5*pi}" />
+          <geometry>
+            <mesh filename="package://hebi_description/meshes/PM-2291-01.stl" scale="0.001 0.001 0.001"/>
+          </geometry>
+        </collision>
+        <inertial>
+          <origin xyz="0 0 0" rpy="0 0 0"/>
+          <mass value="0.010"/>
+          <!-- Approximated as hollow sphere -->
+          <inertia
+            ixx="${0.66*0.010*pow(0.0225, 2)}" ixy="0.0" ixz="0.0"
+            iyy="${0.66*0.010*pow(0.0225, 2)}" iyz="0.0"
+            izz="${0.66*0.010*pow(0.0225, 2)}"/>
+        </inertial>
+      </link>
+      <gazebo reference="${name}/center_pinion">
+        <self_collide>true</self_collide>
+        <xacro:gazebo_silver_material/>
+      </gazebo>
+      <joint name="${name}/center_hub_pinion" type="prismatic">
+        <parent link="${name}/center_hub"/>
+        <child link="${name}/center_pinion"/>
+        <origin xyz="0 0 0" rpy="0 0 0" />
+        <axis xyz="0 0 1" />
+        <limit effort="1000" velocity="1000" lower="-1.0" upper="1.0"/>
+        <physics>
+          <ode>
+            <implicit_spring_damper>true</implicit_spring_damper>
+          </ode>
+        </physics>
+      </joint>
+      <gazebo reference="${name}/center_hub_pinion">
+        <disableFixedJointLumping>true</disableFixedJointLumping>
+        <preserveFixedJoint>true</preserveFixedJoint>
+      </gazebo>
+      <!-- Tree branches for fingers, outer linkages, and grippers -->
+      <xacro:parallel_gripper_outer_subassembly name="${name}" prefix="l"/>
+      <xacro:parallel_gripper_outer_subassembly name="${name}" prefix="r"/>
+      <!-- Tree branches for inner linkages -->
+      <xacro:parallel_gripper_inner_subassembly name="${name}" prefix="l"/>
+      <xacro:parallel_gripper_inner_subassembly name="${name}" prefix="r"/>
+      <gazebo>
+        <joint name="${name}/l_inner_outer_pin" type="revolute">
+          <pose>0 0 0.0439 0 0 0</pose>
+          <parent>${name}/l_gripper_bend</parent>
+          <child>${name}/l_inner_linkage</child>
+          <axis>
+            <xyz>-1 0 0</xyz>
+            <limit>
+              <lower>${-2*pi}</lower>
+              <upper>${2*pi}</upper>
+              <effort>1000</effort>
+              <velocity>1000</velocity>
+            </limit>
+          </axis>
+        </joint>
+        <joint name="${name}/r_inner_outer_pin" type="revolute">
+          <pose>0 0 0.0439 0 0 0</pose>
+          <parent>${name}/r_gripper_bend</parent>
+          <child>${name}/r_inner_linkage</child>
+          <axis>
+            <xyz>-1 0 0</xyz>
+            <limit>
+              <lower>${-2*pi}</lower>
+              <upper>${2*pi}</upper>
+              <effort>1000</effort>
+              <velocity>1000</velocity>
+            </limit>
+          </axis>
+        </joint>
+        <!-- Add constraint between gripper fingers (they mirror each other) using a gearbox -->
+        <joint name="${name}/finger_gearbox" type="gearbox">
+          <parent>${name}/r_finger</parent>
+          <child>${name}/l_finger</child>
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
Commit message: Update dummy end effector masses to improve Gazebo simulation

File: urdf/end_effector.xacro (robot description, xacro)
@@ -197,5 +197,5 @@
     </joint>
   </xacro:macro>
-  <xacro:macro name="gripper" params="name type:=Custom mass:=0.001 com_trans:='0 0 0.0005' output_trans:='0 0 0'">
+  <xacro:macro name="gripper" params="name type:=Custom mass:=0.02 com_trans:='0 0 -0.01' output_trans:='0 0 0'">
     <xacro:property name="com_trans_list" value="${com_trans.split(' ')}"/>
     <xacro:property name="len" value="${sqrt( pow(float(com_trans_list[0]), 2) + pow(float(com_trans_list[1]), 2) + pow(float(com_trans_list[2]), 2) )}"/>

File: urdf/kits/A-2084-01.xacro (robot description, xacro)
@@ -20,4 +20,4 @@
   <xacro:link type="X5" extension="0.325" twist="0" name="elbow_wrist1" child="Arm/J4_wrist1"/>
   <xacro:actuator type="X5_1" name="Arm/J4_wrist1" child="end_effector"/>
-  <xacro:gripper type="Custom" name="end_effector"/>
+  <xacro:gripper type="Custom" name="end_effector" mass="0.02"/>
 </robot>

File: urdf/kits/A-2085-04.xacro (robot description, xacro)
@@ -20,4 +20,4 @@
   <xacro:link type="X5" extension="0.325" twist="${pi}" name="elbow_wrist1" child="Arm/J4_wrist1"/>
   <xacro:actuator type="X5_1" name="Arm/J4_wrist1" child="end_effector"/>
-  <xacro:gripper type="Custom" name="end_effector"/>
+  <xacro:gripper type="Custom" name="end_effector" mass="0.02"/>
 </robot>

File: urdf/kits/A-2085-05.xacro (robot description, xacro)
@@ -22,4 +22,4 @@
   <xacro:bracket type="X5LightRight" name="wrist2_bracket" child="Arm/J5_wrist2"/>
   <xacro:actuator type="X5_1" name="Arm/J5_wrist2" child="end_effector"/>
-  <xacro:gripper type="Custom" name="end_effector"/>
+  <xacro:gripper type="Custom" name="end_effector" mass="0.02"/>
 </robot>

File: urdf/kits/A-2085-06.xacro (robot description, xacro)
@@ -24,4 +24,4 @@
   <xacro:bracket type="X5LightRight" name="wrist3_bracket" child="Arm/J6_wrist3"/>
   <xacro:actuator type="X5_1" name="Arm/J6_wrist3" child="end_effector"/>
-  <xacro:gripper type="Custom" name="end_effector"/>
+  <xacro:gripper type="Custom" name="end_effector" mass="0.02"/>
 </robot>

Commit message: Tweak dummy end effector values to prevent model collapse

File: urdf/end_effector.xacro (robot description, xacro)
@@ -183,5 +183,5 @@
     </link>
     <gazebo reference="${name}/${prefix}_inner_linkage">
-      <xacro:gazebo_black_material/>
+      <xacro:gazebo_black_material />
     </gazebo>
     <joint name="${name}/center_hub_${prefix}_inner_linkage" type="continuous">
@@ -192,33 +192,38 @@
         <origin xyz="0 -0.005 0.023" rpy="${-0.36*pi} 0 ${pi}" />
       </xacro:if>
-      <parent link="${name}/center_hub"/>
-      <child link="${name}/${prefix}_inner_linkage"/>
+      <parent link="${name}/center_hub" />
+      <child link="${name}/${prefix}_inner_linkage" />
       <mimic joint="${name}/input_l_finger" multiplier="1.0" offset="-1.145" />
     </joint>
   </xacro:macro>
-  <xacro:macro name="gripper" params="name type:=Custom mass:=0.02 com_trans:='0 0 -0.01' output_trans:='0 0 0'">
-    <xacro:property name="com_trans_list" value="${com_trans.split(' ')}"/>
-    <xacro:property name="len" value="${sqrt( pow(float(com_trans_list[0]), 2) + pow(float(com_trans_list[1]), 2) + pow(float(com_trans_list[2]), 2) )}"/>
+  <xacro:macro name="gripper" params="name type:=Custom mass:=0.020 com_trans:='0 0 0' output_trans:='0 0 0'">
+    <xacro:property name="com_trans_list" value="${map(float, com_trans.split(' '))}" />
+    <xacro:if value="${ com_trans_list[0] + com_trans_list[1] + com_trans_list[2] >= 0.01 }">
+      <xacro:property name="len" value="${sqrt( pow(com_trans_list[0], 2) + pow(com_trans_list[1], 2) + pow(com_trans_list[2], 2) )}" />
+    </xacro:if>
+    <xacro:unless value="${ com_trans_list[0] + com_trans_list[1] + com_trans_list[2] >= 0.01 }">
+      <xacro:property name="len" value="0.1" />
+    </xacro:unless>
     <xacro:if value="${type == 'Custom'}">
       <link name="${name}/INPUT_INTERFACE">
         <collision>
-          <origin xyz="0 0 0.0005" rpy="0 0 0"/>
-          <geometry>
-            <box size="0.001 0.001 0.001" rpy="0 0 0"/>
+          <origin xyz="0 0 0.0005" rpy="0 0 0" />
+          <geometry>
+            <box size="0.001 0.001 0.001" rpy="0 0 0" />
           </geometry>
         </collision>
         <visual>
-          <origin xyz="0 0 0.0005" rpy="0 0 0"/>
-          <geometry>
-            <box size="0.001 0.001 0.001" rpy="0 0 0"/>
+          <origin xyz="0 0 0.0005" rpy="0 0 0" />
+          <geometry>
+            <box size="0.001 0.001 0.001" rpy="0 0 0" />
           </geometry>
         </visual>
         <inertial>
-          <origin xyz="${com_trans}" rpy="0 0 0"/>
-          <mass value="${mass}"/>
+          <origin xyz="${com_trans}" rpy="0 0 0" />
+          <mass value="${mass}" />
           <inertia
             ixx="${2.0/5.0 * mass * pow(len, 2)}" ixy="0.0" ixz="0.0"
             iyy="${2.0/5.0 * mass * pow(len, 2)}" iyz="0.0"
-            izz="${2.0/5.0 * mass * pow(len, 2)}"/>
+            izz="${2.0/5.0 * mass * pow(len, 2)}" />
         </inertial>
       </link>

Commit message: Updated mimic joints in end effector to match linkage behavior
Was broken by changes for gazebo simulation

File: urdf/end_effector.xacro (robot description, xacro)
@@ -156,8 +156,8 @@
     </joint>
     <joint name="${name}/${prefix}_outer_linkage_${prefix}_gripper" type="revolute">
-      <origin xyz="0 0.025 0.018" rpy="${0.0*pi} 0 0" />
+      <origin xyz="0 0.025 0.018" rpy="0 0 0" />
       <parent link="${name}/${prefix}_outer_linkage"/>
       <child link="${name}/${prefix}_gripper"/>
-      <mimic joint="${name}/input_l_finger" multiplier="-1.0" offset="${pi/2}" />
+      <mimic joint="${name}/input_l_finger" multiplier="-1.0" />
       <limit effort="1000" velocity="1000" lower="${-pi/2}" upper="0"/>
     </joint>
@@ -194,5 +194,5 @@
       <parent link="${name}/center_hub" />
       <child link="${name}/${prefix}_inner_linkage" />
-      <mimic joint="${name}/input_l_finger" multiplier="1.0" offset="-1.145" />
+      <mimic joint="${name}/input_l_finger" multiplier="1.0" />
     </joint>
   </xacro:macro>
@@ -313,4 +313,5 @@
         <axis xyz="0 0 1" />
         <limit effort="1000" velocity="1000" lower="-1.0" upper="1.0"/>
+        <mimic joint="${name}/input_l_finger" multiplier="0.00001" offset="0" />
         <physics>
           <ode>
