Commit message: Fix variable name collision w/ python len

File: urdf/end_effector.xacro (robot description, xacro)
@@ -200,8 +200,8 @@
     <xacro:property name="com_trans_list" value="${map(float, com_trans.split(' '))}" />
     <xacro:if value="${ com_trans_list[0] + com_trans_list[1] + com_trans_list[2] >= 0.01 }">
-      <xacro:property name="len" value="${sqrt( pow(com_trans_list[0], 2) + pow(com_trans_list[1], 2) + pow(com_trans_list[2], 2) )}" />
+      <xacro:property name="gripper_len" value="${sqrt( pow(com_trans_list[0], 2) + pow(com_trans_list[1], 2) + pow(com_trans_list[2], 2) )}" />
     </xacro:if>
     <xacro:unless value="${ com_trans_list[0] + com_trans_list[1] + com_trans_list[2] >= 0.01 }">
-      <xacro:property name="len" value="0.1" />
+      <xacro:property name="gripper_len" value="0.1" />
     </xacro:unless>
     <xacro:if value="${type == 'Custom'}">
@@ -217,7 +217,7 @@
           <mass value="${mass}" />
           <inertia
-            ixx="${2.0/5.0 * mass * pow(len, 2)}" ixy="0.0" ixz="0.0"
-            iyy="${2.0/5.0 * mass * pow(len, 2)}" iyz="0.0"
-            izz="${2.0/5.0 * mass * pow(len, 2)}" />
+            ixx="${2.0/5.0 * mass * pow(gripper_len, 2)}" ixy="0.0" ixz="0.0"
+            iyy="${2.0/5.0 * mass * pow(gripper_len, 2)}" iyz="0.0"
+            izz="${2.0/5.0 * mass * pow(gripper_len, 2)}" />
         </inertial>
       </link>

Commit message: Update end_effector.xacro
<box/> elements don't have an `rpy` attribute, that's handled by the `origin`

File: urdf/end_effector.xacro (robot description, xacro)
@@ -210,5 +210,5 @@
           <origin xyz="0 0 0.0005" rpy="0 0 0" />
           <geometry>
-            <box size="0.001 0.001 0.001" rpy="0 0 0" />
+            <box size="0.001 0.001 0.001" />
           </geometry>
         </visual>

Commit message: Casts map to list
When using the end_effector error I got the error
```
'map' object is not subscriptable 
when evaluating expression ' com_trans_list[0] + com_trans_list[1] + com_trans_list[2] >= 0.01 '
```

Explicitly calling list on the map elements resolved this issue for me.

File: urdf/end_effector.xacro (robot description, xacro)
@@ -198,5 +198,5 @@
   </xacro:macro>
   <xacro:macro name="gripper" params="name type:=Custom mass:=0.0 com_trans:='0 0 0' output_trans:='0 0 0'">
-    <xacro:property name="com_trans_list" value="${map(float, com_trans.split(' '))}" />
+    <xacro:property name="com_trans_list" value="${list(map(float, com_trans.split(' ')))}" />
     <xacro:if value="${ com_trans_list[0] + com_trans_list[1] + com_trans_list[2] >= 0.01 }">
       <xacro:property name="gripper_len" value="${sqrt( pow(com_trans_list[0], 2) + pow(com_trans_list[1], 2) + pow(com_trans_list[2], 2) )}" />
