Commit message: Typo fix.

File: urdf/bracket.xacro (robot description, xacro)
@@ -72,14 +72,8 @@
         </xacro:if>
         <xacro:if value="${bracket_type.endswith('RightInside')}">
-          <origin xyz="0 -.03 .04" rpy="${PI/2} 0 0"/>
-        </xacro:if>
-        <xacro:if value="${bracket_type.endswith('RightInside')}">
           <origin xyz="0 .03 .04" rpy="${PI/2} 0 0"/>
         </xacro:if>
         <xacro:if value="${bracket_type.endswith('LeftOutside')}">
           <origin xyz="0 -.03 .04" rpy="${PI/2} 0 0"/>
-        </xacro:if>
-        <xacro:if value="${bracket_type.endswith('RightInside')}">
-          <origin xyz="0 .03 .04" rpy="${PI/2} 0 ${PI}"/>
         </xacro:if>
         <xacro:if value="${bracket_type.endswith('LeftInside')}">

Commit message: Remove HEBI PI macro in favor or built-in XACRO one

File: urdf/bracket.xacro (robot description, xacro)
@@ -8,5 +8,5 @@
       <visual>
         <xacro:if value="${bracket_type.endswith('Left')}">
-          <origin xyz="0 0 0" rpy="${PI/2} 0 ${PI/2}"/>
+          <origin xyz="0 0 0" rpy="${pi/2} 0 ${pi/2}"/>
           <geometry>
             <mesh filename="package://hebi_description/meshes/PM-2132-01L.stl" scale="0.001 0.001 0.001"/>
@@ -14,5 +14,5 @@
         </xacro:if>
         <xacro:if value="${bracket_type.endswith('Right')}">
-          <origin xyz="0 0 0" rpy="${PI/2} 0 ${-PI/2}"/>
+          <origin xyz="0 0 0" rpy="${pi/2} 0 ${-pi/2}"/>
           <geometry>
             <mesh filename="package://hebi_description/meshes/PM-2132-01R.stl" scale="0.001 0.001 0.001"/>
@@ -23,5 +23,5 @@
       <collision>
         <xacro:if value="${bracket_type.endswith('Left')}">
-          <origin xyz="0 0 0" rpy="${PI/2} 0 ${PI/2}"/>
+          <origin xyz="0 0 0" rpy="${pi/2} 0 ${pi/2}"/>
           <geometry>
             <mesh filename="package://hebi_description/meshes/PM-2132-01L.stl" scale="0.001 0.001 0.001"/>
@@ -29,5 +29,5 @@
         </xacro:if>
         <xacro:if value="${bracket_type.endswith('Right')}">
-          <origin xyz="0 0 0" rpy="${PI/2} 0 ${-PI/2}"/>
+          <origin xyz="0 0 0" rpy="${pi/2} 0 ${-pi/2}"/>
           <geometry>
             <mesh filename="package://hebi_description/meshes/PM-2132-01R.stl" scale="0.001 0.001 0.001"/>
@@ -51,14 +51,14 @@
       <visual>
         <xacro:if value="${bracket_type.endswith('RightOutside')}">
-          <origin xyz="0 0 0.005" rpy="${PI/2} 0 ${PI/2}"/>
+          <origin xyz="0 0 0.005" rpy="${pi/2} 0 ${pi/2}"/>
         </xacro:if>
         <xacro:if value="${bracket_type.endswith('RightInside')}">
-          <origin xyz="0 0 0.005" rpy="${PI/2} 0 ${-PI/2}"/>
+          <origin xyz="0 0 0.005" rpy="${pi/2} 0 ${-pi/2}"/>
         </xacro:if>
         <xacro:if value="${bracket_type.endswith('LeftOutside')}">
-          <origin xyz="0 0 0.005" rpy="${PI/2} 0 ${-PI/2}"/>
+          <origin xyz="0 0 0.005" rpy="${pi/2} 0 ${-pi/2}"/>
         </xacro:if>
         <xacro:if value="${bracket_type.endswith('LeftInside')}">
-          <origin xyz="0 0 0.005" rpy="${PI/2} 0 ${PI/2}"/>
+          <origin xyz="0 0 0.005" rpy="${pi/2} 0 ${pi/2}"/>
         </xacro:if>
         <geometry>
@@ -69,14 +69,14 @@
       <visual>
         <xacro:if value="${bracket_type.endswith('RightOutside')}">
-          <origin xyz="0 -.03 .04" rpy="${PI/2} 0 0"/>
+          <origin xyz="0 -.03 .04" rpy="${pi/2} 0 0"/>
         </xacro:if>
         <xacro:if value="${bracket_type.endswith('RightInside')}">
-          <origin xyz="0 .03 .04" rpy="${PI/2} 0 0"/>
+          <origin xyz="0 .03 .04" rpy="${pi/2} 0 0"/>
         </xacro:if>
         <xacro:if value="${bracket_type.endswith('LeftOutside')}">
-          <origin xyz="0 -.03 .04" rpy="${PI/2} 0 0"/>
+          <origin xyz="0 -.03 .04" rpy="${pi/2} 0 0"/>
         </xacro:if>
         <xacro:if value="${bracket_type.endswith('LeftInside')}">
-          <origin xyz="0 -.03 .04" rpy="${PI/2} 0 ${PI}"/>
+          <origin xyz="0 -.03 .04" rpy="${pi/2} 0 ${pi}"/>
         </xacro:if>
         <geometry>
@@ -92,14 +92,14 @@
       <collision>
         <xacro:if value="${bracket_type.endswith('RightOutside')}">
-          <origin xyz="0 0 0.005" rpy="${PI/2} 0 ${PI/2}"/>
+          <origin xyz="0 0 0.005" rpy="${pi/2} 0 ${pi/2}"/>
         </xacro:if>
         <xacro:if value="${bracket_type.endswith('RightInside')}">
-          <origin xyz="0 0 0.005" rpy="${PI/2} 0 ${-PI/2}"/>
+          <origin xyz="0 0 0.005" rpy="${pi/2} 0 ${-pi/2}"/>
         </xacro:if>
         <xacro:if value="${bracket_type.endswith('LeftOutside')}">
-          <origin xyz="0 0 0.005" rpy="${PI/2} 0 ${-PI/2}"/>
+          <origin xyz="0 0 0.005" rpy="${pi/2} 0 ${-pi/2}"/>
         </xacro:if>
         <xacro:if value="${bracket_type.endswith('LeftInside')}">
-          <origin xyz="0 0 0.005" rpy="${PI/2} 0 ${PI/2}"/>
+          <origin xyz="0 0 0.005" rpy="${pi/2} 0 ${pi/2}"/>
         </xacro:if>
         <geometry>
@@ -109,14 +109,14 @@
       <collision>
         <xacro:if value="${bracket_type.endswith('RightOutside')}">
-          <origin xyz="0 -.03 .04" rpy="${PI/2} 0 0"/>
+          <origin xyz="0 -.03 .04" rpy="${pi/2} 0 0"/>
         </xacro:if>
         <xacro:if value="${bracket_type.endswith('RightInside')}">
-          <origin xyz="0 .03 .04" rpy="${PI/2} 0 0"/>
+          <origin xyz="0 .03 .04" rpy="${pi/2} 0 0"/>
         </xacro:if>
         <xacro:if value="${bracket_type.endswith('LeftOutside')}">
-          <origin xyz="0 .03 .04" rpy="${PI/2} 0 ${PI}"/>
+          <origin xyz="0 .03 .04" rpy="${pi/2} 0 ${pi}"/>
         </xacro:if>
         <xacro:if value="${bracket_type.endswith('LeftInside')}">
-          <origin xyz="0 -.03 .04" rpy="${PI/2} 0 ${PI}"/>
+          <origin xyz="0 -.03 .04" rpy="${pi/2} 0 ${pi}"/>
         </xacro:if>
         <geometry>
@@ -152,20 +152,20 @@
     <child link="${child}/INPUT_INTERFACE"/>
     <xacro:if value="${bracket_type.endswith('RightOutside')}">
-      <origin xyz="0 -.0375 .055" rpy="${PI/2} 0 0"/>
+      <origin xyz="0 -.0375 .055" rpy="${pi/2} 0 0"/>
     </xacro:if>
     <xacro:if value="${bracket_type.endswith('RightInside')}">
-      <origin xyz="0 .0225 .055" rpy="${PI/2} 0 0"/>
+      <origin xyz="0 .0225 .055" rpy="${pi/2} 0 0"/>
     </xacro:if>
     <xacro:if value="${bracket_type.endswith('LeftOutside')}">
-      <origin xyz="0 .0375 .055" rpy="${-PI/2} 0 0"/>
+      <origin xyz="0 .0375 .055" rpy="${-pi/2} 0 0"/>
     </xacro:if>
     <xacro:if value="${bracket_type.endswith('LeftInside')}">
-      <origin xyz="0 -.0225 .055" rpy="${-PI/2} 0 0"/>
+      <origin xyz="0 -.0225 .055" rpy="${-pi/2} 0 0"/>
     </xacro:if>
     <xacro:if value="${bracket_type.endswith('Left')}">
-      <origin xyz="0 .043 .04" rpy="${-PI/2} 0 0"/>
+      <origin xyz="0 .043 .04" rpy="${-pi/2} 0 0"/>
     </xacro:if>
     <xacro:if value="${bracket_type.endswith('Right')}">
-      <origin xyz="0 -.043 .04" rpy="${PI/2} 0 0"/>
+      <origin xyz="0 -.043 .04" rpy="${pi/2} 0 0"/>
     </xacro:if>
   </joint>

File: urdf/hebi.xacro (robot description, xacro)
@@ -3,5 +3,4 @@
   <!-- This is a single xacro file you can include to get
   all of the HEBI components -->
-  <xacro:property name="PI" value="3.1415926535897931" />
   <xacro:macro name="red_material">
     <material name="red">

File: urdf/kits/A-2084-01.xacro (robot description, xacro)
@@ -14,5 +14,5 @@
   <xacro:bracket name="shoulder_bracket" child="HEBI/shoulder" type="X5HeavyRightOutside"/>
   <xacro:actuator name="HEBI/shoulder" child="shoulder_elbow" type="X5_9"/>
-  <xacro:link name="shoulder_elbow" child="HEBI/elbow" extension="0.325" twist="${PI/2}"/>
+  <xacro:link name="shoulder_elbow" child="HEBI/elbow" extension="0.325" twist="${pi/2}"/>
   <xacro:actuator name="HEBI/elbow" child="elbow_wrist1" type="X5_4"/>
   <xacro:link name="elbow_wrist1" child="HEBI/wrist1" extension="0.325" twist="0"/>

File: urdf/kits/A-2085-04.xacro (robot description, xacro)
@@ -14,7 +14,7 @@
   <xacro:bracket name="shoulder_bracket" child="HEBI/shoulder" type="X5HeavyRightOutside"/>
   <xacro:actuator name="HEBI/shoulder" child="shoulder_elbow" type="X5_9"/>
-  <xacro:link name="shoulder_elbow" child="HEBI/elbow" extension="0.325" twist="${PI}"/>
+  <xacro:link name="shoulder_elbow" child="HEBI/elbow" extension="0.325" twist="${pi}"/>
   <xacro:actuator name="HEBI/elbow" child="elbow_wrist1" type="X5_4"/>
-  <xacro:link name="elbow_wrist1" child="HEBI/wrist1" extension="0.325" twist="${PI}"/>
+  <xacro:link name="elbow_wrist1" child="HEBI/wrist1" extension="0.325" twist="${pi}"/>
   <xacro:actuator name="HEBI/wrist1" child="end_effector" type="X5_1"/>
   <!-- end link -->

File: urdf/kits/A-2085-05.xacro (robot description, xacro)
@@ -14,7 +14,7 @@
   <xacro:bracket name="shoulder_bracket" child="HEBI/shoulder" type="X5HeavyRightOutside"/>
   <xacro:actuator name="HEBI/shoulder" child="shoulder_elbow" type="X8_16"/>
-  <xacro:link name="shoulder_elbow" child="HEBI/elbow" extension="0.325" twist="${PI}"/>
+  <xacro:link name="shoulder_elbow" child="HEBI/elbow" extension="0.325" twist="${pi}"/>
   <xacro:actuator name="HEBI/elbow" child="elbow_wrist1" type="X8_9"/>
-  <xacro:link name="elbow_wrist1" child="HEBI/wrist1" extension="0.325" twist="${PI}"/>
+  <xacro:link name="elbow_wrist1" child="HEBI/wrist1" extension="0.325" twist="${pi}"/>
   <xacro:actuator name="HEBI/wrist1" child="wrist1_wrist2" type="X5_1"/>
   <xacro:bracket name="wrist1_wrist2" child="HEBI/wrist2" type="X5LightRight"/>

File: urdf/kits/A-2085-06.xacro (robot description, xacro)
@@ -14,7 +14,7 @@
   <xacro:bracket name="shoulder_bracket" child="HEBI/shoulder" type="X5HeavyRightOutside"/>
   <xacro:actuator name="HEBI/shoulder" child="shoulder_elbow" type="X8_16"/>
-  <xacro:link name="shoulder_elbow" child="HEBI/elbow" extension="0.325" twist="${PI}"/>
+  <xacro:link name="shoulder_elbow" child="HEBI/elbow" extension="0.325" twist="${pi}"/>
   <xacro:actuator name="HEBI/elbow" child="elbow_wrist1" type="X8_9"/>
-  <xacro:link name="elbow_wrist1" child="HEBI/wrist1" extension="0.325" twist="${PI}"/>
+  <xacro:link name="elbow_wrist1" child="HEBI/wrist1" extension="0.325" twist="${pi}"/>
   <xacro:actuator name="HEBI/wrist1" child="wrist1_wrist2" type="X5_1"/>
   <xacro:bracket name="wrist1_wrist2" child="HEBI/wrist2" type="X5LightRight"/>

Commit message: Added gazebo directives to avoid combining fixed links
Naming conventions in sdf files now align better with hrdf

File: urdf/bracket.xacro (robot description, xacro)
@@ -170,4 +170,8 @@
     </xacro:if>
   </joint>
+  <gazebo reference="${name}/OUTPUT_INTERFACE">
+    <disableFixedJointLumping>true</disableFixedJointLumping>
+    <preserveFixedJoint>true</preserveFixedJoint>
+  </gazebo>
   </xacro:macro>
 </robot>

File: urdf/end_effector.xacro (robot description, xacro)
@@ -3,5 +3,26 @@
   <!-- TODO: add collision and inertial elements -->
   <xacro:macro name="null_end_effector" params="name">
-    <link name="${name}/INPUT_INTERFACE"/>
+    <link name="${name}/INPUT_INTERFACE">
+      <collision>
+        <origin xyz="0 0 0.0005" rpy="0 0 0"/>
+	<geometry>
+          <box size="0.001 0.001 0.001" rpy="0 0 0"/>
+	</geometry>
+      </collision>
+      <visual>
+        <origin xyz="0 0 0.0005" rpy="0 0 0"/>
+	<geometry>
+          <box size="0.001 0.001 0.001" rpy="0 0 0"/>
+	</geometry>
+      </visual>
+      <inertial>
+        <origin xyz="0 0 0.0005" rpy="0 0 0"/>
+	<mass value="0.001"/>
+        <inertia
+          ixx="0.1" ixy="0.0" ixz="0.0"
+          iyy="0.1" iyz="0.0"
+          izz="0.1"/>
+      </inertial>
+    </link>
   </xacro:macro>
   <xacro:macro name="parallel_gripper_outer_subassembly" params="name prefix">
@@ -56,4 +77,8 @@
       <child link="${name}/${prefix}_outer_linkage"/>
     </joint>
+    <gazebo reference="${name}/${prefix}_finger_${prefix}_outer_linkage">
+      <disableFixedJointLumping>true</disableFixedJointLumping>
+      <preserveFixedJoint>true</preserveFixedJoint>
+    </gazebo>
     <joint name="${name}/${prefix}_outer_linkage_${prefix}_gripper" type="continuous">
       <origin xyz="0 0.025 0.018" rpy="0 0 0" />
@@ -112,4 +137,8 @@
       <child link="${name}/center_hub"/>
     </joint>
+    <gazebo reference="${name}/input_center_hub">
+      <disableFixedJointLumping>true</disableFixedJointLumping>
+      <preserveFixedJoint>true</preserveFixedJoint>
+    </gazebo>
     <!-- Tree branches for fingers, outer linkages, and grippers -->
     <xacro:parallel_gripper_outer_subassembly name="${name}" prefix="l"/>

File: urdf/link.xacro (robot description, xacro)
@@ -2,5 +2,5 @@
 <robot xmlns:xacro="http://www.ros.org/wiki/xacro">
   <!-- NOTE: joint must match the name of the module -->
-  <xacro:macro name="link" params="name child extension twist">
+  <xacro:macro name="link" params="name child type:=X5 extension twist">
     <xacro:property name="mass" value="${0.4 * (extension + 0.03) + 0.26}"/>
     <xacro:property name="edge_to_center" value="${.02}"/>
@@ -57,4 +57,8 @@
       <origin xyz="${extension} ${-sin(twist) * edge_to_center} ${edge_to_center * (1 + cos(twist))}" rpy="${twist} 0 0"/>
     </joint>
+    <gazebo reference="${name}/OUTPUT_JOINT">
+      <disableFixedJointLumping>true</disableFixedJointLumping>
+      <preserveFixedJoint>true</preserveFixedJoint>
+    </gazebo>
   </xacro:macro>
 </robot>
