Commit message: Added R-Series bracket meshes and inline link caps

File: urdf/bracket.xacro (robot description, xacro)
@@ -5,5 +5,5 @@
   <link name="${name}/INPUT_INTERFACE">
     <!-- Light bracket -->
-    <xacro:if value="${bracket_type.startswith('X5Light') or bracket_type.startswith('R5Light')}">
+    <xacro:if value="${bracket_type.startswith('X5Light')}">
       <visual>
         <xacro:if value="${bracket_type.endswith('Left')}">
@@ -47,6 +47,42 @@
       </inertial>
     </xacro:if>
+    <xacro:if value="${bracket_type.startswith('R8Light')}">
+      <visual>
+        <xacro:if value="${bracket_type.endswith('Left')}">
+          <origin xyz="0 0 0" rpy="0 0 ${pi}"/>
+        </xacro:if>
+        <xacro:if value="${bracket_type.endswith('Right')}">
+          <origin xyz="0 0 0" rpy="0 0 0"/>
+        </xacro:if>
+        <geometry>
+          <mesh filename="package://hebi_description/meshes/A-2220-01.stl" scale="0.001 0.001 0.001"/>
+        </geometry>
+        <xacro:black_material/>
+      </visual>
+      <collision>
+        <xacro:if value="${bracket_type.endswith('Left')}">
+          <origin xyz="0 0 0" rpy="${pi/2} 0 ${pi/2}"/>
+        </xacro:if>
+        <xacro:if value="${bracket_type.endswith('Right')}">
+          <origin xyz="0 0 0" rpy="${pi/2} 0 ${-pi/2}"/>
+        </xacro:if>
+        <geometry>
+          <mesh filename="package://hebi_description/meshes/A-2220-01.stl" scale="0.001 0.001 0.001"/>
+        </geometry>
+      </collision>
+      <!-- NOTE: inertia is just modelled as small sphere, and could be improved. -->
+      <inertial>
+        <xacro:if value="${bracket_type.endswith('Left')}">
+          <origin xyz="0 .0215 .02" rpy="0 0 0" />
+        </xacro:if>
+        <xacro:if value="${bracket_type.endswith('Right')}">
+          <origin xyz="0 -.0215 .02" rpy="0 0 0" />
+        </xacro:if>
+        <mass value="0.1"/>
+        <inertia ixx="${0.4 * 0.1 * 0.06 * 0.06}" ixy="0.0" ixz="0.0" iyy="${0.4 * 0.1 * 0.06 * 0.06}" iyz="0.0" izz="${0.4 * 0.1 * 0.06 * 0.06}"/>
+      </inertial>
+    </xacro:if>
     <!-- Heavy bracket -->
-    <xacro:if value="${bracket_type.startswith('X5Heavy') or bracket_type.startswith('R5Heavy')}">
+    <xacro:if value="${bracket_type.startswith('X5Heavy')}">
       <visual>
         <xacro:if value="${bracket_type.endswith('RightOutside')}">
@@ -147,10 +183,78 @@
       </inertial>
     </xacro:if>
+    <xacro:if value="${bracket_type.startswith('R8Heavy')}">
+      <visual>
+        <xacro:if value="${bracket_type.endswith('RightOutside')}">
+          <!-- <origin xyz="0 0 0.005" rpy="${pi/2} 0 ${pi/2}"/> -->
+          <origin xyz="0 0 0" rpy="0 0 0"/>
+        </xacro:if>
+        <xacro:if value="${bracket_type.endswith('RightInside')}">
+          <!-- <origin xyz="0 0 0.005" rpy="${pi/2} 0 ${-pi/2}"/> -->
+          <origin xyz="0 0 0" rpy="0 0 ${pi}"/>
+        </xacro:if>
+        <xacro:if value="${bracket_type.endswith('LeftOutside')}">
+          <!-- <origin xyz="0 0 0.005" rpy="${pi/2} 0 ${-pi/2}"/> -->
+          <origin xyz="0 0 0" rpy="0 0 ${pi}"/>
+        </xacro:if>
+        <xacro:if value="${bracket_type.endswith('LeftInside')}">
+          <!-- <origin xyz="0 0 0.005" rpy="${pi/2} 0 ${pi/2}"/> -->
+          <origin xyz="0 0 0" rpy="0 0 0"/>
+        </xacro:if>
+        <geometry>
+          <xacro:if value="${bracket_type.endswith('Outside')}">
+            <mesh filename="package://hebi_description/meshes/A-2221-01-Outside.stl" scale="0.001 0.001 0.001"/>
+          </xacro:if>
+          <xacro:if value="${bracket_type.endswith('Inside')}">
+            <mesh filename="package://hebi_description/meshes/A-2221-01-Inside.stl" scale="0.001 0.001 0.001"/>
+          </xacro:if>
+        </geometry>
+        <xacro:black_material/>
+      </visual>
+      <collision>
+        <xacro:if value="${bracket_type.endswith('RightOutside')}">
+          <origin xyz="0 0 0.005" rpy="${pi/2} 0 ${pi/2}"/>
+        </xacro:if>
+        <xacro:if value="${bracket_type.endswith('RightInside')}">
+          <origin xyz="0 0 0.005" rpy="${pi/2} 0 ${-pi/2}"/>
+        </xacro:if>
+        <xacro:if value="${bracket_type.endswith('LeftOutside')}">
+          <origin xyz="0 0 0.005" rpy="${pi/2} 0 ${-pi/2}"/>
+        </xacro:if>
+        <xacro:if value="${bracket_type.endswith('LeftInside')}">
+          <origin xyz="0 0 0.005" rpy="${pi/2} 0 ${pi/2}"/>
+        </xacro:if>
+        <geometry>
+          <xacro:if value="${bracket_type.endswith('Outside')}">
+            <mesh filename="package://hebi_description/meshes/A-2221-01-Outside.stl" scale="0.001 0.001 0.001"/>
+          </xacro:if>
+          <xacro:if value="${bracket_type.endswith('Inside')}">
+            <mesh filename="package://hebi_description/meshes/A-2221-01-Inside.stl" scale="0.001 0.001 0.001"/>
+          </xacro:if>
+        </geometry>
+      </collision>
+      <!-- NOTE: inertia is just modelled as small sphere, and could be improved. -->
+      <inertial>
+        <xacro:if value="${bracket_type.endswith('RightOutside')}">
+          <origin xyz="0 ${0.5 * -.0375} .0275" rpy="0 0 0" />
+        </xacro:if>
+        <xacro:if value="${bracket_type.endswith('RightInside')}">
+          <origin xyz="0 ${0.5 * .0225} .0275" rpy="0 0 0" />
+        </xacro:if>
+        <xacro:if value="${bracket_type.endswith('LeftOutside')}">
+          <origin xyz="0 ${0.5 * .0375} .0275" rpy="0 0 0" />
+        </xacro:if>
+        <xacro:if value="${bracket_type.endswith('LeftInside')}">
+          <origin xyz="0 ${0.5 * -.0225} .0275" rpy="0 0 0" />
+        </xacro:if>
+        <mass value="0.215"/>
+        <inertia ixx="${0.4 * 0.215 * 0.06 * 0.06}" ixy="0.0" ixz="0.0" iyy="${0.4 * 0.215 * 0.06 * 0.06}" iyz="0.0" izz="${0.4 * 0.215 * 0.06 * 0.06}"/>
+      </inertial>
+    </xacro:if>
   </link>
   <gazebo reference="${name}/INPUT_INTERFACE">
-    <xacro:if value="${bracket_type.startswith('X5Light') or bracket_type.startswith('R5Light')}">
+    <xacro:if value="${bracket_type.startswith('X5Light')}">
       <xacro:gazebo_beige_material/>
     </xacro:if>
-    <xacro:if value="${bracket_type.startswith('X5Heavy') or bracket_type.startswith('R5Heavy')}">
+    <xacro:if value="${bracket_type.startswith('X5Heavy') or bracket_type.startswith('R8')}">
       <xacro:gazebo_black_material/>
     </xacro:if>

File: urdf/link.xacro (robot description, xacro)
@@ -2,26 +2,18 @@
 <robot xmlns:xacro="http://www.ros.org/wiki/xacro">
   <!-- NOTE: joint must match the name of the module -->
-  <xacro:macro name="link" params="name child type:=X5 extension twist">
+  <xacro:macro name="link" params="name child type:=X5 input:=RightAngle output:=RightAngle extension twist">
     <xacro:property name="mass" value="${0.4 * (extension + 0.03) + 0.26}"/>
     <xacro:property name="edge_to_center" value="${.02}"/>
     <link name="${name}/INPUT_INTERFACE">
+      <!-- Input Cap -->
       <visual>
         <origin xyz="0 0 0" rpy="0 0 0" />
         <geometry>
-          <mesh filename="package://hebi_description/meshes/A-2038-02.stl"/>
-        </geometry>
-        <xacro:black_material/>
-      </visual>
-      <visual>
-        <origin xyz="${extension/2} 0 ${edge_to_center}" rpy="0 1.57075 0" />
-        <geometry>
-          <cylinder length="${extension-.0254}" radius=".016" />
-        </geometry>
-        <xacro:black_material/>
-      </visual>
-      <visual>
-        <origin xyz="${extension} ${sin(-twist) * edge_to_center} ${edge_to_center * (1 + cos(-twist))}" rpy="${-twist} 0 0"/>
-        <geometry>
-          <mesh filename="package://hebi_description/meshes/A-2039-02.stl"/>
+          <xacro:if value="${input == 'RightAngle'}">
+            <mesh filename="package://hebi_description/meshes/A-2038-02.stl"/>
+          </xacro:if>
+          <xacro:if value="${input == 'Inline'}">
+            <mesh filename="package://hebi_description/meshes/A-2225-01.stl" scale="0.001 0.001 0.001"/>
+          </xacro:if>
         </geometry>
         <xacro:black_material/>
@@ -30,17 +22,80 @@
         <origin xyz="0 0 0" rpy="0 0 0" />
         <geometry>
-          <mesh filename="package://hebi_description/meshes/A-2038-02.stl"/>
+          <xacro:if value="${input == 'RightAngle'}">
+            <mesh filename="package://hebi_description/meshes/A-2038-02.stl"/>
+          </xacro:if>
+          <xacro:if value="${input == 'Inline'}">
+            <mesh filename="package://hebi_description/meshes/A-2225-01.stl" scale="0.001 0.001 0.001"/>
+          </xacro:if>
         </geometry>
       </collision>
+      <!-- Link Pipe -->
+      <visual>
+        <xacro:if value="${input == 'RightAngle'}">
+          <origin xyz="${extension/2} 0 ${edge_to_center}" rpy="0 1.57075 0" />
+        </xacro:if>
+        <xacro:if value="${input == 'Inline'}">
+          <origin xyz="0 0 ${extension/2}" rpy="0 0 0" />
+        </xacro:if>
+        <geometry>
+          <cylinder length="${extension-.0254}" radius=".016" />
+        </geometry>
+        <xacro:black_material/>
+      </visual>
       <collision>
-        <origin xyz="${extension/2} 0 ${edge_to_center}" rpy="0 1.57075 0" />
+        <xacro:if value="${input == 'RightAngle'}">
+          <origin xyz="${extension/2} 0 ${edge_to_center}" rpy="0 1.57075 0" />
+        </xacro:if>
+        <xacro:if value="${input == 'Inline'}">
+          <origin xyz="0 0 ${extension/2}" rpy="0 0 0" />
+        </xacro:if>
         <geometry>
           <cylinder length="${extension-.0254}" radius=".016" />
         </geometry>
       </collision>
+      <!-- Output Cap -->
+      <visual>
+        <xacro:if value="${input == 'RightAngle' and output == 'RightAngle'}">
+          <origin xyz="${extension} ${sin(-twist) * edge_to_center} ${edge_to_center * (1 + cos(-twist))}" rpy="${-twist} 0 0"/>
+        </xacro:if>
+        <xacro:if value="${input == 'RightAngle' and output == 'Inline'}">
+          <origin xyz="${extension} 0 ${edge_to_center}" rpy="${pi/2} ${twist+pi} ${pi/2}"/>
+        </xacro:if>
+        <xacro:if value="${input == 'Inline' and output =='RightAngle'}">
+          <origin xyz="${edge_to_center * sin(twist+pi/2)} ${edge_to_center * -cos(twist+pi/2)} ${extension}" rpy="${pi/2} ${-pi/2} ${twist+pi/2}"/>
+        </xacro:if>
+        <xacro:if value="${input == 'Inline' and output =='Inline'}">
+          <origin xyz="${0} ${0} ${extension}" rpy="${0} ${0} ${twist-pi/2}"/>
+        </xacro:if>
+        <geometry>
+          <xacro:if value="${output == 'RightAngle'}">
+            <mesh filename="package://hebi_description/meshes/A-2039-02.stl"/>
+          </xacro:if>
+          <xacro:if value="${output == 'Inline'}">
+            <mesh filename="package://hebi_description/meshes/A-2226-01.stl" scale="0.001 0.001 0.001"/>
+          </xacro:if>
+        </geometry>
+        <xacro:black_material/>
+      </visual>
       <collision>
-        <origin xyz="${extension} ${sin(-twist) * edge_to_center} ${edge_to_center * (1 + cos(-twist))}" rpy="${-twist} 0 0"/>
+        <xacro:if value="${input == 'RightAngle' and output == 'RightAngle'}">
+          <origin xyz="${extension} ${sin(-twist) * edge_to_center} ${edge_to_center * (1 + cos(-twist))}" rpy="${-twist} 0 0"/>
+        </xacro:if>
+        <xacro:if value="${input == 'RightAngle' and output == 'Inline'}">
+          <origin xyz="${extension} 0 ${edge_to_center}" rpy="${pi/2} ${twist+pi} ${pi/2}"/>
+        </xacro:if>
+        <xacro:if value="${input == 'Inline' and output =='RightAngle'}">
+          <origin xyz="${edge_to_center * sin(twist+pi/2)} ${edge_to_center * -cos(twist+pi/2)} ${extension}" rpy="${pi/2} ${-pi/2} ${twist+pi/2}"/>
+        </xacro:if>
+        <xacro:if value="${input == 'Inline' and output =='Inline'}">
+          <origin xyz="${0} ${0} ${extension}" rpy="${0} ${0} ${twist-pi/2}"/>
+        </xacro:if>
         <geometry>
-          <mesh filename="package://hebi_description/meshes/A-2039-02.stl"/>
+          <xacro:if value="${input == 'RightAngle'}">
+            <mesh filename="package://hebi_description/meshes/A-2039-02.stl"/>
+          </xacro:if>
+          <xacro:if value="${input == 'Inline'}">
+            <mesh filename="package://hebi_description/meshes/A-2226-01.stl" scale="0.001 0.001 0.001"/>
+          </xacro:if>
         </geometry>
       </collision>
@@ -58,5 +113,16 @@
       <parent link="${name}/INPUT_INTERFACE"/>
       <child link="${child}/INPUT_INTERFACE"/>
-      <origin xyz="${extension} ${-sin(twist) * edge_to_center} ${edge_to_center * (1 + cos(twist))}" rpy="${twist} 0 0"/>
+      <xacro:if value="${input == 'RightAngle' and output == 'RightAngle'}">
+        <origin xyz="${extension} ${-sin(twist) * edge_to_center} ${edge_to_center * (1 + cos(twist))}" rpy="${twist} 0 0"/>
+      </xacro:if>
+      <xacro:if value="${input == 'RightAngle' and output == 'Inline'}">
+        <origin xyz="${extension} 0 ${edge_to_center}" rpy="${pi/2} ${twist+pi} ${pi/2}"/>
+      </xacro:if>
+      <xacro:if value="${input == 'Inline' and output =='RightAngle'}">
+        <origin xyz="${edge_to_center * sin(twist+pi/2)} ${edge_to_center * -cos(twist+pi/2)} ${extension}" rpy="${pi/2} ${-pi/2} ${twist+pi/2}"/>
+      </xacro:if>
+      <xacro:if value="${input == 'Inline' and output =='Inline'}">
+        <origin xyz="${0} ${0} ${extension}" rpy="${0} ${0} ${twist-pi/2}"/>
+      </xacro:if>
     </joint>
     <gazebo reference="${name}/OUTPUT_JOINT">

Commit message: Update naming convention of wrist to match convention
Removed hrdf_convert need for redundant hrdf file

File: urdf/bracket.xacro (robot description, xacro)
@@ -186,17 +186,13 @@
       <visual>
         <xacro:if value="${bracket_type.endswith('RightOutside')}">
-          <!-- <origin xyz="0 0 0.005" rpy="${pi/2} 0 ${pi/2}"/> -->
           <origin xyz="0 0 0" rpy="0 0 0"/>
         </xacro:if>
         <xacro:if value="${bracket_type.endswith('RightInside')}">
-          <!-- <origin xyz="0 0 0.005" rpy="${pi/2} 0 ${-pi/2}"/> -->
           <origin xyz="0 0 0" rpy="0 0 ${pi}"/>
         </xacro:if>
         <xacro:if value="${bracket_type.endswith('LeftOutside')}">
-          <!-- <origin xyz="0 0 0.005" rpy="${pi/2} 0 ${-pi/2}"/> -->
           <origin xyz="0 0 0" rpy="0 0 ${pi}"/>
         </xacro:if>
         <xacro:if value="${bracket_type.endswith('LeftInside')}">
-          <!-- <origin xyz="0 0 0.005" rpy="${pi/2} 0 ${pi/2}"/> -->
           <origin xyz="0 0 0" rpy="0 0 0"/>
         </xacro:if>

File: urdf/kits/3-DoF-arm.xacro (robot description, xacro)
@@ -11,13 +11,12 @@
     <origin xyz="0 0 0" rpy="0 0 0"/>
     <parent link="$(arg hebi_base_frame)"/>
-    <child link="Arm/J1_base/INPUT_INTERFACE"/>
+    <child link="Arm/J1/INPUT_INTERFACE"/>
   </joint>
-  <xacro:actuator type="X5_4" name="Arm/J1_base" child="shoulder_bracket"/>
-  <xacro:bracket type="X5HeavyRightOutside" name="shoulder_bracket" child="Arm/J2_shoulder"/>
-  <xacro:actuator type="X5_9" name="Arm/J2_shoulder" child="shoulder_elbow"/>
-  <xacro:link type="X5" extension="0.325" twist="${pi}" name="shoulder_elbow" child="Arm/J3_elbow"/>
-  <xacro:actuator type="X5_4" name="Arm/J3_elbow" child="elbow_wrist"/>
-  <xacro:link type="X5" extension="0.325" twist="${pi}" name="elbow_wrist" child="Arm/J4_wrist"/>
-  <xacro:actuator type="X5_1" name="Arm/J4_wrist" child="end_effector"/>
+  <xacro:actuator type="X5_4" name="Arm/J1" child="shoulder_bracket"/>
+  <xacro:bracket type="X5HeavyRightOutside" name="shoulder_bracket" child="Arm/J2"/>
+  <xacro:actuator type="X5_9" name="Arm/J2" child="shoulder_elbow"/>
+  <xacro:link type="X5" extension="0.325" twist="${pi}" name="shoulder_elbow" child="Arm/J3"/>
+  <xacro:actuator type="X5_4" name="Arm/J3" child="elbow_wrist1"/>
+  <xacro:link type="X5" extension="0.325" twist="${pi}" name="elbow_wrist1" child="end_effector"/>
   <xacro:gripper type="Custom" name="end_effector" mass="0.02"/>
 </robot>

File: urdf/kits/A-2084-01-parallel-gripper.xacro (robot description, xacro)
@@ -17,7 +17,7 @@
   <xacro:actuator type="X5_9" name="Arm/J2_shoulder" child="shoulder_elbow"/>
   <xacro:link type="X5" extension="0.325" twist="${pi/2}" name="shoulder_elbow" child="Arm/J3_elbow"/>
-  <xacro:actuator type="X5_4" name="Arm/J3_elbow" child="elbow_wrist1"/>
-  <xacro:link type="X5" extension="0.325" twist="0" name="elbow_wrist1" child="Arm/J4_wrist1"/>
-  <xacro:actuator type="X5_1" name="Arm/J4_wrist1" child="end_effector"/>
+  <xacro:actuator type="X5_4" name="Arm/J3_elbow" child="elbow_wrist"/>
+  <xacro:link type="X5" extension="0.325" twist="0" name="elbow_wrist" child="Arm/J4_wrist"/>
+  <xacro:actuator type="X5_1" name="Arm/J4_wrist" child="end_effector"/>
   <xacro:gripper type="X5Parallel" name="end_effector"/>
 </robot>

File: urdf/kits/A-2084-01.xacro (robot description, xacro)
@@ -17,7 +17,7 @@
   <xacro:actuator type="X5_9" name="Arm/J2_shoulder" child="shoulder_elbow"/>
   <xacro:link type="X5" extension="0.325" twist="${pi/2}" name="shoulder_elbow" child="Arm/J3_elbow"/>
-  <xacro:actuator type="X5_4" name="Arm/J3_elbow" child="elbow_wrist1"/>
-  <xacro:link type="X5" extension="0.325" twist="0" name="elbow_wrist1" child="Arm/J4_wrist1"/>
-  <xacro:actuator type="X5_1" name="Arm/J4_wrist1" child="end_effector"/>
+  <xacro:actuator type="X5_4" name="Arm/J3_elbow" child="elbow_wrist"/>
+  <xacro:link type="X5" extension="0.325" twist="0" name="elbow_wrist" child="Arm/J4_wrist"/>
+  <xacro:actuator type="X5_1" name="Arm/J4_wrist" child="end_effector"/>
   <xacro:gripper type="Custom" name="end_effector" mass="0.02"/>
 </robot>

File: urdf/kits/A-2085-04-parallel-gripper.xacro (robot description, xacro)
@@ -17,7 +17,7 @@
   <xacro:actuator type="X5_9" name="Arm/J2_shoulder" child="shoulder_elbow"/>
   <xacro:link type="X5" extension="0.325" twist="${pi}" name="shoulder_elbow" child="Arm/J3_elbow"/>
-  <xacro:actuator type="X5_4" name="Arm/J3_elbow" child="elbow_wrist1"/>
-  <xacro:link type="X5" extension="0.325" twist="${pi}" name="elbow_wrist1" child="Arm/J4_wrist1"/>
-  <xacro:actuator type="X5_1" name="Arm/J4_wrist1" child="end_effector"/>
+  <xacro:actuator type="X5_4" name="Arm/J3_elbow" child="elbow_wrist"/>
+  <xacro:link type="X5" extension="0.325" twist="${pi}" name="elbow_wrist" child="Arm/J4_wrist"/>
+  <xacro:actuator type="X5_1" name="Arm/J4_wrist" child="end_effector"/>
   <xacro:gripper type="X5Parallel" name="end_effector"/>
 </robot>

Commit message: Fix LeftOutside.

File: urdf/bracket.xacro (robot description, xacro)
@@ -111,5 +111,5 @@
         </xacro:if>
         <xacro:if value="${bracket_type.endswith('LeftOutside')}">
-          <origin xyz="0 -.03 .04" rpy="${pi/2} 0 0"/>
+          <origin xyz="0 .03 .04" rpy="${pi/2} 0 ${pi}"/>
         </xacro:if>
         <xacro:if value="${bracket_type.endswith('LeftInside')}">

Commit message: hebi_description package for ros2_control - Only A-2085-06 available

File: urdf/bracket.xacro (robot description, xacro)
@@ -35,5 +35,5 @@
         </xacro:if>
       </collision>
-      <!-- NOTE: inertia is just modelled as small sphere, and could be improved. -->
+      <!-- inertia is just modelled as small sphere, and could be improved. -->
       <inertial>
         <xacro:if value="${bracket_type.endswith('Left')}">
@@ -71,5 +71,5 @@
         </geometry>
       </collision>
-      <!-- NOTE: inertia is just modelled as small sphere, and could be improved. -->
+      <!-- inertia is just modelled as small sphere, and could be improved. -->
       <inertial>
         <xacro:if value="${bracket_type.endswith('Left')}">
@@ -165,5 +165,5 @@
         </geometry>
       </collision>
-      <!-- NOTE: inertia is just modelled as small sphere, and could be improved. -->
+      <!-- inertia is just modelled as small sphere, and could be improved. -->
       <inertial>
         <xacro:if value="${bracket_type.endswith('RightOutside')}">
@@ -229,5 +229,5 @@
         </geometry>
       </collision>
-      <!-- NOTE: inertia is just modelled as small sphere, and could be improved. -->
+      <!-- inertia is just modelled as small sphere, and could be improved. -->
       <inertial>
         <xacro:if value="${bracket_type.endswith('RightOutside')}">

File: urdf/link.xacro (robot description, xacro)
@@ -104,5 +104,5 @@
         <origin xyz="${extension/2} 0 ${edge_to_center}" rpy="0 0 0" />
         <mass value="${mass}"/>
-        <inertia  ixx="0.0" ixy="0.0"  ixz="0.0"  iyy="${mass * extension * extension / 12.0}"  iyz="0.0"  izz="${mass * extension * extension / 12.0}"/>
+        <inertia  ixx="${mass * edge_to_center * edge_to_center / 2.0}" ixy="0.0"  ixz="0.0"  iyy="${mass * (extension * extension + 6 * edge_to_center * edge_to_center) / 12.0}"  iyz="0.0"  izz="${mass * (extension * extension + 6 * edge_to_center * edge_to_center) / 12.0}"/>
       </inertial>
     </link>
