Commit message: Fix package namespace

File: urdf/actuator.xacro (robot description, xacro)
@@ -9,8 +9,8 @@
         <geometry>
           <xacro:if value="${model_name.startswith('X5')}">
-            <mesh filename="package://hebiros_description/meshes/x5.stl" scale="0.001 0.001 0.001"/>
+            <mesh filename="package://hebi_description/meshes/x5.stl" scale="0.001 0.001 0.001"/>
           </xacro:if>
           <xacro:if value="${model_name.startswith('X8')}">
-            <mesh filename="package://hebiros_description/meshes/x8.stl" scale="0.001 0.001 0.001"/>
+            <mesh filename="package://hebi_description/meshes/x8.stl" scale="0.001 0.001 0.001"/>
           </xacro:if>
         </geometry>
@@ -21,8 +21,8 @@
         <geometry>
           <xacro:if value="${model_name.startswith('X5')}">
-            <mesh filename="package://hebiros_description/meshes/x5.stl" scale="0.001 0.001 0.001"/>
+            <mesh filename="package://hebi_description/meshes/x5.stl" scale="0.001 0.001 0.001"/>
           </xacro:if>
           <xacro:if value="${model_name.startswith('X8')}">
-            <mesh filename="package://hebiros_description/meshes/x8.stl" scale="0.001 0.001 0.001"/>
+            <mesh filename="package://hebi_description/meshes/x8.stl" scale="0.001 0.001 0.001"/>
           </xacro:if>
         </geometry>

File: urdf/bracket.xacro (robot description, xacro)
@@ -10,5 +10,5 @@
           <origin xyz="0 0 0" rpy="${PI/2} 0 ${PI/2}"/>
           <geometry>
-            <mesh filename="package://hebiros_description/meshes/PM-2132-01L.stl" scale="0.001 0.001 0.001"/>
+            <mesh filename="package://hebi_description/meshes/PM-2132-01L.stl" scale="0.001 0.001 0.001"/>
           </geometry>
         </xacro:if>
@@ -16,5 +16,5 @@
           <origin xyz="0 0 0" rpy="${PI/2} 0 ${-PI/2}"/>
           <geometry>
-            <mesh filename="package://hebiros_description/meshes/PM-2132-01R.stl" scale="0.001 0.001 0.001"/>
+            <mesh filename="package://hebi_description/meshes/PM-2132-01R.stl" scale="0.001 0.001 0.001"/>
           </geometry>
         </xacro:if>
@@ -25,5 +25,5 @@
           <origin xyz="0 0 0" rpy="${PI/2} 0 ${PI/2}"/>
           <geometry>
-            <mesh filename="package://hebiros_description/meshes/PM-2132-01L.stl" scale="0.001 0.001 0.001"/>
+            <mesh filename="package://hebi_description/meshes/PM-2132-01L.stl" scale="0.001 0.001 0.001"/>
           </geometry>
         </xacro:if>
@@ -31,5 +31,5 @@
           <origin xyz="0 0 0" rpy="${PI/2} 0 ${-PI/2}"/>
           <geometry>
-            <mesh filename="package://hebiros_description/meshes/PM-2132-01R.stl" scale="0.001 0.001 0.001"/>
+            <mesh filename="package://hebi_description/meshes/PM-2132-01R.stl" scale="0.001 0.001 0.001"/>
           </geometry>
         </xacro:if>
@@ -63,5 +63,5 @@
         </xacro:if>
         <geometry>
-          <mesh filename="package://hebiros_description/meshes/PM-2149-01.stl" scale="0.001 0.001 0.001"/>
+          <mesh filename="package://hebi_description/meshes/PM-2149-01.stl" scale="0.001 0.001 0.001"/>
         </geometry>
         <xacro:black_material/>
@@ -88,8 +88,8 @@
         <geometry>
           <xacro:if value="${bracket_type.startswith('X5HeavyRight')}">
-            <mesh filename="package://hebiros_description/meshes/PM-2150-01R.stl" scale="0.001 0.001 0.001"/>
+            <mesh filename="package://hebi_description/meshes/PM-2150-01R.stl" scale="0.001 0.001 0.001"/>
           </xacro:if>
           <xacro:if value="${bracket_type.startswith('X5HeavyLeft')}">
-            <mesh filename="package://hebiros_description/meshes/PM-2150-01L.stl" scale="0.001 0.001 0.001"/>
+            <mesh filename="package://hebi_description/meshes/PM-2150-01L.stl" scale="0.001 0.001 0.001"/>
           </xacro:if>
         </geometry>
@@ -110,5 +110,5 @@
         </xacro:if>
         <geometry>
-          <mesh filename="package://hebiros_description/meshes/PM-2149-01.stl" scale="0.001 0.001 0.001"/>
+          <mesh filename="package://hebi_description/meshes/PM-2149-01.stl" scale="0.001 0.001 0.001"/>
         </geometry>
       </collision>
@@ -128,8 +128,8 @@
         <geometry>
           <xacro:if value="${bracket_type.startswith('X5HeavyRight')}">
-            <mesh filename="package://hebiros_description/meshes/PM-2150-01R.stl" scale="0.001 0.001 0.001"/>
+            <mesh filename="package://hebi_description/meshes/PM-2150-01R.stl" scale="0.001 0.001 0.001"/>
           </xacro:if>
           <xacro:if value="${bracket_type.startswith('X5HeavyLeft')}">
-            <mesh filename="package://hebiros_description/meshes/PM-2150-01L.stl" scale="0.001 0.001 0.001"/>
+            <mesh filename="package://hebi_description/meshes/PM-2150-01L.stl" scale="0.001 0.001 0.001"/>
           </xacro:if>
         </geometry>

File: urdf/link.xacro (robot description, xacro)
@@ -9,5 +9,5 @@
         <origin xyz="0 0 0" rpy="0 0 0" />
         <geometry>
-          <mesh filename="package://hebiros_description/meshes/A-2038-02.stl"/>
+          <mesh filename="package://hebi_description/meshes/A-2038-02.stl"/>
         </geometry>
         <xacro:black_material/>
@@ -23,5 +23,5 @@
         <origin xyz="${extension} ${sin(-twist) * edge_to_center} ${edge_to_center * (1 + cos(-twist))}" rpy="${-twist} 0 0"/>
         <geometry>
-          <mesh filename="package://hebiros_description/meshes/A-2039-02.stl"/>
+          <mesh filename="package://hebi_description/meshes/A-2039-02.stl"/>
         </geometry>
         <xacro:black_material/>
@@ -30,5 +30,5 @@
         <origin xyz="0 0 0" rpy="0 0 0" />
         <geometry>
-          <mesh filename="package://hebiros_description/meshes/A-2038-02.stl"/>
+          <mesh filename="package://hebi_description/meshes/A-2038-02.stl"/>
         </geometry>
       </collision>
@@ -42,5 +42,5 @@
         <origin xyz="${extension} ${sin(-twist) * edge_to_center} ${edge_to_center * (1 + cos(-twist))}" rpy="${-twist} 0 0"/>
         <geometry>
-          <mesh filename="package://hebiros_description/meshes/A-2039-02.stl"/>
+          <mesh filename="package://hebi_description/meshes/A-2039-02.stl"/>
         </geometry>
       </collision>

Commit message: Changed .STL name to better match other mesh files

File: urdf/actuator.xacro (robot description, xacro)
@@ -9,8 +9,8 @@
         <geometry>
           <xacro:if value="${model_name.startswith('X5')}">
-            <mesh filename="package://hebi_description/meshes/x5.stl" scale="0.001 0.001 0.001"/>
+            <mesh filename="package://hebi_description/meshes/X5.stl" scale="0.001 0.001 0.001"/>
           </xacro:if>
           <xacro:if value="${model_name.startswith('X8')}">
-            <mesh filename="package://hebi_description/meshes/x8.stl" scale="0.001 0.001 0.001"/>
+            <mesh filename="package://hebi_description/meshes/X8.stl" scale="0.001 0.001 0.001"/>
           </xacro:if>
         </geometry>
@@ -21,8 +21,8 @@
         <geometry>
           <xacro:if value="${model_name.startswith('X5')}">
-            <mesh filename="package://hebi_description/meshes/x5.stl" scale="0.001 0.001 0.001"/>
+            <mesh filename="package://hebi_description/meshes/X5.stl" scale="0.001 0.001 0.001"/>
           </xacro:if>
           <xacro:if value="${model_name.startswith('X8')}">
-            <mesh filename="package://hebi_description/meshes/x8.stl" scale="0.001 0.001 0.001"/>
+            <mesh filename="package://hebi_description/meshes/X8.stl" scale="0.001 0.001 0.001"/>
           </xacro:if>
         </geometry>

Commit message: Improved XACRO parameterization, and added joint limits to actuator elements.

File: urdf/actuator.xacro (robot description, xacro)
@@ -2,16 +2,61 @@
 <robot xmlns:xacro="http://www.ros.org/wiki/xacro">
   <!-- NOTE: joint must match the name of the module -->
-  <xacro:macro name="actuator" params="name child type">
-  <xacro:property name="model_name" value="${type}"/>
+  <xacro:macro name="actuator" params="name child type limits:=${[]}">
+    <xacro:property name="model_name" value="${type}"/>
+    <!-- Continuous joints (no position limits) -->
+    <xacro:if value="${limits == []}">
+      <xacro:property name="urdf_joint_type" value="continuous"/>
+    </xacro:if>
+    <!-- Revolute joints (position limits) -->
+    <xacro:unless value="${limits == []}">
+      <xacro:property name="urdf_joint_type" value="revolute"/>
+    </xacro:unless>
+    <!-- Set properties for model of actuator -->
+    <xacro:if value="${model_name == 'X5_1'}">
+      <xacro:property name="actuator_mass" value="0.315"/>
+      <xacro:property name="effort_limit" value="2.5"/>
+      <xacro:property name="velocity_limit" value="90"/>
+    </xacro:if>
+    <xacro:if value="${model_name == 'X5_4'}">
+      <xacro:property name="actuator_mass" value="0.335"/>
+      <xacro:property name="effort_limit" value="7.0"/>
+      <xacro:property name="velocity_limit" value="32"/>
+    </xacro:if>
+    <xacro:if value="${model_name == 'X5_9'}">
+      <xacro:property name="actuator_mass" value="0.360"/>
+      <xacro:property name="effort_limit" value="13.0"/>
+      <xacro:property name="velocity_limit" value="14"/>
+    </xacro:if>
+    <xacro:if value="${model_name == 'X8_3'}">
+      <xacro:property name="actuator_mass" value="0.460"/>
+      <xacro:property name="effort_limit" value="7"/>
+      <xacro:property name="velocity_limit" value="84"/>
+    </xacro:if>
+    <xacro:if value="${model_name == 'X8_9'}">
+      <xacro:property name="actuator_mass" value="0.480"/>
+      <xacro:property name="effort_limit" value="20"/>
+      <xacro:property name="velocity_limit" value="30"/>
+    </xacro:if>
+    <xacro:if value="${model_name == 'X8_16'}">
+      <xacro:property name="actuator_mass" value="0.500"/>
+      <xacro:property name="effort_limit" value="38"/>
+      <xacro:property name="velocity_limit" value="15"/>
+    </xacro:if>
+    <!-- Note: the frction/damping probably need to be tuned more for accurate simulation -->
+    <xacro:if value="${model_name.startswith('X5')}">
+      <xacro:property name="mesh_filename" value="package://hebi_description/meshes/X5.stl"/>
+      <xacro:property name="damping" value="0.1"/>
+      <xacro:property name="friction" value="0.1"/>
+    </xacro:if>
+    <xacro:if value="${model_name.startswith('X8')}">
+      <xacro:property name="mesh_filename" value="package://hebi_description/meshes/X8.stl"/>
+      <xacro:property name="damping" value="0.5"/>
+      <xacro:property name="friction" value="0.5"/>
+    </xacro:if>
     <link name="${name}/INPUT_INTERFACE">
       <visual>
         <origin xyz="0 0 0" rpy="0 0 0" />
         <geometry>
-          <xacro:if value="${model_name.startswith('X5')}">
-            <mesh filename="package://hebi_description/meshes/X5.stl" scale="0.001 0.001 0.001"/>
-          </xacro:if>
-          <xacro:if value="${model_name.startswith('X8')}">
-            <mesh filename="package://hebi_description/meshes/X8.stl" scale="0.001 0.001 0.001"/>
-          </xacro:if>
+          <mesh filename="${mesh_filename}" scale="0.001 0.001 0.001"/>
         </geometry>
         <xacro:red_material/>
@@ -20,10 +65,5 @@
         <origin xyz="0 0 0" rpy="0 0 0" />
         <geometry>
-          <xacro:if value="${model_name.startswith('X5')}">
-            <mesh filename="package://hebi_description/meshes/X5.stl" scale="0.001 0.001 0.001"/>
-          </xacro:if>
-          <xacro:if value="${model_name.startswith('X8')}">
-            <mesh filename="package://hebi_description/meshes/X8.stl" scale="0.001 0.001 0.001"/>
-          </xacro:if>
+          <mesh filename="${mesh_filename}" scale="0.001 0.001 0.001"/>
         </geometry>
       </collision>
@@ -31,31 +71,15 @@
         <xacro:if value="${model_name.startswith('X5')}">
           <origin xyz="-0.0142 -0.0031 0.0165" rpy="0 0 0" />
-          <xacro:if value="${model_name == 'X5_1'}">
-            <mass value="0.315"/>
-          </xacro:if>
-          <xacro:if value="${model_name == 'X5_4'}">
-            <mass value="0.335"/>
-          </xacro:if>
-          <xacro:if value="${model_name == 'X5_9'}">
-            <mass value="0.360"/>
-          </xacro:if>
+          <mass value="${actuator_mass}"/>
           <inertia ixx="0.00015" iyy="0.000255" izz="0.000350" ixy="0.0000341" ixz="0.0000118" iyz="0.00000229"/>
         </xacro:if>
         <xacro:if value="${model_name.startswith('X8')}">
           <origin xyz="-0.0145 -0.0031 0.0242" rpy="0 0 0" />
-          <xacro:if value="${model_name == 'X8_3'}">
-            <mass value="0.460"/>
-          </xacro:if>
-          <xacro:if value="${model_name == 'X8_9'}">
-            <mass value="0.480"/>
-          </xacro:if>
-          <xacro:if value="${model_name == 'X8_16'}">
-            <mass value="0.500"/>
-          </xacro:if>
+          <mass value="${actuator_mass}"/>
           <inertia ixx="0.000246" iyy="0.000380" izz="0.000463" ixy="0.0000444" ixz="0.0000266" iyz="0.00000422"/>
         </xacro:if>
       </inertial>
     </link>
-    <joint name="${name}/${model_name}" type="continuous">
+    <joint name="${name}/${model_name}" type="${urdf_joint_type}">
       <parent link="${name}/INPUT_INTERFACE"/>
       <child link="${child}/INPUT_INTERFACE"/>
@@ -67,28 +91,13 @@
       </xacro:if>
       <axis xyz="0 0 1"/>
-      <xacro:if value="${model_name == 'X5_1'}">
-        <limit effort="2.5" velocity="90"/>
-        <dynamics damping="0.1" friction="0.1"/>
+      <!-- Continuous joints (no position limits) -->
+      <xacro:if value="${limits == []}">
+        <limit effort="${effort_limit}" velocity="${velocity_limit}"/>
       </xacro:if>
-      <xacro:if value="${model_name == 'X5_4'}">
-        <limit effort="7.0" velocity="32"/>
-        <dynamics damping="0.1" friction="0.1"/>
-      </xacro:if>
-      <xacro:if value="${model_name == 'X5_9'}">
-        <limit effort="13.0" velocity="14"/>
-        <dynamics damping="0.1" friction="0.1"/>
-      </xacro:if>
-      <xacro:if value="${model_name == 'X8_3'}">
-        <limit effort="7" velocity="84"/>
-        <dynamics damping="0.5" friction="0.5"/>
-      </xacro:if>
-      <xacro:if value="${model_name == 'X8_9'}">
-        <limit effort="20" velocity="30"/>
-        <dynamics damping="0.5" friction="0.5"/>
-      </xacro:if>
-      <xacro:if value="${model_name == 'X8_16'}">
-        <limit effort="38" velocity="15"/>
-        <dynamics damping="0.5" friction="0.5"/>
-      </xacro:if>
+      <!-- Revolute joints (position limits) -->
+      <xacro:unless value="${limits == []}">
+        <limit effort="${effort_limit}" velocity="${velocity_limit}" lower="${limits[0]}" upper="${limits[1]}"/>
+      </xacro:unless>
+      <dynamics damping="${damping}" friction="${friction}"/>
     </joint>
   </xacro:macro>
