Commit message: Added Gazebo compatible colors to urdf.xacro macros
changed kit naming to lower case to match moveit configs

File: urdf/actuator.xacro (robot description, xacro)
@@ -81,4 +81,7 @@
       </inertial>
     </link>
+    <gazebo reference="${name}/INPUT_INTERFACE">
+      <xacro:gazebo_red_material/>
+    </gazebo>
     <joint name="${name}/${model_name}" type="${urdf_joint_type}">
       <parent link="${name}/INPUT_INTERFACE"/>

File: urdf/bracket.xacro (robot description, xacro)
@@ -148,4 +148,12 @@
     </xacro:if>
   </link>
+  <gazebo reference="${name}/INPUT_INTERFACE">
+    <xacro:if value="${bracket_type.startswith('X5Light')}">
+      <xacro:gazebo_beige_material/>
+    </xacro:if>
+    <xacro:if value="${bracket_type.startswith('X5Heavy')}">
+      <xacro:gazebo_black_material/>
+    </xacro:if>
+  </gazebo>
   <joint name="${name}/OUTPUT_INTERFACE" type="fixed">
     <parent link="${name}/INPUT_INTERFACE"/>

File: urdf/end_effector.xacro (robot description, xacro)
@@ -1,29 +1,4 @@
 <?xml version="1.0"?>
 <robot xmlns:xacro="http://www.ros.org/wiki/xacro">
-  <!-- TODO: add collision and inertial elements -->
-  <xacro:macro name="null_end_effector" params="name">
-    <link name="${name}/INPUT_INTERFACE">
-      <collision>
-        <origin xyz="0 0 0.0005" rpy="0 0 0"/>
-	<geometry>
-          <box size="0.001 0.001 0.001" rpy="0 0 0"/>
-	</geometry>
-      </collision>
-      <visual>
-        <origin xyz="0 0 0.0005" rpy="0 0 0"/>
-	<geometry>
-          <box size="0.001 0.001 0.001" rpy="0 0 0"/>
-	</geometry>
-      </visual>
-      <inertial>
-        <origin xyz="0 0 0.0005" rpy="0 0 0"/>
-	<mass value="0.001"/>
-        <inertia
-          ixx="0.001" ixy="0.0" ixz="0.0"
-          iyy="0.001" iyz="0.0"
-          izz="0.001"/>
-      </inertial>
-    </link>
-  </xacro:macro>
   <xacro:macro name="parallel_gripper_outer_subassembly" params="name prefix">
     <link name="${name}/${prefix}_finger">
@@ -36,4 +11,7 @@
       </visual>
     </link>
+    <gazebo reference="${name}/${prefix}_finger">
+      <xacro:gazebo_silver_material/>
+    </gazebo>
     <link name="${name}/${prefix}_outer_linkage">
       <visual>
@@ -45,4 +23,7 @@
       </visual>
     </link>
+    <gazebo reference="${name}/${prefix}_outer_linkage">
+      <xacro:gazebo_black_material/>
+    </gazebo>
     <link name="${name}/${prefix}_gripper">
       <visual>
@@ -60,4 +41,7 @@
       </collision>
     </link>
+    <gazebo reference="${name}/${prefix}_gripper">
+      <xacro:gazebo_black_material/>
+    </gazebo>
     <joint name="${name}/input_${prefix}_finger" type="revolute">
       <xacro:if value="${prefix == 'l'}">
@@ -98,4 +82,7 @@
       </visual>
     </link>
+    <gazebo reference="${name}/${prefix}_inner_linkage">
+      <xacro:gazebo_black_material/>
+    </gazebo>
     <joint name="${name}/center_hub_${prefix}_inner_linkage" type="continuous">
       <xacro:if value="${prefix == 'l'}">
@@ -110,41 +97,72 @@
     </joint>
   </xacro:macro>
-  <!-- NOTE: only "parallel" is currently supported for type -->
   <xacro:macro name="gripper" params="name type">
-    <!-- The base body of the gripper -->
-    <link name="${name}/INPUT_INTERFACE">
-      <visual>
-        <origin xyz="0 0 0.00375" />
+    <xacro:if value="${type == 'Custom'}">
+      <link name="${name}/INPUT_INTERFACE">
+        <collision>
+          <origin xyz="0 0 0.0005" rpy="0 0 0"/>
           <geometry>
-          <cylinder length="0.0075" radius=".0225" />
-        </geometry>
-        <xacro:black_material/>
-      </visual>
-    </link>
-    <!-- Tree branch for center hub -->
-    <link name="${name}/center_hub">
-      <visual>
-        <origin xyz="-0.0225 0.0225 0" rpy="${pi/2} 0 0" />
-        <geometry>
-          <mesh filename="package://hebi_description/meshes/PM-2357-02.stl" scale="0.001 0.001 0.001"/>
-        </geometry>
-        <xacro:black_material/>
-      </visual>
-    </link>
-    <joint name="${name}/input_center_hub" type="fixed">
-      <origin xyz="0 0 0.0045" rpy="0 0 0" />
-      <parent link="${name}/INPUT_INTERFACE"/>
-      <child link="${name}/center_hub"/>
-    </joint>
-    <gazebo reference="${name}/input_center_hub">
-      <disableFixedJointLumping>true</disableFixedJointLumping>
-      <preserveFixedJoint>true</preserveFixedJoint>
-    </gazebo>
-    <!-- Tree branches for fingers, outer linkages, and grippers -->
-    <xacro:parallel_gripper_outer_subassembly name="${name}" prefix="l"/>
-    <xacro:parallel_gripper_outer_subassembly name="${name}" prefix="r"/>
-    <!-- Tree branches for inner linkages -->
-    <xacro:parallel_gripper_inner_subassembly name="${name}" prefix="l"/>
-    <xacro:parallel_gripper_inner_subassembly name="${name}" prefix="r"/>
+            <box size="0.001 0.001 0.001" rpy="0 0 0"/>
+          </geometry>
+        </collision>
+        <visual>
+          <origin xyz="0 0 0.0005" rpy="0 0 0"/>
+          <geometry>
+            <box size="0.001 0.001 0.001" rpy="0 0 0"/>
+          </geometry>
+        </visual>
+        <inertial>
+        <origin xyz="0 0 0" rpy="0 0 0"/>
+          <mass value="0.001"/>
+          <inertia
+            ixx="0.001" ixy="0.0" ixz="0.0"
+            iyy="0.001" iyz="0.0"
+            izz="0.001"/>
+        </inertial>
+      </link>
+    </xacro:if>
+    <xacro:if value="${type.endswith('Parallel')}">
+      <!-- The base body of the gripper -->
+      <link name="${name}/INPUT_INTERFACE">
+        <visual>
+          <origin xyz="0 0 0.00375" />
+            <geometry>
+            <cylinder length="0.0075" radius=".0225" />
+          </geometry>
+          <xacro:black_material/>
+        </visual>
+      </link>
+      <gazebo reference="${name}/INPUT_INTERFACE">
+        <xacro:gazebo_black_material/>
+      </gazebo>
+      <!-- Tree branch for center hub -->
+      <link name="${name}/center_hub">
+        <visual>
+          <origin xyz="-0.0225 0.0225 0" rpy="${pi/2} 0 0" />
+          <geometry>
+            <mesh filename="package://hebi_description/meshes/PM-2357-02.stl" scale="0.001 0.001 0.001"/>
+          </geometry>
+          <xacro:black_material/>
+        </visual>
+      </link>
+      <gazebo reference="${name}/center_hub">
+        <xacro:gazebo_black_material/>
+      </gazebo>
+      <joint name="${name}/input_center_hub" type="fixed">
+        <origin xyz="0 0 0.0045" rpy="0 0 0" />
+        <parent link="${name}/INPUT_INTERFACE"/>
+        <child link="${name}/center_hub"/>
+      </joint>
+      <gazebo reference="${name}/input_center_hub">
+        <disableFixedJointLumping>true</disableFixedJointLumping>
+        <preserveFixedJoint>true</preserveFixedJoint>
+      </gazebo>
+      <!-- Tree branches for fingers, outer linkages, and grippers -->
+      <xacro:parallel_gripper_outer_subassembly name="${name}" prefix="l"/>
+      <xacro:parallel_gripper_outer_subassembly name="${name}" prefix="r"/>
+      <!-- Tree branches for inner linkages -->
+      <xacro:parallel_gripper_inner_subassembly name="${name}" prefix="l"/>
+      <xacro:parallel_gripper_inner_subassembly name="${name}" prefix="r"/>
+    </xacro:if>
   </xacro:macro>
 </robot>

File: urdf/hebi.xacro (robot description, xacro)
@@ -8,8 +8,14 @@
     </material>
   </xacro:macro>
+  <xacro:macro name="gazebo_red_material">
+    <material>Gazebo/Red</material>
+  </xacro:macro>
   <xacro:macro name="silver_material">
     <material name="silver">
       <color rgba="0.6 0.6 0.6 1"/>
     </material>
+  </xacro:macro>
+  <xacro:macro name="gazebo_silver_material">
+    <material>Gazebo/Grey</material>
   </xacro:macro>
   <xacro:macro name="black_material">
@@ -18,8 +24,19 @@
     </material>
   </xacro:macro>
+  <xacro:macro name="gazebo_black_material">
+    <material>Gazebo/Black</material>
+  </xacro:macro>
   <xacro:macro name="beige_material">
     <material name="beige">
       <color rgba="0.96 0.945 0.871 1"/>
     </material>
+  </xacro:macro>
+  <xacro:macro name="gazebo_beige_material">
+    <visual>
+      <material>
+          <ambient>0.96 0.945 0.871 1</ambient>
+          <diffuse>0.96 0.945 0.871 1</diffuse>
+      </material>
+    </visual>
   </xacro:macro>
   <xacro:include filename="./actuator.xacro"/>

File: urdf/link.xacro (robot description, xacro)
@@ -18,5 +18,5 @@
           <cylinder length="${extension-.0254}" radius=".016" />
         </geometry>
-        <xacro:silver_material/>
+        <xacro:black_material/>
       </visual>
       <visual>
@@ -52,4 +52,7 @@
       </inertial>
     </link>
+    <gazebo reference="${name}/INPUT_INTERFACE">
+      <xacro:gazebo_black_material/>
+    </gazebo>
     <joint name="${name}/OUTPUT_JOINT" type="fixed">
       <parent link="${name}/INPUT_INTERFACE"/>

Commit message: Add xacros for R-series actuators
Supports R-series brackets/links, though visuals are not updated

File: urdf/actuator.xacro (robot description, xacro)
@@ -43,4 +43,19 @@
       <xacro:property name="velocity_limit" value="15"/>
     </xacro:if>
+    <xacro:if value="${model_name == 'R8_3'}">
+      <xacro:property name="actuator_mass" value="0.670"/>
+      <xacro:property name="effort_limit" value="7"/>
+      <xacro:property name="velocity_limit" value="84"/>
+    </xacro:if>
+    <xacro:if value="${model_name == 'R8_9'}">
+      <xacro:property name="actuator_mass" value="0.685"/>
+      <xacro:property name="effort_limit" value="20"/>
+      <xacro:property name="velocity_limit" value="30"/>
+    </xacro:if>
+    <xacro:if value="${model_name == 'R8_16'}">
+      <xacro:property name="actuator_mass" value="0.715"/>
+      <xacro:property name="effort_limit" value="38"/>
+      <xacro:property name="velocity_limit" value="15"/>
+    </xacro:if>
     <!-- Note: the frction/damping probably need to be tuned more for accurate simulation -->
     <xacro:if value="${model_name.startswith('X5')}">
@@ -54,4 +69,9 @@
       <xacro:property name="friction" value="0.5"/>
     </xacro:if>
+    <xacro:if value="${model_name.startswith('R8')}">
+      <xacro:property name="mesh_filename" value="package://hebi_description/meshes/R8.stl"/>
+      <xacro:property name="damping" value="0.5"/>
+      <xacro:property name="friction" value="0.5"/>
+    </xacro:if>
     <link name="${name}/INPUT_INTERFACE">
       <visual>
@@ -60,5 +80,10 @@
           <mesh filename="${mesh_filename}" scale="0.001 0.001 0.001"/>
         </geometry>
-        <xacro:red_material/>
+        <xacro:unless value="${model_name.startswith('R8')}">
+          <xacro:red_material/>
+        </xacro:unless>
+        <xacro:if value="${model_name.startswith('R8')}">
+          <xacro:black_material/>
+        </xacro:if>
       </visual>
       <collision>
@@ -72,15 +97,31 @@
           <origin xyz="-0.0142 -0.0031 0.0165" rpy="0 0 0" />
           <mass value="${actuator_mass}"/>
-          <inertia ixx="0.00015" iyy="0.000255" izz="0.000350" ixy="0.0000341" ixz="0.0000118" iyz="0.00000229"/>
+          <inertia ixx="0.00015"  ixy="0.0000341"  ixz="0.0000118"
+                   iyy="0.000255" iyz="0.00000229"
+                   izz="0.000350" />
         </xacro:if>
         <xacro:if value="${model_name.startswith('X8')}">
           <origin xyz="-0.0145 -0.0031 0.0242" rpy="0 0 0" />
           <mass value="${actuator_mass}"/>
-          <inertia ixx="0.000246" iyy="0.000380" izz="0.000463" ixy="0.0000444" ixz="0.0000266" iyz="0.00000422"/>
+          <inertia ixx="0.000246" ixy="0.0000444" ixz="0.0000266"
+                   iyy="0.000380" iyz="0.00000422"
+                   izz="0.000463"/>
+        </xacro:if>
+        <xacro:if value="${model_name.startswith('R8')}">
+          <origin xyz="-0.02396 -0.00161 0.02557" rpy="0 0 0" />
+          <mass value="${actuator_mass}"/>
+          <inertia ixx="0.000488" ixy="0.00001297" ixz="0.0000578"
+                   iyy="0.001009" iyz="0.00000494"
+                   izz="0.001186" />
         </xacro:if>
       </inertial>
     </link>
     <gazebo reference="${name}/INPUT_INTERFACE">
-      <xacro:gazebo_red_material/>
+      <xacro:unless value="${model_name.startswith('R8')}">
+        <xacro:gazebo_red_material/>
+      </xacro:unless>
+      <xacro:if value="${model_name.startswith('R8')}">
+        <xacro:gazebo_black_material/>
+      </xacro:if>
     </gazebo>
     <joint name="${name}/${model_name}" type="${urdf_joint_type}">
@@ -92,4 +133,7 @@
       <xacro:if value="${model_name.startswith('X8')}">
         <origin xyz="0 0 0.045" rpy="0 0 0"/>
+      </xacro:if>
+      <xacro:if value="${model_name.startswith('R8')}">
+        <origin xyz="0 0 0.051" rpy="0 0 0"/>
       </xacro:if>
       <axis xyz="0 0 1"/>

File: urdf/bracket.xacro (robot description, xacro)
@@ -5,5 +5,5 @@
   <link name="${name}/INPUT_INTERFACE">
     <!-- Light bracket -->
-    <xacro:if value="${bracket_type.startswith('X5Light')}">
+    <xacro:if value="${bracket_type.startswith('X5Light') or bracket_type.startswith('R5Light')}">
       <visual>
         <xacro:if value="${bracket_type.endswith('Left')}">
@@ -48,5 +48,5 @@
     </xacro:if>
     <!-- Heavy bracket -->
-    <xacro:if value="${bracket_type.startswith('X5Heavy')}">
+    <xacro:if value="${bracket_type.startswith('X5Heavy') or bracket_type.startswith('R5Heavy')}">
       <visual>
         <xacro:if value="${bracket_type.endswith('RightOutside')}">
@@ -81,8 +81,8 @@
         </xacro:if>
         <geometry>
-          <xacro:if value="${bracket_type.startswith('X5HeavyRight')}">
+          <xacro:if value="${bracket_type.startswith('X5HeavyRight') or bracket_type.startswith('R5HeavyRight')}">
             <mesh filename="package://hebi_description/meshes/PM-2150-01R.stl" scale="0.001 0.001 0.001"/>
           </xacro:if>
-          <xacro:if value="${bracket_type.startswith('X5HeavyLeft')}">
+          <xacro:if value="${bracket_type.startswith('X5HeavyLeft') or bracket_type.startswith('R5HeavyLeft')}">
             <mesh filename="package://hebi_description/meshes/PM-2150-01L.stl" scale="0.001 0.001 0.001"/>
           </xacro:if>
@@ -121,8 +121,8 @@
         </xacro:if>
         <geometry>
-          <xacro:if value="${bracket_type.startswith('X5HeavyRight')}">
+          <xacro:if value="${bracket_type.startswith('X5HeavyRight') or bracket_type.startswith('R5HeavyRight')}">
             <mesh filename="package://hebi_description/meshes/PM-2150-01R.stl" scale="0.001 0.001 0.001"/>
           </xacro:if>
-          <xacro:if value="${bracket_type.startswith('X5HeavyLeft')}">
+          <xacro:if value="${bracket_type.startswith('X5HeavyLeft') or bracket_type.startswith('R5HeavyLeft')}">
             <mesh filename="package://hebi_description/meshes/PM-2150-01L.stl" scale="0.001 0.001 0.001"/>
           </xacro:if>
@@ -149,8 +149,8 @@
   </link>
   <gazebo reference="${name}/INPUT_INTERFACE">
-    <xacro:if value="${bracket_type.startswith('X5Light')}">
+    <xacro:if value="${bracket_type.startswith('X5Light') or bracket_type.startswith('R5Light')}">
       <xacro:gazebo_beige_material/>
     </xacro:if>
-    <xacro:if value="${bracket_type.startswith('X5Heavy')}">
+    <xacro:if value="${bracket_type.startswith('X5Heavy') or bracket_type.startswith('R5Heavy')}">
       <xacro:gazebo_black_material/>
     </xacro:if>

Commit message: R-Series xacro update (#7)
* Adds color to Gazebo models (previously only Rviz)

* Add xacros for R-series actuators

Supports R-series brackets/links, though visuals are not updated

File: urdf/actuator.xacro (robot description, xacro)
@@ -43,4 +43,19 @@
       <xacro:property name="velocity_limit" value="15"/>
     </xacro:if>
+    <xacro:if value="${model_name == 'R8_3'}">
+      <xacro:property name="actuator_mass" value="0.670"/>
+      <xacro:property name="effort_limit" value="7"/>
+      <xacro:property name="velocity_limit" value="84"/>
+    </xacro:if>
+    <xacro:if value="${model_name == 'R8_9'}">
+      <xacro:property name="actuator_mass" value="0.685"/>
+      <xacro:property name="effort_limit" value="20"/>
+      <xacro:property name="velocity_limit" value="30"/>
+    </xacro:if>
+    <xacro:if value="${model_name == 'R8_16'}">
+      <xacro:property name="actuator_mass" value="0.715"/>
+      <xacro:property name="effort_limit" value="38"/>
+      <xacro:property name="velocity_limit" value="15"/>
+    </xacro:if>
     <!-- Note: the frction/damping probably need to be tuned more for accurate simulation -->
     <xacro:if value="${model_name.startswith('X5')}">
@@ -54,4 +69,9 @@
       <xacro:property name="friction" value="0.5"/>
     </xacro:if>
+    <xacro:if value="${model_name.startswith('R8')}">
+      <xacro:property name="mesh_filename" value="package://hebi_description/meshes/R8.stl"/>
+      <xacro:property name="damping" value="0.5"/>
+      <xacro:property name="friction" value="0.5"/>
+    </xacro:if>
     <link name="${name}/INPUT_INTERFACE">
       <visual>
@@ -60,5 +80,10 @@
           <mesh filename="${mesh_filename}" scale="0.001 0.001 0.001"/>
         </geometry>
-        <xacro:red_material/>
+        <xacro:unless value="${model_name.startswith('R8')}">
+          <xacro:red_material/>
+        </xacro:unless>
+        <xacro:if value="${model_name.startswith('R8')}">
+          <xacro:black_material/>
+        </xacro:if>
       </visual>
       <collision>
@@ -72,13 +97,32 @@
           <origin xyz="-0.0142 -0.0031 0.0165" rpy="0 0 0" />
           <mass value="${actuator_mass}"/>
-          <inertia ixx="0.00015" iyy="0.000255" izz="0.000350" ixy="0.0000341" ixz="0.0000118" iyz="0.00000229"/>
+          <inertia ixx="0.00015"  ixy="0.0000341"  ixz="0.0000118"
+                   iyy="0.000255" iyz="0.00000229"
+                   izz="0.000350" />
         </xacro:if>
         <xacro:if value="${model_name.startswith('X8')}">
           <origin xyz="-0.0145 -0.0031 0.0242" rpy="0 0 0" />
           <mass value="${actuator_mass}"/>
-          <inertia ixx="0.000246" iyy="0.000380" izz="0.000463" ixy="0.0000444" ixz="0.0000266" iyz="0.00000422"/>
+          <inertia ixx="0.000246" ixy="0.0000444" ixz="0.0000266"
+                   iyy="0.000380" iyz="0.00000422"
+                   izz="0.000463"/>
+        </xacro:if>
+        <xacro:if value="${model_name.startswith('R8')}">
+          <origin xyz="-0.02396 -0.00161 0.02557" rpy="0 0 0" />
+          <mass value="${actuator_mass}"/>
+          <inertia ixx="0.000488" ixy="0.00001297" ixz="0.0000578"
+                   iyy="0.001009" iyz="0.00000494"
+                   izz="0.001186" />
         </xacro:if>
       </inertial>
     </link>
+    <gazebo reference="${name}/INPUT_INTERFACE">
+      <xacro:unless value="${model_name.startswith('R8')}">
+        <xacro:gazebo_red_material/>
+      </xacro:unless>
+      <xacro:if value="${model_name.startswith('R8')}">
+        <xacro:gazebo_black_material/>
+      </xacro:if>
+    </gazebo>
     <joint name="${name}/${model_name}" type="${urdf_joint_type}">
       <parent link="${name}/INPUT_INTERFACE"/>
@@ -89,4 +133,7 @@
       <xacro:if value="${model_name.startswith('X8')}">
         <origin xyz="0 0 0.045" rpy="0 0 0"/>
+      </xacro:if>
+      <xacro:if value="${model_name.startswith('R8')}">
+        <origin xyz="0 0 0.051" rpy="0 0 0"/>
       </xacro:if>
       <axis xyz="0 0 1"/>

File: urdf/bracket.xacro (robot description, xacro)
@@ -5,5 +5,5 @@
   <link name="${name}/INPUT_INTERFACE">
     <!-- Light bracket -->
-    <xacro:if value="${bracket_type.startswith('X5Light')}">
+    <xacro:if value="${bracket_type.startswith('X5Light') or bracket_type.startswith('R5Light')}">
       <visual>
         <xacro:if value="${bracket_type.endswith('Left')}">
@@ -48,5 +48,5 @@
     </xacro:if>
     <!-- Heavy bracket -->
-    <xacro:if value="${bracket_type.startswith('X5Heavy')}">
+    <xacro:if value="${bracket_type.startswith('X5Heavy') or bracket_type.startswith('R5Heavy')}">
       <visual>
         <xacro:if value="${bracket_type.endswith('RightOutside')}">
@@ -81,8 +81,8 @@
         </xacro:if>
         <geometry>
-          <xacro:if value="${bracket_type.startswith('X5HeavyRight')}">
+          <xacro:if value="${bracket_type.startswith('X5HeavyRight') or bracket_type.startswith('R5HeavyRight')}">
             <mesh filename="package://hebi_description/meshes/PM-2150-01R.stl" scale="0.001 0.001 0.001"/>
           </xacro:if>
-          <xacro:if value="${bracket_type.startswith('X5HeavyLeft')}">
+          <xacro:if value="${bracket_type.startswith('X5HeavyLeft') or bracket_type.startswith('R5HeavyLeft')}">
             <mesh filename="package://hebi_description/meshes/PM-2150-01L.stl" scale="0.001 0.001 0.001"/>
           </xacro:if>
@@ -121,8 +121,8 @@
         </xacro:if>
         <geometry>
-          <xacro:if value="${bracket_type.startswith('X5HeavyRight')}">
+          <xacro:if value="${bracket_type.startswith('X5HeavyRight') or bracket_type.startswith('R5HeavyRight')}">
             <mesh filename="package://hebi_description/meshes/PM-2150-01R.stl" scale="0.001 0.001 0.001"/>
           </xacro:if>
-          <xacro:if value="${bracket_type.startswith('X5HeavyLeft')}">
+          <xacro:if value="${bracket_type.startswith('X5HeavyLeft') or bracket_type.startswith('R5HeavyLeft')}">
             <mesh filename="package://hebi_description/meshes/PM-2150-01L.stl" scale="0.001 0.001 0.001"/>
           </xacro:if>
@@ -148,4 +148,12 @@
     </xacro:if>
   </link>
+  <gazebo reference="${name}/INPUT_INTERFACE">
+    <xacro:if value="${bracket_type.startswith('X5Light') or bracket_type.startswith('R5Light')}">
+      <xacro:gazebo_beige_material/>
+    </xacro:if>
+    <xacro:if value="${bracket_type.startswith('X5Heavy') or bracket_type.startswith('R5Heavy')}">
+      <xacro:gazebo_black_material/>
+    </xacro:if>
+  </gazebo>
   <joint name="${name}/OUTPUT_INTERFACE" type="fixed">
     <parent link="${name}/INPUT_INTERFACE"/>
