Commit message: Updates to match simulator plugin changes

File: urdf/actuator.xacro (robot description, xacro)
@@ -2,5 +2,5 @@
 <robot xmlns:xacro="http://www.ros.org/wiki/xacro">
   <!-- NOTE: joint must match the name of the module -->
-  <xacro:macro name="actuator" params="name child type limits:=${[]}">
+  <xacro:macro name="actuator" params="name child:='' type limits:=${[]}">
     <xacro:property name="model_name" value="${type}"/>
     <!-- Continuous joints (no position limits) -->
@@ -94,7 +94,7 @@
       </collision>
       <inertial>
+        <mass value="${actuator_mass}"/>
         <xacro:if value="${model_name.startswith('X5')}">
           <origin xyz="-0.0142 -0.0031 0.0165" rpy="0 0 0" />
-          <mass value="${actuator_mass}"/>
           <inertia ixx="0.00015"  ixy="0.0000341"  ixz="0.0000118"
                    iyy="0.000255" iyz="0.00000229"
@@ -103,5 +103,4 @@
         <xacro:if value="${model_name.startswith('X8')}">
           <origin xyz="-0.0145 -0.0031 0.0242" rpy="0 0 0" />
-          <mass value="${actuator_mass}"/>
           <inertia ixx="0.000246" ixy="0.0000444" ixz="0.0000266"
                    iyy="0.000380" iyz="0.00000422"
@@ -110,5 +109,4 @@
         <xacro:if value="${model_name.startswith('R8')}">
           <origin xyz="-0.02396 -0.00161 0.02557" rpy="0 0 0" />
-          <mass value="${actuator_mass}"/>
           <inertia ixx="0.000488" ixy="0.00001297" ixz="0.0000578"
                    iyy="0.001009" iyz="0.00000494"
@@ -125,5 +123,29 @@
       </xacro:if>
     </gazebo>
-    <joint name="${name}/${model_name}" type="${urdf_joint_type}">
+    <link name="HEBI_SIM/${name}/${model_name}">
+      <visual>
+        <origin xyz="-0.03 0 0.02" rpy="0 0 0" />
+        <geometry>
+          <sphere radius="0.001"/>
+        </geometry>
+      </visual>
+      <inertial>
+        <mass value="0.001"/>
+        <origin xyz="0 0 0" rpy="0 0 0" />
+        <inertia ixx="0.000001" ixy="0" ixz="0"
+                 iyy="0.000001" iyz="0"
+                 izz="0.000001" />
+      </inertial>
+    </link>
+    <joint name="HEBI_SIM_JOINT/${name}" type="fixed">
+      <parent link="${name}/INPUT_INTERFACE"/>
+      <child link="HEBI_SIM/${name}/${model_name}"/>
+      <origin xyz="0 0 0" rpy="0 0 0"/>
+    </joint>
+    <gazebo reference="HEBI_SIM_JOINT/${name}">
+      <disableFixedJointLumping>true</disableFixedJointLumping>
+      <preserveFixedJoint>true</preserveFixedJoint>
+    </gazebo>
+    <joint name="${name}" type="${urdf_joint_type}">
       <parent link="${name}/INPUT_INTERFACE"/>
       <child link="${child}/INPUT_INTERFACE"/>

File: urdf/end_effector.xacro (robot description, xacro)
@@ -197,5 +197,5 @@
     </joint>
   </xacro:macro>
-  <xacro:macro name="gripper" params="name type:=Custom mass:=0.020 com_trans:='0 0 0' output_trans:='0 0 0'">
+  <xacro:macro name="gripper" params="name type:=Custom mass:=0.0 com_trans:='0 0 0' output_trans:='0 0 0'">
     <xacro:property name="com_trans_list" value="${map(float, com_trans.split(' '))}" />
     <xacro:if value="${ com_trans_list[0] + com_trans_list[1] + com_trans_list[2] >= 0.01 }">
@@ -207,10 +207,4 @@
     <xacro:if value="${type == 'Custom'}">
       <link name="${name}/INPUT_INTERFACE">
-        <collision>
-          <origin xyz="0 0 0.0005" rpy="0 0 0" />
-          <geometry>
-            <box size="0.001 0.001 0.001" rpy="0 0 0" />
-          </geometry>
-        </collision>
         <visual>
           <origin xyz="0 0 0.0005" rpy="0 0 0" />

File: urdf/kits/A-2084-01.xacro (robot description, xacro)
@@ -20,4 +20,4 @@
   <xacro:link type="X5" extension="0.325" twist="0" name="elbow_wrist" child="Arm/J4_wrist"/>
   <xacro:actuator type="X5_1" name="Arm/J4_wrist" child="end_effector"/>
-  <xacro:gripper type="Custom" name="end_effector" mass="0.02"/>
+  <xacro:gripper type="Custom" name="end_effector" mass="0.0"/>
 </robot>

File: urdf/kits/A-2085-04.xacro (robot description, xacro)
@@ -18,6 +18,6 @@
   <xacro:link type="X5" extension="0.325" twist="${pi}" name="shoulder_elbow" child="Arm/J3_elbow"/>
   <xacro:actuator type="X5_4" name="Arm/J3_elbow" child="elbow_wrist"/>
-  <xacro:link type="X5" extension="0.325" twist="${pi}" name="elbow_wrist" child="Arm/J4_wrist"/>
+  <xacro:link type="X5" extension="0.325" twist="0" name="elbow_wrist" child="Arm/J4_wrist"/>
   <xacro:actuator type="X5_1" name="Arm/J4_wrist" child="end_effector"/>
-  <xacro:gripper type="Custom" name="end_effector" mass="0.02"/>
+  <xacro:gripper type="Custom" name="end_effector" mass="0.0"/>
 </robot>

File: urdf/kits/A-2085-05.xacro (robot description, xacro)
@@ -22,4 +22,4 @@
   <xacro:bracket type="X5LightRight" name="wrist2_bracket" child="Arm/J5_wrist2"/>
   <xacro:actuator type="X5_1" name="Arm/J5_wrist2" child="end_effector"/>
-  <xacro:gripper type="Custom" name="end_effector" mass="0.02"/>
+  <xacro:gripper type="Custom" name="end_effector" mass="0.0"/>
 </robot>

File: urdf/kits/A-2085-06.xacro (robot description, xacro)
@@ -24,4 +24,4 @@
   <xacro:bracket type="X5LightRight" name="wrist3_bracket" child="Arm/J6_wrist3"/>
   <xacro:actuator type="X5_1" name="Arm/J6_wrist3" child="end_effector"/>
-  <xacro:gripper type="Custom" name="end_effector" mass="0.02"/>
+  <xacro:gripper type="Custom" name="end_effector" mass="0.0"/>
 </robot>

Commit message: Fix units on xacro velocity_limit
previously was rpm, should be rad/s

File: urdf/actuator.xacro (robot description, xacro)
@@ -16,45 +16,45 @@
       <xacro:property name="actuator_mass" value="0.315"/>
       <xacro:property name="effort_limit" value="2.5"/>
-      <xacro:property name="velocity_limit" value="90"/>
+      <xacro:property name="velocity_limit" value="9.425"/>
     </xacro:if>
     <xacro:if value="${model_name == 'X5_4'}">
       <xacro:property name="actuator_mass" value="0.335"/>
       <xacro:property name="effort_limit" value="7.0"/>
-      <xacro:property name="velocity_limit" value="32"/>
+      <xacro:property name="velocity_limit" value="3.351"/>
     </xacro:if>
     <xacro:if value="${model_name == 'X5_9'}">
       <xacro:property name="actuator_mass" value="0.360"/>
       <xacro:property name="effort_limit" value="13.0"/>
-      <xacro:property name="velocity_limit" value="14"/>
+      <xacro:property name="velocity_limit" value="1.466"/>
     </xacro:if>
     <xacro:if value="${model_name == 'X8_3'}">
       <xacro:property name="actuator_mass" value="0.460"/>
       <xacro:property name="effort_limit" value="7"/>
-      <xacro:property name="velocity_limit" value="84"/>
+      <xacro:property name="velocity_limit" value="8.796"/>
     </xacro:if>
     <xacro:if value="${model_name == 'X8_9'}">
       <xacro:property name="actuator_mass" value="0.480"/>
       <xacro:property name="effort_limit" value="20"/>
-      <xacro:property name="velocity_limit" value="30"/>
+      <xacro:property name="velocity_limit" value="3.142"/>
     </xacro:if>
     <xacro:if value="${model_name == 'X8_16'}">
       <xacro:property name="actuator_mass" value="0.500"/>
       <xacro:property name="effort_limit" value="38"/>
-      <xacro:property name="velocity_limit" value="15"/>
+      <xacro:property name="velocity_limit" value="1.571"/>
     </xacro:if>
     <xacro:if value="${model_name == 'R8_3'}">
       <xacro:property name="actuator_mass" value="0.670"/>
       <xacro:property name="effort_limit" value="7"/>
-      <xacro:property name="velocity_limit" value="84"/>
+      <xacro:property name="velocity_limit" value="8.796"/>
     </xacro:if>
     <xacro:if value="${model_name == 'R8_9'}">
       <xacro:property name="actuator_mass" value="0.685"/>
       <xacro:property name="effort_limit" value="20"/>
-      <xacro:property name="velocity_limit" value="30"/>
+      <xacro:property name="velocity_limit" value="3.142"/>
     </xacro:if>
     <xacro:if value="${model_name == 'R8_16'}">
       <xacro:property name="actuator_mass" value="0.715"/>
       <xacro:property name="effort_limit" value="38"/>
-      <xacro:property name="velocity_limit" value="15"/>
+      <xacro:property name="velocity_limit" value="1.571"/>
     </xacro:if>
     <!-- Note: the frction/damping probably need to be tuned more for accurate simulation -->

Commit message: Working kinematic structure for Cricket robot
Some dimensions are placeholders

File: urdf/actuator.xacro (robot description, xacro)
@@ -16,45 +16,45 @@
       <xacro:property name="actuator_mass" value="0.315"/>
       <xacro:property name="effort_limit" value="2.5"/>
-      <xacro:property name="velocity_limit" value="90"/>
+      <xacro:property name="velocity_limit" value="9.425"/>
     </xacro:if>
     <xacro:if value="${model_name == 'X5_4'}">
       <xacro:property name="actuator_mass" value="0.335"/>
       <xacro:property name="effort_limit" value="7.0"/>
-      <xacro:property name="velocity_limit" value="32"/>
+      <xacro:property name="velocity_limit" value="3.351"/>
     </xacro:if>
     <xacro:if value="${model_name == 'X5_9'}">
       <xacro:property name="actuator_mass" value="0.360"/>
       <xacro:property name="effort_limit" value="13.0"/>
-      <xacro:property name="velocity_limit" value="14"/>
+      <xacro:property name="velocity_limit" value="1.466"/>
     </xacro:if>
     <xacro:if value="${model_name == 'X8_3'}">
       <xacro:property name="actuator_mass" value="0.460"/>
       <xacro:property name="effort_limit" value="7"/>
-      <xacro:property name="velocity_limit" value="84"/>
+      <xacro:property name="velocity_limit" value="8.796"/>
     </xacro:if>
     <xacro:if value="${model_name == 'X8_9'}">
       <xacro:property name="actuator_mass" value="0.480"/>
       <xacro:property name="effort_limit" value="20"/>
-      <xacro:property name="velocity_limit" value="30"/>
+      <xacro:property name="velocity_limit" value="3.142"/>
     </xacro:if>
     <xacro:if value="${model_name == 'X8_16'}">
       <xacro:property name="actuator_mass" value="0.500"/>
       <xacro:property name="effort_limit" value="38"/>
-      <xacro:property name="velocity_limit" value="15"/>
+      <xacro:property name="velocity_limit" value="1.571"/>
     </xacro:if>
     <xacro:if value="${model_name == 'R8_3'}">
       <xacro:property name="actuator_mass" value="0.670"/>
       <xacro:property name="effort_limit" value="7"/>
-      <xacro:property name="velocity_limit" value="84"/>
+      <xacro:property name="velocity_limit" value="8.796"/>
     </xacro:if>
     <xacro:if value="${model_name == 'R8_9'}">
       <xacro:property name="actuator_mass" value="0.685"/>
       <xacro:property name="effort_limit" value="20"/>
-      <xacro:property name="velocity_limit" value="30"/>
+      <xacro:property name="velocity_limit" value="3.142"/>
     </xacro:if>
     <xacro:if value="${model_name == 'R8_16'}">
       <xacro:property name="actuator_mass" value="0.715"/>
       <xacro:property name="effort_limit" value="38"/>
-      <xacro:property name="velocity_limit" value="15"/>
+      <xacro:property name="velocity_limit" value="1.571"/>
     </xacro:if>
     <!-- Note: the frction/damping probably need to be tuned more for accurate simulation -->
@@ -171,3 +171,186 @@
     </joint>
   </xacro:macro>
+  <!-- This macro is used when an actuator is "flipped" so parent feeds into input-->
+  <xacro:macro name="reverse_actuator" params="name parent:='' child:='' type limits:=${[]}">
+    <xacro:property name="model_name" value="${type}"/>
+    <!-- Continuous joints (no position limits) -->
+    <xacro:if value="${limits == []}">
+      <xacro:property name="urdf_joint_type" value="continuous"/>
+    </xacro:if>
+    <!-- Revolute joints (position limits) -->
+    <xacro:unless value="${limits == []}">
+      <xacro:property name="urdf_joint_type" value="revolute"/>
+    </xacro:unless>
+    <!-- Set properties for model of actuator -->
+    <xacro:if value="${model_name == 'X5_1'}">
+      <xacro:property name="actuator_mass" value="0.315"/>
+      <xacro:property name="effort_limit" value="2.5"/>
+      <xacro:property name="velocity_limit" value="9.425"/>
+    </xacro:if>
+    <xacro:if value="${model_name == 'X5_4'}">
+      <xacro:property name="actuator_mass" value="0.335"/>
+      <xacro:property name="effort_limit" value="7.0"/>
+      <xacro:property name="velocity_limit" value="3.351"/>
+    </xacro:if>
+    <xacro:if value="${model_name == 'X5_9'}">
+      <xacro:property name="actuator_mass" value="0.360"/>
+      <xacro:property name="effort_limit" value="13.0"/>
+      <xacro:property name="velocity_limit" value="1.466"/>
+    </xacro:if>
+    <xacro:if value="${model_name == 'X8_3'}">
+      <xacro:property name="actuator_mass" value="0.460"/>
+      <xacro:property name="effort_limit" value="7"/>
+      <xacro:property name="velocity_limit" value="8.796"/>
+    </xacro:if>
+    <xacro:if value="${model_name == 'X8_9'}">
+      <xacro:property name="actuator_mass" value="0.480"/>
+      <xacro:property name="effort_limit" value="20"/>
+      <xacro:property name="velocity_limit" value="3.142"/>
+    </xacro:if>
+    <xacro:if value="${model_name == 'X8_16'}">
+      <xacro:property name="actuator_mass" value="0.500"/>
+      <xacro:property name="effort_limit" value="38"/>
+      <xacro:property name="velocity_limit" value="1.571"/>
+    </xacro:if>
+    <xacro:if value="${model_name == 'R8_3'}">
+      <xacro:property name="actuator_mass" value="0.670"/>
+      <xacro:property name="effort_limit" value="7"/>
+      <xacro:property name="velocity_limit" value="8.796"/>
+    </xacro:if>
+    <xacro:if value="${model_name == 'R8_9'}">
+      <xacro:property name="actuator_mass" value="0.685"/>
+      <xacro:property name="effort_limit" value="20"/>
+      <xacro:property name="velocity_limit" value="3.142"/>
+    </xacro:if>
+    <xacro:if value="${model_name == 'R8_16'}">
+      <xacro:property name="actuator_mass" value="0.715"/>
+      <xacro:property name="effort_limit" value="38"/>
+      <xacro:property name="velocity_limit" value="1.571"/>
+    </xacro:if>
+    <!-- Note: the frction/damping probably need to be tuned more for accurate simulation -->
+    <xacro:if value="${model_name.startswith('X5')}">
+      <xacro:property name="mesh_filename" value="package://hebi_description/meshes/X5.stl"/>
+      <xacro:property name="damping" value="0.1"/>
+      <xacro:property name="friction" value="0.1"/>
+    </xacro:if>
+    <xacro:if value="${model_name.startswith('X8')}">
+      <xacro:property name="mesh_filename" value="package://hebi_description/meshes/X8.stl"/>
+      <xacro:property name="damping" value="0.5"/>
+      <xacro:property name="friction" value="0.5"/>
+    </xacro:if>
+    <xacro:if value="${model_name.startswith('R8')}">
+      <xacro:property name="mesh_filename" value="package://hebi_description/meshes/R8.stl"/>
+      <xacro:property name="damping" value="0.5"/>
+      <xacro:property name="friction" value="0.5"/>
+    </xacro:if>
+    <link name="${name}/INPUT_INTERFACE">
+      <visual>
+        <origin xyz="0 0 0" rpy="0 0 0" />
+        <geometry>
+          <mesh filename="${mesh_filename}" scale="0.001 0.001 0.001"/>
+        </geometry>
+        <xacro:unless value="${model_name.startswith('R8')}">
+          <xacro:red_material/>
+        </xacro:unless>
+        <xacro:if value="${model_name.startswith('R8')}">
+          <xacro:black_material/>
+        </xacro:if>
+      </visual>
+      <collision>
+        <origin xyz="0 0 0" rpy="0 0 0" />
+        <geometry>
+          <mesh filename="${mesh_filename}" scale="0.001 0.001 0.001"/>
+        </geometry>
+      </collision>
+      <inertial>
+        <mass value="${actuator_mass}"/>
+        <xacro:if value="${model_name.startswith('X5')}">
+          <origin xyz="-0.0142 -0.0031 0.0165" rpy="0 0 0" />
+          <inertia ixx="0.00015"  ixy="0.0000341"  ixz="0.0000118"
+                   iyy="0.000255" iyz="0.00000229"
+                   izz="0.000350" />
+        </xacro:if>
+        <xacro:if value="${model_name.startswith('X8')}">
+          <origin xyz="-0.0145 -0.0031 0.0242" rpy="0 0 0" />
+          <inertia ixx="0.000246" ixy="0.0000444" ixz="0.0000266"
+                   iyy="0.000380" iyz="0.00000422"
+                   izz="0.000463"/>
+        </xacro:if>
+        <xacro:if value="${model_name.startswith('R8')}">
+          <origin xyz="-0.02396 -0.00161 0.02557" rpy="0 0 0" />
+          <inertia ixx="0.000488" ixy="0.00001297" ixz="0.0000578"
+                   iyy="0.001009" iyz="0.00000494"
+                   izz="0.001186" />
+        </xacro:if>
+      </inertial>
+    </link>
+    <gazebo reference="${name}/INPUT_INTERFACE">
+      <xacro:unless value="${model_name.startswith('R8')}">
+        <xacro:gazebo_red_material/>
+      </xacro:unless>
+      <xacro:if value="${model_name.startswith('R8')}">
+        <xacro:gazebo_black_material/>
+      </xacro:if>
+    </gazebo>
+    <link name="HEBI_SIM/${name}/${model_name}">
+      <visual>
+        <origin xyz="-0.03 0 0.02" rpy="0 0 0" />
+        <geometry>
+          <sphere radius="0.001"/>
+        </geometry>
+      </visual>
+      <inertial>
+        <mass value="0.001"/>
+        <origin xyz="0 0 0" rpy="0 0 0" />
+        <inertia ixx="0.000001" ixy="0" ixz="0"
+                 iyy="0.000001" iyz="0"
+                 izz="0.000001" />
+      </inertial>
+    </link>
+    <joint name="HEBI_SIM_JOINT/${name}" type="fixed">
+      <parent link="${name}/INPUT_INTERFACE"/>
+      <child link="HEBI_SIM/${name}/${model_name}"/>
+      <origin xyz="0 0 0" rpy="0 0 0"/>
+    </joint>
+    <gazebo reference="HEBI_SIM_JOINT/${name}">
+      <disableFixedJointLumping>true</disableFixedJointLumping>
+      <preserveFixedJoint>true</preserveFixedJoint>
+    </gazebo>
+    <joint name="${name}" type="${urdf_joint_type}">
+      <parent link="${parent}/INPUT_INTERFACE"/>
+      <child link="${name}/INPUT_INTERFACE"/>
+      <xacro:if value="${model_name.startswith('X5')}">
+        <origin xyz="0 0 0.031" rpy="0 ${pi} 0"/>
+      </xacro:if>
+      <xacro:if value="${model_name.startswith('X8')}">
+        <origin xyz="0 0 0.045" rpy="0 ${pi} 0"/>
+      </xacro:if>
+      <xacro:if value="${model_name.startswith('R8')}">
+        <origin xyz="0 0 0.051" rpy="0 ${pi} 0"/>
+      </xacro:if>
+      <axis xyz="0 0 1"/>
+      <!-- Continuous joints (no position limits) -->
+      <xacro:if value="${limits == []}">
+        <limit effort="${effort_limit}" velocity="${velocity_limit}"/>
+      </xacro:if>
+      <!-- Revolute joints (position limits) -->
+      <xacro:unless value="${limits == []}">
+        <limit effort="${effort_limit}" velocity="${velocity_limit}" lower="${limits[0]}" upper="${limits[1]}"/>
+      </xacro:unless>
+      <dynamics damping="${damping}" friction="${friction}"/>
+    </joint>
+    <joint name="${name}_fixed" type="fixed">
+      <parent link="${name}/INPUT_INTERFACE"/>
+      <child link="${child}/INPUT_INTERFACE"/>
+      <xacro:if value="${model_name.startswith('X5')}">
+        <origin xyz="0 0 0" rpy="0 0 0"/>
+      </xacro:if>
+      <xacro:if value="${model_name.startswith('X8')}">
+        <origin xyz="0 0 0" rpy="0 0 0"/>
+      </xacro:if>
+      <xacro:if value="${model_name.startswith('R8')}">
+        <origin xyz="0 0 0" rpy="0 0 0"/>
+      </xacro:if>
+    </joint>
+  </xacro:macro>
 </robot>
