Commit message: Add plugin parameters to example xacros

File: urdf/actuator.xacro (robot description, xacro)
@@ -123,28 +123,4 @@
       </xacro:if>
     </gazebo>
-    <link name="HEBI_SIM/${name}/${model_name}">
-      <visual>
-        <origin xyz="-0.03 0 0.02" rpy="0 0 0" />
-        <geometry>
-          <sphere radius="0.001"/>
-        </geometry>
-      </visual>
-      <inertial>
-        <mass value="0.001"/>
-        <origin xyz="0 0 0" rpy="0 0 0" />
-        <inertia ixx="0.000001" ixy="0" ixz="0"
-                 iyy="0.000001" iyz="0"
-                 izz="0.000001" />
-      </inertial>
-    </link>
-    <joint name="HEBI_SIM_JOINT/${name}" type="fixed">
-      <parent link="${name}/INPUT_INTERFACE"/>
-      <child link="HEBI_SIM/${name}/${model_name}"/>
-      <origin xyz="0 0 0" rpy="0 0 0"/>
-    </joint>
-    <gazebo reference="HEBI_SIM_JOINT/${name}">
-      <disableFixedJointLumping>true</disableFixedJointLumping>
-      <preserveFixedJoint>true</preserveFixedJoint>
-    </gazebo>
     <joint name="${name}" type="${urdf_joint_type}">
       <parent link="${name}/INPUT_INTERFACE"/>
@@ -293,28 +269,4 @@
       </xacro:if>
     </gazebo>
-    <link name="HEBI_SIM/${name}/${model_name}">
-      <visual>
-        <origin xyz="-0.03 0 0.02" rpy="0 0 0" />
-        <geometry>
-          <sphere radius="0.001"/>
-        </geometry>
-      </visual>
-      <inertial>
-        <mass value="0.001"/>
-        <origin xyz="0 0 0" rpy="0 0 0" />
-        <inertia ixx="0.000001" ixy="0" ixz="0"
-                 iyy="0.000001" iyz="0"
-                 izz="0.000001" />
-      </inertial>
-    </link>
-    <joint name="HEBI_SIM_JOINT/${name}" type="fixed">
-      <parent link="${name}/INPUT_INTERFACE"/>
-      <child link="HEBI_SIM/${name}/${model_name}"/>
-      <origin xyz="0 0 0" rpy="0 0 0"/>
-    </joint>
-    <gazebo reference="HEBI_SIM_JOINT/${name}">
-      <disableFixedJointLumping>true</disableFixedJointLumping>
-      <preserveFixedJoint>true</preserveFixedJoint>
-    </gazebo>
     <joint name="${name}" type="${urdf_joint_type}">
       <parent link="${parent}/INPUT_INTERFACE"/>

File: urdf/bracket.xacro (robot description, xacro)
@@ -278,8 +278,4 @@
     </xacro:if>
   </joint>
-  <gazebo reference="${name}/OUTPUT_INTERFACE">
-    <disableFixedJointLumping>true</disableFixedJointLumping>
-    <preserveFixedJoint>true</preserveFixedJoint>
-  </gazebo>
   </xacro:macro>
 </robot>

File: urdf/hebi.xacro (robot description, xacro)
@@ -44,8 +44,3 @@
   <xacro:include filename="./bracket.xacro"/>
   <xacro:include filename="./end_effector.xacro"/>
-  <!-- This automatically loads the gazebo plugin for xacro models
-       which include hebi.xacro -->
-  <gazebo>
-    <plugin name="hebi_gazebo_plugin" filename="libhebi_gazebo_plugin.so"/>
-  </gazebo>
 </robot>

File: urdf/kits/A-2084-01-parallel-gripper.xacro (robot description, xacro)
@@ -3,4 +3,14 @@
   <!-- HEBI A-2084-01-parallel-gripper Arm Kit -->
   <xacro:include filename="$(find hebi_description)/urdf/hebi.xacro"/>
+  <gazebo>
+    <plugin name="hebi_gazebo_plugin" filename="libhebi_gazebo_plugin.so">
+      <actuators>
+        <actuator family="Arm" name="J1_base"     type="X5_4" mocked="false"/>
+        <actuator family="Arm" name="J2_shoulder" type="X5_9" mocked="false"/>
+        <actuator family="Arm" name="J3_elbow"    type="X5_4" mocked="false"/>
+        <actuator family="Arm" name="J4_wrist"    type="X5_1" mocked="true"/>
+      </actuators>
+    </plugin>
+  </gazebo>
   <xacro:arg name="hebi_base_frame" default="world"/>
   <xacro:property name="hebi_base_frame" value="$(arg hebi_base_frame)"/>

File: urdf/kits/A-2084-01.xacro (robot description, xacro)
@@ -3,4 +3,14 @@
   <!-- HEBI A-2084-01 Arm Kit -->
   <xacro:include filename="$(find hebi_description)/urdf/hebi.xacro"/>
+  <gazebo>
+    <plugin name="hebi_gazebo_plugin" filename="libhebi_gazebo_plugin.so">
+      <actuators>
+        <actuator family="Arm" name="J1_base"     type="X5_4" mocked="false"/>
+        <actuator family="Arm" name="J2_shoulder" type="X5_9" mocked="false"/>
+        <actuator family="Arm" name="J3_elbow"    type="X5_4" mocked="false"/>
+        <actuator family="Arm" name="J4_wrist"    type="X5_1" mocked="true"/>
+      </actuators>
+    </plugin>
+  </gazebo>
   <xacro:arg name="hebi_base_frame" default="world"/>
   <xacro:property name="hebi_base_frame" value="$(arg hebi_base_frame)"/>

File: urdf/kits/A-2085-04-parallel-gripper.xacro (robot description, xacro)
@@ -3,4 +3,14 @@
   <!-- HEBI A-2085-04-parallel-gripper Arm Kit -->
   <xacro:include filename="$(find hebi_description)/urdf/hebi.xacro"/>
+  <gazebo>
+    <plugin name="hebi_gazebo_plugin" filename="libhebi_gazebo_plugin.so">
+      <actuators>
+        <actuator family="Arm" name="J1_base"     type="X5_4" mocked="false"/>
+        <actuator family="Arm" name="J2_shoulder" type="X5_9" mocked="false"/>
+        <actuator family="Arm" name="J3_elbow"    type="X5_4" mocked="false"/>
+        <actuator family="Arm" name="J4_wrist"    type="X5_1" mocked="true"/>
+      </actuators>
+    </plugin>
+  </gazebo>
   <xacro:arg name="hebi_base_frame" default="world"/>
   <xacro:property name="hebi_base_frame" value="$(arg hebi_base_frame)"/>

File: urdf/kits/A-2085-04.xacro (robot description, xacro)
@@ -3,4 +3,14 @@
   <!-- HEBI A-2085-04 Arm Kit -->
   <xacro:include filename="$(find hebi_description)/urdf/hebi.xacro"/>
+  <gazebo>
+    <plugin name="hebi_gazebo_plugin" filename="libhebi_gazebo_plugin.so">
+      <actuators>
+        <actuator family="Arm" name="J1_base"     type="X5_4" mocked="false"/>
+        <actuator family="Arm" name="J2_shoulder" type="X5_9" mocked="false"/>
+        <actuator family="Arm" name="J3_elbow"    type="X5_4" mocked="false"/>
+        <actuator family="Arm" name="J4_wrist"    type="X5_1" mocked="true"/>
+      </actuators>
+    </plugin>
+  </gazebo>
   <xacro:arg name="hebi_base_frame" default="world"/>
   <xacro:property name="hebi_base_frame" value="$(arg hebi_base_frame)"/>

File: urdf/kits/A-2085-05-parallel-gripper.xacro (robot description, xacro)
@@ -3,4 +3,15 @@
   <!-- HEBI A-2085-05-parallel-gripper Arm Kit -->
   <xacro:include filename="$(find hebi_description)/urdf/hebi.xacro"/>
+  <gazebo>
+    <plugin name="hebi_gazebo_plugin" filename="libhebi_gazebo_plugin.so">
+      <actuators>
+        <actuator family="Arm" name="J1_base"     type="X8_9" mocked="false"/>
+        <actuator family="Arm" name="J2_shoulder" type="X8_16" mocked="false"/>
+        <actuator family="Arm" name="J3_elbow"    type="X8_9" mocked="false"/>
+        <actuator family="Arm" name="J4_wrist1"    type="X5_1" mocked="true"/>
+        <actuator family="Arm" name="J5_wrist2"    type="X5_1" mocked="true"/>
+      </actuators>
+    </plugin>
+  </gazebo>
   <xacro:arg name="hebi_base_frame" default="world"/>
   <xacro:property name="hebi_base_frame" value="$(arg hebi_base_frame)"/>

File: urdf/kits/A-2085-05.xacro (robot description, xacro)
@@ -3,4 +3,15 @@
   <!-- HEBI A-2085-05 Arm Kit -->
   <xacro:include filename="$(find hebi_description)/urdf/hebi.xacro"/>
+  <gazebo>
+    <plugin name="hebi_gazebo_plugin" filename="libhebi_gazebo_plugin.so">
+      <actuators>
+        <actuator family="Arm" name="J1_base"     type="X8_9" mocked="false"/>
+        <actuator family="Arm" name="J2_shoulder" type="X8_16" mocked="false"/>
+        <actuator family="Arm" name="J3_elbow"    type="X8_9" mocked="false"/>
+        <actuator family="Arm" name="J4_wrist1"    type="X5_1" mocked="true"/>
+        <actuator family="Arm" name="J5_wrist2"    type="X5_1" mocked="true"/>
+      </actuators>
+    </plugin>
+  </gazebo>
   <xacro:arg name="hebi_base_frame" default="world"/>
   <xacro:property name="hebi_base_frame" value="$(arg hebi_base_frame)"/>

File: urdf/kits/A-2085-06-parallel-gripper.xacro (robot description, xacro)
@@ -3,4 +3,16 @@
   <!-- HEBI A-2085-06-parallel-gripper Arm Kit -->
   <xacro:include filename="$(find hebi_description)/urdf/hebi.xacro"/>
+  <gazebo>
+    <plugin name="hebi_gazebo_plugin" filename="libhebi_gazebo_plugin.so">
+      <actuators>
+        <actuator family="Arm" name="J1_base"     type="X8_9" mocked="false"/>
+        <actuator family="Arm" name="J2_shoulder" type="X8_16" mocked="false"/>
+        <actuator family="Arm" name="J3_elbow"    type="X8_9" mocked="false"/>
+        <actuator family="Arm" name="J4_wrist1"    type="X5_1" mocked="true"/>
+        <actuator family="Arm" name="J5_wrist2"    type="X5_1" mocked="true"/>
+        <actuator family="Arm" name="J6_wrist3"    type="X5_1" mocked="true"/>
+      </actuators>
+    </plugin>
+  </gazebo>
   <xacro:arg name="hebi_base_frame" default="world"/>
   <xacro:property name="hebi_base_frame" value="$(arg hebi_base_frame)"/>

File: urdf/kits/A-2085-06.xacro (robot description, xacro)
@@ -3,4 +3,16 @@
   <!-- HEBI A-2085-06 Arm Kit -->
   <xacro:include filename="$(find hebi_description)/urdf/hebi.xacro"/>
+  <gazebo>
+    <plugin name="hebi_gazebo_plugin" filename="libhebi_gazebo_plugin.so">
+      <actuators>
+        <actuator family="Arm" name="J1_base"     type="X8_9" mocked="false"/>
+        <actuator family="Arm" name="J2_shoulder" type="X8_16" mocked="false"/>
+        <actuator family="Arm" name="J3_elbow"    type="X8_9" mocked="false"/>
+        <actuator family="Arm" name="J4_wrist1"    type="X5_1" mocked="true"/>
+        <actuator family="Arm" name="J5_wrist2"    type="X5_1" mocked="true"/>
+        <actuator family="Arm" name="J6_wrist3"    type="X5_1" mocked="true"/>
+      </actuators>
+    </plugin>
+  </gazebo>
   <xacro:arg name="hebi_base_frame" default="world"/>
   <xacro:property name="hebi_base_frame" value="$(arg hebi_base_frame)"/>

File: urdf/kits/cricket.xacro (robot description, xacro)
@@ -3,4 +3,30 @@
   <!-- HEBI Lily Hexapod Kit -->
   <xacro:include filename="$(find hebi_description)/urdf/hebi.xacro"/>
+  <gazebo>
+    <plugin name="hebi_gazebo_plugin" filename="libhebi_gazebo_plugin.so">
+      <actuators>
+        <actuator family="Cricket" name="L1_J1_shoulder1" type="X8_16" mocked="false"/>
+        <actuator family="Cricket" name="L1_J2_shoulder2" type="X8_16" mocked="false"/>
+        <actuator family="Cricket" name="L1_J3_knee"      type="X8_16" mocked="false"/>
+        <actuator family="Cricket" name="L1_J4_ankle"     type="X8_16" mocked="false"/>
+        <actuator family="Cricket" name="L1_J5_tread"     type="X8_16" mocked="false"/>
+        <actuator family="Cricket" name="L2_J1_shoulder1" type="X8_16" mocked="false"/>
+        <actuator family="Cricket" name="L2_J2_shoulder2" type="X8_16" mocked="false"/>
+        <actuator family="Cricket" name="L2_J3_knee"      type="X8_16" mocked="false"/>
+        <actuator family="Cricket" name="L2_J4_ankle"     type="X8_16" mocked="false"/>
+        <actuator family="Cricket" name="L2_J5_tread"     type="X8_16" mocked="false"/>
+        <actuator family="Cricket" name="L3_J1_shoulder1" type="X8_16" mocked="false"/>
+        <actuator family="Cricket" name="L3_J2_shoulder2" type="X8_16" mocked="false"/>
+        <actuator family="Cricket" name="L3_J3_knee"      type="X8_16" mocked="false"/>
+        <actuator family="Cricket" name="L3_J4_ankle"     type="X8_16" mocked="false"/>
+        <actuator family="Cricket" name="L3_J5_tread"     type="X8_16" mocked="false"/>
+        <actuator family="Cricket" name="L4_J1_shoulder1" type="X8_16" mocked="false"/>
+        <actuator family="Cricket" name="L4_J2_shoulder2" type="X8_16" mocked="false"/>
+        <actuator family="Cricket" name="L4_J3_knee"      type="X8_16" mocked="false"/>
+        <actuator family="Cricket" name="L4_J4_ankle"     type="X8_16" mocked="false"/>
+        <actuator family="Cricket" name="L4_J5_tread"     type="X8_16" mocked="false"/>
+      </actuators>
+    </plugin>
+  </gazebo>
   <xacro:macro name="rigid_body" params="mass size output_trans output_rot:='0 0 0' name child">
     <xacro:property name="output_trans_prop" value="${[float(x) for x in output_trans.split(' ')]}"/>
@@ -41,5 +67,5 @@
     <link name="${name}/INPUT_INTERFACE">
       <visual>
-        <origin xyz="0 0 0" rpy="0 0 0" />
+        <origin xyz="0 0 0.020" rpy="0 0 0" />
         <geometry>
           <cylinder radius="${radius}" length="${width}"/>
@@ -48,5 +74,5 @@
       </visual>
       <collision>
-        <origin xyz="0 0 0" rpy="0 0 0" />
+        <origin xyz="0 0 0.020" rpy="0 0 0" />
         <geometry>
           <cylinder radius="${radius}" length="${width}"/>
@@ -65,5 +91,5 @@
     <link name="${name}">
       <visual>
-        <origin xyz="0 0 ${-width}" rpy="0 0 0" />
+        <origin xyz="0.0 0.0 -0.03" rpy="0 0 0" />
         <geometry>
           <cylinder radius="${radius}" length="${width}"/>
@@ -83,4 +109,5 @@
       <parent link="${parent}/INPUT_INTERFACE"/>
       <child link="${name}"/>
+      <axis xyz="0 0 1"/>
     </joint>
   </xacro:macro>
@@ -128,5 +155,5 @@
     <xacro:drive_pulley mass="0.1" radius="0.068" width="0.033" name="leg${leg_num}_drive_pulley"/>
     <xacro:idle_pulley mass="0.1" radius="0.068" width="0.033"
-	    name="leg${leg_num}_drive_pulley" parent="leg${leg_num}_tread_bracket_1"/>
+	    name="leg${leg_num}_idle_pulley" parent="${family}/L${leg_num}_J4_ankle"/>
   </xacro:macro>
   <link name="cricket_base">
@@ -155,6 +182,6 @@
   </link>
   <joint name="cricket_base_inertia_joint" type="fixed">
-	  <parent link="cricket_base"/>
-	  <child link="cricket_base_inertia"/>
+    <parent link="cricket_base"/>
+    <child link="cricket_base_inertia"/>
   </joint>
   <xacro:cricket_leg type="left"  family="Cricket" leg_num="1" angle="${-pi/2} 0 0" offset="0.135 0.100 0.030" />

File: urdf/link.xacro (robot description, xacro)
@@ -126,8 +126,4 @@
       </xacro:if>
     </joint>
-    <gazebo reference="${name}/OUTPUT_JOINT">
-      <disableFixedJointLumping>true</disableFixedJointLumping>
-      <preserveFixedJoint>true</preserveFixedJoint>
-    </gazebo>
   </xacro:macro>
 </robot>

Commit message: Cwbollinger/update plugin urdf (#18)
* Update xacros for new plugin parameter

* Add plugin parameters to example xacros

* Update generator script to include new plugin parameters

File: urdf/actuator.xacro (robot description, xacro)
@@ -123,28 +123,4 @@
       </xacro:if>
     </gazebo>
-    <link name="HEBI_SIM/${name}/${model_name}">
-      <visual>
-        <origin xyz="-0.03 0 0.02" rpy="0 0 0" />
-        <geometry>
-          <sphere radius="0.001"/>
-        </geometry>
-      </visual>
-      <inertial>
-        <mass value="0.001"/>
-        <origin xyz="0 0 0" rpy="0 0 0" />
-        <inertia ixx="0.000001" ixy="0" ixz="0"
-                 iyy="0.000001" iyz="0"
-                 izz="0.000001" />
-      </inertial>
-    </link>
-    <joint name="HEBI_SIM_JOINT/${name}" type="fixed">
-      <parent link="${name}/INPUT_INTERFACE"/>
-      <child link="HEBI_SIM/${name}/${model_name}"/>
-      <origin xyz="0 0 0" rpy="0 0 0"/>
-    </joint>
-    <gazebo reference="HEBI_SIM_JOINT/${name}">
-      <disableFixedJointLumping>true</disableFixedJointLumping>
-      <preserveFixedJoint>true</preserveFixedJoint>
-    </gazebo>
     <joint name="${name}" type="${urdf_joint_type}">
       <parent link="${name}/INPUT_INTERFACE"/>
@@ -171,3 +147,162 @@
     </joint>
   </xacro:macro>
+  <!-- This macro is used when an actuator is "flipped" so parent feeds into input-->
+  <xacro:macro name="reverse_actuator" params="name parent:='' child:='' type limits:=${[]}">
+    <xacro:property name="model_name" value="${type}"/>
+    <!-- Continuous joints (no position limits) -->
+    <xacro:if value="${limits == []}">
+      <xacro:property name="urdf_joint_type" value="continuous"/>
+    </xacro:if>
+    <!-- Revolute joints (position limits) -->
+    <xacro:unless value="${limits == []}">
+      <xacro:property name="urdf_joint_type" value="revolute"/>
+    </xacro:unless>
+    <!-- Set properties for model of actuator -->
+    <xacro:if value="${model_name == 'X5_1'}">
+      <xacro:property name="actuator_mass" value="0.315"/>
+      <xacro:property name="effort_limit" value="2.5"/>
+      <xacro:property name="velocity_limit" value="9.425"/>
+    </xacro:if>
+    <xacro:if value="${model_name == 'X5_4'}">
+      <xacro:property name="actuator_mass" value="0.335"/>
+      <xacro:property name="effort_limit" value="7.0"/>
+      <xacro:property name="velocity_limit" value="3.351"/>
+    </xacro:if>
+    <xacro:if value="${model_name == 'X5_9'}">
+      <xacro:property name="actuator_mass" value="0.360"/>
+      <xacro:property name="effort_limit" value="13.0"/>
+      <xacro:property name="velocity_limit" value="1.466"/>
+    </xacro:if>
+    <xacro:if value="${model_name == 'X8_3'}">
+      <xacro:property name="actuator_mass" value="0.460"/>
+      <xacro:property name="effort_limit" value="7"/>
+      <xacro:property name="velocity_limit" value="8.796"/>
+    </xacro:if>
+    <xacro:if value="${model_name == 'X8_9'}">
+      <xacro:property name="actuator_mass" value="0.480"/>
+      <xacro:property name="effort_limit" value="20"/>
+      <xacro:property name="velocity_limit" value="3.142"/>
+    </xacro:if>
+    <xacro:if value="${model_name == 'X8_16'}">
+      <xacro:property name="actuator_mass" value="0.500"/>
+      <xacro:property name="effort_limit" value="38"/>
+      <xacro:property name="velocity_limit" value="1.571"/>
+    </xacro:if>
+    <xacro:if value="${model_name == 'R8_3'}">
+      <xacro:property name="actuator_mass" value="0.670"/>
+      <xacro:property name="effort_limit" value="7"/>
+      <xacro:property name="velocity_limit" value="8.796"/>
+    </xacro:if>
+    <xacro:if value="${model_name == 'R8_9'}">
+      <xacro:property name="actuator_mass" value="0.685"/>
+      <xacro:property name="effort_limit" value="20"/>
+      <xacro:property name="velocity_limit" value="3.142"/>
+    </xacro:if>
+    <xacro:if value="${model_name == 'R8_16'}">
+      <xacro:property name="actuator_mass" value="0.715"/>
+      <xacro:property name="effort_limit" value="38"/>
+      <xacro:property name="velocity_limit" value="1.571"/>
+    </xacro:if>
+    <!-- Note: the frction/damping probably need to be tuned more for accurate simulation -->
+    <xacro:if value="${model_name.startswith('X5')}">
+      <xacro:property name="mesh_filename" value="package://hebi_description/meshes/X5.stl"/>
+      <xacro:property name="damping" value="0.1"/>
+      <xacro:property name="friction" value="0.1"/>
+    </xacro:if>
+    <xacro:if value="${model_name.startswith('X8')}">
+      <xacro:property name="mesh_filename" value="package://hebi_description/meshes/X8.stl"/>
+      <xacro:property name="damping" value="0.5"/>
+      <xacro:property name="friction" value="0.5"/>
+    </xacro:if>
+    <xacro:if value="${model_name.startswith('R8')}">
+      <xacro:property name="mesh_filename" value="package://hebi_description/meshes/R8.stl"/>
+      <xacro:property name="damping" value="0.5"/>
+      <xacro:property name="friction" value="0.5"/>
+    </xacro:if>
+    <link name="${name}/INPUT_INTERFACE">
+      <visual>
+        <origin xyz="0 0 0" rpy="0 0 0" />
+        <geometry>
+          <mesh filename="${mesh_filename}" scale="0.001 0.001 0.001"/>
+        </geometry>
+        <xacro:unless value="${model_name.startswith('R8')}">
+          <xacro:red_material/>
+        </xacro:unless>
+        <xacro:if value="${model_name.startswith('R8')}">
+          <xacro:black_material/>
+        </xacro:if>
+      </visual>
+      <collision>
+        <origin xyz="0 0 0" rpy="0 0 0" />
+        <geometry>
+          <mesh filename="${mesh_filename}" scale="0.001 0.001 0.001"/>
+        </geometry>
+      </collision>
+      <inertial>
+        <mass value="${actuator_mass}"/>
+        <xacro:if value="${model_name.startswith('X5')}">
+          <origin xyz="-0.0142 -0.0031 0.0165" rpy="0 0 0" />
+          <inertia ixx="0.00015"  ixy="0.0000341"  ixz="0.0000118"
+                   iyy="0.000255" iyz="0.00000229"
+                   izz="0.000350" />
+        </xacro:if>
+        <xacro:if value="${model_name.startswith('X8')}">
+          <origin xyz="-0.0145 -0.0031 0.0242" rpy="0 0 0" />
+          <inertia ixx="0.000246" ixy="0.0000444" ixz="0.0000266"
+                   iyy="0.000380" iyz="0.00000422"
+                   izz="0.000463"/>
+        </xacro:if>
+        <xacro:if value="${model_name.startswith('R8')}">
+          <origin xyz="-0.02396 -0.00161 0.02557" rpy="0 0 0" />
+          <inertia ixx="0.000488" ixy="0.00001297" ixz="0.0000578"
+                   iyy="0.001009" iyz="0.00000494"
+                   izz="0.001186" />
+        </xacro:if>
+      </inertial>
+    </link>
+    <gazebo reference="${name}/INPUT_INTERFACE">
+      <xacro:unless value="${model_name.startswith('R8')}">
+        <xacro:gazebo_red_material/>
+      </xacro:unless>
+      <xacro:if value="${model_name.startswith('R8')}">
+        <xacro:gazebo_black_material/>
+      </xacro:if>
+    </gazebo>
+    <joint name="${name}" type="${urdf_joint_type}">
+      <parent link="${parent}/INPUT_INTERFACE"/>
+      <child link="${name}/INPUT_INTERFACE"/>
+      <xacro:if value="${model_name.startswith('X5')}">
+        <origin xyz="0 0 0.031" rpy="0 ${pi} 0"/>
+      </xacro:if>
+      <xacro:if value="${model_name.startswith('X8')}">
+        <origin xyz="0 0 0.045" rpy="0 ${pi} 0"/>
+      </xacro:if>
+      <xacro:if value="${model_name.startswith('R8')}">
+        <origin xyz="0 0 0.051" rpy="0 ${pi} 0"/>
+      </xacro:if>
+      <axis xyz="0 0 1"/>
+      <!-- Continuous joints (no position limits) -->
+      <xacro:if value="${limits == []}">
+        <limit effort="${effort_limit}" velocity="${velocity_limit}"/>
+      </xacro:if>
+      <!-- Revolute joints (position limits) -->
+      <xacro:unless value="${limits == []}">
+        <limit effort="${effort_limit}" velocity="${velocity_limit}" lower="${limits[0]}" upper="${limits[1]}"/>
+      </xacro:unless>
+      <dynamics damping="${damping}" friction="${friction}"/>
+    </joint>
+    <joint name="${name}_fixed" type="fixed">
+      <parent link="${name}/INPUT_INTERFACE"/>
+      <child link="${child}/INPUT_INTERFACE"/>
+      <xacro:if value="${model_name.startswith('X5')}">
+        <origin xyz="0 0 0" rpy="0 0 0"/>
+      </xacro:if>
+      <xacro:if value="${model_name.startswith('X8')}">
+        <origin xyz="0 0 0" rpy="0 0 0"/>
+      </xacro:if>
+      <xacro:if value="${model_name.startswith('R8')}">
+        <origin xyz="0 0 0" rpy="0 0 0"/>
+      </xacro:if>
+    </joint>
+  </xacro:macro>
 </robot>

Commit message: Fix rotation direction of inverse actuator URDF

File: urdf/actuator.xacro (robot description, xacro)
@@ -281,5 +281,5 @@
         <origin xyz="0 0 0.051" rpy="0 ${pi} 0"/>
       </xacro:if>
-      <axis xyz="0 0 1"/>
+      <axis xyz="0 0 -1"/>
       <!-- Continuous joints (no position limits) -->
       <xacro:if value="${limits == []}">
