Commit message: Sort of stable behavior in Copellia

File: urdf/actuator.xacro (robot description, xacro)
@@ -14,45 +14,45 @@
     <!-- Set properties for model of actuator -->
     <xacro:if value="${model_name == 'X5_1'}">
-      <xacro:property name="actuator_mass" value="0.315"/>
+      <xacro:property name="actuator_mass" value="1.0"/>
       <xacro:property name="effort_limit" value="2.5"/>
       <xacro:property name="velocity_limit" value="9.425"/>
     </xacro:if>
     <xacro:if value="${model_name == 'X5_4'}">
-      <xacro:property name="actuator_mass" value="0.335"/>
+      <xacro:property name="actuator_mass" value="1.0"/>
       <xacro:property name="effort_limit" value="7.0"/>
       <xacro:property name="velocity_limit" value="3.351"/>
     </xacro:if>
     <xacro:if value="${model_name == 'X5_9'}">
-      <xacro:property name="actuator_mass" value="0.360"/>
+      <xacro:property name="actuator_mass" value="1.0"/>
       <xacro:property name="effort_limit" value="13.0"/>
       <xacro:property name="velocity_limit" value="1.466"/>
     </xacro:if>
     <xacro:if value="${model_name == 'X8_3'}">
-      <xacro:property name="actuator_mass" value="0.460"/>
+      <xacro:property name="actuator_mass" value="1.0"/>
       <xacro:property name="effort_limit" value="7"/>
       <xacro:property name="velocity_limit" value="8.796"/>
     </xacro:if>
     <xacro:if value="${model_name == 'X8_9'}">
-      <xacro:property name="actuator_mass" value="0.480"/>
+      <xacro:property name="actuator_mass" value="1.0"/>
       <xacro:property name="effort_limit" value="20"/>
       <xacro:property name="velocity_limit" value="3.142"/>
     </xacro:if>
     <xacro:if value="${model_name == 'X8_16'}">
-      <xacro:property name="actuator_mass" value="0.500"/>
+      <xacro:property name="actuator_mass" value="1.0"/>
       <xacro:property name="effort_limit" value="38"/>
       <xacro:property name="velocity_limit" value="1.571"/>
     </xacro:if>
     <xacro:if value="${model_name == 'R8_3'}">
-      <xacro:property name="actuator_mass" value="0.670"/>
+      <xacro:property name="actuator_mass" value="1.0"/>
       <xacro:property name="effort_limit" value="7"/>
       <xacro:property name="velocity_limit" value="8.796"/>
     </xacro:if>
     <xacro:if value="${model_name == 'R8_9'}">
-      <xacro:property name="actuator_mass" value="0.685"/>
+      <xacro:property name="actuator_mass" value="1.0"/>
       <xacro:property name="effort_limit" value="20"/>
       <xacro:property name="velocity_limit" value="3.142"/>
     </xacro:if>
     <xacro:if value="${model_name == 'R8_16'}">
-      <xacro:property name="actuator_mass" value="0.715"/>
+      <xacro:property name="actuator_mass" value="1.0"/>
       <xacro:property name="effort_limit" value="38"/>
       <xacro:property name="velocity_limit" value="1.571"/>
@@ -61,4 +61,6 @@
     <xacro:if value="${model_name.startswith('X5')}">
       <xacro:property name="mesh_filename" value="package://hebi_description/meshes/X5.stl"/>
+      <xacro:property name="collision_box_origin" value="-0.0185 0 0.0155"/>
+      <xacro:property name="collision_box_size" value="0.110 0.073 0.031"/>
       <xacro:property name="damping" value="0.1"/>
       <xacro:property name="friction" value="0.1"/>
@@ -66,4 +68,6 @@
     <xacro:if value="${model_name.startswith('X8')}">
       <xacro:property name="mesh_filename" value="package://hebi_description/meshes/X8.stl"/>
+      <xacro:property name="collision_box_origin" value="-0.0185 0 0.0225"/>
+      <xacro:property name="collision_box_size" value="0.110 0.073 0.045"/>
       <xacro:property name="damping" value="0.5"/>
       <xacro:property name="friction" value="0.5"/>
@@ -71,4 +75,6 @@
     <xacro:if value="${model_name.startswith('R8')}">
       <xacro:property name="mesh_filename" value="package://hebi_description/meshes/R8.stl"/>
+      <xacro:property name="collision_box_origin" value="-0.039 0.0 0.0255"/>
+      <xacro:property name="collision_box_size" value="0.156 0.078 0.051"/>
       <xacro:property name="damping" value="0.5"/>
       <xacro:property name="friction" value="0.5"/>
@@ -88,7 +94,7 @@
       </visual>
       <collision>
-        <origin xyz="0 0 0" rpy="0 0 0" />
+        <origin xyz="${collision_box_origin}" rpy="0 0 0" />
         <geometry>
-          <mesh filename="${mesh_filename}" scale="0.001 0.001 0.001"/>
+	  <box size="${collision_box_size}"/>
         </geometry>
       </collision>
@@ -97,30 +103,22 @@
         <xacro:if value="${model_name.startswith('X5')}">
           <origin xyz="-0.0142 -0.0031 0.0165" rpy="0 0 0" />
-          <inertia ixx="0.00015"  ixy="0.0000341"  ixz="0.0000118"
-                   iyy="0.000255" iyz="0.00000229"
-                   izz="0.000350" />
+          <inertia ixx="0.001" ixy="0.0"  ixz="0.0"
+                   iyy="0.001" iyz="0.0"
+                   izz="0.001" />
         </xacro:if>
         <xacro:if value="${model_name.startswith('X8')}">
           <origin xyz="-0.0145 -0.0031 0.0242" rpy="0 0 0" />
-          <inertia ixx="0.000246" ixy="0.0000444" ixz="0.0000266"
-                   iyy="0.000380" iyz="0.00000422"
-                   izz="0.000463"/>
+          <inertia ixx="0.001" ixy="0.0" ixz="0.0"
+                   iyy="0.001" iyz="0.0"
+                   izz="0.001"/>
         </xacro:if>
         <xacro:if value="${model_name.startswith('R8')}">
           <origin xyz="-0.02396 -0.00161 0.02557" rpy="0 0 0" />
-          <inertia ixx="0.000488" ixy="0.00001297" ixz="0.0000578"
-                   iyy="0.001009" iyz="0.00000494"
-                   izz="0.001186" />
+          <inertia ixx="0.001" ixy="0.0" ixz="0.0"
+                   iyy="0.001" iyz="0.0"
+                   izz="0.001" />
         </xacro:if>
       </inertial>
     </link>
-    <gazebo reference="${name}/INPUT_INTERFACE">
-      <xacro:unless value="${model_name.startswith('R8')}">
-        <xacro:gazebo_red_material/>
-      </xacro:unless>
-      <xacro:if value="${model_name.startswith('R8')}">
-        <xacro:gazebo_black_material/>
-      </xacro:if>
-    </gazebo>
     <joint name="${name}" type="${urdf_joint_type}">
       <parent link="${name}/INPUT_INTERFACE"/>
@@ -160,45 +158,45 @@
     <!-- Set properties for model of actuator -->
     <xacro:if value="${model_name == 'X5_1'}">
-      <xacro:property name="actuator_mass" value="0.315"/>
+      <xacro:property name="actuator_mass" value="1.0"/>
       <xacro:property name="effort_limit" value="2.5"/>
       <xacro:property name="velocity_limit" value="9.425"/>
     </xacro:if>
     <xacro:if value="${model_name == 'X5_4'}">
-      <xacro:property name="actuator_mass" value="0.335"/>
+      <xacro:property name="actuator_mass" value="1.0"/>
       <xacro:property name="effort_limit" value="7.0"/>
       <xacro:property name="velocity_limit" value="3.351"/>
     </xacro:if>
     <xacro:if value="${model_name == 'X5_9'}">
-      <xacro:property name="actuator_mass" value="0.360"/>
+      <xacro:property name="actuator_mass" value="1.0"/>
       <xacro:property name="effort_limit" value="13.0"/>
       <xacro:property name="velocity_limit" value="1.466"/>
     </xacro:if>
     <xacro:if value="${model_name == 'X8_3'}">
-      <xacro:property name="actuator_mass" value="0.460"/>
+      <xacro:property name="actuator_mass" value="1.0"/>
       <xacro:property name="effort_limit" value="7"/>
       <xacro:property name="velocity_limit" value="8.796"/>
     </xacro:if>
     <xacro:if value="${model_name == 'X8_9'}">
-      <xacro:property name="actuator_mass" value="0.480"/>
+      <xacro:property name="actuator_mass" value="1.0"/>
       <xacro:property name="effort_limit" value="20"/>
       <xacro:property name="velocity_limit" value="3.142"/>
     </xacro:if>
     <xacro:if value="${model_name == 'X8_16'}">
-      <xacro:property name="actuator_mass" value="0.500"/>
+      <xacro:property name="actuator_mass" value="1.0"/>
       <xacro:property name="effort_limit" value="38"/>
       <xacro:property name="velocity_limit" value="1.571"/>
     </xacro:if>
     <xacro:if value="${model_name == 'R8_3'}">
-      <xacro:property name="actuator_mass" value="0.670"/>
+      <xacro:property name="actuator_mass" value="1.0"/>
       <xacro:property name="effort_limit" value="7"/>
       <xacro:property name="velocity_limit" value="8.796"/>
     </xacro:if>
     <xacro:if value="${model_name == 'R8_9'}">
-      <xacro:property name="actuator_mass" value="0.685"/>
+      <xacro:property name="actuator_mass" value="1.0"/>
       <xacro:property name="effort_limit" value="20"/>
       <xacro:property name="velocity_limit" value="3.142"/>
     </xacro:if>
     <xacro:if value="${model_name == 'R8_16'}">
-      <xacro:property name="actuator_mass" value="0.715"/>
+      <xacro:property name="actuator_mass" value="1.0"/>
       <xacro:property name="effort_limit" value="38"/>
       <xacro:property name="velocity_limit" value="1.571"/>
@@ -207,4 +205,5 @@
     <xacro:if value="${model_name.startswith('X5')}">
       <xacro:property name="mesh_filename" value="package://hebi_description/meshes/X5.stl"/>
+      <xacro:property name="collision_box_size" value="0.031 0.073 0.110"/>
       <xacro:property name="damping" value="0.1"/>
       <xacro:property name="friction" value="0.1"/>
@@ -212,4 +211,5 @@
     <xacro:if value="${model_name.startswith('X8')}">
       <xacro:property name="mesh_filename" value="package://hebi_description/meshes/X8.stl"/>
+      <xacro:property name="collision_box_size" value="0.045 0.073 0.110"/>
       <xacro:property name="damping" value="0.5"/>
       <xacro:property name="friction" value="0.5"/>
@@ -217,4 +217,5 @@
     <xacro:if value="${model_name.startswith('R8')}">
       <xacro:property name="mesh_filename" value="package://hebi_description/meshes/R8.stl"/>
+      <xacro:property name="collision_box_size" value="0.051 0.078 0.156"/>
       <xacro:property name="damping" value="0.5"/>
       <xacro:property name="friction" value="0.5"/>
@@ -236,5 +237,5 @@
         <origin xyz="0 0 0" rpy="0 0 0" />
         <geometry>
-          <mesh filename="${mesh_filename}" scale="0.001 0.001 0.001"/>
+	  <box size="${collision_box_size}"/>
         </geometry>
       </collision>
@@ -261,12 +262,4 @@
       </inertial>
     </link>
-    <gazebo reference="${name}/INPUT_INTERFACE">
-      <xacro:unless value="${model_name.startswith('R8')}">
-        <xacro:gazebo_red_material/>
-      </xacro:unless>
-      <xacro:if value="${model_name.startswith('R8')}">
-        <xacro:gazebo_black_material/>
-      </xacro:if>
-    </gazebo>
     <joint name="${name}" type="${urdf_joint_type}">
       <parent link="${parent}/INPUT_INTERFACE"/>

File: urdf/bracket.xacro (robot description, xacro)
@@ -43,5 +43,5 @@
           <origin xyz="0 -.0215 .02" rpy="0 0 0" />
         </xacro:if>
-        <mass value="0.1"/>
+        <mass value="1.0"/>
         <inertia ixx="${0.4 * 0.1 * 0.06 * 0.06}" ixy="0.0" ixz="0.0" iyy="${0.4 * 0.1 * 0.06 * 0.06}" iyz="0.0" izz="${0.4 * 0.1 * 0.06 * 0.06}"/>
       </inertial>
@@ -79,5 +79,5 @@
           <origin xyz="0 -.0215 .02" rpy="0 0 0" />
         </xacro:if>
-        <mass value="0.1"/>
+        <mass value="1.0"/>
         <inertia ixx="${0.4 * 0.1 * 0.06 * 0.06}" ixy="0.0" ixz="0.0" iyy="${0.4 * 0.1 * 0.06 * 0.06}" iyz="0.0" izz="${0.4 * 0.1 * 0.06 * 0.06}"/>
       </inertial>
@@ -179,5 +179,5 @@
           <origin xyz="0 ${0.5 * -.0225} .0275" rpy="0 0 0" />
         </xacro:if>
-        <mass value="0.215"/>
+        <mass value="1.0"/>
         <inertia ixx="${0.4 * 0.215 * 0.06 * 0.06}" ixy="0.0" ixz="0.0" iyy="${0.4 * 0.215 * 0.06 * 0.06}" iyz="0.0" izz="${0.4 * 0.215 * 0.06 * 0.06}"/>
       </inertial>
@@ -209,23 +209,27 @@
       <collision>
         <xacro:if value="${bracket_type.endswith('RightOutside')}">
-          <origin xyz="0 0 0.005" rpy="${pi/2} 0 ${pi/2}"/>
-        </xacro:if>
-        <xacro:if value="${bracket_type.endswith('RightInside')}">
-          <origin xyz="0 0 0.005" rpy="${pi/2} 0 ${-pi/2}"/>
-        </xacro:if>
-        <xacro:if value="${bracket_type.endswith('LeftOutside')}">
-          <origin xyz="0 0 0.005" rpy="${pi/2} 0 ${-pi/2}"/>
-        </xacro:if>
-        <xacro:if value="${bracket_type.endswith('LeftInside')}">
-          <origin xyz="0 0 0.005" rpy="${pi/2} 0 ${pi/2}"/>
-        </xacro:if>
-        <geometry>
-          <xacro:if value="${bracket_type.endswith('Outside')}">
-            <mesh filename="package://hebi_description/meshes/A-2221-01-Outside.stl" scale="0.001 0.001 0.001"/>
-          </xacro:if>
-          <xacro:if value="${bracket_type.endswith('Inside')}">
-            <mesh filename="package://hebi_description/meshes/A-2221-01-Inside.stl" scale="0.001 0.001 0.001"/>
-          </xacro:if>
-        </geometry>
+          <origin xyz="0 -0.032 0.045" rpy="0 0 0"/>
+          <geometry>
+	    <box size="0.10 0.01 0.09"/>
+          </geometry>
+        </xacro:if>
+        <xacro:if value="${bracket_type.endswith('RightInside')}">
+          <origin xyz="0 0.028 0.045" rpy="0 0 0"/>
+          <geometry>
+	    <box size="0.10 0.01 0.09"/>
+          </geometry>
+        </xacro:if>
+        <xacro:if value="${bracket_type.endswith('LeftOutside')}">
+          <origin xyz="0 0.032 0.045" rpy="0 0 0"/>
+          <geometry>
+	    <box size="0.10 0.01 0.09"/>
+          </geometry>
+        </xacro:if>
+        <xacro:if value="${bracket_type.endswith('LeftInside')}">
+          <origin xyz="0 -0.028 0.045" rpy="0 0 0"/>
+          <geometry>
+	    <box size="0.10 0.01 0.09"/>
+          </geometry>
+        </xacro:if>
       </collision>
       <!-- NOTE: inertia is just modelled as small sphere, and could be improved. -->
@@ -243,17 +247,9 @@
           <origin xyz="0 ${0.5 * -.0225} .0275" rpy="0 0 0" />
         </xacro:if>
-        <mass value="0.215"/>
+        <mass value="1.0"/>
         <inertia ixx="${0.4 * 0.215 * 0.06 * 0.06}" ixy="0.0" ixz="0.0" iyy="${0.4 * 0.215 * 0.06 * 0.06}" iyz="0.0" izz="${0.4 * 0.215 * 0.06 * 0.06}"/>
       </inertial>
     </xacro:if>
   </link>
-  <gazebo reference="${name}/INPUT_INTERFACE">
-    <xacro:if value="${bracket_type.startswith('X5Light')}">
-      <xacro:gazebo_beige_material/>
-    </xacro:if>
-    <xacro:if value="${bracket_type.startswith('X5Heavy') or bracket_type.startswith('R8')}">
-      <xacro:gazebo_black_material/>
-    </xacro:if>
-  </gazebo>
   <joint name="${name}/OUTPUT_INTERFACE" type="fixed">
     <parent link="${name}/INPUT_INTERFACE"/>

File: urdf/end_effector.xacro (robot description, xacro)
@@ -51,7 +51,4 @@
       <self_collide>true</self_collide>
     </link>
-    <gazebo reference="${name}/${prefix}_finger">
-      <xacro:gazebo_silver_material/>
-    </gazebo>
     <link name="${name}/${prefix}_outer_linkage">
       <visual>
@@ -72,7 +69,4 @@
       </inertial>
     </link>
-    <gazebo reference="${name}/${prefix}_outer_linkage">
-      <xacro:gazebo_black_material/>
-    </gazebo>
     <link name="${name}/${prefix}_gripper">
       <visual>
@@ -98,7 +92,4 @@
       </inertial>
     </link>
-    <gazebo reference="${name}/${prefix}_gripper">
-      <xacro:gazebo_black_material/>
-    </gazebo>
     <link name="${name}/${prefix}_gripper_bend">
       <visual>
@@ -119,7 +110,4 @@
       </inertial>
     </link>
-    <gazebo reference="${name}/${prefix}_gripper_bend">
-      <xacro:gazebo_silver_material/>
-    </gazebo>
     <joint name="${name}/${prefix}_gripper_finger_${prefix}_gripper_bend" type="fixed">
       <origin xyz="0.0 -0.0075 0.0165" rpy="0 0 0" />
@@ -127,8 +115,4 @@
       <child link="${name}/${prefix}_gripper_bend"/>
     </joint>
-    <gazebo reference="${name}/${prefix}_gripper_finger_${prefix}_gripper_bend">
-      <disableFixedJointLumping>true</disableFixedJointLumping>
-      <preserveFixedJoint>true</preserveFixedJoint>
-    </gazebo>
     <joint name="${name}/input_${prefix}_finger" type="revolute">
       <xacro:if value="${prefix == 'l'}">
@@ -143,11 +127,4 @@
       <limit effort="1000" velocity="1000" lower="0" upper="${0.37*pi}"/>
     </joint>
-    <gazebo reference="${name}/input_${prefix}_finger">
-      <physics>
-        <ode>
-          <implicit_spring_damper>true</implicit_spring_damper>
-        </ode>
-      </physics>
-    </gazebo>
     <joint name="${name}/${prefix}_finger_${prefix}_outer_linkage" type="fixed">
       <origin xyz="0 0.015 0" rpy="0 0 0" />
@@ -182,7 +159,4 @@
       </inertial>
     </link>
-    <gazebo reference="${name}/${prefix}_inner_linkage">
-      <xacro:gazebo_black_material />
-    </gazebo>
     <joint name="${name}/center_hub_${prefix}_inner_linkage" type="continuous">
       <xacro:if value="${prefix == 'l'}">
@@ -243,7 +217,4 @@
         </inertial>
       </link>
-      <gazebo reference="${name}/INPUT_INTERFACE">
-        <xacro:gazebo_black_material/>
-      </gazebo>
       <!-- Tree branch for center hub -->
       <link name="${name}/center_hub">
@@ -265,7 +236,4 @@
         </inertial>
       </link>
-      <gazebo reference="${name}/center_hub">
-        <xacro:gazebo_black_material/>
-      </gazebo>
       <joint name="${name}/input_center_hub" type="fixed">
         <origin xyz="0 0 0.0045" rpy="0 0 0" />
@@ -297,8 +265,4 @@
         </inertial>
       </link>
-      <gazebo reference="${name}/center_pinion">
-        <self_collide>true</self_collide>
-        <xacro:gazebo_silver_material/>
-      </gazebo>
       <joint name="${name}/center_hub_pinion" type="prismatic">
         <parent link="${name}/center_hub"/>
@@ -307,5 +271,5 @@
         <axis xyz="0 0 1" />
         <limit effort="1000" velocity="1000" lower="-1.0" upper="1.0"/>
-        <!-- Don't actually want the pinion to move (only needed fore gazebo)
+        <!-- Don't actually want the pinion to move (only needed for gazebo)
              so set multiplier very small -->
         <mimic joint="${name}/input_l_finger" multiplier="0.00001" offset="0" />
@@ -316,8 +280,4 @@
         </physics>
       </joint>
-      <gazebo reference="${name}/center_hub_pinion">
-        <disableFixedJointLumping>true</disableFixedJointLumping>
-        <preserveFixedJoint>true</preserveFixedJoint>
-      </gazebo>
       <!-- Tree branches for fingers, outer linkages, and grippers -->
       <xacro:parallel_gripper_outer_subassembly name="${name}" prefix="l"/>
@@ -326,47 +286,4 @@
       <xacro:parallel_gripper_inner_subassembly name="${name}" prefix="l"/>
       <xacro:parallel_gripper_inner_subassembly name="${name}" prefix="r"/>
-      <gazebo>
-        <joint name="${name}/l_inner_outer_pin" type="revolute">
-          <pose>0 0 0.0439 0 0 0</pose>
-          <parent>${name}/l_gripper_bend</parent>
-          <child>${name}/l_inner_linkage</child>
-          <axis>
-            <xyz>-1 0 0</xyz>
-            <limit>
-              <lower>${-2*pi}</lower>
-              <upper>${2*pi}</upper>
-              <effort>1000</effort>
-              <velocity>1000</velocity>
-            </limit>
-          </axis>
-        </joint>
-        <joint name="${name}/r_inner_outer_pin" type="revolute">
-          <pose>0 0 0.0439 0 0 0</pose>
-          <parent>${name}/r_gripper_bend</parent>
-          <child>${name}/r_inner_linkage</child>
-          <axis>
-            <xyz>-1 0 0</xyz>
-            <limit>
-              <lower>${-2*pi}</lower>
-              <upper>${2*pi}</upper>
-              <effort>1000</effort>
-              <velocity>1000</velocity>
-            </limit>
-          </axis>
-        </joint>
-        <!-- Add constraint between gripper fingers (they mirror each other) using a gearbox -->
-        <joint name="${name}/finger_gearbox" type="gearbox">
-          <parent>${name}/r_finger</parent>
-          <child>${name}/l_finger</child>
-          <gearbox_reference_body>${name}/INPUT_INTERFACE</gearbox_reference_body>
-          <gearbox_ratio>1</gearbox_ratio>
-          <axis>
-            <xyz>1 0 0</xyz>
-          </axis>
-          <axis2>
-            <xyz>1 0 0</xyz>
-          </axis2>
-        </joint>
-      </gazebo>
     </xacro:if>
   </xacro:macro>
