Commit message: Sort of stable behavior in Copellia

File: urdf/link.xacro (robot description, xacro)
@@ -3,5 +3,5 @@
   <!-- NOTE: joint must match the name of the module -->
   <xacro:macro name="link" params="name child type:=X5 input:=RightAngle output:=RightAngle extension twist">
-    <xacro:property name="mass" value="${0.4 * (extension + 0.03) + 0.26}"/>
+    <xacro:property name="mass" value="${2 * (extension + 0.03) + 0.26}"/>
     <xacro:property name="edge_to_center" value="${.02}"/>
     <link name="${name}/INPUT_INTERFACE">
@@ -20,13 +20,16 @@
       </visual>
       <collision>
+        <xacro:if value="${input == 'RightAngle'}">
+        <origin xyz="0.006 0 0.01875" rpy="0 0 0" />
+        <geometry>
+            <box size="0.059 0.048 0.0375" />
+        </geometry>
+        </xacro:if>
+        <xacro:if value="${input == 'Inline'}">
         <origin xyz="0 0 0" rpy="0 0 0" />
         <geometry>
-          <xacro:if value="${input == 'RightAngle'}">
-            <mesh filename="package://hebi_description/meshes/A-2038-02.stl"/>
-          </xacro:if>
-          <xacro:if value="${input == 'Inline'}">
             <mesh filename="package://hebi_description/meshes/A-2225-01.stl" scale="0.001 0.001 0.001"/>
-          </xacro:if>
         </geometry>
+        </xacro:if>
       </collision>
       <!-- Link Pipe -->
@@ -57,46 +60,66 @@
       <visual>
         <xacro:if value="${input == 'RightAngle' and output == 'RightAngle'}">
-          <origin xyz="${extension} ${sin(-twist) * edge_to_center} ${edge_to_center * (1 + cos(-twist))}" rpy="${-twist} 0 0"/>
+          <origin xyz="${extension} ${sin(-twist) * edge_to_center} ${edge_to_center * (1 + cos(twist))}" rpy="${twist} 0 0"/>
+          <geometry>
+            <mesh filename="package://hebi_description/meshes/A-2039-02.stl"/>
+          </geometry>
         </xacro:if>
         <xacro:if value="${input == 'RightAngle' and output == 'Inline'}">
           <origin xyz="${extension} 0 ${edge_to_center}" rpy="${pi/2} ${twist+pi} ${pi/2}"/>
+          <geometry>
+            <mesh filename="package://hebi_description/meshes/A-2226-01.stl" scale="0.001 0.001 0.001"/>
+          </geometry>
+        </xacro:if>
+        <xacro:if value="${input == 'RightAngle' and output == 'None'}">
+          <origin xyz="${extension - 0.035} 0 ${edge_to_center}" rpy="0 ${pi/2} 0"/>
+          <geometry>
+            <cylinder length="0.05" radius="0.02" />
+          </geometry>
         </xacro:if>
         <xacro:if value="${input == 'Inline' and output =='RightAngle'}">
           <origin xyz="${edge_to_center * sin(twist+pi/2)} ${edge_to_center * -cos(twist+pi/2)} ${extension}" rpy="${pi/2} ${-pi/2} ${twist+pi/2}"/>
+          <geometry>
+            <mesh filename="package://hebi_description/meshes/A-2039-02.stl"/>
+          </geometry>
         </xacro:if>
         <xacro:if value="${input == 'Inline' and output =='Inline'}">
           <origin xyz="${0} ${0} ${extension}" rpy="${0} ${0} ${twist-pi/2}"/>
+          <geometry>
+            <mesh filename="package://hebi_description/meshes/A-2226-01.stl" scale="0.001 0.001 0.001"/>
+          </geometry>
         </xacro:if>
-        <geometry>
-          <xacro:if value="${output == 'RightAngle'}">
-            <mesh filename="package://hebi_description/meshes/A-2039-02.stl"/>
-          </xacro:if>
-          <xacro:if value="${output == 'Inline'}">
-            <mesh filename="package://hebi_description/meshes/A-2226-01.stl" scale="0.001 0.001 0.001"/>
-          </xacro:if>
-        </geometry>
         <xacro:black_material/>
       </visual>
       <collision>
         <xacro:if value="${input == 'RightAngle' and output == 'RightAngle'}">
-          <origin xyz="${extension} ${sin(-twist) * edge_to_center} ${edge_to_center * (1 + cos(-twist))}" rpy="${-twist} 0 0"/>
+          <origin xyz="${extension - 0.0015} ${-0.001 * sin(twist)} ${edge_to_center + 0.001 * cos(twist)}" rpy="${twist} 0 0"/>
+          <geometry>
+	    <box size="0.0685 0.065 0.0375" />
+	  </geometry>
         </xacro:if>
         <xacro:if value="${input == 'RightAngle' and output == 'Inline'}">
           <origin xyz="${extension} 0 ${edge_to_center}" rpy="${pi/2} ${twist+pi} ${pi/2}"/>
+          <geometry>
+            <mesh filename="package://hebi_description/meshes/A-2226-01.stl" scale="0.001 0.001 0.001"/>
+          </geometry>
+        </xacro:if>
+        <xacro:if value="${input == 'RightAngle' and output == 'None'}">
+          <origin xyz="${extension - 0.035} 0 ${edge_to_center}" rpy="0 ${pi/2} 0"/>
+          <geometry>
+            <cylinder length="0.05" radius="0.02" />
+          </geometry>
         </xacro:if>
         <xacro:if value="${input == 'Inline' and output =='RightAngle'}">
           <origin xyz="${edge_to_center * sin(twist+pi/2)} ${edge_to_center * -cos(twist+pi/2)} ${extension}" rpy="${pi/2} ${-pi/2} ${twist+pi/2}"/>
+          <geometry>
+	    <box size="0.0685 0.065 0.0375" />
+	  </geometry>
         </xacro:if>
         <xacro:if value="${input == 'Inline' and output =='Inline'}">
           <origin xyz="${0} ${0} ${extension}" rpy="${0} ${0} ${twist-pi/2}"/>
+          <geometry>
+            <mesh filename="package://hebi_description/meshes/A-2226-01.stl" scale="0.001 0.001 0.001"/>
+          </geometry>
         </xacro:if>
-        <geometry>
-          <xacro:if value="${input == 'RightAngle'}">
-            <mesh filename="package://hebi_description/meshes/A-2039-02.stl"/>
-          </xacro:if>
-          <xacro:if value="${input == 'Inline'}">
-            <mesh filename="package://hebi_description/meshes/A-2226-01.stl" scale="0.001 0.001 0.001"/>
-          </xacro:if>
-        </geometry>
       </collision>
       <!-- Approximate inertia as thin rod about x axis -->
@@ -104,10 +127,10 @@
         <origin xyz="${extension/2} 0 ${edge_to_center}" rpy="0 0 0" />
         <mass value="${mass}"/>
-        <inertia  ixx="0.0" ixy="0.0"  ixz="0.0"  iyy="${mass * extension * extension / 12.0}"  iyz="0.0"  izz="${mass * extension * extension / 12.0}"/>
+	<inertia ixx="0.0004" ixy="0.0"  ixz="0.0"
+                 iyy="${mass * extension * extension / 12.0}"  iyz="0.0"
+                 izz="${mass * extension * extension / 12.0}"/>
       </inertial>
     </link>
-    <gazebo reference="${name}/INPUT_INTERFACE">
-      <xacro:gazebo_black_material/>
-    </gazebo>
+    <xacro:unless value="${output == 'None'}">
     <joint name="${name}/OUTPUT_JOINT" type="fixed">
       <parent link="${name}/INPUT_INTERFACE"/>
@@ -126,4 +149,5 @@
       </xacro:if>
     </joint>
+    </xacro:unless>
   </xacro:macro>
 </robot>
