Commit message: Changes for Rviz and Gazebo

File: urdf/actuator.xacro (robot description, xacro)
@@ -60,15 +60,15 @@
     <!-- Note: the frction/damping probably need to be tuned more for accurate simulation -->
     <xacro:if value="${model_name.startswith('X5')}">
-      <xacro:property name="mesh_filename" value="package://hebi_description/meshes/X5.stl"/>
+      <xacro:property name="mesh_filename" value="file://$(find hebi_description)/meshes/X5.stl"/>
       <xacro:property name="damping" value="0.1"/>
       <xacro:property name="friction" value="0.1"/>
     </xacro:if>
     <xacro:if value="${model_name.startswith('X8')}">
-      <xacro:property name="mesh_filename" value="package://hebi_description/meshes/X8.stl"/>
+      <xacro:property name="mesh_filename" value="file://$(find hebi_description)/meshes/X8.stl"/>
       <xacro:property name="damping" value="0.5"/>
       <xacro:property name="friction" value="0.5"/>
     </xacro:if>
     <xacro:if value="${model_name.startswith('R8')}">
-      <xacro:property name="mesh_filename" value="package://hebi_description/meshes/R8.stl"/>
+      <xacro:property name="mesh_filename" value="file://$(find hebi_description)/meshes/R8.stl"/>
       <xacro:property name="damping" value="0.5"/>
       <xacro:property name="friction" value="0.5"/>
@@ -206,15 +206,15 @@
     <!-- Note: the frction/damping probably need to be tuned more for accurate simulation -->
     <xacro:if value="${model_name.startswith('X5')}">
-      <xacro:property name="mesh_filename" value="package://hebi_description/meshes/X5.stl"/>
+      <xacro:property name="mesh_filename" value="file://$(find hebi_description)/meshes/X5.stl"/>
       <xacro:property name="damping" value="0.1"/>
       <xacro:property name="friction" value="0.1"/>
     </xacro:if>
     <xacro:if value="${model_name.startswith('X8')}">
-      <xacro:property name="mesh_filename" value="package://hebi_description/meshes/X8.stl"/>
+      <xacro:property name="mesh_filename" value="file://$(find hebi_description)/meshes/X8.stl"/>
       <xacro:property name="damping" value="0.5"/>
       <xacro:property name="friction" value="0.5"/>
     </xacro:if>
     <xacro:if value="${model_name.startswith('R8')}">
-      <xacro:property name="mesh_filename" value="package://hebi_description/meshes/R8.stl"/>
+      <xacro:property name="mesh_filename" value="file://$(find hebi_description)/meshes/R8.stl"/>
       <xacro:property name="damping" value="0.5"/>
       <xacro:property name="friction" value="0.5"/>

File: urdf/bracket.xacro (robot description, xacro)
@@ -10,5 +10,5 @@
           <origin xyz="0 0 0" rpy="${pi/2} 0 ${pi/2}"/>
           <geometry>
-            <mesh filename="package://hebi_description/meshes/PM-2132-01L.stl" scale="0.001 0.001 0.001"/>
+            <mesh filename="file://$(find hebi_description)/meshes/PM-2132-01L.stl" scale="0.001 0.001 0.001"/>
           </geometry>
         </xacro:if>
@@ -16,5 +16,5 @@
           <origin xyz="0 0 0" rpy="${pi/2} 0 ${-pi/2}"/>
           <geometry>
-            <mesh filename="package://hebi_description/meshes/PM-2132-01R.stl" scale="0.001 0.001 0.001"/>
+            <mesh filename="file://$(find hebi_description)/meshes/PM-2132-01R.stl" scale="0.001 0.001 0.001"/>
           </geometry>
         </xacro:if>
@@ -25,5 +25,5 @@
           <origin xyz="0 0 0" rpy="${pi/2} 0 ${pi/2}"/>
           <geometry>
-            <mesh filename="package://hebi_description/meshes/PM-2132-01L.stl" scale="0.001 0.001 0.001"/>
+            <mesh filename="file://$(find hebi_description)/meshes/PM-2132-01L.stl" scale="0.001 0.001 0.001"/>
           </geometry>
         </xacro:if>
@@ -31,5 +31,5 @@
           <origin xyz="0 0 0" rpy="${pi/2} 0 ${-pi/2}"/>
           <geometry>
-            <mesh filename="package://hebi_description/meshes/PM-2132-01R.stl" scale="0.001 0.001 0.001"/>
+            <mesh filename="file://$(find hebi_description)/meshes/PM-2132-01R.stl" scale="0.001 0.001 0.001"/>
           </geometry>
         </xacro:if>
@@ -56,5 +56,5 @@
         </xacro:if>
         <geometry>
-          <mesh filename="package://hebi_description/meshes/A-2220-01.stl" scale="0.001 0.001 0.001"/>
+          <mesh filename="file://$(find hebi_description)/meshes/A-2220-01.stl" scale="0.001 0.001 0.001"/>
         </geometry>
         <xacro:black_material/>
@@ -68,5 +68,5 @@
         </xacro:if>
         <geometry>
-          <mesh filename="package://hebi_description/meshes/A-2220-01.stl" scale="0.001 0.001 0.001"/>
+          <mesh filename="file://$(find hebi_description)/meshes/A-2220-01.stl" scale="0.001 0.001 0.001"/>
         </geometry>
       </collision>
@@ -99,5 +99,5 @@
         </xacro:if>
         <geometry>
-          <mesh filename="package://hebi_description/meshes/PM-2149-01.stl" scale="0.001 0.001 0.001"/>
+          <mesh filename="file://$(find hebi_description)/meshes/PM-2149-01.stl" scale="0.001 0.001 0.001"/>
         </geometry>
         <xacro:black_material/>
@@ -118,27 +118,27 @@
         <geometry>
           <xacro:if value="${bracket_type.startswith('X5HeavyRight') or bracket_type.startswith('R5HeavyRight')}">
-            <mesh filename="package://hebi_description/meshes/PM-2150-01R.stl" scale="0.001 0.001 0.001"/>
+            <mesh filename="file://$(find hebi_description)/meshes/PM-2150-01R.stl" scale="0.001 0.001 0.001"/>
           </xacro:if>
           <xacro:if value="${bracket_type.startswith('X5HeavyLeft') or bracket_type.startswith('R5HeavyLeft')}">
-            <mesh filename="package://hebi_description/meshes/PM-2150-01L.stl" scale="0.001 0.001 0.001"/>
-          </xacro:if>
-        </geometry>
-        <xacro:black_material/>
-      </visual>
-      <collision>
-        <xacro:if value="${bracket_type.endswith('RightOutside')}">
-          <origin xyz="0 0 0.005" rpy="${pi/2} 0 ${pi/2}"/>
-        </xacro:if>
-        <xacro:if value="${bracket_type.endswith('RightInside')}">
-          <origin xyz="0 0 0.005" rpy="${pi/2} 0 ${-pi/2}"/>
-        </xacro:if>
-        <xacro:if value="${bracket_type.endswith('LeftOutside')}">
-          <origin xyz="0 0 0.005" rpy="${pi/2} 0 ${-pi/2}"/>
-        </xacro:if>
-        <xacro:if value="${bracket_type.endswith('LeftInside')}">
-          <origin xyz="0 0 0.005" rpy="${pi/2} 0 ${pi/2}"/>
-        </xacro:if>
-        <geometry>
-          <mesh filename="package://hebi_description/meshes/PM-2149-01.stl" scale="0.001 0.001 0.001"/>
+            <mesh filename="file://$(find hebi_description)/meshes/PM-2150-01L.stl" scale="0.001 0.001 0.001"/>
+          </xacro:if>
+        </geometry>
+        <xacro:black_material/>
+      </visual>
+      <collision>
+        <xacro:if value="${bracket_type.endswith('RightOutside')}">
+          <origin xyz="0 0 0.005" rpy="${pi/2} 0 ${pi/2}"/>
+        </xacro:if>
+        <xacro:if value="${bracket_type.endswith('RightInside')}">
+          <origin xyz="0 0 0.005" rpy="${pi/2} 0 ${-pi/2}"/>
+        </xacro:if>
+        <xacro:if value="${bracket_type.endswith('LeftOutside')}">
+          <origin xyz="0 0 0.005" rpy="${pi/2} 0 ${-pi/2}"/>
+        </xacro:if>
+        <xacro:if value="${bracket_type.endswith('LeftInside')}">
+          <origin xyz="0 0 0.005" rpy="${pi/2} 0 ${pi/2}"/>
+        </xacro:if>
+        <geometry>
+          <mesh filename="file://$(find hebi_description)/meshes/PM-2149-01.stl" scale="0.001 0.001 0.001"/>
         </geometry>
       </collision>
@@ -158,8 +158,8 @@
         <geometry>
           <xacro:if value="${bracket_type.startswith('X5HeavyRight') or bracket_type.startswith('R5HeavyRight')}">
-            <mesh filename="package://hebi_description/meshes/PM-2150-01R.stl" scale="0.001 0.001 0.001"/>
+            <mesh filename="file://$(find hebi_description)/meshes/PM-2150-01R.stl" scale="0.001 0.001 0.001"/>
           </xacro:if>
           <xacro:if value="${bracket_type.startswith('X5HeavyLeft') or bracket_type.startswith('R5HeavyLeft')}">
-            <mesh filename="package://hebi_description/meshes/PM-2150-01L.stl" scale="0.001 0.001 0.001"/>
+            <mesh filename="file://$(find hebi_description)/meshes/PM-2150-01L.stl" scale="0.001 0.001 0.001"/>
           </xacro:if>
         </geometry>
@@ -199,8 +199,8 @@
         <geometry>
           <xacro:if value="${bracket_type.endswith('Outside')}">
-            <mesh filename="package://hebi_description/meshes/A-2221-01-Outside.stl" scale="0.001 0.001 0.001"/>
+            <mesh filename="file://$(find hebi_description)/meshes/A-2221-01-Outside.stl" scale="0.001 0.001 0.001"/>
           </xacro:if>
           <xacro:if value="${bracket_type.endswith('Inside')}">
-            <mesh filename="package://hebi_description/meshes/A-2221-01-Inside.stl" scale="0.001 0.001 0.001"/>
+            <mesh filename="file://$(find hebi_description)/meshes/A-2221-01-Inside.stl" scale="0.001 0.001 0.001"/>
           </xacro:if>
         </geometry>
@@ -222,8 +222,8 @@
         <geometry>
           <xacro:if value="${bracket_type.endswith('Outside')}">
-            <mesh filename="package://hebi_description/meshes/A-2221-01-Outside.stl" scale="0.001 0.001 0.001"/>
+            <mesh filename="file://$(find hebi_description)/meshes/A-2221-01-Outside.stl" scale="0.001 0.001 0.001"/>
           </xacro:if>
           <xacro:if value="${bracket_type.endswith('Inside')}">
-            <mesh filename="package://hebi_description/meshes/A-2221-01-Inside.stl" scale="0.001 0.001 0.001"/>
+            <mesh filename="file://$(find hebi_description)/meshes/A-2221-01-Inside.stl" scale="0.001 0.001 0.001"/>
           </xacro:if>
         </geometry>

File: urdf/end_effector.xacro (robot description, xacro)
@@ -30,5 +30,5 @@
         <origin xyz="-0.006 -0.0055 -0.0045" rpy="${pi/2} 0 ${pi/2}" />
         <geometry>
-          <mesh filename="package://hebi_description/meshes/PM-2221-01.stl" scale="0.001 0.001 0.001"/>
+          <mesh filename="file://$(find hebi_description)/meshes/PM-2221-01.stl" scale="0.001 0.001 0.001"/>
         </geometry>
         <xacro:silver_material/>
@@ -37,5 +37,5 @@
         <origin xyz="-0.006 -0.0055 -0.0045" rpy="${pi/2} 0 ${pi/2}" />
         <geometry>
-          <mesh filename="package://hebi_description/meshes/PM-2221-01.stl" scale="0.001 0.001 0.001"/>
+          <mesh filename="file://$(find hebi_description)/meshes/PM-2221-01.stl" scale="0.001 0.001 0.001"/>
         </geometry>
       </collision>
@@ -58,5 +58,5 @@
         <origin xyz="-0.0115 0.029 -0.004" rpy="${pi/2} 0 0" />
         <geometry>
-          <mesh filename="package://hebi_description/meshes/PM-2358-02.stl" scale="0.001 0.001 0.001"/>
+          <mesh filename="file://$(find hebi_description)/meshes/PM-2358-02.stl" scale="0.001 0.001 0.001"/>
         </geometry>
         <xacro:black_material/>
@@ -79,5 +79,5 @@
         <origin xyz="-0.006 -0.0115 -0.0036" rpy="${0.5*pi} ${0.0*pi} ${0.5*pi}" />
         <geometry>
-          <mesh filename="package://hebi_description/meshes/PM-2360-02.stl" scale="0.001 0.001 0.001"/>
+          <mesh filename="file://$(find hebi_description)/meshes/PM-2360-02.stl" scale="0.001 0.001 0.001"/>
         </geometry>
         <xacro:black_material/>
@@ -86,5 +86,5 @@
         <origin xyz="-0.006 -0.0115 -0.0036" rpy="${0.5*pi} ${0.0*pi} ${0.5*pi}" />
         <geometry>
-          <mesh filename="package://hebi_description/meshes/PM-2360-02.stl" scale="0.001 0.001 0.001"/>
+          <mesh filename="file://$(find hebi_description)/meshes/PM-2360-02.stl" scale="0.001 0.001 0.001"/>
         </geometry>
       </collision>
@@ -168,5 +168,5 @@
         <origin xyz="-0.0115 -0.004 -0.004" rpy="0 0 0" />
         <geometry>
-          <mesh filename="package://hebi_description/meshes/PM-2359-02.stl" scale="0.001 0.001 0.001"/>
+          <mesh filename="file://$(find hebi_description)/meshes/PM-2359-02.stl" scale="0.001 0.001 0.001"/>
         </geometry>
         <xacro:black_material/>
@@ -251,5 +251,5 @@
           <origin xyz="-0.0225 0.0225 0" rpy="${pi/2} 0 0" />
           <geometry>
-            <mesh filename="package://hebi_description/meshes/PM-2357-02.stl" scale="0.001 0.001 0.001"/>
+            <mesh filename="file://$(find hebi_description)/meshes/PM-2357-02.stl" scale="0.001 0.001 0.001"/>
           </geometry>
           <xacro:black_material/>
@@ -277,5 +277,5 @@
           <origin xyz="-0.0145 -0.008 0.0038" rpy="${0.5*pi} ${0.0*pi} ${0.5*pi}" />
           <geometry>
-            <mesh filename="package://hebi_description/meshes/PM-2291-01.stl" scale="0.001 0.001 0.001"/>
+            <mesh filename="file://$(find hebi_description)/meshes/PM-2291-01.stl" scale="0.001 0.001 0.001"/>
           </geometry>
           <xacro:silver_material/>
@@ -284,5 +284,5 @@
           <origin xyz="-0.0145 -0.008 0.004" rpy="${0.5*pi} ${0.0*pi} ${0.5*pi}" />
           <geometry>
-            <mesh filename="package://hebi_description/meshes/PM-2291-01.stl" scale="0.001 0.001 0.001"/>
+            <mesh filename="file://$(find hebi_description)/meshes/PM-2291-01.stl" scale="0.001 0.001 0.001"/>
           </geometry>
         </collision>

File: urdf/kits/ros2_control/A-2085-06_macro.ros2_control.xacro (robot description, xacro)
@@ -34,125 +34,54 @@
       </hardware>
       <joint name="J1_base">
-        <command_interface name="position">     <!-- Add/Remove interfaces as needed -->
-          <param name="min">-3.1428</param>
-          <param name="max">3.1428</param>
-        </command_interface>
+        <command_interface name="position" />
         <state_interface name="position">
           <param name="initial_value">0.0</param>
         </state_interface>
-        <state_interface name="velocity">
-          <param name="initial_value">0.0</param>
-        </state_interface>
-        <state_interface name="effort">
-          <param name="initial_value">0.0</param>
-        </state_interface>
+        <state_interface name="velocity" />
       </joint>
       <joint name="J2_shoulder">
-        <command_interface name="position">     <!-- Add/Remove interfaces as needed -->
-          <param name="min">-3.1428</param>
-          <param name="max">3.1428</param>
-        </command_interface>
+        <command_interface name="position" />
         <state_interface name="position">
           <param name="initial_value">0.0</param>
         </state_interface>
-        <state_interface name="velocity">
-          <param name="initial_value">0.0</param>
-        </state_interface>
-        <state_interface name="effort">
-          <param name="initial_value">0.0</param>
-        </state_interface>
+        <state_interface name="velocity" />
       </joint>
       <joint name="J3_elbow">
-        <command_interface name="position">     <!-- Add/Remove interfaces as needed -->
-          <param name="min">-3.1428</param>
-          <param name="max">3.1428</param>
-        </command_interface>
+        <command_interface name="position" />
         <state_interface name="position">
           <param name="initial_value">0.0</param>
         </state_interface>
-        <state_interface name="velocity">
-          <param name="initial_value">0.0</param>
-        </state_interface>
-        <state_interface name="effort">
-          <param name="initial_value">0.0</param>
-        </state_interface>
+        <state_interface name="velocity" />
       </joint>
       <joint name="J4_wrist1">
-        <command_interface name="position">     <!-- Add/Remove interfaces as needed -->
-          <param name="min">-3.1428</param>
-          <param name="max">3.1428</param>
-        </command_interface>
+        <command_interface name="position" />
         <state_interface name="position">
           <param name="initial_value">0.0</param>
         </state_interface>
-        <state_interface name="velocity">
-          <param name="initial_value">0.0</param>
-        </state_interface>
-        <state_interface name="effort">
-          <param name="initial_value">0.0</param>
-        </state_interface>
+        <state_interface name="velocity" />
       </joint>
       <joint name="J5_wrist2">
-        <command_interface name="position">     <!-- Add/Remove interfaces as needed -->
-          <param name="min">-3.1428</param>
-          <param name="max">3.1428</param>
-        </command_interface>
+        <command_interface name="position" />
         <state_interface name="position">
           <param name="initial_value">0.0</param>
         </state_interface>
-        <state_interface name="velocity">
-          <param name="initial_value">0.0</param>
-        </state_interface>
-        <state_interface name="effort">
-          <param name="initial_value">0.0</param>
-        </state_interface>
+        <state_interface name="velocity" />
       </joint>
       <joint name="J6_wrist3">
-        <command_interface name="position">     <!-- Add/Remove interfaces as needed -->
-          <param name="min">-3.1428</param>
-          <param name="max">3.1428</param>
-        </command_interface>
+        <command_interface name="position" />
         <state_interface name="position">
           <param name="initial_value">0.0</param>
         </state_interface>
-        <state_interface name="velocity">
-          <param name="initial_value">0.0</param>
-        </state_interface>
-        <state_interface name="effort">
-          <param name="initial_value">0.0</param>
-        </state_interface>
+        <state_interface name="velocity" />
       </joint>
-      <!-- <sensor name="tcp_fts_sensor">
-        <state_interface name="fx"/>
-        <state_interface name="fy"/>
-        <state_interface name="fz"/>
-        <state_interface name="tx"/>
-        <state_interface name="ty"/>
-        <state_interface name="tz"/>
-        <param name="frame_id">end_effector</param>
-        <param name="min_fx">-100</param>
-        <param name="max_fx">100</param>
-        <param name="min_fy">-100</param>
-        <param name="max_fy">100</param>
-        <param name="min_fz">-200</param>
-        <param name="max_fz">200</param>
-        <param name="min_tx">-10</param>
-        <param name="max_tx">10</param>
-        <param name="min_ty">-10</param>
-        <param name="max_ty">10</param>
-        <param name="min_tz">-15</param>
-        <param name="max_tz">15</param>
-      </sensor> -->
     </ros2_control>
-    <xacro:if value="$(arg sim_gazebo_classic)">
-      <!-- Gazebo plugins -->
-      <gazebo reference="world">
-      </gazebo>
+    <!-- Gazebo plugins -->
+    <!-- <xacro:if value="$(arg sim_gazebo_classic)">
       <gazebo>
         <plugin filename="libgazebo_ros2_control.so" name="gazebo_ros2_control">
-          <parameters>${simulation_controllers}</parameters>
+          <parameters>$(find hebi_bringup)/config/A-2085-06_controllers.yaml</parameters>
         </plugin>
       </gazebo>
-    </xacro:if>
+    </xacro:if> -->
     <xacro:if value="$(arg sim_gazebo)">
       <!-- Gazebo plugins -->

File: urdf/link.xacro (robot description, xacro)
@@ -11,8 +11,8 @@
         <geometry>
           <xacro:if value="${input == 'RightAngle'}">
-            <mesh filename="package://hebi_description/meshes/A-2038-02.stl"/>
+            <mesh filename="file://$(find hebi_description)/meshes/A-2038-02.stl"/>
           </xacro:if>
           <xacro:if value="${input == 'Inline'}">
-            <mesh filename="package://hebi_description/meshes/A-2225-01.stl" scale="0.001 0.001 0.001"/>
+            <mesh filename="file://$(find hebi_description)/meshes/A-2225-01.stl" scale="0.001 0.001 0.001"/>
           </xacro:if>
         </geometry>
@@ -23,8 +23,8 @@
         <geometry>
           <xacro:if value="${input == 'RightAngle'}">
-            <mesh filename="package://hebi_description/meshes/A-2038-02.stl"/>
+            <mesh filename="file://$(find hebi_description)/meshes/A-2038-02.stl"/>
           </xacro:if>
           <xacro:if value="${input == 'Inline'}">
-            <mesh filename="package://hebi_description/meshes/A-2225-01.stl" scale="0.001 0.001 0.001"/>
+            <mesh filename="file://$(find hebi_description)/meshes/A-2225-01.stl" scale="0.001 0.001 0.001"/>
           </xacro:if>
         </geometry>
@@ -70,8 +70,8 @@
         <geometry>
           <xacro:if value="${output == 'RightAngle'}">
-            <mesh filename="package://hebi_description/meshes/A-2039-02.stl"/>
+            <mesh filename="file://$(find hebi_description)/meshes/A-2039-02.stl"/>
           </xacro:if>
           <xacro:if value="${output == 'Inline'}">
-            <mesh filename="package://hebi_description/meshes/A-2226-01.stl" scale="0.001 0.001 0.001"/>
+            <mesh filename="file://$(find hebi_description)/meshes/A-2226-01.stl" scale="0.001 0.001 0.001"/>
           </xacro:if>
         </geometry>
@@ -93,8 +93,8 @@
         <geometry>
           <xacro:if value="${input == 'RightAngle'}">
-            <mesh filename="package://hebi_description/meshes/A-2039-02.stl"/>
+            <mesh filename="file://$(find hebi_description)/meshes/A-2039-02.stl"/>
           </xacro:if>
           <xacro:if value="${input == 'Inline'}">
-            <mesh filename="package://hebi_description/meshes/A-2226-01.stl" scale="0.001 0.001 0.001"/>
+            <mesh filename="file://$(find hebi_description)/meshes/A-2226-01.stl" scale="0.001 0.001 0.001"/>
           </xacro:if>
         </geometry>
