Commit message: Updated pipeline to follow new naming conventions

File: urdf/kits/A-2084-01.xacro (robot description, xacro)
@@ -1,22 +1,19 @@
-<?xml version="1.0"?>
-<!-- HEBI A-2084-01 4-DoF Robot SCARA Style Arm Kit -->
-<robot xmlns:xacro="http://www.ros.org/wiki/xacro" name="A-2084-01">
+<?xml version='1.0' encoding='UTF-8'?>
+<robot xmlns:xacro="http://www.ros.org/wiki/xacro" version="1.1.0" name="A-2084-01">
   <xacro:include filename="$(find hebi_description)/urdf/hebi.xacro"/>
-  <!-- world -->
-  <link name="world" />
-  <joint name="world_joint"  type="fixed">
-    <origin xyz="0 0 0" rpy="0 0 0" />
+  <!-- HEBI A-2084-01 Style Arm Kit -->
+  <link name="world"/>
+  <joint name="world_joint" type="fixed">
+    <origin xyz="0 0 0" rpy="0 0 0"/>
     <parent link="world"/>
-    <child link="HEBI/base/INPUT_INTERFACE"/>
+    <child link="Arm/J1_base/INPUT_INTERFACE"/>
   </joint>
-  <!-- robot -->
-  <xacro:actuator name="HEBI/base" child="shoulder_bracket" type="X5_4"/>
-  <xacro:bracket name="shoulder_bracket" child="HEBI/shoulder" type="X5HeavyRightOutside"/>
-  <xacro:actuator name="HEBI/shoulder" child="shoulder_elbow" type="X5_9"/>
-  <xacro:link name="shoulder_elbow" child="HEBI/elbow" extension="0.325" twist="${pi/2}"/>
-  <xacro:actuator name="HEBI/elbow" child="elbow_wrist1" type="X5_4"/>
-  <xacro:link name="elbow_wrist1" child="HEBI/wrist1" extension="0.325" twist="0"/>
-  <xacro:actuator name="HEBI/wrist1" child="end_effector" type="X5_1"/>
-  <!-- placeholder end link at end of arm -->
+  <xacro:actuator type="X5_4" name="Arm/J1_base" child="shoulder_bracket"/>
+  <xacro:bracket type="X5HeavyRightOutside" name="shoulder_bracket" child="Arm/J2_shoulder"/>
+  <xacro:actuator type="X5_9" name="Arm/J2_shoulder" child="shoulder_elbow"/>
+  <xacro:link type="X5" extension="0.325" twist="${pi/2}" name="shoulder_elbow" child="Arm/J3_elbow"/>
+  <xacro:actuator type="X5_4" name="Arm/J3_elbow" child="elbow_wrist1"/>
+  <xacro:link type="X5" extension="0.325" twist="0" name="elbow_wrist1" child="Arm/J4_wrist1"/>
+  <xacro:actuator type="X5_1" name="Arm/J4_wrist1" child="end_effector"/>
   <xacro:null_end_effector name="end_effector"/>
 </robot>

File: urdf/kits/A-2085-04.xacro (robot description, xacro)
@@ -1,22 +1,19 @@
-<?xml version="1.0"?>
-<!-- HEBI A-2085-04 4-DoF Robot Arm Kit -->
-<robot xmlns:xacro="http://www.ros.org/wiki/xacro" name="A-2085-04">
+<?xml version='1.0' encoding='UTF-8'?>
+<robot xmlns:xacro="http://www.ros.org/wiki/xacro" version="1.1.0" name="A-2085-04">
   <xacro:include filename="$(find hebi_description)/urdf/hebi.xacro"/>
-  <!-- world -->
-  <link name="world" />
-  <joint name="world_joint"  type="fixed">
-    <origin xyz="0 0 0" rpy="0 0 0" />
+  <!-- HEBI A-2085-04 Style Arm Kit -->
+  <link name="world"/>
+  <joint name="world_joint" type="fixed">
+    <origin xyz="0 0 0" rpy="0 0 0"/>
     <parent link="world"/>
-    <child link="HEBI/base/INPUT_INTERFACE"/>
+    <child link="Arm/J1_base/INPUT_INTERFACE"/>
   </joint>
-  <!-- robot -->
-  <xacro:actuator name="HEBI/base" child="shoulder_bracket" type="X5_4" limits="${[-pi,pi]}"/>
-  <xacro:bracket name="shoulder_bracket" child="HEBI/shoulder" type="X5HeavyRightOutside"/>
-  <xacro:actuator name="HEBI/shoulder" child="shoulder_elbow" type="X5_9" limits="${[-0.5,pi]}"/>
-  <xacro:link name="shoulder_elbow" child="HEBI/elbow" extension="0.325" twist="${pi}"/>
-  <xacro:actuator name="HEBI/elbow" child="elbow_wrist1" type="X5_4" limits="${[-3,3]}"/>
-  <xacro:link name="elbow_wrist1" child="HEBI/wrist1" extension="0.325" twist="${pi}"/>
-  <xacro:actuator name="HEBI/wrist1" child="end_effector" type="X5_1"/>
-  <!-- placeholder end link at end of arm -->
+  <xacro:actuator type="X5_4" name="Arm/J1_base" child="shoulder_bracket"/>
+  <xacro:bracket type="X5HeavyRightOutside" name="shoulder_bracket" child="Arm/J2_shoulder"/>
+  <xacro:actuator type="X5_9" name="Arm/J2_shoulder" child="shoulder_elbow"/>
+  <xacro:link type="X5" extension="0.325" twist="${pi}" name="shoulder_elbow" child="Arm/J3_elbow"/>
+  <xacro:actuator type="X5_4" name="Arm/J3_elbow" child="elbow_wrist1"/>
+  <xacro:link type="X5" extension="0.325" twist="${pi}" name="elbow_wrist1" child="Arm/J4_wrist1"/>
+  <xacro:actuator type="X5_1" name="Arm/J4_wrist1" child="end_effector"/>
   <xacro:null_end_effector name="end_effector"/>
 </robot>

File: urdf/kits/A-2085-05.xacro (robot description, xacro)
@@ -1,24 +1,21 @@
-<?xml version="1.0"?>
-<!-- HEBI A-2085-05 5-DoF Robot Arm Kit -->
-<robot xmlns:xacro="http://www.ros.org/wiki/xacro" name="A-2085-05">
+<?xml version='1.0' encoding='UTF-8'?>
+<robot xmlns:xacro="http://www.ros.org/wiki/xacro" version="1.1.0" name="A-2085-05">
   <xacro:include filename="$(find hebi_description)/urdf/hebi.xacro"/>
-  <!-- world -->
-  <link name="world" />
-  <joint name="world_joint"  type="fixed">
-    <origin xyz="0 0 0" rpy="0 0 0" />
+  <!-- HEBI A-2085-05 Style Arm Kit -->
+  <link name="world"/>
+  <joint name="world_joint" type="fixed">
+    <origin xyz="0 0 0" rpy="0 0 0"/>
     <parent link="world"/>
-    <child link="HEBI/base/INPUT_INTERFACE"/>
+    <child link="Arm/J1_base/INPUT_INTERFACE"/>
   </joint>
-  <!-- robot -->
-  <xacro:actuator name="HEBI/base" child="shoulder_bracket" type="X8_9" limits="${[-pi,pi]}"/>
-  <xacro:bracket name="shoulder_bracket" child="HEBI/shoulder" type="X5HeavyRightOutside"/>
-  <xacro:actuator name="HEBI/shoulder" child="shoulder_elbow" type="X8_16" limits="${[-0.5,pi]}"/>
-  <xacro:link name="shoulder_elbow" child="HEBI/elbow" extension="0.325" twist="${pi}"/>
-  <xacro:actuator name="HEBI/elbow" child="elbow_wrist1" type="X8_9" limits="${[-3,3]}"/>
-  <xacro:link name="elbow_wrist1" child="HEBI/wrist1" extension="0.325" twist="${pi}"/>
-  <xacro:actuator name="HEBI/wrist1" child="wrist1_wrist2" type="X5_1" limits="${[-2 * pi,2 * pi]}"/>
-  <xacro:bracket name="wrist1_wrist2" child="HEBI/wrist2" type="X5LightRight"/>
-  <xacro:actuator name="HEBI/wrist2" child="end_effector" type="X5_1"/>
-  <!-- placeholder end link at end of arm -->
+  <xacro:actuator type="X8_9" name="Arm/J1_base" child="shoulder_bracket"/>
+  <xacro:bracket type="X5HeavyRightOutside" name="shoulder_bracket" child="Arm/J2_shoulder"/>
+  <xacro:actuator type="X8_16" name="Arm/J2_shoulder" child="shoulder_elbow"/>
+  <xacro:link type="X5" extension="0.325" twist="${pi}" name="shoulder_elbow" child="Arm/J3_elbow"/>
+  <xacro:actuator type="X8_9" name="Arm/J3_elbow" child="elbow_wrist1"/>
+  <xacro:link type="X5" extension="0.325" twist="${pi}" name="elbow_wrist1" child="Arm/J4_wrist1"/>
+  <xacro:actuator type="X5_1" name="Arm/J4_wrist1" child="wrist2_bracket"/>
+  <xacro:bracket type="X5LightRight" name="wrist2_bracket" child="Arm/J5_wrist2"/>
+  <xacro:actuator type="X5_1" name="Arm/J5_wrist2" child="end_effector"/>
   <xacro:null_end_effector name="end_effector"/>
 </robot>

File: urdf/kits/A-2085-06.xacro (robot description, xacro)
@@ -1,26 +1,23 @@
-<?xml version="1.0"?>
-<!-- HEBI A-2085-06 6-DoF Robot Arm Kit -->
-<robot xmlns:xacro="http://www.ros.org/wiki/xacro" name="A-2085-06">
+<?xml version='1.0' encoding='UTF-8'?>
+<robot xmlns:xacro="http://www.ros.org/wiki/xacro" version="1.1.0" name="A-2085-06">
   <xacro:include filename="$(find hebi_description)/urdf/hebi.xacro"/>
-  <!-- world -->
-  <link name="world" />
-  <joint name="world_joint"  type="fixed">
-    <origin xyz="0 0 0" rpy="0 0 0" />
+  <!-- HEBI A-2085-06 Style Arm Kit -->
+  <link name="world"/>
+  <joint name="world_joint" type="fixed">
+    <origin xyz="0 0 0" rpy="0 0 0"/>
     <parent link="world"/>
-    <child link="HEBI/base/INPUT_INTERFACE"/>
+    <child link="Arm/J1_base/INPUT_INTERFACE"/>
   </joint>
-  <!-- robot -->
-  <xacro:actuator name="HEBI/base" child="shoulder_bracket" type="X8_9" limits="${[-pi,pi]}"/>
-  <xacro:bracket name="shoulder_bracket" child="HEBI/shoulder" type="X5HeavyRightOutside"/>
-  <xacro:actuator name="HEBI/shoulder" child="shoulder_elbow" type="X8_16" limits="${[-0.5,pi]}"/>
-  <xacro:link name="shoulder_elbow" child="HEBI/elbow" extension="0.325" twist="${pi}"/>
-  <xacro:actuator name="HEBI/elbow" child="elbow_wrist1" type="X8_9" limits="${[-3,3]}"/>
-  <xacro:link name="elbow_wrist1" child="HEBI/wrist1" extension="0.325" twist="${pi}"/>
-  <xacro:actuator name="HEBI/wrist1" child="wrist1_wrist2" type="X5_1" limits="${[-2 * pi, 2 * pi]}"/>
-  <xacro:bracket name="wrist1_wrist2" child="HEBI/wrist2" type="X5LightRight"/>
-  <xacro:actuator name="HEBI/wrist2" child="wrist2_wrist3" type="X5_1" limits="${[-1.5 * pi, 1.5 * pi]}"/>
-  <xacro:bracket name="wrist2_wrist3" child="HEBI/wrist3" type="X5LightRight"/>
-  <xacro:actuator name="HEBI/wrist3" child="end_effector" type="X5_1"/>
-  <!-- placeholder end link at end of arm -->
+  <xacro:actuator type="X8_9" name="Arm/J1_base" child="shoulder_bracket"/>
+  <xacro:bracket type="X5HeavyRightOutside" name="shoulder_bracket" child="Arm/J2_shoulder"/>
+  <xacro:actuator type="X8_16" name="Arm/J2_shoulder" child="shoulder_elbow"/>
+  <xacro:link type="X5" extension="0.325" twist="${pi}" name="shoulder_elbow" child="Arm/J3_elbow"/>
+  <xacro:actuator type="X8_9" name="Arm/J3_elbow" child="elbow_wrist1"/>
+  <xacro:link type="X5" extension="0.325" twist="${pi}" name="elbow_wrist1" child="Arm/J4_wrist1"/>
+  <xacro:actuator type="X5_1" name="Arm/J4_wrist1" child="wrist2_bracket"/>
+  <xacro:bracket type="X5LightRight" name="wrist2_bracket" child="Arm/J5_wrist2"/>
+  <xacro:actuator type="X5_1" name="Arm/J5_wrist2" child="wrist3_bracket"/>
+  <xacro:bracket type="X5LightRight" name="wrist3_bracket" child="Arm/J6_wrist3"/>
+  <xacro:actuator type="X5_1" name="Arm/J6_wrist3" child="end_effector"/>
   <xacro:null_end_effector name="end_effector"/>
 </robot>
