Commit message: Forgot to update xacros for gripper configs

File: urdf/kits/A-2084-01-parallel-gripper.xacro (robot description, xacro)
@@ -8,14 +8,14 @@
     <origin xyz="0 0 0" rpy="0 0 0" />
     <parent link="world"/>
-    <child link="HEBI/base/INPUT_INTERFACE"/>
+    <child link="Arm/J1_base/INPUT_INTERFACE"/>
   </joint>
   <!-- robot -->
-  <xacro:actuator name="HEBI/base" child="shoulder_bracket" type="X5_4"/>
-  <xacro:bracket name="shoulder_bracket" child="HEBI/shoulder" type="X5HeavyRightOutside"/>
-  <xacro:actuator name="HEBI/shoulder" child="shoulder_elbow" type="X5_9"/>
-  <xacro:link name="shoulder_elbow" child="HEBI/elbow" extension="0.325" twist="${pi/2}"/>
-  <xacro:actuator name="HEBI/elbow" child="elbow_wrist1" type="X5_4"/>
-  <xacro:link name="elbow_wrist1" child="HEBI/wrist1" extension="0.325" twist="0"/>
-  <xacro:actuator name="HEBI/wrist1" child="end_effector" type="X5_1"/>
+  <xacro:actuator name="Arm/J1_base" child="shoulder_bracket" type="X5_4"/>
+  <xacro:bracket name="shoulder_bracket" child="Arm/J2_shoulder" type="X5HeavyRightOutside"/>
+  <xacro:actuator name="Arm/J2_shoulder" child="shoulder_elbow" type="X5_9"/>
+  <xacro:link name="shoulder_elbow" child="Arm/J3_elbow" extension="0.325" twist="${pi/2}"/>
+  <xacro:actuator name="Arm/J3_elbow" child="elbow_wrist1" type="X5_4"/>
+  <xacro:link name="elbow_wrist1" child="Arm/J4_wrist1" extension="0.325" twist="0"/>
+  <xacro:actuator name="Arm/J4_wrist1" child="end_effector" type="X5_1"/>
   <!-- parallel gripper end effector -->
   <xacro:gripper name="end_effector" type="parallel"/>

File: urdf/kits/A-2085-04-parallel-gripper.xacro (robot description, xacro)
@@ -8,14 +8,14 @@
     <origin xyz="0 0 0" rpy="0 0 0" />
     <parent link="world"/>
-    <child link="HEBI/base/INPUT_INTERFACE"/>
+    <child link="Arm/J1_base/INPUT_INTERFACE"/>
   </joint>
   <!-- robot -->
-  <xacro:actuator name="HEBI/base" child="shoulder_bracket" type="X5_4" limits="${[-pi,pi]}"/>
-  <xacro:bracket name="shoulder_bracket" child="HEBI/shoulder" type="X5HeavyRightOutside"/>
-  <xacro:actuator name="HEBI/shoulder" child="shoulder_elbow" type="X5_9" limits="${[-0.5,pi]}"/>
-  <xacro:link name="shoulder_elbow" child="HEBI/elbow" extension="0.325" twist="${pi}"/>
-  <xacro:actuator name="HEBI/elbow" child="elbow_wrist1" type="X5_4" limits="${[-3,3]}"/>
-  <xacro:link name="elbow_wrist1" child="HEBI/wrist1" extension="0.325" twist="${pi}"/>
-  <xacro:actuator name="HEBI/wrist1" child="end_effector" type="X5_1"/>
+  <xacro:actuator name="Arm/J1_base" child="shoulder_bracket" type="X5_4" limits="${[-pi,pi]}"/>
+  <xacro:bracket name="shoulder_bracket" child="Arm/J2_shoulder" type="X5HeavyRightOutside"/>
+  <xacro:actuator name="Arm/J2_shoulder" child="shoulder_elbow" type="X5_9" limits="${[-0.5,pi]}"/>
+  <xacro:link name="shoulder_elbow" child="Arm/J3_elbow" extension="0.325" twist="${pi}"/>
+  <xacro:actuator name="Arm/J3_elbow" child="elbow_wrist1" type="X5_4" limits="${[-3,3]}"/>
+  <xacro:link name="elbow_wrist1" child="Arm/J4_wrist1" extension="0.325" twist="${pi}"/>
+  <xacro:actuator name="Arm/J4_wrist1" child="end_effector" type="X5_1"/>
   <!-- parallel gripper end effector -->
   <xacro:gripper name="end_effector" type="parallel"/>

File: urdf/kits/A-2085-05-parallel-gripper.xacro (robot description, xacro)
@@ -8,16 +8,16 @@
     <origin xyz="0 0 0" rpy="0 0 0" />
     <parent link="world"/>
-    <child link="HEBI/base/INPUT_INTERFACE"/>
+    <child link="Arm/J1_base/INPUT_INTERFACE"/>
   </joint>
   <!-- robot -->
-  <xacro:actuator name="HEBI/base" child="shoulder_bracket" type="X8_9" limits="${[-pi,pi]}"/>
-  <xacro:bracket name="shoulder_bracket" child="HEBI/shoulder" type="X5HeavyRightOutside"/>
-  <xacro:actuator name="HEBI/shoulder" child="shoulder_elbow" type="X8_16" limits="${[-0.5,pi]}"/>
-  <xacro:link name="shoulder_elbow" child="HEBI/elbow" extension="0.325" twist="${pi}"/>
-  <xacro:actuator name="HEBI/elbow" child="elbow_wrist1" type="X8_9" limits="${[-3,3]}"/>
-  <xacro:link name="elbow_wrist1" child="HEBI/wrist1" extension="0.325" twist="${pi}"/>
-  <xacro:actuator name="HEBI/wrist1" child="wrist1_wrist2" type="X5_1" limits="${[-2 * pi,2 * pi]}"/>
-  <xacro:bracket name="wrist1_wrist2" child="HEBI/wrist2" type="X5LightRight"/>
-  <xacro:actuator name="HEBI/wrist2" child="end_effector" type="X5_1"/>
+  <xacro:actuator name="Arm/J1_base" child="shoulder_bracket" type="X8_9" limits="${[-pi,pi]}"/>
+  <xacro:bracket name="shoulder_bracket" child="Arm/J2_shoulder" type="X5HeavyRightOutside"/>
+  <xacro:actuator name="Arm/J2_shoulder" child="shoulder_elbow" type="X8_16" limits="${[-0.5,pi]}"/>
+  <xacro:link name="shoulder_elbow" child="Arm/J3_elbow" extension="0.325" twist="${pi}"/>
+  <xacro:actuator name="Arm/J3_elbow" child="elbow_wrist1" type="X8_9" limits="${[-3,3]}"/>
+  <xacro:link name="elbow_wrist1" child="Arm/J4_wrist1" extension="0.325" twist="${pi}"/>
+  <xacro:actuator name="Arm/J4_wrist1" child="wrist1_wrist2" type="X5_1" limits="${[-2 * pi,2 * pi]}"/>
+  <xacro:bracket name="wrist1_wrist2" child="Arm/J5_wrist2" type="X5LightRight"/>
+  <xacro:actuator name="Arm/J5_wrist2" child="end_effector" type="X5_1"/>
   <!-- parallel gripper end effector -->
   <xacro:gripper name="end_effector" type="parallel"/>

File: urdf/kits/A-2085-06-parallel-gripper.xacro (robot description, xacro)
@@ -8,18 +8,18 @@
     <origin xyz="0 0 0" rpy="0 0 0" />
     <parent link="world"/>
-    <child link="HEBI/base/INPUT_INTERFACE"/>
+    <child link="Arm/J1_base/INPUT_INTERFACE"/>
   </joint>
   <!-- robot -->
-  <xacro:actuator name="HEBI/base" child="shoulder_bracket" type="X8_9" limits="${[-pi,pi]}"/>
-  <xacro:bracket name="shoulder_bracket" child="HEBI/shoulder" type="X5HeavyRightOutside"/>
-  <xacro:actuator name="HEBI/shoulder" child="shoulder_elbow" type="X8_16" limits="${[-0.5,pi]}"/>
-  <xacro:link name="shoulder_elbow" child="HEBI/elbow" extension="0.325" twist="${pi}"/>
-  <xacro:actuator name="HEBI/elbow" child="elbow_wrist1" type="X8_9" limits="${[-3,3]}"/>
-  <xacro:link name="elbow_wrist1" child="HEBI/wrist1" extension="0.325" twist="${pi}"/>
-  <xacro:actuator name="HEBI/wrist1" child="wrist1_wrist2" type="X5_1" limits="${[-2 * pi, 2 * pi]}"/>
-  <xacro:bracket name="wrist1_wrist2" child="HEBI/wrist2" type="X5LightRight"/>
-  <xacro:actuator name="HEBI/wrist2" child="wrist2_wrist3" type="X5_1" limits="${[-1.5 * pi, 1.5 * pi]}"/>
-  <xacro:bracket name="wrist2_wrist3" child="HEBI/wrist3" type="X5LightRight"/>
-  <xacro:actuator name="HEBI/wrist3" child="end_effector" type="X5_1"/>
+  <xacro:actuator name="Arm/J1_base" child="shoulder_bracket" type="X8_9" limits="${[-pi,pi]}"/>
+  <xacro:bracket name="shoulder_bracket" child="Arm/J2_shoulder" type="X5HeavyRightOutside"/>
+  <xacro:actuator name="Arm/J2_shoulder" child="shoulder_elbow" type="X8_16" limits="${[-0.5,pi]}"/>
+  <xacro:link name="shoulder_elbow" child="Arm/J3_elbow" extension="0.325" twist="${pi}"/>
+  <xacro:actuator name="Arm/J3_elbow" child="elbow_wrist1" type="X8_9" limits="${[-3,3]}"/>
+  <xacro:link name="elbow_wrist1" child="Arm/J4_wrist1" extension="0.325" twist="${pi}"/>
+  <xacro:actuator name="Arm/J4_wrist1" child="wrist1_wrist2" type="X5_1" limits="${[-2 * pi, 2 * pi]}"/>
+  <xacro:bracket name="wrist1_wrist2" child="Arm/J5_wrist2" type="X5LightRight"/>
+  <xacro:actuator name="Arm/J5_wrist2" child="wrist2_wrist3" type="X5_1" limits="${[-1.5 * pi, 1.5 * pi]}"/>
+  <xacro:bracket name="wrist2_wrist3" child="Arm/J6_wrist3" type="X5LightRight"/>
+  <xacro:actuator name="Arm/J6_wrist3" child="end_effector" type="X5_1"/>
   <!-- parallel gripper end effector -->
   <xacro:gripper name="end_effector" type="parallel"/>

Commit message: Updated template to allow attaching arms to other models
'world' frame can be changed by xacro arg to mount on
another robot. Tested and working with Clearpath jackal.

File: urdf/kits/A-2084-01-parallel-gripper.xacro (robot description, xacro)
@@ -1,11 +1,14 @@
 <?xml version="1.0"?>
-<!-- HEBI A-2084-01 4-DoF Robot SCARA Style Arm Kit -->
 <robot xmlns:xacro="http://www.ros.org/wiki/xacro" name="A-2084-01">
+  <!-- HEBI A-2084-01-parallel-gripper Arm Kit -->
   <xacro:include filename="$(find hebi_description)/urdf/hebi.xacro"/>
-  <!-- world -->
-  <link name="world" />
-  <joint name="world_joint"  type="fixed">
-    <origin xyz="0 0 0" rpy="0 0 0" />
-    <parent link="world"/>
+  <xacro:arg name="hebi_base_frame" default="world"/>
+  <xacro:property name="hebi_base_frame" value="$(arg hebi_base_frame)"/>
+  <xacro:if value="${hebi_base_frame == 'world'}">
+    <link name="$(arg hebi_base_frame)"/>
+  </xacro:if>
+  <joint name="$(arg hebi_base_frame)_arm_joint" type="fixed">
+    <origin xyz="0 0 0" rpy="0 0 0"/>
+    <parent link="$(arg hebi_base_frame)"/>
     <child link="Arm/J1_base/INPUT_INTERFACE"/>
   </joint>

File: urdf/kits/A-2084-01.xacro (robot description, xacro)
@@ -1,10 +1,14 @@
 <?xml version='1.0' encoding='UTF-8'?>
 <robot xmlns:xacro="http://www.ros.org/wiki/xacro" version="1.1.0" name="A-2084-01">
+  <!-- HEBI A-2084-01 Arm Kit -->
   <xacro:include filename="$(find hebi_description)/urdf/hebi.xacro"/>
-  <!-- HEBI A-2084-01 Style Arm Kit -->
-  <link name="world"/>
-  <joint name="world_joint" type="fixed">
-    <origin xyz="0 0 0" rpy="0 0 0"/>
-    <parent link="world"/>
+  <xacro:arg default="world" name="hebi_base_frame"/>
+  <xacro:property name="hebi_base_frame" value="$(arg hebi_base_frame)"/>
+  <xacro:if value="${hebi_base_frame == 'world'}">
+    <link name="$(arg hebi_base_frame)"/>
+  </xacro:if>
+  <joint name="$(arg hebi_base_frame)_joint" type="fixed">
+    <origin rpy="0 0 0" xyz="0 0 0"/>
+    <parent link="$(arg hebi_base_frame)"/>
     <child link="Arm/J1_base/INPUT_INTERFACE"/>
   </joint>

File: urdf/kits/A-2085-04-parallel-gripper.xacro (robot description, xacro)
@@ -1,11 +1,14 @@
 <?xml version="1.0"?>
-<!-- HEBI A-2085-04 4-DoF Robot Arm Kit -->
 <robot xmlns:xacro="http://www.ros.org/wiki/xacro" name="A-2085-04">
+  <!-- HEBI A-2085-04 Arm Kit -->
   <xacro:include filename="$(find hebi_description)/urdf/hebi.xacro"/>
-  <!-- world -->
-  <link name="world" />
-  <joint name="world_joint"  type="fixed">
-    <origin xyz="0 0 0" rpy="0 0 0" />
-    <parent link="world"/>
+  <xacro:arg name="hebi_base_frame" default="world"/>
+  <xacro:property name="hebi_base_frame" value="$(arg hebi_base_frame)"/>
+  <xacro:if value="${hebi_base_frame == 'world'}">
+    <link name="$(arg hebi_base_frame)"/>
+  </xacro:if>
+  <joint name="$(arg hebi_base_frame)_arm_joint" type="fixed">
+    <origin xyz="0 0 0" rpy="0 0 0"/>
+    <parent link="$(arg hebi_base_frame)"/>
     <child link="Arm/J1_base/INPUT_INTERFACE"/>
   </joint>

File: urdf/kits/A-2085-04.xacro (robot description, xacro)
@@ -1,10 +1,14 @@
 <?xml version='1.0' encoding='UTF-8'?>
 <robot xmlns:xacro="http://www.ros.org/wiki/xacro" version="1.1.0" name="A-2085-04">
+  <!-- HEBI A-2085-04 Arm Kit -->
   <xacro:include filename="$(find hebi_description)/urdf/hebi.xacro"/>
-  <!-- HEBI A-2085-04 Style Arm Kit -->
-  <link name="world"/>
-  <joint name="world_joint" type="fixed">
-    <origin xyz="0 0 0" rpy="0 0 0"/>
-    <parent link="world"/>
+  <xacro:arg default="world" name="hebi_base_frame"/>
+  <xacro:property name="hebi_base_frame" value="$(arg hebi_base_frame)"/>
+  <xacro:if value="${hebi_base_frame == 'world'}">
+    <link name="$(arg hebi_base_frame)"/>
+  </xacro:if>
+  <joint name="$(arg hebi_base_frame)_joint" type="fixed">
+    <origin rpy="0 0 0" xyz="0 0 0"/>
+    <parent link="$(arg hebi_base_frame)"/>
     <child link="Arm/J1_base/INPUT_INTERFACE"/>
   </joint>

File: urdf/kits/A-2085-05-parallel-gripper.xacro (robot description, xacro)
@@ -1,11 +1,14 @@
 <?xml version="1.0"?>
-<!-- HEBI A-2085-05 5-DoF Robot Arm Kit -->
 <robot xmlns:xacro="http://www.ros.org/wiki/xacro" name="A-2085-05">
+  <!-- HEBI A-2085-05-parallel-gripper Arm Kit -->
   <xacro:include filename="$(find hebi_description)/urdf/hebi.xacro"/>
-  <!-- world -->
-  <link name="world" />
-  <joint name="world_joint"  type="fixed">
-    <origin xyz="0 0 0" rpy="0 0 0" />
-    <parent link="world"/>
+  <xacro:arg name="hebi_base_frame" default="world"/>
+  <xacro:property name="hebi_base_frame" value="$(arg hebi_base_frame)"/>
+  <xacro:if value="${hebi_base_frame == 'world'}">
+    <link name="$(arg hebi_base_frame)"/>
+  </xacro:if>
+  <joint name="$(arg hebi_base_frame)_arm_joint" type="fixed">
+    <origin xyz="0 0 0" rpy="0 0 0"/>
+    <parent link="$(arg hebi_base_frame)"/>
     <child link="Arm/J1_base/INPUT_INTERFACE"/>
   </joint>

File: urdf/kits/A-2085-05.xacro (robot description, xacro)
@@ -1,10 +1,14 @@
 <?xml version='1.0' encoding='UTF-8'?>
 <robot xmlns:xacro="http://www.ros.org/wiki/xacro" version="1.1.0" name="A-2085-05">
+  <!-- HEBI A-2085-05 Arm Kit -->
   <xacro:include filename="$(find hebi_description)/urdf/hebi.xacro"/>
-  <!-- HEBI A-2085-05 Style Arm Kit -->
-  <link name="world"/>
-  <joint name="world_joint" type="fixed">
-    <origin xyz="0 0 0" rpy="0 0 0"/>
-    <parent link="world"/>
+  <xacro:arg default="world" name="hebi_base_frame"/>
+  <xacro:property name="hebi_base_frame" value="$(arg hebi_base_frame)"/>
+  <xacro:if value="${hebi_base_frame == 'world'}">
+    <link name="$(arg hebi_base_frame)"/>
+  </xacro:if>
+  <joint name="$(arg hebi_base_frame)_joint" type="fixed">
+    <origin rpy="0 0 0" xyz="0 0 0"/>
+    <parent link="$(arg hebi_base_frame)"/>
     <child link="Arm/J1_base/INPUT_INTERFACE"/>
   </joint>

File: urdf/kits/A-2085-06-parallel-gripper.xacro (robot description, xacro)
@@ -1,11 +1,14 @@
 <?xml version="1.0"?>
-<!-- HEBI A-2085-06 6-DoF Robot Arm Kit -->
 <robot xmlns:xacro="http://www.ros.org/wiki/xacro" name="A-2085-06">
+  <!-- HEBI A-2085-06-parallel-gripper Arm Kit -->
   <xacro:include filename="$(find hebi_description)/urdf/hebi.xacro"/>
-  <!-- world -->
-  <link name="world" />
-  <joint name="world_joint"  type="fixed">
-    <origin xyz="0 0 0" rpy="0 0 0" />
-    <parent link="world"/>
+  <xacro:arg name="hebi_base_frame" default="world"/>
+  <xacro:property name="hebi_base_frame" value="$(arg hebi_base_frame)"/>
+  <xacro:if value="${hebi_base_frame == 'world'}">
+    <link name="$(arg hebi_base_frame)"/>
+  </xacro:if>
+  <joint name="$(arg hebi_base_frame)_arm_joint" type="fixed">
+    <origin xyz="0 0 0" rpy="0 0 0"/>
+    <parent link="$(arg hebi_base_frame)"/>
     <child link="Arm/J1_base/INPUT_INTERFACE"/>
   </joint>

File: urdf/kits/A-2085-06.xacro (robot description, xacro)
@@ -1,10 +1,14 @@
 <?xml version='1.0' encoding='UTF-8'?>
 <robot xmlns:xacro="http://www.ros.org/wiki/xacro" version="1.1.0" name="A-2085-06">
+  <!-- HEBI A-2085-06 Arm Kit -->
   <xacro:include filename="$(find hebi_description)/urdf/hebi.xacro"/>
-  <!-- HEBI A-2085-06 Style Arm Kit -->
-  <link name="world"/>
-  <joint name="world_joint" type="fixed">
-    <origin xyz="0 0 0" rpy="0 0 0"/>
-    <parent link="world"/>
+  <xacro:arg default="world" name="hebi_base_frame"/>
+  <xacro:property name="hebi_base_frame" value="$(arg hebi_base_frame)"/>
+  <xacro:if value="${hebi_base_frame == 'world'}">
+    <link name="$(arg hebi_base_frame)"/>
+  </xacro:if>
+  <joint name="$(arg hebi_base_frame)_joint" type="fixed">
+    <origin rpy="0 0 0" xyz="0 0 0"/>
+    <parent link="$(arg hebi_base_frame)"/>
     <child link="Arm/J1_base/INPUT_INTERFACE"/>
   </joint>
