Commit message: Add hrdf for gripper configs.
New scripts to enable directly loading hrdf to robot_description
in launchfiles

File: urdf/kits/A-2084-01-parallel-gripper.xacro (robot description, xacro)
@@ -1,25 +1,23 @@
-<?xml version="1.0"?>
-<robot xmlns:xacro="http://www.ros.org/wiki/xacro" name="A-2084-01">
+<?xml version='1.0' encoding='UTF-8'?>
+<robot xmlns:xacro="http://www.ros.org/wiki/xacro" version="1.2.0" name="A-2084-01-parallel-gripper">
   <!-- HEBI A-2084-01-parallel-gripper Arm Kit -->
   <xacro:include filename="$(find hebi_description)/urdf/hebi.xacro"/>
-  <xacro:arg name="hebi_base_frame" default="world"/>
+  <xacro:arg default="world" name="hebi_base_frame"/>
   <xacro:property name="hebi_base_frame" value="$(arg hebi_base_frame)"/>
   <xacro:if value="${hebi_base_frame == 'world'}">
     <link name="$(arg hebi_base_frame)"/>
   </xacro:if>
-  <joint name="$(arg hebi_base_frame)_arm_joint" type="fixed">
-    <origin xyz="0 0 0" rpy="0 0 0"/>
+  <joint name="$(arg hebi_base_frame)_joint" type="fixed">
+    <origin rpy="0 0 0" xyz="0 0 0"/>
     <parent link="$(arg hebi_base_frame)"/>
     <child link="Arm/J1_base/INPUT_INTERFACE"/>
   </joint>
-  <!-- robot -->
-  <xacro:actuator name="Arm/J1_base" child="shoulder_bracket" type="X5_4"/>
-  <xacro:bracket name="shoulder_bracket" child="Arm/J2_shoulder" type="X5HeavyRightOutside"/>
-  <xacro:actuator name="Arm/J2_shoulder" child="shoulder_elbow" type="X5_9"/>
-  <xacro:link name="shoulder_elbow" child="Arm/J3_elbow" extension="0.325" twist="${pi/2}"/>
-  <xacro:actuator name="Arm/J3_elbow" child="elbow_wrist1" type="X5_4"/>
-  <xacro:link name="elbow_wrist1" child="Arm/J4_wrist1" extension="0.325" twist="0"/>
-  <xacro:actuator name="Arm/J4_wrist1" child="end_effector" type="X5_1"/>
-  <!-- parallel gripper end effector -->
-  <xacro:gripper name="end_effector" type="parallel"/>
+  <xacro:actuator type="X5_4" name="Arm/J1_base" child="shoulder_bracket"/>
+  <xacro:bracket type="X5HeavyRightOutside" name="shoulder_bracket" child="Arm/J2_shoulder"/>
+  <xacro:actuator type="X5_9" name="Arm/J2_shoulder" child="shoulder_elbow"/>
+  <xacro:link type="X5" extension="0.325" twist="${pi/2}" name="shoulder_elbow" child="Arm/J3_elbow"/>
+  <xacro:actuator type="X5_4" name="Arm/J3_elbow" child="elbow_wrist1"/>
+  <xacro:link type="X5" extension="0.325" twist="0" name="elbow_wrist1" child="Arm/J4_wrist1"/>
+  <xacro:actuator type="X5_1" name="Arm/J4_wrist1" child="end_effector"/>
+  <xacro:gripper type="X5Parallel" name="end_effector"/>
 </robot>

File: urdf/kits/A-2084-01.xacro (robot description, xacro)
@@ -20,4 +20,4 @@
   <xacro:link type="X5" extension="0.325" twist="0" name="elbow_wrist1" child="Arm/J4_wrist1"/>
   <xacro:actuator type="X5_1" name="Arm/J4_wrist1" child="end_effector"/>
-  <xacro:null_end_effector name="end_effector"/>
+  <xacro:gripper name="end_effector" type="Custom"/>
 </robot>

File: urdf/kits/A-2085-04-parallel-gripper.xacro (robot description, xacro)
@@ -1,25 +1,23 @@
-<?xml version="1.0"?>
-<robot xmlns:xacro="http://www.ros.org/wiki/xacro" name="A-2085-04">
-  <!-- HEBI A-2085-04 Arm Kit -->
+<?xml version='1.0' encoding='UTF-8'?>
+<robot xmlns:xacro="http://www.ros.org/wiki/xacro" version="1.2.0" name="A-2085-04-parallel-gripper">
+  <!-- HEBI A-2085-04-parallel-gripper Arm Kit -->
   <xacro:include filename="$(find hebi_description)/urdf/hebi.xacro"/>
-  <xacro:arg name="hebi_base_frame" default="world"/>
+  <xacro:arg default="world" name="hebi_base_frame"/>
   <xacro:property name="hebi_base_frame" value="$(arg hebi_base_frame)"/>
   <xacro:if value="${hebi_base_frame == 'world'}">
     <link name="$(arg hebi_base_frame)"/>
   </xacro:if>
-  <joint name="$(arg hebi_base_frame)_arm_joint" type="fixed">
-    <origin xyz="0 0 0" rpy="0 0 0"/>
+  <joint name="$(arg hebi_base_frame)_joint" type="fixed">
+    <origin rpy="0 0 0" xyz="0 0 0"/>
     <parent link="$(arg hebi_base_frame)"/>
     <child link="Arm/J1_base/INPUT_INTERFACE"/>
   </joint>
-  <!-- robot -->
-  <xacro:actuator name="Arm/J1_base" child="shoulder_bracket" type="X5_4" limits="${[-pi,pi]}"/>
-  <xacro:bracket name="shoulder_bracket" child="Arm/J2_shoulder" type="X5HeavyRightOutside"/>
-  <xacro:actuator name="Arm/J2_shoulder" child="shoulder_elbow" type="X5_9" limits="${[-0.5,pi]}"/>
-  <xacro:link name="shoulder_elbow" child="Arm/J3_elbow" extension="0.325" twist="${pi}"/>
-  <xacro:actuator name="Arm/J3_elbow" child="elbow_wrist1" type="X5_4" limits="${[-3,3]}"/>
-  <xacro:link name="elbow_wrist1" child="Arm/J4_wrist1" extension="0.325" twist="${pi}"/>
-  <xacro:actuator name="Arm/J4_wrist1" child="end_effector" type="X5_1"/>
-  <!-- parallel gripper end effector -->
-  <xacro:gripper name="end_effector" type="parallel"/>
+  <xacro:actuator type="X5_4" name="Arm/J1_base" child="shoulder_bracket"/>
+  <xacro:bracket type="X5HeavyRightOutside" name="shoulder_bracket" child="Arm/J2_shoulder"/>
+  <xacro:actuator type="X5_9" name="Arm/J2_shoulder" child="shoulder_elbow"/>
+  <xacro:link type="X5" extension="0.325" twist="${pi}" name="shoulder_elbow" child="Arm/J3_elbow"/>
+  <xacro:actuator type="X5_4" name="Arm/J3_elbow" child="elbow_wrist1"/>
+  <xacro:link type="X5" extension="0.325" twist="${pi}" name="elbow_wrist1" child="Arm/J4_wrist1"/>
+  <xacro:actuator type="X5_1" name="Arm/J4_wrist1" child="end_effector"/>
+  <xacro:gripper type="X5Parallel" name="end_effector"/>
 </robot>

File: urdf/kits/A-2085-04.xacro (robot description, xacro)
@@ -20,4 +20,4 @@
   <xacro:link type="X5" extension="0.325" twist="${pi}" name="elbow_wrist1" child="Arm/J4_wrist1"/>
   <xacro:actuator type="X5_1" name="Arm/J4_wrist1" child="end_effector"/>
-  <xacro:null_end_effector name="end_effector"/>
+  <xacro:gripper name="end_effector" type="Custom"/>
 </robot>

File: urdf/kits/A-2085-05-parallel-gripper.xacro (robot description, xacro)
@@ -1,27 +1,25 @@
-<?xml version="1.0"?>
-<robot xmlns:xacro="http://www.ros.org/wiki/xacro" name="A-2085-05">
+<?xml version='1.0' encoding='UTF-8'?>
+<robot xmlns:xacro="http://www.ros.org/wiki/xacro" version="1.2.0" name="A-2085-05-parallel-gripper">
   <!-- HEBI A-2085-05-parallel-gripper Arm Kit -->
   <xacro:include filename="$(find hebi_description)/urdf/hebi.xacro"/>
-  <xacro:arg name="hebi_base_frame" default="world"/>
+  <xacro:arg default="world" name="hebi_base_frame"/>
   <xacro:property name="hebi_base_frame" value="$(arg hebi_base_frame)"/>
   <xacro:if value="${hebi_base_frame == 'world'}">
     <link name="$(arg hebi_base_frame)"/>
   </xacro:if>
-  <joint name="$(arg hebi_base_frame)_arm_joint" type="fixed">
-    <origin xyz="0 0 0" rpy="0 0 0"/>
+  <joint name="$(arg hebi_base_frame)_joint" type="fixed">
+    <origin rpy="0 0 0" xyz="0 0 0"/>
     <parent link="$(arg hebi_base_frame)"/>
     <child link="Arm/J1_base/INPUT_INTERFACE"/>
   </joint>
-  <!-- robot -->
-  <xacro:actuator name="Arm/J1_base" child="shoulder_bracket" type="X8_9" limits="${[-pi,pi]}"/>
-  <xacro:bracket name="shoulder_bracket" child="Arm/J2_shoulder" type="X5HeavyRightOutside"/>
-  <xacro:actuator name="Arm/J2_shoulder" child="shoulder_elbow" type="X8_16" limits="${[-0.5,pi]}"/>
-  <xacro:link name="shoulder_elbow" child="Arm/J3_elbow" extension="0.325" twist="${pi}"/>
-  <xacro:actuator name="Arm/J3_elbow" child="elbow_wrist1" type="X8_9" limits="${[-3,3]}"/>
-  <xacro:link name="elbow_wrist1" child="Arm/J4_wrist1" extension="0.325" twist="${pi}"/>
-  <xacro:actuator name="Arm/J4_wrist1" child="wrist1_wrist2" type="X5_1" limits="${[-2 * pi,2 * pi]}"/>
-  <xacro:bracket name="wrist1_wrist2" child="Arm/J5_wrist2" type="X5LightRight"/>
-  <xacro:actuator name="Arm/J5_wrist2" child="end_effector" type="X5_1"/>
-  <!-- parallel gripper end effector -->
-  <xacro:gripper name="end_effector" type="parallel"/>
+  <xacro:actuator type="X8_9" name="Arm/J1_base" child="shoulder_bracket"/>
+  <xacro:bracket type="X5HeavyRightOutside" name="shoulder_bracket" child="Arm/J2_shoulder"/>
+  <xacro:actuator type="X8_16" name="Arm/J2_shoulder" child="shoulder_elbow"/>
+  <xacro:link type="X5" extension="0.325" twist="${pi}" name="shoulder_elbow" child="Arm/J3_elbow"/>
+  <xacro:actuator type="X8_9" name="Arm/J3_elbow" child="elbow_wrist1"/>
+  <xacro:link type="X5" extension="0.325" twist="${pi}" name="elbow_wrist1" child="Arm/J4_wrist1"/>
+  <xacro:actuator type="X5_1" name="Arm/J4_wrist1" child="wrist2_bracket"/>
+  <xacro:bracket type="X5LightRight" name="wrist2_bracket" child="Arm/J5_wrist2"/>
+  <xacro:actuator type="X5_1" name="Arm/J5_wrist2" child="end_effector"/>
+  <xacro:gripper type="X5Parallel" name="end_effector"/>
 </robot>

File: urdf/kits/A-2085-05.xacro (robot description, xacro)
@@ -22,4 +22,4 @@
   <xacro:bracket type="X5LightRight" name="wrist2_bracket" child="Arm/J5_wrist2"/>
   <xacro:actuator type="X5_1" name="Arm/J5_wrist2" child="end_effector"/>
-  <xacro:null_end_effector name="end_effector"/>
+  <xacro:gripper name="end_effector" type="Custom"/>
 </robot>

File: urdf/kits/A-2085-06-parallel-gripper.xacro (robot description, xacro)
@@ -1,29 +1,27 @@
-<?xml version="1.0"?>
-<robot xmlns:xacro="http://www.ros.org/wiki/xacro" name="A-2085-06">
+<?xml version='1.0' encoding='UTF-8'?>
+<robot xmlns:xacro="http://www.ros.org/wiki/xacro" version="1.2.0" name="A-2085-06-parallel-gripper">
   <!-- HEBI A-2085-06-parallel-gripper Arm Kit -->
   <xacro:include filename="$(find hebi_description)/urdf/hebi.xacro"/>
-  <xacro:arg name="hebi_base_frame" default="world"/>
+  <xacro:arg default="world" name="hebi_base_frame"/>
   <xacro:property name="hebi_base_frame" value="$(arg hebi_base_frame)"/>
   <xacro:if value="${hebi_base_frame == 'world'}">
     <link name="$(arg hebi_base_frame)"/>
   </xacro:if>
-  <joint name="$(arg hebi_base_frame)_arm_joint" type="fixed">
-    <origin xyz="0 0 0" rpy="0 0 0"/>
+  <joint name="$(arg hebi_base_frame)_joint" type="fixed">
+    <origin rpy="0 0 0" xyz="0 0 0"/>
     <parent link="$(arg hebi_base_frame)"/>
     <child link="Arm/J1_base/INPUT_INTERFACE"/>
   </joint>
-  <!-- robot -->
-  <xacro:actuator name="Arm/J1_base" child="shoulder_bracket" type="X8_9" limits="${[-pi,pi]}"/>
-  <xacro:bracket name="shoulder_bracket" child="Arm/J2_shoulder" type="X5HeavyRightOutside"/>
-  <xacro:actuator name="Arm/J2_shoulder" child="shoulder_elbow" type="X8_16" limits="${[-0.5,pi]}"/>
-  <xacro:link name="shoulder_elbow" child="Arm/J3_elbow" extension="0.325" twist="${pi}"/>
-  <xacro:actuator name="Arm/J3_elbow" child="elbow_wrist1" type="X8_9" limits="${[-3,3]}"/>
-  <xacro:link name="elbow_wrist1" child="Arm/J4_wrist1" extension="0.325" twist="${pi}"/>
-  <xacro:actuator name="Arm/J4_wrist1" child="wrist1_wrist2" type="X5_1" limits="${[-2 * pi, 2 * pi]}"/>
-  <xacro:bracket name="wrist1_wrist2" child="Arm/J5_wrist2" type="X5LightRight"/>
-  <xacro:actuator name="Arm/J5_wrist2" child="wrist2_wrist3" type="X5_1" limits="${[-1.5 * pi, 1.5 * pi]}"/>
-  <xacro:bracket name="wrist2_wrist3" child="Arm/J6_wrist3" type="X5LightRight"/>
-  <xacro:actuator name="Arm/J6_wrist3" child="end_effector" type="X5_1"/>
-  <!-- parallel gripper end effector -->
-  <xacro:gripper name="end_effector" type="parallel"/>
+  <xacro:actuator type="X8_9" name="Arm/J1_base" child="shoulder_bracket"/>
+  <xacro:bracket type="X5HeavyRightOutside" name="shoulder_bracket" child="Arm/J2_shoulder"/>
+  <xacro:actuator type="X8_16" name="Arm/J2_shoulder" child="shoulder_elbow"/>
+  <xacro:link type="X5" extension="0.325" twist="${pi}" name="shoulder_elbow" child="Arm/J3_elbow"/>
+  <xacro:actuator type="X8_9" name="Arm/J3_elbow" child="elbow_wrist1"/>
+  <xacro:link type="X5" extension="0.325" twist="${pi}" name="elbow_wrist1" child="Arm/J4_wrist1"/>
+  <xacro:actuator type="X5_1" name="Arm/J4_wrist1" child="wrist2_bracket"/>
+  <xacro:bracket type="X5LightRight" name="wrist2_bracket" child="Arm/J5_wrist2"/>
+  <xacro:actuator type="X5_1" name="Arm/J5_wrist2" child="wrist3_bracket"/>
+  <xacro:bracket type="X5LightRight" name="wrist3_bracket" child="Arm/J6_wrist3"/>
+  <xacro:actuator type="X5_1" name="Arm/J6_wrist3" child="end_effector"/>
+  <xacro:gripper type="X5Parallel" name="end_effector"/>
 </robot>

File: urdf/kits/A-2085-06.xacro (robot description, xacro)
@@ -24,4 +24,4 @@
   <xacro:bracket type="X5LightRight" name="wrist3_bracket" child="Arm/J6_wrist3"/>
   <xacro:actuator type="X5_1" name="Arm/J6_wrist3" child="end_effector"/>
-  <xacro:null_end_effector name="end_effector"/>
+  <xacro:gripper name="end_effector" type="Custom"/>
 </robot>

Commit message: Regenerate urdf/sdf from Melodic to match previous version

File: urdf/kits/A-2084-01-parallel-gripper.xacro (robot description, xacro)
@@ -3,5 +3,5 @@
   <!-- HEBI A-2084-01-parallel-gripper Arm Kit -->
   <xacro:include filename="$(find hebi_description)/urdf/hebi.xacro"/>
-  <xacro:arg default="world" name="hebi_base_frame"/>
+  <xacro:arg name="hebi_base_frame" default="world"/>
   <xacro:property name="hebi_base_frame" value="$(arg hebi_base_frame)"/>
   <xacro:if value="${hebi_base_frame == 'world'}">
@@ -9,5 +9,5 @@
   </xacro:if>
   <joint name="$(arg hebi_base_frame)_joint" type="fixed">
-    <origin rpy="0 0 0" xyz="0 0 0"/>
+    <origin xyz="0 0 0" rpy="0 0 0"/>
     <parent link="$(arg hebi_base_frame)"/>
     <child link="Arm/J1_base/INPUT_INTERFACE"/>

File: urdf/kits/A-2084-01.xacro (robot description, xacro)
@@ -3,5 +3,5 @@
   <!-- HEBI A-2084-01 Arm Kit -->
   <xacro:include filename="$(find hebi_description)/urdf/hebi.xacro"/>
-  <xacro:arg default="world" name="hebi_base_frame"/>
+  <xacro:arg name="hebi_base_frame" default="world"/>
   <xacro:property name="hebi_base_frame" value="$(arg hebi_base_frame)"/>
   <xacro:if value="${hebi_base_frame == 'world'}">
@@ -9,5 +9,5 @@
   </xacro:if>
   <joint name="$(arg hebi_base_frame)_joint" type="fixed">
-    <origin rpy="0 0 0" xyz="0 0 0"/>
+    <origin xyz="0 0 0" rpy="0 0 0"/>
     <parent link="$(arg hebi_base_frame)"/>
     <child link="Arm/J1_base/INPUT_INTERFACE"/>
@@ -20,4 +20,4 @@
   <xacro:link type="X5" extension="0.325" twist="0" name="elbow_wrist1" child="Arm/J4_wrist1"/>
   <xacro:actuator type="X5_1" name="Arm/J4_wrist1" child="end_effector"/>
-  <xacro:gripper name="end_effector" type="Custom"/>
+  <xacro:gripper type="Custom" name="end_effector"/>
 </robot>

File: urdf/kits/A-2085-04-parallel-gripper.xacro (robot description, xacro)
@@ -3,5 +3,5 @@
   <!-- HEBI A-2085-04-parallel-gripper Arm Kit -->
   <xacro:include filename="$(find hebi_description)/urdf/hebi.xacro"/>
-  <xacro:arg default="world" name="hebi_base_frame"/>
+  <xacro:arg name="hebi_base_frame" default="world"/>
   <xacro:property name="hebi_base_frame" value="$(arg hebi_base_frame)"/>
   <xacro:if value="${hebi_base_frame == 'world'}">
@@ -9,5 +9,5 @@
   </xacro:if>
   <joint name="$(arg hebi_base_frame)_joint" type="fixed">
-    <origin rpy="0 0 0" xyz="0 0 0"/>
+    <origin xyz="0 0 0" rpy="0 0 0"/>
     <parent link="$(arg hebi_base_frame)"/>
     <child link="Arm/J1_base/INPUT_INTERFACE"/>

File: urdf/kits/A-2085-04.xacro (robot description, xacro)
@@ -3,5 +3,5 @@
   <!-- HEBI A-2085-04 Arm Kit -->
   <xacro:include filename="$(find hebi_description)/urdf/hebi.xacro"/>
-  <xacro:arg default="world" name="hebi_base_frame"/>
+  <xacro:arg name="hebi_base_frame" default="world"/>
   <xacro:property name="hebi_base_frame" value="$(arg hebi_base_frame)"/>
   <xacro:if value="${hebi_base_frame == 'world'}">
@@ -9,5 +9,5 @@
   </xacro:if>
   <joint name="$(arg hebi_base_frame)_joint" type="fixed">
-    <origin rpy="0 0 0" xyz="0 0 0"/>
+    <origin xyz="0 0 0" rpy="0 0 0"/>
     <parent link="$(arg hebi_base_frame)"/>
     <child link="Arm/J1_base/INPUT_INTERFACE"/>
@@ -20,4 +20,4 @@
   <xacro:link type="X5" extension="0.325" twist="${pi}" name="elbow_wrist1" child="Arm/J4_wrist1"/>
   <xacro:actuator type="X5_1" name="Arm/J4_wrist1" child="end_effector"/>
-  <xacro:gripper name="end_effector" type="Custom"/>
+  <xacro:gripper type="Custom" name="end_effector"/>
 </robot>

File: urdf/kits/A-2085-05-parallel-gripper.xacro (robot description, xacro)
@@ -3,5 +3,5 @@
   <!-- HEBI A-2085-05-parallel-gripper Arm Kit -->
   <xacro:include filename="$(find hebi_description)/urdf/hebi.xacro"/>
-  <xacro:arg default="world" name="hebi_base_frame"/>
+  <xacro:arg name="hebi_base_frame" default="world"/>
   <xacro:property name="hebi_base_frame" value="$(arg hebi_base_frame)"/>
   <xacro:if value="${hebi_base_frame == 'world'}">
@@ -9,5 +9,5 @@
   </xacro:if>
   <joint name="$(arg hebi_base_frame)_joint" type="fixed">
-    <origin rpy="0 0 0" xyz="0 0 0"/>
+    <origin xyz="0 0 0" rpy="0 0 0"/>
     <parent link="$(arg hebi_base_frame)"/>
     <child link="Arm/J1_base/INPUT_INTERFACE"/>

File: urdf/kits/A-2085-05.xacro (robot description, xacro)
@@ -3,5 +3,5 @@
   <!-- HEBI A-2085-05 Arm Kit -->
   <xacro:include filename="$(find hebi_description)/urdf/hebi.xacro"/>
-  <xacro:arg default="world" name="hebi_base_frame"/>
+  <xacro:arg name="hebi_base_frame" default="world"/>
   <xacro:property name="hebi_base_frame" value="$(arg hebi_base_frame)"/>
   <xacro:if value="${hebi_base_frame == 'world'}">
@@ -9,5 +9,5 @@
   </xacro:if>
   <joint name="$(arg hebi_base_frame)_joint" type="fixed">
-    <origin rpy="0 0 0" xyz="0 0 0"/>
+    <origin xyz="0 0 0" rpy="0 0 0"/>
     <parent link="$(arg hebi_base_frame)"/>
     <child link="Arm/J1_base/INPUT_INTERFACE"/>
@@ -22,4 +22,4 @@
   <xacro:bracket type="X5LightRight" name="wrist2_bracket" child="Arm/J5_wrist2"/>
   <xacro:actuator type="X5_1" name="Arm/J5_wrist2" child="end_effector"/>
-  <xacro:gripper name="end_effector" type="Custom"/>
+  <xacro:gripper type="Custom" name="end_effector"/>
 </robot>

File: urdf/kits/A-2085-06-parallel-gripper.xacro (robot description, xacro)
@@ -3,5 +3,5 @@
   <!-- HEBI A-2085-06-parallel-gripper Arm Kit -->
   <xacro:include filename="$(find hebi_description)/urdf/hebi.xacro"/>
-  <xacro:arg default="world" name="hebi_base_frame"/>
+  <xacro:arg name="hebi_base_frame" default="world"/>
   <xacro:property name="hebi_base_frame" value="$(arg hebi_base_frame)"/>
   <xacro:if value="${hebi_base_frame == 'world'}">
@@ -9,5 +9,5 @@
   </xacro:if>
   <joint name="$(arg hebi_base_frame)_joint" type="fixed">
-    <origin rpy="0 0 0" xyz="0 0 0"/>
+    <origin xyz="0 0 0" rpy="0 0 0"/>
     <parent link="$(arg hebi_base_frame)"/>
     <child link="Arm/J1_base/INPUT_INTERFACE"/>

File: urdf/kits/A-2085-06.xacro (robot description, xacro)
@@ -3,5 +3,5 @@
   <!-- HEBI A-2085-06 Arm Kit -->
   <xacro:include filename="$(find hebi_description)/urdf/hebi.xacro"/>
-  <xacro:arg default="world" name="hebi_base_frame"/>
+  <xacro:arg name="hebi_base_frame" default="world"/>
   <xacro:property name="hebi_base_frame" value="$(arg hebi_base_frame)"/>
   <xacro:if value="${hebi_base_frame == 'world'}">
@@ -9,5 +9,5 @@
   </xacro:if>
   <joint name="$(arg hebi_base_frame)_joint" type="fixed">
-    <origin rpy="0 0 0" xyz="0 0 0"/>
+    <origin xyz="0 0 0" rpy="0 0 0"/>
     <parent link="$(arg hebi_base_frame)"/>
     <child link="Arm/J1_base/INPUT_INTERFACE"/>
@@ -24,4 +24,4 @@
   <xacro:bracket type="X5LightRight" name="wrist3_bracket" child="Arm/J6_wrist3"/>
   <xacro:actuator type="X5_1" name="Arm/J6_wrist3" child="end_effector"/>
-  <xacro:gripper name="end_effector" type="Custom"/>
+  <xacro:gripper type="Custom" name="end_effector"/>
 </robot>
