Commit message: Add collsion geometry

File: urdf/kits/cricket.xacro (robot description, xacro)
@@ -27,5 +27,5 @@
     </joint>
   </xacro:macro>
-  <xacro:macro name="double_input_spacer" params="mass size output_trans name output_name">
+  <xacro:macro name="dummy_spacer" params="mass size output_trans name">
     <link name="${name}/INPUT_INTERFACE">
       <visual>
@@ -44,11 +44,4 @@
       </inertial>
     </link>
-    <link name="${output_name}/INPUT_INTERFACE">
-    </link>
-    <joint name="${name}_child_joint" type="fixed">
-      <origin xyz="${output_trans}" rpy="0 0 0" />
-      <parent link="${name}/INPUT_INTERFACE"/>
-      <child link="${output_name}/INPUT_INTERFACE"/>
-    </joint>
   </xacro:macro>
   <xacro:macro name="drive_pulley" params="mass radius width name">
@@ -61,4 +54,10 @@
         <xacro:black_material/>
       </visual>
+      <collision>
+        <origin xyz="0 0 0" rpy="0 0 0" />
+        <geometry>
+          <cylinder radius="${radius}" length="${width}"/>
+        </geometry>
+      </collision>
       <inertial>
         <mass value="${mass}"/>
@@ -123,8 +122,8 @@
     <xacro:link type="X5" extension="0.275" twist="0"
 	    name="leg${leg_num}_knee_ankle" child="leg${leg_num}_ankle_spacer"/>
-    <xacro:double_input_spacer mass="0.5" size="0.01" output_trans="0 0 0"
-	    name="leg${leg_num}_ankle_spacer" output_name="leg${leg_num}_ankle_spacer_output"/>
+    <xacro:dummy_spacer mass="0.05" size="0.0" output_trans="0 0 0"
+	    name="leg${leg_num}_ankle_spacer"/>
     <xacro:reverse_actuator type="X8_16"
-	    name="${family}/L${leg_num}_J4_ankle" parent="leg${leg_num}_ankle_spacer_output" child="leg${leg_num}_tread_bracket_1"/>
+	    name="${family}/L${leg_num}_J4_ankle" parent="leg${leg_num}_ankle_spacer" child="leg${leg_num}_tread_bracket_1"/>
     <xacro:rigid_body mass="0.3" size="0.15 0.05 0.01" output_trans="-0.137 0 -0.01"
 	    name="leg${leg_num}_tread_bracket_1" child="leg${leg_num}_tread_bracket_2"/>
@@ -147,4 +146,10 @@
       <xacro:black_material/>
     </visual>
+    <collision>
+      <origin xyz="0 0 0" rpy="0 0 0" />
+      <geometry>
+        <box size="0.370 0.285 0.150"/>
+      </geometry>
+    </collision>
     <inertial>
       <mass value="2.0"/>

Commit message: Fix zero size collision box bug

File: urdf/kits/cricket.xacro (robot description, xacro)
@@ -27,13 +27,6 @@
     </joint>
   </xacro:macro>
-  <xacro:macro name="dummy_spacer" params="mass size output_trans name">
+  <xacro:macro name="dummy_spacer" params="mass name">
     <link name="${name}/INPUT_INTERFACE">
-      <visual>
-        <origin xyz="0 0 0" rpy="0 0 0" />
-        <geometry>
-		<cylinder radius="${0.025}" length="${size}"/>
-        </geometry>
-        <xacro:beige_material/>
-      </visual>
       <inertial>
         <mass value="${mass}"/>
@@ -122,6 +115,5 @@
     <xacro:link type="X5" extension="0.275" twist="0"
 	    name="leg${leg_num}_knee_ankle" child="leg${leg_num}_ankle_spacer"/>
-    <xacro:dummy_spacer mass="0.05" size="0.0" output_trans="0 0 0"
-	    name="leg${leg_num}_ankle_spacer"/>
+    <xacro:dummy_spacer mass="0.01" name="leg${leg_num}_ankle_spacer"/>
     <xacro:reverse_actuator type="X8_16"
 	    name="${family}/L${leg_num}_J4_ankle" parent="leg${leg_num}_ankle_spacer" child="leg${leg_num}_tread_bracket_1"/>
@@ -152,4 +144,6 @@
       </geometry>
     </collision>
+  </link>
+  <link name="cricket_base_inertia">
     <inertial>
       <mass value="2.0"/>
@@ -160,4 +154,8 @@
     </inertial>
   </link>
+  <joint name="cricket_base_inertia_joint" type="fixed">
+	  <parent link="cricket_base"/>
+	  <child link="cricket_base_inertia"/>
+  </joint>
   <xacro:cricket_leg type="left"  family="Cricket" leg_num="1" angle="${-pi/2} 0 0" offset="0.135 0.100 0.030" />
   <xacro:cricket_leg type="right" family="Cricket" leg_num="2" angle="${pi/2} 0 0" offset="0.135 -0.100 0.030" />
