Commit message: Use up-to-date macros

File: urdf/kits/rosie.xacro (robot description, xacro)
@@ -1,5 +1,5 @@
 <?xml version="1.0" ?>
 <robot name="rosie_test" xmlns:xacro="http://www.ros.org/wiki/xacro">
-  <xacro:include filename="$(find hebiros_description)/urdf/hebi.xacro"/>
+  <xacro:include filename="$(find hebi_description)/urdf/hebi.xacro"/>
   <link name="base_footprint"/>
   <joint name="base_joint" type="fixed">
@@ -13,5 +13,5 @@
       <geometry>
         <!--box size="0.50 0.50 0.10"/-->
-        <mesh filename="package://hebiros_description/meshes/rosie_base.stl" scale="0.001 0.001 0.001"/>
+        <mesh filename="package://hebi_description/meshes/rosie_base.stl" scale="0.001 0.001 0.001"/>
       </geometry>
       <material name="light_black"/>
@@ -42,7 +42,7 @@
     <axis xyz="0 0 1"/>
   </joint>
-  <xacro:x5 joint="HEBI/Wheel1" child="omniwheel1" model="X5_4"/>
-  <xacro:x5 joint="HEBI/Wheel2" child="omniwheel2" model="X5_4"/>
-  <xacro:x5 joint="HEBI/Wheel3" child="omniwheel3" model="X5_4"/>
+  <xacro:actuator type="X5_4" name="HEBI/Wheel1" child="omniwheel1"/>
+  <xacro:actuator type="X5_4" name="HEBI/Wheel2" child="omniwheel2"/>
+  <xacro:actuator type="X5_4" name="HEBI/Wheel3" child="omniwheel3"/>
   <link name="omniwheel1/INPUT_INTERFACE">
     <visual>
@@ -50,5 +50,5 @@
       <geometry>
         <!--box size="0.50 0.50 0.10"/-->
-        <mesh filename="package://hebiros_description/meshes/omniwheel.stl" scale="0.001 0.001 0.001"/>
+        <mesh filename="package://hebi_description/meshes/omniwheel.stl" scale="0.001 0.001 0.001"/>
       </geometry>
     </visual>
@@ -59,5 +59,5 @@
       <geometry>
         <!--box size="0.50 0.50 0.10"/-->
-        <mesh filename="package://hebiros_description/meshes/omni_25k.stl" scale="0.001 0.001 0.001"/>
+        <mesh filename="package://hebi_description/meshes/omni_25k.stl" scale="0.001 0.001 0.001"/>
       </geometry>
     </visual>
@@ -68,5 +68,5 @@
       <geometry>
         <!--box size="0.50 0.50 0.10"/-->
-        <mesh filename="package://hebiros_description/meshes/omni_25k.stl" scale="0.001 0.001 0.001"/>
+        <mesh filename="package://hebi_description/meshes/omni_25k.stl" scale="0.001 0.001 0.001"/>
       </geometry>
     </visual>
