Commit message: Updated script to generate URDF from HRDF - Regenerated URDFs for kits using new script

File: urdf/kits/A-2084-01-parallel-gripper.urdf.xacro (robot description, xacro)
@@ -1,19 +1,20 @@
 <?xml version='1.0' encoding='UTF-8'?>
-<robot xmlns:xacro="http://www.ros.org/wiki/xacro" name="A-2084-01-parallel-gripper">
+<robot xmlns:xacro="http://wiki.ros.org/xacro" version="1.2.0" name="A-2084-01-parallel-gripper">
+  <xacro:arg name="prefix" default=""/>
   <!-- HEBI A-2084-01-parallel-gripper Arm Kit -->
   <xacro:include filename="$(find hebi_description)/urdf/components/hebi.xacro"/>
-  <link name="base_link" />
-  <joint name="base_joint" type="fixed">
+  <link name="$(arg prefix)base_link"/>
+  <joint name="$(arg prefix)base_joint" type="fixed">
     <origin xyz="0 0 0" rpy="0 0 0"/>
-    <parent link="base_link" />
-    <child link="J1_base/INPUT_INTERFACE"/>
+    <parent link="$(arg prefix)base_link"/>
+    <child link="$(arg prefix)J1_base/INPUT_INTERFACE"/>
   </joint>
-  <xacro:actuator type="X5_4" name="J1_base" child="shoulder_bracket"/>
-  <xacro:bracket type="X5HeavyRightOutside" name="shoulder_bracket" child="J2_shoulder"/>
-  <xacro:actuator type="X5_9" name="J2_shoulder" child="shoulder_elbow"/>
-  <xacro:link type="X5" extension="0.325" twist="${pi/2}" name="shoulder_elbow" child="J3_elbow"/>
-  <xacro:actuator type="X5_4" name="J3_elbow" child="elbow_wrist"/>
-  <xacro:link type="X5" extension="0.325" twist="0" name="elbow_wrist" child="J4_wrist"/>
-  <xacro:actuator type="X5_1" name="J4_wrist" child="end_effector"/>
-  <xacro:gripper type="X5Parallel" name="end_effector"/>
+  <xacro:actuator type="X5_4" name="$(arg prefix)J1_base" child="$(arg prefix)shoulder_bracket"/>
+  <xacro:bracket type="X5HeavyRightOutside" name="$(arg prefix)shoulder_bracket" child="$(arg prefix)J2_shoulder"/>
+  <xacro:actuator type="X5_9" name="$(arg prefix)J2_shoulder" child="$(arg prefix)shoulder_elbow"/>
+  <xacro:link type="X5" extension="0.325" twist="${pi/2}" name="$(arg prefix)shoulder_elbow" child="$(arg prefix)J3_elbow"/>
+  <xacro:actuator type="X5_4" name="$(arg prefix)J3_elbow" child="$(arg prefix)elbow_wrist"/>
+  <xacro:link type="X5" extension="0.325" twist="0" name="$(arg prefix)elbow_wrist" child="$(arg prefix)J4_wrist"/>
+  <xacro:actuator type="X5_1" name="$(arg prefix)J4_wrist" child="$(arg prefix)end_effector"/>
+  <xacro:gripper type="X5Parallel" name="$(arg prefix)end_effector"/>
 </robot>

File: urdf/kits/A-2084-01.urdf.xacro (robot description, xacro)
@@ -1,19 +1,20 @@
 <?xml version='1.0' encoding='UTF-8'?>
-<robot xmlns:xacro="http://www.ros.org/wiki/xacro" name="A-2084-01">
+<robot xmlns:xacro="http://wiki.ros.org/xacro" version="1.1.0" name="A-2084-01">
+  <xacro:arg name="prefix" default=""/>
   <!-- HEBI A-2084-01 Arm Kit -->
   <xacro:include filename="$(find hebi_description)/urdf/components/hebi.xacro"/>
-  <link name="base_link" />
-  <joint name="base_joint" type="fixed">
+  <link name="$(arg prefix)base_link"/>
+  <joint name="$(arg prefix)base_joint" type="fixed">
     <origin xyz="0 0 0" rpy="0 0 0"/>
-    <parent link="base_link" />
-    <child link="J1_base/INPUT_INTERFACE"/>
+    <parent link="$(arg prefix)base_link"/>
+    <child link="$(arg prefix)J1_base/INPUT_INTERFACE"/>
   </joint>
-  <xacro:actuator type="X5_4" name="J1_base" child="shoulder_bracket"/>
-  <xacro:bracket type="X5HeavyRightOutside" name="shoulder_bracket" child="J2_shoulder"/>
-  <xacro:actuator type="X5_9" name="J2_shoulder" child="shoulder_elbow"/>
-  <xacro:link type="X5" extension="0.325" twist="${pi/2}" name="shoulder_elbow" child="J3_elbow"/>
-  <xacro:actuator type="X5_4" name="J3_elbow" child="elbow_wrist"/>
-  <xacro:link type="X5" extension="0.325" twist="0" name="elbow_wrist" child="J4_wrist"/>
-  <xacro:actuator type="X5_1" name="J4_wrist" child="end_effector"/>
+  <xacro:actuator type="X5_4" name="$(arg prefix)J1_base" child="$(arg prefix)shoulder_bracket"/>
+  <xacro:bracket type="X5HeavyRightOutside" name="$(arg prefix)shoulder_bracket" child="$(arg prefix)J2_shoulder"/>
+  <xacro:actuator type="X5_9" name="$(arg prefix)J2_shoulder" child="$(arg prefix)shoulder_elbow"/>
+  <xacro:link type="X5" extension="0.325" twist="${pi/2}" name="$(arg prefix)shoulder_elbow" child="$(arg prefix)J3_elbow"/>
+  <xacro:actuator type="X5_4" name="$(arg prefix)J3_elbow" child="$(arg prefix)elbow_wrist"/>
+  <xacro:link type="X5" extension="0.325" twist="0" name="$(arg prefix)elbow_wrist" child="$(arg prefix)J4_wrist"/>
+  <xacro:actuator type="X5_1" name="$(arg prefix)J4_wrist" child="end_effector"/>
   <xacro:gripper type="Custom" name="end_effector" mass="0.005"/>
 </robot>

File: urdf/kits/A-2085-04-parallel-gripper.urdf.xacro (robot description, xacro)
@@ -1,19 +1,20 @@
 <?xml version='1.0' encoding='UTF-8'?>
-<robot xmlns:xacro="http://www.ros.org/wiki/xacro" name="A-2085-04-parallel-gripper">
+<robot xmlns:xacro="http://wiki.ros.org/xacro" version="1.2.0" name="A-2085-04-parallel-gripper">
+  <xacro:arg name="prefix" default=""/>
   <!-- HEBI A-2085-04-parallel-gripper Arm Kit -->
   <xacro:include filename="$(find hebi_description)/urdf/components/hebi.xacro"/>
-  <link name="base_link" />
-  <joint name="base_joint" type="fixed">
+  <link name="$(arg prefix)base_link"/>
+  <joint name="$(arg prefix)base_joint" type="fixed">
     <origin xyz="0 0 0" rpy="0 0 0"/>
-    <parent link="base_link" />
-    <child link="J1_base/INPUT_INTERFACE"/>
+    <parent link="$(arg prefix)base_link"/>
+    <child link="$(arg prefix)J1_base/INPUT_INTERFACE"/>
   </joint>
-  <xacro:actuator type="X5_4" name="J1_base" child="shoulder_bracket"/>
-  <xacro:bracket type="X5HeavyRightOutside" name="shoulder_bracket" child="J2_shoulder"/>
-  <xacro:actuator type="X5_9" name="J2_shoulder" child="shoulder_elbow"/>
-  <xacro:link type="X5" extension="0.325" twist="${pi}" name="shoulder_elbow" child="J3_elbow"/>
-  <xacro:actuator type="X5_4" name="J3_elbow" child="elbow_wrist"/>
-  <xacro:link type="X5" extension="0.325" twist="${pi}" name="elbow_wrist" child="J4_wrist"/>
-  <xacro:actuator type="X5_1" name="J4_wrist" child="end_effector"/>
-  <xacro:gripper type="X5Parallel" name="end_effector"/>
+  <xacro:actuator type="X5_4" name="$(arg prefix)J1_base" child="$(arg prefix)shoulder_bracket"/>
+  <xacro:bracket type="X5HeavyRightOutside" name="$(arg prefix)shoulder_bracket" child="$(arg prefix)J2_shoulder"/>
+  <xacro:actuator type="X5_9" name="$(arg prefix)J2_shoulder" child="$(arg prefix)shoulder_elbow"/>
+  <xacro:link type="X5" extension="0.325" twist="${pi}" name="$(arg prefix)shoulder_elbow" child="$(arg prefix)J3_elbow"/>
+  <xacro:actuator type="X5_4" name="$(arg prefix)J3_elbow" child="$(arg prefix)elbow_wrist"/>
+  <xacro:link type="X5" extension="0.325" twist="${pi}" name="$(arg prefix)elbow_wrist" child="$(arg prefix)J4_wrist"/>
+  <xacro:actuator type="X5_1" name="$(arg prefix)J4_wrist" child="$(arg prefix)end_effector"/>
+  <xacro:gripper type="X5Parallel" name="$(arg prefix)end_effector"/>
 </robot>

File: urdf/kits/A-2085-04.urdf.xacro (robot description, xacro)
@@ -1,19 +1,20 @@
 <?xml version='1.0' encoding='UTF-8'?>
-<robot xmlns:xacro="http://www.ros.org/wiki/xacro" name="A-2085-04">
+<robot xmlns:xacro="http://wiki.ros.org/xacro" version="1.1.0" name="A-2085-04">
+  <xacro:arg name="prefix" default=""/>
   <!-- HEBI A-2085-04 Arm Kit -->
   <xacro:include filename="$(find hebi_description)/urdf/components/hebi.xacro"/>
-  <link name="base_link" />
-  <joint name="base_joint" type="fixed">
+  <link name="$(arg prefix)base_link"/>
+  <joint name="$(arg prefix)base_joint" type="fixed">
     <origin xyz="0 0 0" rpy="0 0 0"/>
-    <parent link="base_link" />
-    <child link="J1_base/INPUT_INTERFACE"/>
+    <parent link="$(arg prefix)base_link"/>
+    <child link="$(arg prefix)J1_base/INPUT_INTERFACE"/>
   </joint>
-  <xacro:actuator type="X5_4" name="J1_base" child="shoulder_bracket"/>
-  <xacro:bracket type="X5HeavyRightOutside" name="shoulder_bracket" child="J2_shoulder"/>
-  <xacro:actuator type="X5_9" name="J2_shoulder" child="shoulder_elbow"/>
-  <xacro:link type="X5" extension="0.325" twist="${pi}" name="shoulder_elbow" child="J3_elbow"/>
-  <xacro:actuator type="X5_4" name="J3_elbow" child="elbow_wrist"/>
-  <xacro:link type="X5" extension="0.325" twist="${pi}" name="elbow_wrist" child="J4_wrist"/>
-  <xacro:actuator type="X5_1" name="J4_wrist" child="end_effector"/>
+  <xacro:actuator type="X5_4" name="$(arg prefix)J1_base" child="$(arg prefix)shoulder_bracket"/>
+  <xacro:bracket type="X5HeavyRightOutside" name="$(arg prefix)shoulder_bracket" child="$(arg prefix)J2_shoulder"/>
+  <xacro:actuator type="X5_9" name="$(arg prefix)J2_shoulder" child="$(arg prefix)shoulder_elbow"/>
+  <xacro:link type="X5" extension="0.325" twist="${pi}" name="$(arg prefix)shoulder_elbow" child="$(arg prefix)J3_elbow"/>
+  <xacro:actuator type="X5_4" name="$(arg prefix)J3_elbow" child="$(arg prefix)elbow_wrist"/>
+  <xacro:link type="X5" extension="0.325" twist="${pi}" name="$(arg prefix)elbow_wrist" child="$(arg prefix)J4_wrist"/>
+  <xacro:actuator type="X5_1" name="$(arg prefix)J4_wrist" child="end_effector"/>
   <xacro:gripper type="Custom" name="end_effector" mass="0.005"/>
 </robot>

File: urdf/kits/A-2085-05-parallel-gripper.urdf.xacro (robot description, xacro)
@@ -1,21 +1,22 @@
 <?xml version='1.0' encoding='UTF-8'?>
-<robot xmlns:xacro="http://www.ros.org/wiki/xacro" name="A-2085-05-parallel-gripper">
+<robot xmlns:xacro="http://wiki.ros.org/xacro" version="1.2.0" name="A-2085-05-parallel-gripper">
+  <xacro:arg name="prefix" default=""/>
   <!-- HEBI A-2085-05-parallel-gripper Arm Kit -->
   <xacro:include filename="$(find hebi_description)/urdf/components/hebi.xacro"/>
-  <link name="base_link" />
-  <joint name="base_joint" type="fixed">
+  <link name="$(arg prefix)base_link"/>
+  <joint name="$(arg prefix)base_joint" type="fixed">
     <origin xyz="0 0 0" rpy="0 0 0"/>
-    <parent link="base_link" />
-    <child link="J1_base/INPUT_INTERFACE"/>
+    <parent link="$(arg prefix)base_link"/>
+    <child link="$(arg prefix)J1_base/INPUT_INTERFACE"/>
   </joint>
-  <xacro:actuator type="X8_9" name="J1_base" child="shoulder_bracket"/>
-  <xacro:bracket type="X5HeavyRightOutside" name="shoulder_bracket" child="J2_shoulder"/>
-  <xacro:actuator type="X8_16" name="J2_shoulder" child="shoulder_elbow"/>
-  <xacro:link type="X5" extension="0.325" twist="${pi}" name="shoulder_elbow" child="J3_elbow"/>
-  <xacro:actuator type="X8_9" name="J3_elbow" child="elbow_wrist1"/>
-  <xacro:link type="X5" extension="0.325" twist="${pi}" name="elbow_wrist1" child="J4_wrist1"/>
-  <xacro:actuator type="X5_1" name="J4_wrist1" child="wrist2_bracket"/>
-  <xacro:bracket type="X5LightRight" name="wrist2_bracket" child="J5_wrist2"/>
-  <xacro:actuator type="X5_1" name="J5_wrist2" child="end_effector"/>
-  <xacro:gripper type="X5Parallel" name="end_effector"/>
+  <xacro:actuator type="X8_9" name="$(arg prefix)J1_base" child="$(arg prefix)shoulder_bracket"/>
+  <xacro:bracket type="X5HeavyRightOutside" name="$(arg prefix)shoulder_bracket" child="$(arg prefix)J2_shoulder"/>
+  <xacro:actuator type="X8_16" name="$(arg prefix)J2_shoulder" child="$(arg prefix)shoulder_elbow"/>
+  <xacro:link type="X5" extension="0.325" twist="${pi}" name="$(arg prefix)shoulder_elbow" child="$(arg prefix)J3_elbow"/>
+  <xacro:actuator type="X8_9" name="$(arg prefix)J3_elbow" child="$(arg prefix)elbow_wrist1"/>
+  <xacro:link type="X5" extension="0.325" twist="${pi}" name="$(arg prefix)elbow_wrist1" child="$(arg prefix)J4_wrist1"/>
+  <xacro:actuator type="X5_1" name="$(arg prefix)J4_wrist1" child="$(arg prefix)wrist2_bracket"/>
+  <xacro:bracket type="X5LightRight" name="$(arg prefix)wrist2_bracket" child="$(arg prefix)J5_wrist2"/>
+  <xacro:actuator type="X5_1" name="$(arg prefix)J5_wrist2" child="$(arg prefix)end_effector"/>
+  <xacro:gripper type="X5Parallel" name="$(arg prefix)end_effector"/>
 </robot>

File: urdf/kits/A-2085-05.urdf.xacro (robot description, xacro)
@@ -1,11 +1,11 @@
 <?xml version='1.0' encoding='UTF-8'?>
-<robot xmlns:xacro="http://www.ros.org/wiki/xacro" name="A-2085-05">
-  <xacro:arg name="prefix" default="" />
+<robot xmlns:xacro="http://wiki.ros.org/xacro" version="1.2.0" name="A-2085-05">
+  <xacro:arg name="prefix" default=""/>
   <!-- HEBI A-2085-05 Arm Kit -->
   <xacro:include filename="$(find hebi_description)/urdf/components/hebi.xacro"/>
-  <link name="$(arg prefix)base_link" />
+  <link name="$(arg prefix)base_link"/>
   <joint name="$(arg prefix)base_joint" type="fixed">
     <origin xyz="0 0 0" rpy="0 0 0"/>
-    <parent link="$(arg prefix)base_link" />
+    <parent link="$(arg prefix)base_link"/>
     <child link="$(arg prefix)J1_base/INPUT_INTERFACE"/>
   </joint>

File: urdf/kits/A-2085-06-parallel-gripper.urdf.xacro (robot description, xacro)
@@ -1,23 +1,24 @@
 <?xml version='1.0' encoding='UTF-8'?>
-<robot xmlns:xacro="http://www.ros.org/wiki/xacro" name="A-2085-06-parallel-gripper">
+<robot xmlns:xacro="http://wiki.ros.org/xacro" version="1.2.0" name="A-2085-06-parallel-gripper">
+  <xacro:arg name="prefix" default=""/>
   <!-- HEBI A-2085-06-parallel-gripper Arm Kit -->
   <xacro:include filename="$(find hebi_description)/urdf/components/hebi.xacro"/>
-  <link name="base_link" />
-  <joint name="base_joint" type="fixed">
+  <link name="$(arg prefix)base_link"/>
+  <joint name="$(arg prefix)base_joint" type="fixed">
     <origin xyz="0 0 0" rpy="0 0 0"/>
-    <parent link="base_link" />
-    <child link="J1_base/INPUT_INTERFACE"/>
+    <parent link="$(arg prefix)base_link"/>
+    <child link="$(arg prefix)J1_base/INPUT_INTERFACE"/>
   </joint>
-  <xacro:actuator type="X8_9" name="J1_base" child="shoulder_bracket"/>
-  <xacro:bracket type="X5HeavyRightOutside" name="shoulder_bracket" child="J2_shoulder"/>
-  <xacro:actuator type="X8_16" name="J2_shoulder" child="shoulder_elbow"/>
-  <xacro:link type="X5" extension="0.325" twist="${pi}" name="shoulder_elbow" child="J3_elbow"/>
-  <xacro:actuator type="X8_9" name="J3_elbow" child="elbow_wrist1"/>
-  <xacro:link type="X5" extension="0.325" twist="${pi}" name="elbow_wrist1" child="J4_wrist1"/>
-  <xacro:actuator type="X5_1" name="J4_wrist1" child="wrist2_bracket"/>
-  <xacro:bracket type="X5LightRight" name="wrist2_bracket" child="J5_wrist2"/>
-  <xacro:actuator type="X5_1" name="J5_wrist2" child="wrist3_bracket"/>
-  <xacro:bracket type="X5LightRight" name="wrist3_bracket" child="J6_wrist3"/>
-  <xacro:actuator type="X5_1" name="J6_wrist3" child="end_effector"/>
-  <xacro:gripper type="X5Parallel" name="end_effector"/>
+  <xacro:actuator type="X8_9" name="$(arg prefix)J1_base" child="$(arg prefix)shoulder_bracket"/>
+  <xacro:bracket type="X5HeavyRightOutside" name="$(arg prefix)shoulder_bracket" child="$(arg prefix)J2_shoulder"/>
+  <xacro:actuator type="X8_16" name="$(arg prefix)J2_shoulder" child="$(arg prefix)shoulder_elbow"/>
+  <xacro:link type="X5" extension="0.325" twist="${pi}" name="$(arg prefix)shoulder_elbow" child="$(arg prefix)J3_elbow"/>
+  <xacro:actuator type="X8_9" name="$(arg prefix)J3_elbow" child="$(arg prefix)elbow_wrist1"/>
+  <xacro:link type="X5" extension="0.325" twist="${pi}" name="$(arg prefix)elbow_wrist1" child="$(arg prefix)J4_wrist1"/>
+  <xacro:actuator type="X5_1" name="$(arg prefix)J4_wrist1" child="$(arg prefix)wrist2_bracket"/>
+  <xacro:bracket type="X5LightRight" name="$(arg prefix)wrist2_bracket" child="$(arg prefix)J5_wrist2"/>
+  <xacro:actuator type="X5_1" name="$(arg prefix)J5_wrist2" child="$(arg prefix)wrist3_bracket"/>
+  <xacro:bracket type="X5LightRight" name="$(arg prefix)wrist3_bracket" child="$(arg prefix)J6_wrist3"/>
+  <xacro:actuator type="X5_1" name="$(arg prefix)J6_wrist3" child="$(arg prefix)end_effector"/>
+  <xacro:gripper type="X5Parallel" name="$(arg prefix)end_effector"/>
 </robot>

File: urdf/kits/A-2085-06.urdf.xacro (robot description, xacro)
@@ -1,11 +1,11 @@
-<?xml version="1.0" encoding="UTF-8"?>
-<robot xmlns:xacro="http://wiki.ros.org/xacro" name="A-2085-06">
-  <xacro:arg name="prefix" default="" />
+<?xml version='1.0' encoding='UTF-8'?>
+<robot xmlns:xacro="http://wiki.ros.org/xacro" version="1.2.0" name="A-2085-06">
+  <xacro:arg name="prefix" default=""/>
   <!-- HEBI A-2085-06 Arm Kit -->
-  <xacro:include filename="$(find hebi_description)/urdf/components/hebi.xacro" />
-  <link name="$(arg prefix)base_link" />
+  <xacro:include filename="$(find hebi_description)/urdf/components/hebi.xacro"/>
+  <link name="$(arg prefix)base_link"/>
   <joint name="$(arg prefix)base_joint" type="fixed">
     <origin xyz="0 0 0" rpy="0 0 0"/>
-    <parent link="$(arg prefix)base_link" />
+    <parent link="$(arg prefix)base_link"/>
     <child link="$(arg prefix)J1_base/INPUT_INTERFACE"/>
   </joint>
