Commit message: New URDF files for kits including the new T-Series

File: urdf/kits/A-2085-03.urdf.xacro (robot description, xacro)
@@ -1,6 +1,6 @@
 <?xml version='1.0' encoding='UTF-8'?>
-<robot xmlns:xacro="http://wiki.ros.org/xacro" name="A-2084-01">
+<robot xmlns:xacro="http://wiki.ros.org/xacro" name="A-2085-03">
   <xacro:arg name="prefix" default=""/>
-  <!-- HEBI A-2084-01 Arm Kit -->
+  <!-- HEBI A-2085-03 Arm Kit -->
   <xacro:include filename="$(find hebi_description)/urdf/components/hebi.xacro"/>
   <link name="$(arg prefix)base_link"/>
@@ -14,8 +14,6 @@
   <xacro:output type="X5HeavyRightOutside" parent="$(arg prefix)B1" child="$(arg prefix)J2_shoulder" name="$(arg prefix)B1_J2_shoulder"/>
   <xacro:actuator type="X5_9" name="$(arg prefix)J2_shoulder" child="$(arg prefix)L1"/>
-  <xacro:link type="X5" extension="0.325" twist="${-pi/2}" name="$(arg prefix)L1" child="$(arg prefix)J3_elbow" output="RightAngle"/>
-  <xacro:actuator type="X5_4" name="$(arg prefix)J3_elbow" child="$(arg prefix)L2"/>
-  <xacro:link type="X5" extension="0.325" twist="0" name="$(arg prefix)L2" child="$(arg prefix)J4_wrist" output="RightAngle"/>
-  <xacro:actuator type="X5_1" name="$(arg prefix)J4_wrist" child="$(arg prefix)EE1"/>
+  <xacro:link type="X5" extension="0.325" twist="${pi}" name="$(arg prefix)L1" child="$(arg prefix)J3_elbow" output="RightAngle"/>
+  <xacro:actuator type="X5_4" name="$(arg prefix)J3_elbow" child="$(arg prefix)EE1"/>
   <xacro:gripper name="$(arg prefix)EE1" type="Custom" mass="0.01"/>
 </robot>

File: urdf/kits/A-2085-04.urdf.xacro (robot description, xacro)
@@ -8,13 +8,14 @@
     <origin xyz="0 0 0" rpy="0 0 0"/>
     <parent link="$(arg prefix)base_link"/>
-    <child link="$(arg prefix)J1_base/INPUT_INTERFACE"/>
+    <child link="$(arg prefix)J1_base"/>
   </joint>
-  <xacro:actuator type="X5_4" name="$(arg prefix)J1_base" child="$(arg prefix)shoulder_bracket"/>
-  <xacro:bracket type="X5HeavyRightOutside" name="$(arg prefix)shoulder_bracket" child="$(arg prefix)J2_shoulder"/>
-  <xacro:actuator type="X5_9" name="$(arg prefix)J2_shoulder" child="$(arg prefix)shoulder_elbow"/>
-  <xacro:link type="X5" extension="0.325" twist="${pi}" name="$(arg prefix)shoulder_elbow" child="$(arg prefix)J3_elbow"/>
-  <xacro:actuator type="X5_4" name="$(arg prefix)J3_elbow" child="$(arg prefix)elbow_wrist"/>
-  <xacro:link type="X5" extension="0.325" twist="${pi}" name="$(arg prefix)elbow_wrist" child="$(arg prefix)J4_wrist"/>
-  <xacro:actuator type="X5_1" name="$(arg prefix)J4_wrist" child="end_effector"/>
-  <xacro:gripper type="Custom" name="end_effector" mass="0.005"/>
+  <xacro:actuator type="X5_4" name="$(arg prefix)J1_base" child="$(arg prefix)B1"/>
+  <xacro:bracket type="X5HeavyRightOutside" name="$(arg prefix)B1"/>
+  <xacro:output type="X5HeavyRightOutside" parent="$(arg prefix)B1" child="$(arg prefix)J2_shoulder" name="$(arg prefix)B1_J2_shoulder"/>
+  <xacro:actuator type="X5_9" name="$(arg prefix)J2_shoulder" child="$(arg prefix)L1"/>
+  <xacro:link type="X5" extension="0.325" twist="${pi}" name="$(arg prefix)L1" child="$(arg prefix)J3_elbow" input="Inline" output="RightAngle"/>
+  <xacro:actuator type="X5_4" name="$(arg prefix)J3_elbow" child="$(arg prefix)L2"/>
+  <xacro:link type="X5" extension="0.325" twist="${pi}" name="$(arg prefix)L2" child="$(arg prefix)J4_wrist" output="RightAngle"/>
+  <xacro:actuator type="X5_1" name="$(arg prefix)J4_wrist" child="$(arg prefix)EE1"/>
+  <xacro:gripper name="$(arg prefix)EE1" type="Custom" mass="0.01"/>
 </robot>

File: urdf/kits/A-2085-05.urdf.xacro (robot description, xacro)
@@ -8,15 +8,17 @@
     <origin xyz="0 0 0" rpy="0 0 0"/>
     <parent link="$(arg prefix)base_link"/>
-    <child link="$(arg prefix)J1_base/INPUT_INTERFACE"/>
+    <child link="$(arg prefix)J1_base"/>
   </joint>
-  <xacro:actuator type="X8_9" name="$(arg prefix)J1_base" child="$(arg prefix)shoulder_bracket"/>
-  <xacro:bracket type="X5HeavyRightOutside" name="$(arg prefix)shoulder_bracket" child="$(arg prefix)J2_shoulder"/>
-  <xacro:actuator type="X8_16" name="$(arg prefix)J2_shoulder" child="$(arg prefix)shoulder_elbow"/>
-  <xacro:link type="X5" extension="0.325" twist="${pi}" name="$(arg prefix)shoulder_elbow" child="$(arg prefix)J3_elbow"/>
-  <xacro:actuator type="X8_9" name="$(arg prefix)J3_elbow" child="$(arg prefix)elbow_wrist1"/>
-  <xacro:link type="X5" extension="0.325" twist="${pi}" name="$(arg prefix)elbow_wrist1" child="$(arg prefix)J4_wrist1"/>
-  <xacro:actuator type="X5_1" name="$(arg prefix)J4_wrist1" child="$(arg prefix)wrist2_bracket"/>
-  <xacro:bracket type="X5LightRight" name="$(arg prefix)wrist2_bracket" child="$(arg prefix)J5_wrist2"/>
-  <xacro:actuator type="X5_1" name="$(arg prefix)J5_wrist2" child="$(arg prefix)end_effector"/>
-  <xacro:gripper type="Custom" name="$(arg prefix)end_effector" mass="0.005"/>
+  <xacro:actuator type="X8_9" name="$(arg prefix)J1_base" child="$(arg prefix)B1"/>
+  <xacro:bracket type="X5HeavyRightOutside" name="$(arg prefix)B1"/>
+  <xacro:output type="X5HeavyRightOutside" parent="$(arg prefix)B1" child="$(arg prefix)J2_shoulder" name="$(arg prefix)B1_J2_shoulder"/>
+  <xacro:actuator type="X8_16" name="$(arg prefix)J2_shoulder" child="$(arg prefix)L1"/>
+  <xacro:link type="X5" extension="0.325" twist="${pi}" name="$(arg prefix)L1" child="$(arg prefix)J3_elbow" output="RightAngle"/>
+  <xacro:actuator type="X8_9" name="$(arg prefix)J3_elbow" child="$(arg prefix)L2"/>
+  <xacro:link type="X5" extension="0.325" twist="${pi}" name="$(arg prefix)L2" child="$(arg prefix)J4_wrist1" output="RightAngle"/>
+  <xacro:actuator type="X5_1" name="$(arg prefix)J4_wrist1" child="$(arg prefix)B2"/>
+  <xacro:bracket type="X5LightRight" name="$(arg prefix)B2"/>
+  <xacro:output type="X5LightRight" parent="$(arg prefix)B2" child="$(arg prefix)J5_wrist2" name="$(arg prefix)B2_J5_wrist2"/>
+  <xacro:actuator type="X5_1" name="$(arg prefix)J5_wrist2" child="$(arg prefix)EE1"/>
+  <xacro:gripper name="$(arg prefix)EE1" type="Custom" mass="0.01"/>
 </robot>

File: urdf/kits/A-2085-05G.urdf.xacro (robot description, xacro)
@@ -1,6 +1,6 @@
 <?xml version='1.0' encoding='UTF-8'?>
-<robot xmlns:xacro="http://wiki.ros.org/xacro" name="A-2085-06">
+<robot xmlns:xacro="http://wiki.ros.org/xacro" name="A-2085-05G">
   <xacro:arg name="prefix" default=""/>
-  <!-- HEBI A-2085-06 Arm Kit -->
+  <!-- HEBI A-2085-05G Arm Kit -->
   <xacro:include filename="$(find hebi_description)/urdf/components/hebi.xacro"/>
   <link name="$(arg prefix)base_link"/>
@@ -20,8 +20,5 @@
   <xacro:bracket type="X5LightRight" name="$(arg prefix)B2"/>
   <xacro:output type="X5LightRight" parent="$(arg prefix)B2" child="$(arg prefix)J5_wrist2" name="$(arg prefix)B2_J5_wrist2"/>
-  <xacro:actuator type="X5_1" name="$(arg prefix)J5_wrist2" child="$(arg prefix)B3"/>
-  <xacro:bracket type="X5LightRight" name="$(arg prefix)B3"/>
-  <xacro:output type="X5LightRight" parent="$(arg prefix)B3" child="$(arg prefix)J6_wrist3" name="$(arg prefix)B3_J6_wrist3"/>
-  <xacro:actuator type="X5_1" name="$(arg prefix)J6_wrist3" child="$(arg prefix)EE1"/>
-  <xacro:gripper name="$(arg prefix)EE1" type="Custom" mass="0.01"/>
+  <xacro:actuator type="X5_1" name="$(arg prefix)J5_wrist2" child="$(arg prefix)EE1"/>
+  <xacro:gripper type="X5Parallel" name="$(arg prefix)EE1" mass="0.01"/>
 </robot>

File: urdf/kits/A-2085-06G.urdf.xacro (robot description, xacro)
@@ -1,6 +1,6 @@
 <?xml version='1.0' encoding='UTF-8'?>
-<robot xmlns:xacro="http://wiki.ros.org/xacro" name="A-2085-06">
+<robot xmlns:xacro="http://wiki.ros.org/xacro" name="A-2085-06G">
   <xacro:arg name="prefix" default=""/>
-  <!-- HEBI A-2085-06 Arm Kit -->
+  <!-- HEBI A-2085-06G Arm Kit -->
   <xacro:include filename="$(find hebi_description)/urdf/components/hebi.xacro"/>
   <link name="$(arg prefix)base_link"/>
@@ -24,4 +24,4 @@
   <xacro:output type="X5LightRight" parent="$(arg prefix)B3" child="$(arg prefix)J6_wrist3" name="$(arg prefix)B3_J6_wrist3"/>
   <xacro:actuator type="X5_1" name="$(arg prefix)J6_wrist3" child="$(arg prefix)EE1"/>
-  <xacro:gripper name="$(arg prefix)EE1" type="Custom" mass="0.01"/>
+  <xacro:gripper type="X5Parallel" name="$(arg prefix)EE1" mass="0.01"/>
 </robot>
