Commit message: Updated URDF and HRDF

File: urdf/kits/A-2240-06.urdf.xacro (robot description, xacro)
@@ -23,23 +23,7 @@
   <xacro:bracket type="R8LightRight" name="$(arg prefix)bracket_3"/>
   <xacro:output type="R8LightRight" parent="$(arg prefix)bracket_3" child="$(arg prefix)J6_wrist3/body" name="$(arg prefix)bracket_3_J6_wrist3"/>
-  <xacro:actuator type="R8_3" name="$(arg prefix)J6_wrist3" child="$(arg prefix)link_3"/>
-  <link name="$(arg prefix)link_3">
-    <visual>
-      <geometry>
-        <cylinder length="0.0005" radius="0.0075"/>
-      </geometry>
-    </visual>
-    <collision>
-      <geometry>
-        <cylinder length="0.0005" radius="0.0075"/>
-      </geometry>
-    </collision>
-  </link>
-  <joint name="link3_to_ee" type="fixed">
-    <parent link="$(arg prefix)link_3"/>
-    <child link="$(arg prefix)rigid_body_1"/>
-  </joint>
-  <xacro:rigid-body mass="0.001" mesh_path="file://$(find hebi_description)/meshes/end_effector.stl" mesh_trans="-0.1 0.08 0.1725" mesh_rot="0 ${pi} ${pi}" mesh_scale="1 1 1" name="$(arg prefix)rigid_body_1"/>
+  <xacro:actuator type="R8_3" name="$(arg prefix)J6_wrist3" child="$(arg prefix)rigid_body_1"/>
+  <xacro:rigid-body mass="1.068" mesh_path="file://$(find hebi_description)/meshes/end_effector.stl" mesh_scale="1 1 1" name="$(arg prefix)rigid_body_1"/>
   <xacro:output trans="0 0 0" rot="0 0 0" parent="$(arg prefix)rigid_body_1" child="$(arg prefix)end_effector_1" name="$(arg prefix)rigid_body_1_end_effector_1"/>
-  <xacro:null_end_effector name="$(arg prefix)end_effector_1" output_trans="0.005 0 0.13"/>
+  <xacro:null_end_effector name="$(arg prefix)end_effector_1"/>
 </robot>
