Commit message: Updated mecanum wheels

File: urdf/kits/mecanum_base.urdf.xacro (robot description, xacro)
@@ -50,5 +50,5 @@
       <origin xyz="0 0 0" rpy="0 0 0" />
       <geometry>
-        <mesh filename="file://$(find hebi_description)/meshes/mecanum_wheel.stl"/>
+        <mesh filename="file://$(find hebi_description)/meshes/mecanum_wheel_right.obj"/>
       </geometry>
     </visual>
@@ -56,5 +56,5 @@
       <origin xyz="0 0 0" rpy="0 0 0" />
       <geometry>
-        <mesh filename="file://$(find hebi_description)/meshes/mecanum_wheel.stl"/>
+        <mesh filename="file://$(find hebi_description)/meshes/mecanum_wheel_right.obj"/>
       </geometry>
     </collision>
@@ -78,5 +78,5 @@
       <origin xyz="0 0 0" rpy="0 0 0" />
       <geometry>
-        <mesh filename="file://$(find hebi_description)/meshes/mecanum_wheel.stl"/>
+        <mesh filename="file://$(find hebi_description)/meshes/mecanum_wheel_left.obj"/>
       </geometry>
     </visual>
@@ -84,5 +84,5 @@
       <origin xyz="0 0 0" rpy="0 0 0" />
       <geometry>
-        <mesh filename="file://$(find hebi_description)/meshes/mecanum_wheel.stl"/>
+        <mesh filename="file://$(find hebi_description)/meshes/mecanum_wheel_left.obj"/>
       </geometry>
     </collision>
@@ -106,5 +106,5 @@
       <origin xyz="0 0 0" rpy="0 0 0" />
       <geometry>
-        <mesh filename="file://$(find hebi_description)/meshes/mecanum_wheel.stl"/>
+        <mesh filename="file://$(find hebi_description)/meshes/mecanum_wheel_left.obj"/>
       </geometry>
     </visual>
@@ -112,5 +112,5 @@
       <origin xyz="0 0 0" rpy="0 0 0" />
       <geometry>
-        <mesh filename="file://$(find hebi_description)/meshes/mecanum_wheel.stl"/>
+        <mesh filename="file://$(find hebi_description)/meshes/mecanum_wheel_left.obj"/>
       </geometry>
     </collision>
@@ -134,5 +134,5 @@
       <origin xyz="0 0 0" rpy="0 0 0" />
       <geometry>
-        <mesh filename="file://$(find hebi_description)/meshes/mecanum_wheel.stl"/>
+        <mesh filename="file://$(find hebi_description)/meshes/mecanum_wheel_right.obj"/>
       </geometry>
     </visual>
@@ -140,5 +140,5 @@
       <origin xyz="0 0 0" rpy="0 0 0" />
       <geometry>
-        <mesh filename="file://$(find hebi_description)/meshes/mecanum_wheel.stl"/>
+        <mesh filename="file://$(find hebi_description)/meshes/mecanum_wheel_right.obj"/>
       </geometry>
     </collision>
