Commit message: Added ROS2 Control for 5-dof arm (A_2085-05)

File: urdf/kits/ros2_control/A-2085-05.urdf.xacro (robot description, xacro)
@@ -1,4 +1,4 @@
 <?xml version="1.0" encoding="UTF-8"?>
-<robot xmlns:xacro="http://wiki.ros.org/xacro" name="A-2085-06">
+<robot xmlns:xacro="http://wiki.ros.org/xacro" name="A-2085-05">
   <xacro:arg name="families" default="" />
   <xacro:arg name="names" default="" />
@@ -10,5 +10,5 @@
   <xacro:arg name="mock_sensor_commands" default="false" />
   <xacro:arg name="sim_gazebo" default="false" />
-  <xacro:include filename="$(find hebi_description)/urdf/kits/ros2_control/A-2085-06_macro.ros2_control.xacro"/>
+  <xacro:include filename="$(find hebi_description)/urdf/kits/ros2_control/A-2085-05_macro.ros2_control.xacro"/>
   <!-- create link fixed to the "world" -->
   <link name="world" />
@@ -18,7 +18,7 @@
     <child link="base_link"/>
   </joint>
-  <xacro:include filename="$(find hebi_description)/urdf/kits/A-2085-06.urdf.xacro"/>
-  <xacro:A-2085-06_ros2_control
-    name="A-2085-06"
+  <xacro:include filename="$(find hebi_description)/urdf/kits/A-2085-05.urdf.xacro"/>
+  <xacro:A-2085-05_ros2_control
+    name="A-2085-05"
     use_mock_hardware="$(arg use_mock_hardware)"
     mock_sensor_commands="$(arg mock_sensor_commands)"

File: urdf/kits/ros2_control/A-2085-05_macro.ros2_control.xacro (robot description, xacro)
@@ -1,5 +1,5 @@
 <?xml version="1.0" encoding="UTF-8"?>
 <robot xmlns:xacro="http://wiki.ros.org/xacro">
-  <xacro:macro name="A-2085-06_ros2_control" params="
+  <xacro:macro name="A-2085-05_ros2_control" params="
                 name
                 use_mock_hardware:=^|false
@@ -67,11 +67,4 @@
         <state_interface name="velocity" />
       </joint>
-      <joint name="J6_wrist3">
-        <command_interface name="position" />
-        <state_interface name="position">
-          <param name="initial_value">0.0</param>
-        </state_interface>
-        <state_interface name="velocity" />
-      </joint>
     </ros2_control>
     <!-- Gazebo Classic plugins -->
@@ -79,5 +72,5 @@
       <gazebo>
         <plugin filename="libgazebo_ros2_control.so" name="gazebo_ros2_control">
-          <parameters>$(find hebi_bringup)/config/A-2085-06_controllers.yaml</parameters>
+          <parameters>$(find hebi_bringup)/config/A-2085-05_controllers.yaml</parameters>
         </plugin>
       </gazebo>
