Commit message: Fixed ros2 control xacros

File: urdf/kits/ros2_control/A-2085-05_macro.ros2_control.xacro (robot description, xacro)
@@ -91,5 +91,5 @@
     </ros2_control>
     <!-- Gazebo Classic plugins -->
-    <xacro:if value="$(arg sim_gazebo_classic)">
+    <xacro:if value="${sim_gazebo_classic}">
       <gazebo>
         <plugin filename="libgazebo_ros2_control.so" name="gazebo_ros2_control">
@@ -99,5 +99,5 @@
     </xacro:if>
     <!-- Gazebo plugins -->
-    <xacro:if value="$(arg sim_gazebo)">
+    <xacro:if value="${sim_gazebo}">
       <gazebo>
         <plugin filename="gz_ros2_control-system" name="gz_ros2_control::GazeboSimROS2ControlPlugin">

File: urdf/kits/ros2_control/A-2240-06_macro.ros2_control.xacro (robot description, xacro)
@@ -1,5 +1,5 @@
 <?xml version="1.0" encoding="UTF-8"?>
 <robot xmlns:xacro="http://wiki.ros.org/xacro">
-  <xacro:macro name="A-2085-06_ros2_control" params="
+  <xacro:macro name="A-2240-06_ros2_control" params="
                 name
                 prefix
@@ -26,5 +26,5 @@
         </xacro:if>
         <xacro:if value="${sim_gazebo}">
-          <plugin>gz_ros2_control/GazeboSimSystem</plugin>
+          <plugin>ign_ros2_control/IgnitionSystem</plugin>
         </xacro:if>
         <xacro:unless value="${use_mock_hardware or sim_gazebo_classic or sim_gazebo}">
@@ -104,5 +104,5 @@
       <gazebo>
         <plugin filename="libgazebo_ros2_control.so" name="gazebo_ros2_control">
-          <parameters>$(find hebi_bringup)/config/A-2085-06_controllers.yaml</parameters>
+          <parameters>$(find hebi_bringup)/config/A-2240-06_controllers.yaml</parameters>
         </plugin>
       </gazebo>
@@ -111,6 +111,6 @@
     <xacro:if value="${sim_gazebo}">
       <gazebo>
-        <plugin filename="gz_ros2_control-system" name="gz_ros2_control::GazeboSimROS2ControlPlugin">
-          <parameters>$(find hebi_bringup)/config/A-2085-06_controllers.yaml</parameters>
+        <plugin filename="ign_ros2_control-system" name="ign_ros2_control::IgnitionROS2ControlPlugin">
+          <parameters>$(find hebi_bringup)/config/A-2240-06_controllers.yaml</parameters>
         </plugin>
       </gazebo>
