Commit message: Fixed ros2 control xacros

File: urdf/kits/ros2_control/A-2085-06_macro.ros2_control.xacro (robot description, xacro)
@@ -97,5 +97,5 @@
     </ros2_control>
     <!-- Gazebo plugins -->
-    <xacro:if value="$(arg sim_gazebo)">
+    <xacro:if value="${sim_gazebo}">
       <gazebo>
         <plugin filename="gz_ros2_control-system" name="gz_ros2_control::GazeboSimROS2ControlPlugin">

File: urdf/kits/ros2_control/A-2240-06_macro.ros2_control.xacro (robot description, xacro)
@@ -1,5 +1,5 @@
 <?xml version="1.0" encoding="UTF-8"?>
 <robot xmlns:xacro="http://wiki.ros.org/xacro">
-  <xacro:macro name="A-2085-05_ros2_control" params="
+  <xacro:macro name="A-2240-06_ros2_control" params="
                 name
                 prefix
@@ -85,4 +85,14 @@
         </state_interface>
       </joint>
+      <joint name="${prefix}J6_wrist3">
+        <command_interface name="position" />
+        <command_interface name="velocity" />
+        <state_interface name="position">
+          <param name="initial_value">0.0</param>
+        </state_interface>
+        <state_interface name="velocity">
+          <param name="initial_value">0.0</param>
+        </state_interface>
+      </joint>
     </ros2_control>
     <!-- Gazebo plugins -->
@@ -90,5 +100,5 @@
       <gazebo>
         <plugin filename="gz_ros2_control-system" name="gz_ros2_control::GazeboSimROS2ControlPlugin">
-          <parameters>$(find hebi_bringup)/config/A-2085-05_controllers.yaml</parameters>
+          <parameters>$(find hebi_bringup)/config/A-2240-06_controllers.yaml</parameters>
         </plugin>
       </gazebo>
