Commit message: Updated ROS2 Control URDFs

File: urdf/kits/ros2_control/A-2084-01.ros2_control.xacro (robot description, xacro)
@@ -1,5 +1,5 @@
 <?xml version="1.0" encoding="UTF-8"?>
 <robot xmlns:xacro="http://wiki.ros.org/xacro">
-  <xacro:macro name="A-2085-06_ros2_control" params="
+  <xacro:macro name="A-2084-01_ros2_control" params="
                 name
                 prefix
@@ -10,5 +10,5 @@
                 config_pkg
                 config_file"
-               >
+  >
     <ros2_control name="${name}" type="system">
       <hardware>
@@ -59,25 +59,5 @@
         </state_interface>
       </joint>
-      <joint name="${prefix}J4_wrist1">
-        <command_interface name="position" />
-        <command_interface name="velocity" />
-        <state_interface name="position">
-          <param name="initial_value">0.0</param>
-        </state_interface>
-        <state_interface name="velocity">
-          <param name="initial_value">0.0</param>
-        </state_interface>
-      </joint>
-      <joint name="${prefix}J5_wrist2">
-        <command_interface name="position" />
-        <command_interface name="velocity" />
-        <state_interface name="position">
-          <param name="initial_value">0.0</param>
-        </state_interface>
-        <state_interface name="velocity">
-          <param name="initial_value">0.0</param>
-        </state_interface>
-      </joint>
-      <joint name="${prefix}J6_wrist3">
+      <joint name="${prefix}J4_wrist">
         <command_interface name="position" />
         <command_interface name="velocity" />
@@ -94,5 +74,5 @@
       <gazebo>
         <plugin filename="libgazebo_ros2_control.so" name="gazebo_ros2_control">
-          <parameters>$(find hebi_bringup)/config/A-2085-06_controllers.yaml</parameters>
+          <parameters>$(find hebi_bringup)/config/A-2084-01_controllers.yaml</parameters>
         </plugin>
       </gazebo>
@@ -102,5 +82,5 @@
       <gazebo>
         <plugin filename="ign_ros2_control-system" name="ign_ros2_control::IgnitionROS2ControlPlugin">
-          <parameters>$(find hebi_bringup)/config/A-2085-06_controllers.yaml</parameters>
+          <parameters>$(find hebi_bringup)/config/A-2084-01_controllers.yaml</parameters>
         </plugin>
       </gazebo>

File: urdf/kits/ros2_control/A-2084-01.urdf.xacro (robot description, xacro)
@@ -1,4 +1,4 @@
 <?xml version="1.0" encoding="UTF-8"?>
-<robot xmlns:xacro="http://wiki.ros.org/xacro" name="A-2240-06">
+<robot xmlns:xacro="http://wiki.ros.org/xacro" name="A-2084-01">
   <xacro:arg name="config_pkg" default="" />
   <xacro:arg name="config_file" default="" />
@@ -8,5 +8,5 @@
   <xacro:arg name="sim_gazebo_classic" default="false" />
   <xacro:arg name="sim_gazebo" default="false" />
-  <xacro:include filename="$(find hebi_description)/urdf/kits/ros2_control/A-2240-06.ros2_control.xacro" />
+  <xacro:include filename="$(find hebi_description)/urdf/kits/ros2_control/A-2084-01.ros2_control.xacro" />
   <!-- create link fixed to the "world" -->
   <link name="world" />
@@ -16,7 +16,7 @@
     <child link="base_link" />
   </joint>
-  <xacro:include filename="$(find hebi_description)/urdf/kits/A-2240-06.urdf.xacro" />
-  <xacro:A-2240-06_ros2_control
-    name="A-2240-06"
+  <xacro:include filename="$(find hebi_description)/urdf/kits/A-2084-01.urdf.xacro" />
+  <xacro:A-2084-01_ros2_control
+    name="A-2084-01"
     use_mock_hardware="$(arg use_mock_hardware)"
     mock_sensor_commands="$(arg mock_sensor_commands)"

File: urdf/kits/ros2_control/A-2084-01G.urdf.xacro (robot description, xacro)
@@ -1,4 +1,4 @@
 <?xml version="1.0" encoding="UTF-8"?>
-<robot xmlns:xacro="http://wiki.ros.org/xacro" name="A-2240-06">
+<robot xmlns:xacro="http://wiki.ros.org/xacro" name="A-2084-01G">
   <xacro:arg name="config_pkg" default="" />
   <xacro:arg name="config_file" default="" />
@@ -8,5 +8,5 @@
   <xacro:arg name="sim_gazebo_classic" default="false" />
   <xacro:arg name="sim_gazebo" default="false" />
-  <xacro:include filename="$(find hebi_description)/urdf/kits/ros2_control/A-2240-06.ros2_control.xacro" />
+  <xacro:include filename="$(find hebi_description)/urdf/kits/ros2_control/A-2084-01G.ros2_control.xacro" />
   <!-- create link fixed to the "world" -->
   <link name="world" />
@@ -16,7 +16,7 @@
     <child link="base_link" />
   </joint>
-  <xacro:include filename="$(find hebi_description)/urdf/kits/A-2240-06.urdf.xacro" />
-  <xacro:A-2240-06_ros2_control
-    name="A-2240-06"
+  <xacro:include filename="$(find hebi_description)/urdf/kits/A-2084-01G.urdf.xacro" />
+  <xacro:A-2084-01G_ros2_control
+    name="A-2084-01G"
     use_mock_hardware="$(arg use_mock_hardware)"
     mock_sensor_commands="$(arg mock_sensor_commands)"

File: urdf/kits/ros2_control/A-2085-03.urdf.xacro (robot description, xacro)
@@ -1,4 +1,4 @@
 <?xml version="1.0" encoding="UTF-8"?>
-<robot xmlns:xacro="http://wiki.ros.org/xacro" name="A-2240-06">
+<robot xmlns:xacro="http://wiki.ros.org/xacro" name="A-2085-03">
   <xacro:arg name="config_pkg" default="" />
   <xacro:arg name="config_file" default="" />
@@ -8,5 +8,5 @@
   <xacro:arg name="sim_gazebo_classic" default="false" />
   <xacro:arg name="sim_gazebo" default="false" />
-  <xacro:include filename="$(find hebi_description)/urdf/kits/ros2_control/A-2240-06.ros2_control.xacro" />
+  <xacro:include filename="$(find hebi_description)/urdf/kits/ros2_control/A-2085-03.ros2_control.xacro" />
   <!-- create link fixed to the "world" -->
   <link name="world" />
@@ -16,7 +16,7 @@
     <child link="base_link" />
   </joint>
-  <xacro:include filename="$(find hebi_description)/urdf/kits/A-2240-06.urdf.xacro" />
-  <xacro:A-2240-06_ros2_control
-    name="A-2240-06"
+  <xacro:include filename="$(find hebi_description)/urdf/kits/A-2085-03.urdf.xacro" />
+  <xacro:A-2085-03_ros2_control
+    name="A-2085-03"
     use_mock_hardware="$(arg use_mock_hardware)"
     mock_sensor_commands="$(arg mock_sensor_commands)"

File: urdf/kits/ros2_control/A-2085-04.ros2_control.xacro (robot description, xacro)
@@ -1,5 +1,5 @@
 <?xml version="1.0" encoding="UTF-8"?>
 <robot xmlns:xacro="http://wiki.ros.org/xacro">
-  <xacro:macro name="A-2085-05_ros2_control" params="
+  <xacro:macro name="A-2085-04_ros2_control" params="
                 name
                 prefix
@@ -10,5 +10,5 @@
                 config_pkg
                 config_file"
-               >
+  >
     <ros2_control name="${name}" type="system">
       <hardware>
@@ -59,15 +59,5 @@
         </state_interface>
       </joint>
-      <joint name="${prefix}J4_wrist1">
-        <command_interface name="position" />
-        <command_interface name="velocity" />
-        <state_interface name="position">
-          <param name="initial_value">0.0</param>
-        </state_interface>
-        <state_interface name="velocity">
-          <param name="initial_value">0.0</param>
-        </state_interface>
-      </joint>
-      <joint name="${prefix}J5_wrist2">
+      <joint name="${prefix}J4_wrist">
         <command_interface name="position" />
         <command_interface name="velocity" />
@@ -84,5 +74,5 @@
       <gazebo>
         <plugin filename="libgazebo_ros2_control.so" name="gazebo_ros2_control">
-          <parameters>$(find hebi_bringup)/config/A-2085-05_controllers.yaml</parameters>
+          <parameters>$(find hebi_bringup)/config/A-2085-04_controllers.yaml</parameters>
         </plugin>
       </gazebo>
@@ -92,5 +82,5 @@
       <gazebo>
         <plugin filename="ign_ros2_control-system" name="ign_ros2_control::IgnitionROS2ControlPlugin">
-          <parameters>$(find hebi_bringup)/config/A-2085-05_controllers.yaml</parameters>
+          <parameters>$(find hebi_bringup)/config/A-2085-04_controllers.yaml</parameters>
         </plugin>
       </gazebo>

File: urdf/kits/ros2_control/A-2085-04.urdf.xacro (robot description, xacro)
@@ -1,4 +1,4 @@
 <?xml version="1.0" encoding="UTF-8"?>
-<robot xmlns:xacro="http://wiki.ros.org/xacro" name="A-2240-06">
+<robot xmlns:xacro="http://wiki.ros.org/xacro" name="A-2085-04">
   <xacro:arg name="config_pkg" default="" />
   <xacro:arg name="config_file" default="" />
@@ -8,5 +8,5 @@
   <xacro:arg name="sim_gazebo_classic" default="false" />
   <xacro:arg name="sim_gazebo" default="false" />
-  <xacro:include filename="$(find hebi_description)/urdf/kits/ros2_control/A-2240-06.ros2_control.xacro" />
+  <xacro:include filename="$(find hebi_description)/urdf/kits/ros2_control/A-2085-04.ros2_control.xacro" />
   <!-- create link fixed to the "world" -->
   <link name="world" />
@@ -16,7 +16,7 @@
     <child link="base_link" />
   </joint>
-  <xacro:include filename="$(find hebi_description)/urdf/kits/A-2240-06.urdf.xacro" />
-  <xacro:A-2240-06_ros2_control
-    name="A-2240-06"
+  <xacro:include filename="$(find hebi_description)/urdf/kits/A-2085-04.urdf.xacro" />
+  <xacro:A-2085-04_ros2_control
+    name="A-2085-04"
     use_mock_hardware="$(arg use_mock_hardware)"
     mock_sensor_commands="$(arg mock_sensor_commands)"

File: urdf/kits/ros2_control/A-2085-05.urdf.xacro (robot description, xacro)
@@ -8,13 +8,13 @@
   <xacro:arg name="sim_gazebo_classic" default="false" />
   <xacro:arg name="sim_gazebo" default="false" />
-  <xacro:include filename="$(find hebi_description)/urdf/kits/ros2_control/A-2085-05_macro.ros2_control.xacro"/>
+  <xacro:include filename="$(find hebi_description)/urdf/kits/ros2_control/A-2085-05.ros2_control.xacro" />
   <!-- create link fixed to the "world" -->
   <link name="world" />
   <joint name="world_to_base_joint" type="fixed">
-    <origin xyz="0 0 0" rpy="0 0 0"/>
+    <origin xyz="0 0 0" rpy="0 0 0" />
     <parent link="world" />
-    <child link="base_link"/>
+    <child link="base_link" />
   </joint>
-  <xacro:include filename="$(find hebi_description)/urdf/kits/A-2085-05.urdf.xacro"/>
+  <xacro:include filename="$(find hebi_description)/urdf/kits/A-2085-05.urdf.xacro" />
   <xacro:A-2085-05_ros2_control
     name="A-2085-05"

File: urdf/kits/ros2_control/A-2085-05G.urdf.xacro (robot description, xacro)
@@ -1,4 +1,4 @@
 <?xml version="1.0" encoding="UTF-8"?>
-<robot xmlns:xacro="http://wiki.ros.org/xacro" name="A-2240-06">
+<robot xmlns:xacro="http://wiki.ros.org/xacro" name="A-2085-05G">
   <xacro:arg name="config_pkg" default="" />
   <xacro:arg name="config_file" default="" />
@@ -8,5 +8,5 @@
   <xacro:arg name="sim_gazebo_classic" default="false" />
   <xacro:arg name="sim_gazebo" default="false" />
-  <xacro:include filename="$(find hebi_description)/urdf/kits/ros2_control/A-2240-06.ros2_control.xacro" />
+  <xacro:include filename="$(find hebi_description)/urdf/kits/ros2_control/A-2085-05G.ros2_control.xacro" />
   <!-- create link fixed to the "world" -->
   <link name="world" />
@@ -16,7 +16,7 @@
     <child link="base_link" />
   </joint>
-  <xacro:include filename="$(find hebi_description)/urdf/kits/A-2240-06.urdf.xacro" />
-  <xacro:A-2240-06_ros2_control
-    name="A-2240-06"
+  <xacro:include filename="$(find hebi_description)/urdf/kits/A-2085-05G.urdf.xacro" />
+  <xacro:A-2085-05G_ros2_control
+    name="A-2085-05G"
     use_mock_hardware="$(arg use_mock_hardware)"
     mock_sensor_commands="$(arg mock_sensor_commands)"

File: urdf/kits/ros2_control/A-2085-06.urdf.xacro (robot description, xacro)
@@ -8,13 +8,13 @@
   <xacro:arg name="sim_gazebo_classic" default="false" />
   <xacro:arg name="sim_gazebo" default="false" />
-  <xacro:include filename="$(find hebi_description)/urdf/kits/ros2_control/A-2085-06_macro.ros2_control.xacro"/>
+  <xacro:include filename="$(find hebi_description)/urdf/kits/ros2_control/A-2085-06.ros2_control.xacro" />
   <!-- create link fixed to the "world" -->
   <link name="world" />
   <joint name="world_to_base_joint" type="fixed">
-    <origin xyz="0 0 0" rpy="0 0 0"/>
+    <origin xyz="0 0 0" rpy="0 0 0" />
     <parent link="world" />
-    <child link="base_link"/>
+    <child link="base_link" />
   </joint>
-  <xacro:include filename="$(find hebi_description)/urdf/kits/A-2085-06.urdf.xacro"/>
+  <xacro:include filename="$(find hebi_description)/urdf/kits/A-2085-06.urdf.xacro" />
   <xacro:A-2085-06_ros2_control
     name="A-2085-06"

File: urdf/kits/ros2_control/A-2085-06G.urdf.xacro (robot description, xacro)
@@ -1,4 +1,4 @@
 <?xml version="1.0" encoding="UTF-8"?>
-<robot xmlns:xacro="http://wiki.ros.org/xacro" name="A-2240-06">
+<robot xmlns:xacro="http://wiki.ros.org/xacro" name="A-2085-06G">
   <xacro:arg name="config_pkg" default="" />
   <xacro:arg name="config_file" default="" />
@@ -8,5 +8,5 @@
   <xacro:arg name="sim_gazebo_classic" default="false" />
   <xacro:arg name="sim_gazebo" default="false" />
-  <xacro:include filename="$(find hebi_description)/urdf/kits/ros2_control/A-2240-06.ros2_control.xacro" />
+  <xacro:include filename="$(find hebi_description)/urdf/kits/ros2_control/A-2085-06G.ros2_control.xacro" />
   <!-- create link fixed to the "world" -->
   <link name="world" />
@@ -16,7 +16,7 @@
     <child link="base_link" />
   </joint>
-  <xacro:include filename="$(find hebi_description)/urdf/kits/A-2240-06.urdf.xacro" />
-  <xacro:A-2240-06_ros2_control
-    name="A-2240-06"
+  <xacro:include filename="$(find hebi_description)/urdf/kits/A-2085-06G.urdf.xacro" />
+  <xacro:A-2085-06G_ros2_control
+    name="A-2085-06G"
     use_mock_hardware="$(arg use_mock_hardware)"
     mock_sensor_commands="$(arg mock_sensor_commands)"

File: urdf/kits/ros2_control/A-2240-04.urdf.xacro (robot description, xacro)
@@ -1,4 +1,4 @@
 <?xml version="1.0" encoding="UTF-8"?>
-<robot xmlns:xacro="http://wiki.ros.org/xacro" name="A-2240-06">
+<robot xmlns:xacro="http://wiki.ros.org/xacro" name="A-2240-04">
   <xacro:arg name="config_pkg" default="" />
   <xacro:arg name="config_file" default="" />
@@ -8,5 +8,5 @@
   <xacro:arg name="sim_gazebo_classic" default="false" />
   <xacro:arg name="sim_gazebo" default="false" />
-  <xacro:include filename="$(find hebi_description)/urdf/kits/ros2_control/A-2240-06.ros2_control.xacro" />
+  <xacro:include filename="$(find hebi_description)/urdf/kits/ros2_control/A-2240-04.ros2_control.xacro" />
   <!-- create link fixed to the "world" -->
   <link name="world" />
@@ -16,7 +16,7 @@
     <child link="base_link" />
   </joint>
-  <xacro:include filename="$(find hebi_description)/urdf/kits/A-2240-06.urdf.xacro" />
-  <xacro:A-2240-06_ros2_control
-    name="A-2240-06"
+  <xacro:include filename="$(find hebi_description)/urdf/kits/A-2240-04.urdf.xacro" />
+  <xacro:A-2240-04_ros2_control
+    name="A-2240-04"
     use_mock_hardware="$(arg use_mock_hardware)"
     mock_sensor_commands="$(arg mock_sensor_commands)"

File: urdf/kits/ros2_control/A-2240-05.urdf.xacro (robot description, xacro)
@@ -1,4 +1,4 @@
 <?xml version="1.0" encoding="UTF-8"?>
-<robot xmlns:xacro="http://wiki.ros.org/xacro" name="A-2240-06">
+<robot xmlns:xacro="http://wiki.ros.org/xacro" name="A-2240-05">
   <xacro:arg name="config_pkg" default="" />
   <xacro:arg name="config_file" default="" />
@@ -8,5 +8,5 @@
   <xacro:arg name="sim_gazebo_classic" default="false" />
   <xacro:arg name="sim_gazebo" default="false" />
-  <xacro:include filename="$(find hebi_description)/urdf/kits/ros2_control/A-2240-06.ros2_control.xacro" />
+  <xacro:include filename="$(find hebi_description)/urdf/kits/ros2_control/A-2240-05.ros2_control.xacro" />
   <!-- create link fixed to the "world" -->
   <link name="world" />
@@ -16,7 +16,7 @@
     <child link="base_link" />
   </joint>
-  <xacro:include filename="$(find hebi_description)/urdf/kits/A-2240-06.urdf.xacro" />
-  <xacro:A-2240-06_ros2_control
-    name="A-2240-06"
+  <xacro:include filename="$(find hebi_description)/urdf/kits/A-2240-05.urdf.xacro" />
+  <xacro:A-2240-05_ros2_control
+    name="A-2240-05"
     use_mock_hardware="$(arg use_mock_hardware)"
     mock_sensor_commands="$(arg mock_sensor_commands)"

File: urdf/kits/ros2_control/A-2240-05G.urdf.xacro (robot description, xacro)
@@ -1,4 +1,4 @@
 <?xml version="1.0" encoding="UTF-8"?>
-<robot xmlns:xacro="http://wiki.ros.org/xacro" name="A-2240-06">
+<robot xmlns:xacro="http://wiki.ros.org/xacro" name="A-2240-05G">
   <xacro:arg name="config_pkg" default="" />
   <xacro:arg name="config_file" default="" />
@@ -8,5 +8,5 @@
   <xacro:arg name="sim_gazebo_classic" default="false" />
   <xacro:arg name="sim_gazebo" default="false" />
-  <xacro:include filename="$(find hebi_description)/urdf/kits/ros2_control/A-2240-06.ros2_control.xacro" />
+  <xacro:include filename="$(find hebi_description)/urdf/kits/ros2_control/A-2240-05G.ros2_control.xacro" />
   <!-- create link fixed to the "world" -->
   <link name="world" />
@@ -16,7 +16,7 @@
     <child link="base_link" />
   </joint>
-  <xacro:include filename="$(find hebi_description)/urdf/kits/A-2240-06.urdf.xacro" />
-  <xacro:A-2240-06_ros2_control
-    name="A-2240-06"
+  <xacro:include filename="$(find hebi_description)/urdf/kits/A-2240-05G.urdf.xacro" />
+  <xacro:A-2240-05G_ros2_control
+    name="A-2240-05G"
     use_mock_hardware="$(arg use_mock_hardware)"
     mock_sensor_commands="$(arg mock_sensor_commands)"

File: urdf/kits/ros2_control/A-2240-06G.urdf.xacro (robot description, xacro)
@@ -1,4 +1,4 @@
 <?xml version="1.0" encoding="UTF-8"?>
-<robot xmlns:xacro="http://wiki.ros.org/xacro" name="A-2240-06">
+<robot xmlns:xacro="http://wiki.ros.org/xacro" name="A-2240-06G">
   <xacro:arg name="config_pkg" default="" />
   <xacro:arg name="config_file" default="" />
@@ -8,5 +8,5 @@
   <xacro:arg name="sim_gazebo_classic" default="false" />
   <xacro:arg name="sim_gazebo" default="false" />
-  <xacro:include filename="$(find hebi_description)/urdf/kits/ros2_control/A-2240-06.ros2_control.xacro" />
+  <xacro:include filename="$(find hebi_description)/urdf/kits/ros2_control/A-2240-06G.ros2_control.xacro" />
   <!-- create link fixed to the "world" -->
   <link name="world" />
@@ -16,7 +16,7 @@
     <child link="base_link" />
   </joint>
-  <xacro:include filename="$(find hebi_description)/urdf/kits/A-2240-06.urdf.xacro" />
-  <xacro:A-2240-06_ros2_control
-    name="A-2240-06"
+  <xacro:include filename="$(find hebi_description)/urdf/kits/A-2240-06G.urdf.xacro" />
+  <xacro:A-2240-06G_ros2_control
+    name="A-2240-06G"
     use_mock_hardware="$(arg use_mock_hardware)"
     mock_sensor_commands="$(arg mock_sensor_commands)"

File: urdf/kits/ros2_control/A-2302-01.urdf.xacro (robot description, xacro)
@@ -1,4 +1,4 @@
 <?xml version="1.0" encoding="UTF-8"?>
-<robot xmlns:xacro="http://wiki.ros.org/xacro" name="A-2240-06">
+<robot xmlns:xacro="http://wiki.ros.org/xacro" name="A-2302-01">
   <xacro:arg name="config_pkg" default="" />
   <xacro:arg name="config_file" default="" />
@@ -8,5 +8,5 @@
   <xacro:arg name="sim_gazebo_classic" default="false" />
   <xacro:arg name="sim_gazebo" default="false" />
-  <xacro:include filename="$(find hebi_description)/urdf/kits/ros2_control/A-2240-06.ros2_control.xacro" />
+  <xacro:include filename="$(find hebi_description)/urdf/kits/ros2_control/A-2302-01.ros2_control.xacro" />
   <!-- create link fixed to the "world" -->
   <link name="world" />
@@ -16,7 +16,7 @@
     <child link="base_link" />
   </joint>
-  <xacro:include filename="$(find hebi_description)/urdf/kits/A-2240-06.urdf.xacro" />
-  <xacro:A-2240-06_ros2_control
-    name="A-2240-06"
+  <xacro:include filename="$(find hebi_description)/urdf/kits/A-2302-01.urdf.xacro" />
+  <xacro:A-2302-01_ros2_control
+    name="A-2302-01"
     use_mock_hardware="$(arg use_mock_hardware)"
     mock_sensor_commands="$(arg mock_sensor_commands)"

File: urdf/kits/ros2_control/A-2302-01G.urdf.xacro (robot description, xacro)
@@ -1,4 +1,4 @@
 <?xml version="1.0" encoding="UTF-8"?>
-<robot xmlns:xacro="http://wiki.ros.org/xacro" name="A-2240-06">
+<robot xmlns:xacro="http://wiki.ros.org/xacro" name="A-2302-01G">
   <xacro:arg name="config_pkg" default="" />
   <xacro:arg name="config_file" default="" />
@@ -8,5 +8,5 @@
   <xacro:arg name="sim_gazebo_classic" default="false" />
   <xacro:arg name="sim_gazebo" default="false" />
-  <xacro:include filename="$(find hebi_description)/urdf/kits/ros2_control/A-2240-06.ros2_control.xacro" />
+  <xacro:include filename="$(find hebi_description)/urdf/kits/ros2_control/A-2302-01G.ros2_control.xacro" />
   <!-- create link fixed to the "world" -->
   <link name="world" />
@@ -16,7 +16,7 @@
     <child link="base_link" />
   </joint>
-  <xacro:include filename="$(find hebi_description)/urdf/kits/A-2240-06.urdf.xacro" />
-  <xacro:A-2240-06_ros2_control
-    name="A-2240-06"
+  <xacro:include filename="$(find hebi_description)/urdf/kits/A-2302-01G.urdf.xacro" />
+  <xacro:A-2302-01G_ros2_control
+    name="A-2302-01G"
     use_mock_hardware="$(arg use_mock_hardware)"
     mock_sensor_commands="$(arg mock_sensor_commands)"

File: urdf/kits/ros2_control/A-2580-04.urdf.xacro (robot description, xacro)
@@ -1,4 +1,4 @@
 <?xml version="1.0" encoding="UTF-8"?>
-<robot xmlns:xacro="http://wiki.ros.org/xacro" name="A-2240-06">
+<robot xmlns:xacro="http://wiki.ros.org/xacro" name="A-2580-04">
   <xacro:arg name="config_pkg" default="" />
   <xacro:arg name="config_file" default="" />
@@ -8,5 +8,5 @@
   <xacro:arg name="sim_gazebo_classic" default="false" />
   <xacro:arg name="sim_gazebo" default="false" />
-  <xacro:include filename="$(find hebi_description)/urdf/kits/ros2_control/A-2240-06.ros2_control.xacro" />
+  <xacro:include filename="$(find hebi_description)/urdf/kits/ros2_control/A-2580-04.ros2_control.xacro" />
   <!-- create link fixed to the "world" -->
   <link name="world" />
@@ -16,7 +16,7 @@
     <child link="base_link" />
   </joint>
-  <xacro:include filename="$(find hebi_description)/urdf/kits/A-2240-06.urdf.xacro" />
-  <xacro:A-2240-06_ros2_control
-    name="A-2240-06"
+  <xacro:include filename="$(find hebi_description)/urdf/kits/A-2580-04.urdf.xacro" />
+  <xacro:A-2580-04_ros2_control
+    name="A-2580-04"
     use_mock_hardware="$(arg use_mock_hardware)"
     mock_sensor_commands="$(arg mock_sensor_commands)"
