Commit message: Updated ROS2 Control URDFs

File: urdf/kits/ros2_control/A-2085-05G.ros2_control.xacro (robot description, xacro)
@@ -1,5 +1,5 @@
 <?xml version="1.0" encoding="UTF-8"?>
 <robot xmlns:xacro="http://wiki.ros.org/xacro">
-  <xacro:macro name="A-2085-06_ros2_control" params="
+  <xacro:macro name="A-2085-05G_ros2_control" params="
                 name
                 prefix
@@ -10,5 +10,5 @@
                 config_pkg
                 config_file"
-               >
+  >
     <ros2_control name="${name}" type="system">
       <hardware>
@@ -21,5 +21,5 @@
         </xacro:if>
         <xacro:if value="${sim_gazebo}">
-          <plugin>gz_ros2_control/GazeboSimSystem</plugin>
+          <plugin>ign_ros2_control/IgnitionSystem</plugin>
         </xacro:if>
         <xacro:unless value="${use_mock_hardware or sim_gazebo_classic or sim_gazebo}">
@@ -79,5 +79,5 @@
         </state_interface>
       </joint>
-      <joint name="${prefix}J6_wrist3">
+      <joint name="${prefix}end_effector_1/input_l_finger">
         <command_interface name="position" />
         <command_interface name="velocity" />
@@ -94,5 +94,5 @@
       <gazebo>
         <plugin filename="libgazebo_ros2_control.so" name="gazebo_ros2_control">
-          <parameters>$(find hebi_bringup)/config/A-2085-06_controllers.yaml</parameters>
+          <parameters>$(find hebi_bringup)/config/A-2085-05G_controllers.yaml</parameters>
         </plugin>
       </gazebo>
@@ -102,5 +102,5 @@
       <gazebo>
         <plugin filename="gz_ros2_control-system" name="gz_ros2_control::GazeboSimROS2ControlPlugin">
-          <parameters>$(find hebi_bringup)/config/A-2085-06_controllers.yaml</parameters>
+          <parameters>$(find hebi_bringup)/config/A-2085-05G_controllers.yaml</parameters>
         </plugin>
       </gazebo>

File: urdf/kits/ros2_control/A-2302-01.ros2_control.xacro (robot description, xacro)
@@ -1,5 +1,5 @@
 <?xml version="1.0" encoding="UTF-8"?>
 <robot xmlns:xacro="http://wiki.ros.org/xacro">
-  <xacro:macro name="A-2240-06_ros2_control" params="
+  <xacro:macro name="A-2302-01_ros2_control" params="
                 name
                 prefix
@@ -10,5 +10,5 @@
                 config_pkg
                 config_file"
-               >
+  >
     <ros2_control name="${name}" type="system">
       <hardware>
@@ -21,5 +21,5 @@
         </xacro:if>
         <xacro:if value="${sim_gazebo}">
-          <plugin>gz_ros2_control/GazeboSimSystem</plugin>
+          <plugin>ign_ros2_control/IgnitionSystem</plugin>
         </xacro:if>
         <xacro:unless value="${use_mock_hardware or sim_gazebo_classic or sim_gazebo}">
@@ -59,25 +59,5 @@
         </state_interface>
       </joint>
-      <joint name="${prefix}J4_wrist1">
-        <command_interface name="position" />
-        <command_interface name="velocity" />
-        <state_interface name="position">
-          <param name="initial_value">0.0</param>
-        </state_interface>
-        <state_interface name="velocity">
-          <param name="initial_value">0.0</param>
-        </state_interface>
-      </joint>
-      <joint name="${prefix}J5_wrist2">
-        <command_interface name="position" />
-        <command_interface name="velocity" />
-        <state_interface name="position">
-          <param name="initial_value">0.0</param>
-        </state_interface>
-        <state_interface name="velocity">
-          <param name="initial_value">0.0</param>
-        </state_interface>
-      </joint>
-      <joint name="${prefix}J6_wrist3">
+      <joint name="${prefix}J4_wrist">
         <command_interface name="position" />
         <command_interface name="velocity" />
@@ -94,5 +74,5 @@
       <gazebo>
         <plugin filename="libgazebo_ros2_control.so" name="gazebo_ros2_control">
-          <parameters>$(find hebi_bringup)/config/A-2240-06_controllers.yaml</parameters>
+          <parameters>$(find hebi_bringup)/config/A-2302-01_controllers.yaml</parameters>
         </plugin>
       </gazebo>
@@ -102,5 +82,5 @@
       <gazebo>
         <plugin filename="gz_ros2_control-system" name="gz_ros2_control::GazeboSimROS2ControlPlugin">
-          <parameters>$(find hebi_bringup)/config/A-2240-06_controllers.yaml</parameters>
+          <parameters>$(find hebi_bringup)/config/A-2302-01_controllers.yaml</parameters>
         </plugin>
       </gazebo>

File: urdf/kits/ros2_control/A-2580-06G.ros2_control.xacro (robot description, xacro)
@@ -1,5 +1,5 @@
 <?xml version="1.0" encoding="UTF-8"?>
 <robot xmlns:xacro="http://wiki.ros.org/xacro">
-  <xacro:macro name="A-2085-05_ros2_control" params="
+  <xacro:macro name="A-2580-06G_ros2_control" params="
                 name
                 prefix
@@ -10,5 +10,5 @@
                 config_pkg
                 config_file"
-               >
+  >
     <ros2_control name="${name}" type="system">
       <hardware>
@@ -21,5 +21,5 @@
         </xacro:if>
         <xacro:if value="${sim_gazebo}">
-          <plugin>gz_ros2_control/GazeboSimSystem</plugin>
+          <plugin>ign_ros2_control/IgnitionSystem</plugin>
         </xacro:if>
         <xacro:unless value="${use_mock_hardware or sim_gazebo_classic or sim_gazebo}">
@@ -79,4 +79,24 @@
         </state_interface>
       </joint>
+      <joint name="${prefix}J6_wrist3">
+        <command_interface name="position" />
+        <command_interface name="velocity" />
+        <state_interface name="position">
+          <param name="initial_value">0.0</param>
+        </state_interface>
+        <state_interface name="velocity">
+          <param name="initial_value">0.0</param>
+        </state_interface>
+      </joint>
+      <joint name="${prefix}end_effector_1/input_l_finger">
+        <command_interface name="position" />
+        <command_interface name="velocity" />
+        <state_interface name="position">
+          <param name="initial_value">0.0</param>
+        </state_interface>
+        <state_interface name="velocity">
+          <param name="initial_value">0.0</param>
+        </state_interface>
+      </joint>
     </ros2_control>
     <!-- Gazebo Classic plugins -->
@@ -84,5 +104,5 @@
       <gazebo>
         <plugin filename="libgazebo_ros2_control.so" name="gazebo_ros2_control">
-          <parameters>$(find hebi_bringup)/config/A-2085-05_controllers.yaml</parameters>
+          <parameters>$(find hebi_bringup)/config/A-2580-06G_controllers.yaml</parameters>
         </plugin>
       </gazebo>
@@ -92,5 +112,5 @@
       <gazebo>
         <plugin filename="gz_ros2_control-system" name="gz_ros2_control::GazeboSimROS2ControlPlugin">
-          <parameters>$(find hebi_bringup)/config/A-2085-05_controllers.yaml</parameters>
+          <parameters>$(find hebi_bringup)/config/A-2580-06G_controllers.yaml</parameters>
         </plugin>
       </gazebo>
