Commit message: Updated ROS2 Control URDFs

File: urdf/kits/ros2_control/A-2580-05.urdf.xacro (robot description, xacro)
@@ -1,4 +1,4 @@
 <?xml version="1.0" encoding="UTF-8"?>
-<robot xmlns:xacro="http://wiki.ros.org/xacro" name="A-2085-06">
+<robot xmlns:xacro="http://wiki.ros.org/xacro" name="A-2580-05">
   <xacro:arg name="config_pkg" default="" />
   <xacro:arg name="config_file" default="" />
@@ -7,5 +7,5 @@
   <xacro:arg name="mock_sensor_commands" default="false" />
   <xacro:arg name="sim_gazebo" default="false" />
-  <xacro:include filename="$(find hebi_description)/urdf/kits/ros2_control/A-2085-06.ros2_control.xacro" />
+  <xacro:include filename="$(find hebi_description)/urdf/kits/ros2_control/A-2580-05.ros2_control.xacro" />
   <!-- create link fixed to the "world" -->
   <link name="world" />
@@ -15,7 +15,7 @@
     <child link="base_link" />
   </joint>
-  <xacro:include filename="$(find hebi_description)/urdf/kits/A-2085-06.urdf.xacro" />
-  <xacro:A-2085-06_ros2_control
-    name="A-2085-06"
+  <xacro:include filename="$(find hebi_description)/urdf/kits/A-2580-05.urdf.xacro" />
+  <xacro:A-2580-05_ros2_control
+    name="A-2580-05"
     use_mock_hardware="$(arg use_mock_hardware)"
     mock_sensor_commands="$(arg mock_sensor_commands)"

File: urdf/kits/ros2_control/A-2580-05G.urdf.xacro (robot description, xacro)
@@ -1,4 +1,4 @@
 <?xml version="1.0" encoding="UTF-8"?>
-<robot xmlns:xacro="http://wiki.ros.org/xacro" name="A-2085-06">
+<robot xmlns:xacro="http://wiki.ros.org/xacro" name="A-2580-05G">
   <xacro:arg name="config_pkg" default="" />
   <xacro:arg name="config_file" default="" />
@@ -7,5 +7,5 @@
   <xacro:arg name="mock_sensor_commands" default="false" />
   <xacro:arg name="sim_gazebo" default="false" />
-  <xacro:include filename="$(find hebi_description)/urdf/kits/ros2_control/A-2085-06.ros2_control.xacro" />
+  <xacro:include filename="$(find hebi_description)/urdf/kits/ros2_control/A-2580-05G.ros2_control.xacro" />
   <!-- create link fixed to the "world" -->
   <link name="world" />
@@ -15,7 +15,7 @@
     <child link="base_link" />
   </joint>
-  <xacro:include filename="$(find hebi_description)/urdf/kits/A-2085-06.urdf.xacro" />
-  <xacro:A-2085-06_ros2_control
-    name="A-2085-06"
+  <xacro:include filename="$(find hebi_description)/urdf/kits/A-2580-05G.urdf.xacro" />
+  <xacro:A-2580-05G_ros2_control
+    name="A-2580-05G"
     use_mock_hardware="$(arg use_mock_hardware)"
     mock_sensor_commands="$(arg mock_sensor_commands)"
