Commit message: Fixed rosie URDF

File: urdf/components/omnibase.xacro (robot description, xacro)
@@ -3,5 +3,5 @@
   <xacro:macro name="omnibase" params="child">
     <joint name="base_child_joint" type="fixed">
-      <origin xyz="0 0 0.21" rpy="0 0 0"/>
+      <origin xyz="0 0 0.135" rpy="0 0 0"/>
       <parent link="omni_base" />
       <child link="${child}"/>
@@ -10,5 +10,5 @@
       <origin xyz="0 0 0" rpy="0 0 0" />
     </link>
-    <joint name="base_joint" type="fixed">
+    <joint name="omnibase_joint" type="fixed">
       <origin xyz="0 0 0" rpy="0 0 0"/>
       <parent link="base_link" />
@@ -17,5 +17,5 @@
     <link name="omni_base">
       <visual>
-        <origin xyz="0 0 0.075" rpy="${pi/2} 0 0" />
+        <origin xyz="0 0 0" rpy="${pi/2} 0 0" />
         <geometry>
           <mesh filename="file://$(find hebi_description)/meshes/A-2121-01_Export.obj" />
@@ -23,5 +23,5 @@
       </visual>
       <collision>
-        <origin xyz="0 0 0.075" rpy="${pi/2} 0 0" />
+        <origin xyz="0 0 0" rpy="${pi/2} 0 0" />
         <geometry>
           <mesh filename="file://$(find hebi_description)/meshes/A-2121-01_Export.obj" />
@@ -30,5 +30,5 @@
       <inertial>
         <mass value="5"/>
-        <origin xyz="0 0 0.075" rpy="0 0 0" />
+        <origin xyz="0 0 0" rpy="0 0 0" />
           <inertia ixx="0.00015"  ixy="0.0000341"  ixz="0.0000118"
                     iyy="0.000255" iyz="0.00000229"
@@ -37,15 +37,15 @@
     </link>
     <joint name="wheel_1_joint" type="fixed">
-      <origin xyz="0.0788 -0.1364 0.0750" rpy="0 ${pi/2} ${-pi/3}" />
+      <origin xyz="0.0788 -0.1364 0" rpy="0 ${pi/2} ${-pi/3}" />
       <parent link="omni_base" />
       <child link="wheel_1/INPUT_INTERFACE"/>
     </joint>
     <joint name="wheel_2_joint" type="fixed">
-      <origin xyz="0.0788 0.1364 0.0750" rpy="0 ${pi/2} ${pi/3}" />
+      <origin xyz="0.0788 0.1364 0" rpy="0 ${pi/2} ${pi/3}" />
       <parent link="omni_base" />
       <child link="wheel_2/INPUT_INTERFACE"/>
     </joint>
     <joint name="wheel_3_joint" type="fixed">
-      <origin xyz="-0.1575 0 0.0750" rpy="0 ${pi/2} ${pi}" />
+      <origin xyz="-0.1575 0 0" rpy="0 ${pi/2} ${pi}" />
       <parent link="omni_base" />
       <child link="wheel_3/INPUT_INTERFACE"/>

File: urdf/kits/rosie.urdf.xacro (robot description, xacro)
@@ -2,7 +2,15 @@
 <robot xmlns:xacro="http://www.ros.org/wiki/xacro" name="rosie">
   <xacro:include filename="$(find hebi_description)/urdf/components/hebi.xacro" />
-  <xacro:arg name="prefix" default="arm/" />
-  <!-- HEBI A-2085-05 Arm Kit -->
-  <xacro:include filename="$(find hebi_description)/urdf/kits/A-2085-05.urdf.xacro" />
+  <xacro:arg name="prefix" default="" />
+  <xacro:arg name="hebi_arm" default="A-2085-06" />
+  <!-- HEBI Arm Kit -->
+  <xacro:include filename="$(find hebi_description)/urdf/kits/$(arg hebi_arm).urdf.xacro" />
   <xacro:omnibase child="$(arg prefix)base_link" />
+  <!-- Robot Footprint -->
+  <link name="base_footprint"/>
+  <joint name="base_joint" type="fixed">
+    <parent link="base_footprint"/>
+    <child link="base_link"/>
+    <origin xyz="0.0 0.0 0.075" rpy="0 0 0"/>
+  </joint>
 </robot>
