Commit message: Fixed rigid-body xacro to include mesh transforms

File: urdf/components/rigid_body.xacro (robot description, xacro)
@@ -5,5 +5,5 @@
       <xacro:if value="${mesh_path != ''}">
         <visual>
-          <origin xyz="0 0 0" rpy="0 0 0"/>
+          <origin xyz="${mesh_trans}" rpy="${mesh_rot}"/>
           <geometry>
             <mesh filename="${mesh_path}"/>
@@ -12,5 +12,5 @@
         </visual>
         <collision>
-          <origin xyz="0 0 0" rpy="0 0 0"/>
+          <origin xyz="${mesh_trans}" rpy="${mesh_rot}"/>
           <geometry>
             <mesh filename="${mesh_path}"/>
