Commit message: Added every HEBI kit xacro - Debugged link xacro twist - ros2_control completed only for one arm - README updated

File: urdf/components/link.xacro (robot description, xacro)
@@ -57,5 +57,5 @@
       <visual>
         <xacro:if value="${input == 'RightAngle' and output == 'RightAngle'}">
-          <origin xyz="${extension} ${sin(-twist) * edge_to_center} ${edge_to_center * (1 + cos(-twist))}" rpy="${-twist} 0 0"/>
+          <origin xyz="${extension} ${sin(-twist) * edge_to_center} ${edge_to_center * (1 + cos(-twist))}" rpy="${twist} 0 0"/>
         </xacro:if>
         <xacro:if value="${input == 'RightAngle' and output == 'Inline'}">
@@ -80,5 +80,5 @@
       <collision>
         <xacro:if value="${input == 'RightAngle' and output == 'RightAngle'}">
-          <origin xyz="${extension} ${sin(-twist) * edge_to_center} ${edge_to_center * (1 + cos(-twist))}" rpy="${-twist} 0 0"/>
+          <origin xyz="${extension} ${sin(-twist) * edge_to_center} ${edge_to_center * (1 + cos(-twist))}" rpy="${twist} 0 0"/>
         </xacro:if>
         <xacro:if value="${input == 'RightAngle' and output == 'Inline'}">

File: urdf/kits/A-2085-05-parallel-gripper.urdf.xacro (robot description, xacro)
@@ -1,6 +1,6 @@
-<?xml version="1.0" encoding="UTF-8"?>
-<robot xmlns:xacro="http://wiki.ros.org/xacro" name="A-2085-06">
-  <!-- HEBI A-2085-06 Arm Kit -->
-  <xacro:include filename="$(find hebi_description)/urdf/components/hebi.xacro" />
+<?xml version='1.0' encoding='UTF-8'?>
+<robot xmlns:xacro="http://www.ros.org/wiki/xacro" name="A-2085-05-parallel-gripper">
+  <!-- HEBI A-2085-05-parallel-gripper Arm Kit -->
+  <xacro:include filename="$(find hebi_description)/urdf/components/hebi.xacro"/>
   <link name="base_link" />
   <joint name="base_joint" type="fixed">
@@ -17,7 +17,5 @@
   <xacro:actuator type="X5_1" name="J4_wrist1" child="wrist2_bracket"/>
   <xacro:bracket type="X5LightRight" name="wrist2_bracket" child="J5_wrist2"/>
-  <xacro:actuator type="X5_1" name="J5_wrist2" child="wrist3_bracket"/>
-  <xacro:bracket type="X5LightRight" name="wrist3_bracket" child="J6_wrist3"/>
-  <xacro:actuator type="X5_1" name="J6_wrist3" child="end_effector"/>
-  <xacro:gripper type="Custom" name="end_effector" mass="0.005"/>
+  <xacro:actuator type="X5_1" name="J5_wrist2" child="end_effector"/>
+  <xacro:gripper type="X5Parallel" name="end_effector"/>
 </robot>

File: urdf/kits/A-2085-05.urdf.xacro (robot description, xacro)
@@ -1,5 +1,6 @@
-<?xml version="1.0" encoding="UTF-8"?>
-<robot xmlns:xacro="http://wiki.ros.org/xacro" name="A-2085-06">
-  <xacro:include filename="$(find hebi_description)/urdf/hebi.xacro" />
+<?xml version='1.0' encoding='UTF-8'?>
+<robot xmlns:xacro="http://www.ros.org/wiki/xacro" name="A-2085-05">
+  <!-- HEBI A-2085-05 Arm Kit -->
+  <xacro:include filename="$(find hebi_description)/urdf/components/hebi.xacro"/>
   <link name="base_link" />
   <joint name="base_joint" type="fixed">
@@ -16,7 +17,5 @@
   <xacro:actuator type="X5_1" name="J4_wrist1" child="wrist2_bracket"/>
   <xacro:bracket type="X5LightRight" name="wrist2_bracket" child="J5_wrist2"/>
-  <xacro:actuator type="X5_1" name="J5_wrist2" child="wrist3_bracket"/>
-  <xacro:bracket type="X5LightRight" name="wrist3_bracket" child="J6_wrist3"/>
-  <xacro:actuator type="X5_1" name="J6_wrist3" child="end_effector"/>
-  <xacro:gripper type="Custom" name="end_effector" mass="0.05"/>
+  <xacro:actuator type="X5_1" name="J5_wrist2" child="end_effector"/>
+  <xacro:gripper type="Custom" name="end_effector" mass="0.005"/>
 </robot>

File: urdf/kits/A-2085-06-parallel-gripper.urdf.xacro (robot description, xacro)
@@ -1,6 +1,6 @@
-<?xml version="1.0" encoding="UTF-8"?>
-<robot xmlns:xacro="http://wiki.ros.org/xacro" name="A-2085-06">
-  <!-- HEBI A-2085-06 Arm Kit -->
-  <xacro:include filename="$(find hebi_description)/urdf/components/hebi.xacro" />
+<?xml version='1.0' encoding='UTF-8'?>
+<robot xmlns:xacro="http://www.ros.org/wiki/xacro" name="A-2085-06-parallel-gripper">
+  <!-- HEBI A-2085-06-parallel-gripper Arm Kit -->
+  <xacro:include filename="$(find hebi_description)/urdf/components/hebi.xacro"/>
   <link name="base_link" />
   <joint name="base_joint" type="fixed">
@@ -20,4 +20,4 @@
   <xacro:bracket type="X5LightRight" name="wrist3_bracket" child="J6_wrist3"/>
   <xacro:actuator type="X5_1" name="J6_wrist3" child="end_effector"/>
-  <xacro:gripper type="Custom" name="end_effector" mass="0.005"/>
+  <xacro:gripper type="X5Parallel" name="end_effector"/>
 </robot>

File: urdf/kits/ros2_control/A-2085-06.urdf.xacro (robot description, xacro)
@@ -1,6 +1,23 @@
 <?xml version="1.0" encoding="UTF-8"?>
 <robot xmlns:xacro="http://wiki.ros.org/xacro" name="A-2085-06">
-  <!-- HEBI A-2085-06 Arm Kit -->
+  <!-- Use this if parameters are set from the launch file, otherwise delete -->
+  <xacro:arg name="prefix" default="" />
+  <xacro:arg name="families" default="" />
+  <xacro:arg name="names" default="" />
+  <xacro:arg name="config_pkg" default="" />
+  <xacro:arg name="use_mock_hardware" default="false" />
+  <xacro:arg name="mock_sensor_commands" default="false" />
+  <xacro:arg name="sim_gazebo_classic" default="false" />
+  <xacro:arg name="sim_gazebo" default="false" />
+  <xacro:arg name="simulation_controllers" default="" />
   <xacro:include filename="$(find hebi_description)/urdf/components/hebi.xacro" />
+  <xacro:include filename="$(find hebi_description)/urdf/kits/ros2_control/A-2085-06_macro.ros2_control.xacro"/>
+  <!-- create link fixed to the "world" -->
+  <link name="world" />
+  <joint name="world_to_base_joint" type="fixed">
+    <origin xyz="0 0 0" rpy="0 0 0"/>
+    <parent link="world" />
+    <child link="base_link"/>
+  </joint>
   <link name="base_link" />
   <joint name="base_joint" type="fixed">
@@ -21,3 +38,13 @@
   <xacro:actuator type="X5_1" name="J6_wrist3" child="end_effector"/>
   <xacro:gripper type="Custom" name="end_effector" mass="0.005"/>
+  <xacro:A-2085-06_ros2_control
+    name="A-2085-06"
+    prefix="$(arg prefix)"
+    use_mock_hardware="$(arg use_mock_hardware)"
+    mock_sensor_commands="$(arg mock_sensor_commands)"
+    sim_gazebo_classic="$(arg sim_gazebo_classic)"
+    sim_gazebo="$(arg sim_gazebo)"
+    families="$(arg families)"
+    names="$(arg names)"
+    config_pkg="$(arg config_pkg)" />
 </robot>

File: urdf/kits/ros2_control/A-2085-06_macro.ros2_control.xacro (robot description, xacro)
@@ -8,5 +8,4 @@
                 sim_gazebo_classic:=^|false
                 sim_gazebo:=^|false
-                simulation_controllers
                 families
                 names
@@ -15,8 +14,4 @@
     <ros2_control name="${name}" type="system">
       <hardware>
-        <!-- Parameters to initialize the Components -->
-        <param name="families">${families}</param>
-        <param name="names">${names}</param>
-        <param name="config_pkg">${config_pkg}</param>
         <xacro:if value="${use_mock_hardware}">
           <plugin>mock_components/GenericSystem</plugin>
@@ -30,4 +25,8 @@
         </xacro:if>
         <xacro:unless value="${use_mock_hardware or sim_gazebo_classic or sim_gazebo}">
+          <!-- Parameters to initialize the Components -->
+          <param name="families">${families}</param>
+          <param name="names">${names}</param>
+          <param name="config_pkg">${config_pkg}</param>
           <plugin>hebi_hardware/HEBIHardwareInterface</plugin>
         </xacro:unless>
@@ -76,6 +75,6 @@
       </joint>
     </ros2_control>
-    <!-- Gazebo plugins -->
-    <!-- <xacro:if value="$(arg sim_gazebo_classic)">
+    <!-- Gazebo Classic plugins -->
+    <xacro:if value="$(arg sim_gazebo_classic)">
       <gazebo>
         <plugin filename="libgazebo_ros2_control.so" name="gazebo_ros2_control">
@@ -83,12 +82,12 @@
         </plugin>
       </gazebo>
-    </xacro:if> -->
+    </xacro:if>
+    <!-- Gazebo Ignition plugins -->
     <xacro:if value="$(arg sim_gazebo)">
-      <!-- Gazebo plugins -->
       <gazebo reference="world">
       </gazebo>
       <gazebo>
         <plugin filename="libign_ros2_control-system.so" name="ign_ros2_control::IgnitionROS2ControlPlugin">
-          <parameters>${simulation_controllers}</parameters>
+          <parameters>$(find hebi_bringup)/config/A-2085-06_controllers.yaml</parameters>
           <controller_manager_node_name>controller_manager</controller_manager_node_name>
         </plugin>

Commit message: Added missing URDFs and final documentation

File: urdf/components/link.xacro (robot description, xacro)
@@ -112,5 +112,5 @@
       <xacro:gazebo_black_material/>
     </gazebo>
-    <joint name="${name}_joint" type="fixed">
+    <joint name="${name}/joint" type="fixed">
       <parent link="${name}"/>
       <child link="${child}"/>
