Commit message: - Prefix option for the arm urdf - Added omnibase files (mesh ingnored due to size) - Added home position as hardware param

File: urdf/components/hebi.xacro (robot description, xacro)
@@ -44,3 +44,4 @@
   <xacro:include filename="./bracket.xacro"/>
   <xacro:include filename="./end_effector.xacro"/>
+  <xacro:include filename="./omnibase.xacro"/>
 </robot>

File: urdf/kits/A-2085-05.urdf.xacro (robot description, xacro)
@@ -1,21 +1,22 @@
 <?xml version='1.0' encoding='UTF-8'?>
 <robot xmlns:xacro="http://www.ros.org/wiki/xacro" name="A-2085-05">
+  <xacro:arg name="prefix" default="" />
   <!-- HEBI A-2085-05 Arm Kit -->
   <xacro:include filename="$(find hebi_description)/urdf/components/hebi.xacro"/>
-  <link name="base_link" />
-  <joint name="base_joint" type="fixed">
+  <link name="$(arg prefix)base_link" />
+  <joint name="$(arg prefix)base_joint" type="fixed">
     <origin xyz="0 0 0" rpy="0 0 0"/>
-    <parent link="base_link" />
-    <child link="J1_base/INPUT_INTERFACE"/>
+    <parent link="$(arg prefix)base_link" />
+    <child link="$(arg prefix)J1_base/INPUT_INTERFACE"/>
   </joint>
-  <xacro:actuator type="X8_9" name="J1_base" child="shoulder_bracket"/>
-  <xacro:bracket type="X5HeavyRightOutside" name="shoulder_bracket" child="J2_shoulder"/>
-  <xacro:actuator type="X8_16" name="J2_shoulder" child="shoulder_elbow"/>
-  <xacro:link type="X5" extension="0.325" twist="${pi}" name="shoulder_elbow" child="J3_elbow"/>
-  <xacro:actuator type="X8_9" name="J3_elbow" child="elbow_wrist1"/>
-  <xacro:link type="X5" extension="0.325" twist="${pi}" name="elbow_wrist1" child="J4_wrist1"/>
-  <xacro:actuator type="X5_1" name="J4_wrist1" child="wrist2_bracket"/>
-  <xacro:bracket type="X5LightRight" name="wrist2_bracket" child="J5_wrist2"/>
-  <xacro:actuator type="X5_1" name="J5_wrist2" child="end_effector"/>
-  <xacro:gripper type="Custom" name="end_effector" mass="0.005"/>
+  <xacro:actuator type="X8_9" name="$(arg prefix)J1_base" child="$(arg prefix)shoulder_bracket"/>
+  <xacro:bracket type="X5HeavyRightOutside" name="$(arg prefix)shoulder_bracket" child="$(arg prefix)J2_shoulder"/>
+  <xacro:actuator type="X8_16" name="$(arg prefix)J2_shoulder" child="$(arg prefix)shoulder_elbow"/>
+  <xacro:link type="X5" extension="0.325" twist="${pi}" name="$(arg prefix)shoulder_elbow" child="$(arg prefix)J3_elbow"/>
+  <xacro:actuator type="X8_9" name="$(arg prefix)J3_elbow" child="$(arg prefix)elbow_wrist1"/>
+  <xacro:link type="X5" extension="0.325" twist="${pi}" name="$(arg prefix)elbow_wrist1" child="$(arg prefix)J4_wrist1"/>
+  <xacro:actuator type="X5_1" name="$(arg prefix)J4_wrist1" child="$(arg prefix)wrist2_bracket"/>
+  <xacro:bracket type="X5LightRight" name="$(arg prefix)wrist2_bracket" child="$(arg prefix)J5_wrist2"/>
+  <xacro:actuator type="X5_1" name="$(arg prefix)J5_wrist2" child="$(arg prefix)end_effector"/>
+  <xacro:gripper type="Custom" name="$(arg prefix)end_effector" mass="0.005"/>
 </robot>

File: urdf/kits/A-2085-06.urdf.xacro (robot description, xacro)
@@ -1,23 +1,24 @@
 <?xml version="1.0" encoding="UTF-8"?>
 <robot xmlns:xacro="http://wiki.ros.org/xacro" name="A-2085-06">
+  <xacro:arg name="prefix" default="" />
   <!-- HEBI A-2085-06 Arm Kit -->
   <xacro:include filename="$(find hebi_description)/urdf/components/hebi.xacro" />
-  <link name="base_link" />
-  <joint name="base_joint" type="fixed">
+  <link name="$(arg prefix)base_link" />
+  <joint name="$(arg prefix)base_joint" type="fixed">
     <origin xyz="0 0 0" rpy="0 0 0"/>
-    <parent link="base_link" />
-    <child link="J1_base/INPUT_INTERFACE"/>
+    <parent link="$(arg prefix)base_link" />
+    <child link="$(arg prefix)J1_base/INPUT_INTERFACE"/>
   </joint>
-  <xacro:actuator type="X8_9" name="J1_base" child="shoulder_bracket"/>
-  <xacro:bracket type="X5HeavyRightOutside" name="shoulder_bracket" child="J2_shoulder"/>
-  <xacro:actuator type="X8_16" name="J2_shoulder" child="shoulder_elbow"/>
-  <xacro:link type="X5" extension="0.325" twist="${pi}" name="shoulder_elbow" child="J3_elbow"/>
-  <xacro:actuator type="X8_9" name="J3_elbow" child="elbow_wrist1"/>
-  <xacro:link type="X5" extension="0.325" twist="${pi}" name="elbow_wrist1" child="J4_wrist1"/>
-  <xacro:actuator type="X5_1" name="J4_wrist1" child="wrist2_bracket"/>
-  <xacro:bracket type="X5LightRight" name="wrist2_bracket" child="J5_wrist2"/>
-  <xacro:actuator type="X5_1" name="J5_wrist2" child="wrist3_bracket"/>
-  <xacro:bracket type="X5LightRight" name="wrist3_bracket" child="J6_wrist3"/>
-  <xacro:actuator type="X5_1" name="J6_wrist3" child="end_effector"/>
-  <xacro:gripper type="Custom" name="end_effector" mass="0.005"/>
+  <xacro:actuator type="X8_9" name="$(arg prefix)J1_base" child="$(arg prefix)shoulder_bracket"/>
+  <xacro:bracket type="X5HeavyRightOutside" name="$(arg prefix)shoulder_bracket" child="$(arg prefix)J2_shoulder"/>
+  <xacro:actuator type="X8_16" name="$(arg prefix)J2_shoulder" child="$(arg prefix)shoulder_elbow"/>
+  <xacro:link type="X5" extension="0.325" twist="${pi}" name="$(arg prefix)shoulder_elbow" child="$(arg prefix)J3_elbow"/>
+  <xacro:actuator type="X8_9" name="$(arg prefix)J3_elbow" child="$(arg prefix)elbow_wrist1"/>
+  <xacro:link type="X5" extension="0.325" twist="${pi}" name="$(arg prefix)elbow_wrist1" child="$(arg prefix)J4_wrist1"/>
+  <xacro:actuator type="X5_1" name="$(arg prefix)J4_wrist1" child="$(arg prefix)wrist2_bracket"/>
+  <xacro:bracket type="X5LightRight" name="$(arg prefix)wrist2_bracket" child="$(arg prefix)J5_wrist2"/>
+  <xacro:actuator type="X5_1" name="$(arg prefix)J5_wrist2" child="$(arg prefix)wrist3_bracket"/>
+  <xacro:bracket type="X5LightRight" name="$(arg prefix)wrist3_bracket" child="$(arg prefix)J6_wrist3"/>
+  <xacro:actuator type="X5_1" name="$(arg prefix)J6_wrist3" child="$(arg prefix)end_effector"/>
+  <xacro:gripper type="Custom" name="$(arg prefix)end_effector" mass="0.005"/>
 </robot>

File: urdf/kits/ros2_control/A-2085-05_macro.ros2_control.xacro (robot description, xacro)
@@ -3,4 +3,5 @@
   <xacro:macro name="A-2085-05_ros2_control" params="
                 name
+                prefix
                 use_mock_hardware:=^|false
                 mock_sensor_commands:=^|false
@@ -32,38 +33,53 @@
         </xacro:unless>
       </hardware>
-      <joint name="J1_base">
+      <joint name="${prefix}J1_base">
         <command_interface name="position" />
+        <command_interface name="velocity" />
         <state_interface name="position">
           <param name="initial_value">0.0</param>
         </state_interface>
-        <state_interface name="velocity" />
+        <state_interface name="velocity">
+          <param name="initial_value">0.0</param>
+        </state_interface>
       </joint>
-      <joint name="J2_shoulder">
+      <joint name="${prefix}J2_shoulder">
         <command_interface name="position" />
+        <command_interface name="velocity" />
         <state_interface name="position">
           <param name="initial_value">0.0</param>
         </state_interface>
-        <state_interface name="velocity" />
+        <state_interface name="velocity">
+          <param name="initial_value">0.0</param>
+        </state_interface>
       </joint>
-      <joint name="J3_elbow">
+      <joint name="${prefix}J3_elbow">
         <command_interface name="position" />
+        <command_interface name="velocity" />
         <state_interface name="position">
           <param name="initial_value">0.0</param>
         </state_interface>
-        <state_interface name="velocity" />
+        <state_interface name="velocity">
+          <param name="initial_value">0.0</param>
+        </state_interface>
       </joint>
-      <joint name="J4_wrist1">
+      <joint name="${prefix}J4_wrist1">
         <command_interface name="position" />
+        <command_interface name="velocity" />
         <state_interface name="position">
           <param name="initial_value">0.0</param>
         </state_interface>
-        <state_interface name="velocity" />
+        <state_interface name="velocity">
+          <param name="initial_value">0.0</param>
+        </state_interface>
       </joint>
-      <joint name="J5_wrist2">
+      <joint name="${prefix}J5_wrist2">
         <command_interface name="position" />
+        <command_interface name="velocity" />
         <state_interface name="position">
           <param name="initial_value">0.0</param>
         </state_interface>
-        <state_interface name="velocity" />
+        <state_interface name="velocity">
+          <param name="initial_value">0.0</param>
+        </state_interface>
       </joint>
     </ros2_control>

File: urdf/kits/ros2_control/A-2085-06.urdf.xacro (robot description, xacro)
@@ -7,4 +7,6 @@
   <xacro:arg name="gains_pkg" default="" />
   <xacro:arg name="gains_file" default="" />
+  <xacro:arg name="prefix" default="" />
+  <xacro:arg name="home_position" default="" />
   <xacro:arg name="use_mock_hardware" default="false" />
   <xacro:arg name="mock_sensor_commands" default="false" />
@@ -29,4 +31,6 @@
     hrdf_file="$(arg hrdf_file)"
     gains_pkg="$(arg gains_pkg)"
-    gains_file="$(arg gains_file)" />
+    gains_file="$(arg gains_file)"
+    prefix="$(arg prefix)"
+    home_position="$(arg home_position)" />
 </robot>

File: urdf/kits/ros2_control/A-2085-06_macro.ros2_control.xacro (robot description, xacro)
@@ -3,4 +3,5 @@
   <xacro:macro name="A-2085-06_ros2_control" params="
                 name
+                prefix
                 use_mock_hardware:=^|false
                 mock_sensor_commands:=^|false
@@ -11,5 +12,6 @@
                 hrdf_file
                 gains_pkg
-                gains_file"
+                gains_file
+                home_position"
                >
     <ros2_control name="${name}" type="system">
@@ -29,48 +31,67 @@
           <param name="gains_pkg">${gains_pkg}</param>
           <param name="gains_file">${gains_file}</param>
+          <param name="home_position">${home_position}</param>
           <plugin>hebi_hardware/HEBIHardwareInterface</plugin>
         </xacro:unless>
       </hardware>
-      <joint name="J1_base">
+      <joint name="${prefix}J1_base">
         <command_interface name="position" />
+        <command_interface name="velocity" />
         <state_interface name="position">
           <param name="initial_value">0.0</param>
         </state_interface>
-        <state_interface name="velocity" />
+        <state_interface name="velocity">
+          <param name="initial_value">0.0</param>
+        </state_interface>
       </joint>
-      <joint name="J2_shoulder">
+      <joint name="${prefix}J2_shoulder">
         <command_interface name="position" />
+        <command_interface name="velocity" />
         <state_interface name="position">
           <param name="initial_value">0.0</param>
         </state_interface>
-        <state_interface name="velocity" />
+        <state_interface name="velocity">
+          <param name="initial_value">0.0</param>
+        </state_interface>
       </joint>
-      <joint name="J3_elbow">
+      <joint name="${prefix}J3_elbow">
         <command_interface name="position" />
+        <command_interface name="velocity" />
         <state_interface name="position">
           <param name="initial_value">0.0</param>
         </state_interface>
-        <state_interface name="velocity" />
+        <state_interface name="velocity">
+          <param name="initial_value">0.0</param>
+        </state_interface>
       </joint>
-      <joint name="J4_wrist1">
+      <joint name="${prefix}J4_wrist1">
         <command_interface name="position" />
+        <command_interface name="velocity" />
         <state_interface name="position">
           <param name="initial_value">0.0</param>
         </state_interface>
-        <state_interface name="velocity" />
+        <state_interface name="velocity">
+          <param name="initial_value">0.0</param>
+        </state_interface>
       </joint>
-      <joint name="J5_wrist2">
+      <joint name="${prefix}J5_wrist2">
         <command_interface name="position" />
+        <command_interface name="velocity" />
         <state_interface name="position">
           <param name="initial_value">0.0</param>
         </state_interface>
-        <state_interface name="velocity" />
+        <state_interface name="velocity">
+          <param name="initial_value">0.0</param>
+        </state_interface>
       </joint>
-      <joint name="J6_wrist3">
+      <joint name="${prefix}J6_wrist3">
         <command_interface name="position" />
+        <command_interface name="velocity" />
         <state_interface name="position">
           <param name="initial_value">0.0</param>
         </state_interface>
-        <state_interface name="velocity" />
+        <state_interface name="velocity">
+          <param name="initial_value">0.0</param>
+        </state_interface>
       </joint>
     </ros2_control>

Commit message: Added mecanum base URDF and updated omnibase

File: urdf/components/hebi.xacro (robot description, xacro)
@@ -59,4 +59,3 @@
   <xacro:include filename="./rigid_body.xacro"/>
   <xacro:include filename="./output.xacro"/>
-  <xacro:include filename="./omnibase.xacro"/>
 </robot>

File: urdf/kits/rosie.urdf.xacro (robot description, xacro)
@@ -1,16 +1,16 @@
 <?xml version='1.0' encoding='UTF-8'?>
 <robot xmlns:xacro="http://www.ros.org/wiki/xacro" name="rosie">
-  <xacro:include filename="$(find hebi_description)/urdf/components/hebi.xacro" />
-  <xacro:arg name="prefix" default="" />
-  <xacro:arg name="hebi_arm" default="A-2085-06" />
+  <!-- HEBI Omnidirectional Mobile Base -->
+  <xacro:include filename="$(find hebi_description)/urdf/kits/omnibase.urdf.xacro" />
+  <!-- Arguments for HEBI Arm -->
+  <xacro:arg name="prefix" default="arm/" />
+  <xacro:arg name="hebi_arm" default="A-2580-06" />
+  <!-- Base-Arm Joint -->
+  <joint name="base_arm_joint" type="fixed">
+    <origin xyz="0 0 0.135" rpy="0 0 0"/>
+    <parent link="omni_base" />
+    <child link="$(arg prefix)base_link"/>
+  </joint>
   <!-- HEBI Arm Kit -->
   <xacro:include filename="$(find hebi_description)/urdf/kits/$(arg hebi_arm).urdf.xacro" />
-  <xacro:omnibase child="$(arg prefix)base_link" />
-  <!-- Robot Footprint -->
-  <link name="base_footprint"/>
-  <joint name="base_joint" type="fixed">
-    <parent link="base_footprint"/>
-    <child link="base_link"/>
-    <origin xyz="0.0 0.0 0.075" rpy="0 0 0"/>
-  </joint>
 </robot>
