Commit message: Fixed bugs in bracket and link xacro

File: urdf/components/bracket.xacro (robot description, xacro)
@@ -147,5 +147,5 @@
         </xacro:if>
         <xacro:if value="${bracket_type.endswith('LeftOutside')}">
-          <origin xyz="0 -.03 .04" rpy="${pi/2} 0 0"/>
+          <origin xyz="0 .03 .04" rpy="${pi/2} 0 ${pi}"/>
         </xacro:if>
         <xacro:if value="${bracket_type.endswith('LeftInside')}">

File: urdf/components/link.xacro (robot description, xacro)
@@ -61,11 +61,11 @@
           </xacro:if>
           <xacro:if value="${input == 'RightAngle' and output == 'Inline'}">
-            <origin xyz="${extension} 0 ${edge_to_center}" rpy="${pi/2} ${twist+pi} ${pi/2}"/>
+            <origin xyz="${extension} 0 ${edge_to_center}" rpy="${pi/2} ${twist} ${pi/2}"/>
           </xacro:if>
           <xacro:if value="${input == 'Inline' and output =='RightAngle'}">
-            <origin xyz="${edge_to_center * sin(twist+pi/2)} ${edge_to_center * -cos(twist+pi/2)} ${extension}" rpy="${pi/2} ${-pi/2} ${twist+pi/2}"/>
+            <origin xyz="${edge_to_center * sin(twist-pi/2)} ${edge_to_center * -cos(twist-pi/2)} ${extension}" rpy="${pi/2} ${-pi/2} ${twist-pi/2}"/>
           </xacro:if>
           <xacro:if value="${input == 'Inline' and output =='Inline'}">
-            <origin xyz="${0} ${0} ${extension}" rpy="${0} ${0} ${twist-pi/2}"/>
+            <origin xyz="${0} ${0} ${extension}" rpy="${0} ${0} ${twist+pi/2}"/>
           </xacro:if>
           <geometry>
@@ -84,11 +84,11 @@
           </xacro:if>
           <xacro:if value="${input == 'RightAngle' and output == 'Inline'}">
-            <origin xyz="${extension} 0 ${edge_to_center}" rpy="${pi/2} ${twist+pi} ${pi/2}"/>
+            <origin xyz="${extension} 0 ${edge_to_center}" rpy="${pi/2} ${twist} ${pi/2}"/>
           </xacro:if>
           <xacro:if value="${input == 'Inline' and output =='RightAngle'}">
-            <origin xyz="${edge_to_center * sin(twist+pi/2)} ${edge_to_center * -cos(twist+pi/2)} ${extension}" rpy="${pi/2} ${-pi/2} ${twist+pi/2}"/>
+            <origin xyz="${edge_to_center * sin(twist-pi/2)} ${edge_to_center * -cos(twist-pi/2)} ${extension}" rpy="${pi/2} ${-pi/2} ${twist-pi/2}"/>
           </xacro:if>
           <xacro:if value="${input == 'Inline' and output =='Inline'}">
-            <origin xyz="${0} ${0} ${extension}" rpy="${0} ${0} ${twist-pi/2}"/>
+            <origin xyz="${0} ${0} ${extension}" rpy="${0} ${0} ${twist+pi/2}"/>
           </xacro:if>
           <geometry>
@@ -119,17 +119,17 @@
       </xacro:if>
       <xacro:if value="${input == 'RightAngle' and output == 'Inline'}">
-        <origin xyz="${extension} 0 ${edge_to_center}" rpy="${pi/2} ${twist+pi} ${pi/2}"/>
+        <origin xyz="${extension} 0 ${edge_to_center}" rpy="${pi/2} ${twist+pi/2} ${pi/2}"/>
       </xacro:if>
       <xacro:if value="${input == 'Inline' and output =='RightAngle'}">
-        <origin xyz="${edge_to_center * sin(twist+pi/2)} ${edge_to_center * -cos(twist+pi/2)} ${extension}" rpy="${pi/2} ${-pi/2} ${twist+pi/2}"/>
+        <origin xyz="${edge_to_center * sin(twist-pi/2)} ${edge_to_center * -cos(twist-pi/2)} ${extension}" rpy="${pi/2} ${-pi/2} ${twist-pi/2}"/>
       </xacro:if>
       <xacro:if value="${input == 'Inline' and output =='Inline'}">
-        <origin xyz="${0} ${0} ${extension}" rpy="${0} ${0} ${twist-pi/2}"/>
+        <origin xyz="${0} ${0} ${extension}" rpy="${0} ${0} ${twist}"/>
       </xacro:if>
       <xacro:if value="${input == 'RightAngle' and output =='None'}">
-        <origin xyz="${extension} 0 ${edge_to_center}" rpy="${pi/2} ${twist+pi} ${pi/2}"/>
+        <origin xyz="${extension} 0 ${edge_to_center}" rpy="${pi/2} ${twist+pi/2} ${pi/2}"/>
       </xacro:if>
       <xacro:if value="${input == 'Inline' and output =='None'}">
-        <origin xyz="${0} ${0} ${extension}" rpy="${0} ${0} ${twist-pi/2}"/>
+        <origin xyz="${0} ${0} ${extension}" rpy="${0} ${0} ${twist}"/>
       </xacro:if>
     </joint>

Commit message: Corrected link and bracket xacros

File: urdf/components/bracket.xacro (robot description, xacro)
@@ -111,5 +111,5 @@
         </xacro:if>
         <xacro:if value="${bracket_type.endswith('LeftOutside')}">
-          <origin xyz="0 -.03 .04" rpy="${pi/2} 0 0"/>
+          <origin xyz="0 .03 .04" rpy="${pi/2} 0 ${pi}"/>
         </xacro:if>
         <xacro:if value="${bracket_type.endswith('LeftInside')}">
@@ -259,23 +259,23 @@
     <parent link="${name}/INPUT_INTERFACE"/>
     <child link="${child}/INPUT_INTERFACE"/>
-    <xacro:if value="${bracket_type.endswith('RightOutside')}">
-      <origin xyz="0 -.0375 .055" rpy="${pi/2} 0 0"/>
-    </xacro:if>
-    <xacro:if value="${bracket_type.endswith('RightInside')}">
-      <origin xyz="0 .0225 .055" rpy="${pi/2} 0 0"/>
-    </xacro:if>
-    <xacro:if value="${bracket_type.endswith('LeftOutside')}">
-      <origin xyz="0 .0375 .055" rpy="${-pi/2} 0 0"/>
-    </xacro:if>
-    <xacro:if value="${bracket_type.endswith('LeftInside')}">
-      <origin xyz="0 -.0225 .055" rpy="${-pi/2} 0 0"/>
-    </xacro:if>
-    <xacro:if value="${bracket_type.endswith('Left')}">
-      <origin xyz="0 .043 .04" rpy="${-pi/2} 0 0"/>
-    </xacro:if>
-    <xacro:if value="${bracket_type.endswith('Right')}">
-      <origin xyz="0 -.043 .04" rpy="${pi/2} 0 0"/>
-    </xacro:if>
-  </joint>
+      <xacro:if value="${bracket_type.endswith('RightOutside')}">
+        <origin xyz="0 -.0375 .055" rpy="${pi/2} 0 0"/>
+      </xacro:if>
+      <xacro:if value="${bracket_type.endswith('RightInside')}">
+        <origin xyz="0 .0225 .055" rpy="${pi/2} 0 0"/>
+      </xacro:if>
+      <xacro:if value="${bracket_type.endswith('LeftOutside')}">
+        <origin xyz="0 .0375 .055" rpy="${-pi/2} 0 0"/>
+      </xacro:if>
+      <xacro:if value="${bracket_type.endswith('LeftInside')}">
+        <origin xyz="0 -.0225 .055" rpy="${-pi/2} 0 0"/>
+      </xacro:if>
+      <xacro:if value="${bracket_type.endswith('Left')}">
+        <origin xyz="0 .043 .04" rpy="${-pi/2} 0 0"/>
+      </xacro:if>
+      <xacro:if value="${bracket_type.endswith('Right')}">
+        <origin xyz="0 -.043 .04" rpy="${pi/2} 0 0"/>
+      </xacro:if>
+    </joint>
   </xacro:macro>
 </robot>

File: urdf/components/link.xacro (robot description, xacro)
@@ -60,11 +60,11 @@
         </xacro:if>
         <xacro:if value="${input == 'RightAngle' and output == 'Inline'}">
-          <origin xyz="${extension} 0 ${edge_to_center}" rpy="${pi/2} ${twist+pi} ${pi/2}"/>
+          <origin xyz="${extension} 0 ${edge_to_center}" rpy="${pi/2} ${twist} ${pi/2}"/>
         </xacro:if>
         <xacro:if value="${input == 'Inline' and output =='RightAngle'}">
-          <origin xyz="${edge_to_center * sin(twist+pi/2)} ${edge_to_center * -cos(twist+pi/2)} ${extension}" rpy="${pi/2} ${-pi/2} ${twist+pi/2}"/>
+          <origin xyz="${edge_to_center * sin(twist-pi/2)} ${edge_to_center * -cos(twist-pi/2)} ${extension}" rpy="${pi/2} ${-pi/2} ${twist-pi/2}"/>
         </xacro:if>
         <xacro:if value="${input == 'Inline' and output =='Inline'}">
-          <origin xyz="${0} ${0} ${extension}" rpy="${0} ${0} ${twist-pi/2}"/>
+          <origin xyz="${0} ${0} ${extension}" rpy="${0} ${0} ${twist+pi/2}"/>
         </xacro:if>
         <geometry>
@@ -83,11 +83,11 @@
         </xacro:if>
         <xacro:if value="${input == 'RightAngle' and output == 'Inline'}">
-          <origin xyz="${extension} 0 ${edge_to_center}" rpy="${pi/2} ${twist+pi} ${pi/2}"/>
+          <origin xyz="${extension} 0 ${edge_to_center}" rpy="${pi/2} ${twist} ${pi/2}"/>
         </xacro:if>
         <xacro:if value="${input == 'Inline' and output =='RightAngle'}">
-          <origin xyz="${edge_to_center * sin(twist+pi/2)} ${edge_to_center * -cos(twist+pi/2)} ${extension}" rpy="${pi/2} ${-pi/2} ${twist+pi/2}"/>
+          <origin xyz="${edge_to_center * sin(twist-pi/2)} ${edge_to_center * -cos(twist-pi/2)} ${extension}" rpy="${pi/2} ${-pi/2} ${twist-pi/2}"/>
         </xacro:if>
         <xacro:if value="${input == 'Inline' and output =='Inline'}">
-          <origin xyz="${0} ${0} ${extension}" rpy="${0} ${0} ${twist-pi/2}"/>
+          <origin xyz="${0} ${0} ${extension}" rpy="${0} ${0} ${twist+pi/2}"/>
         </xacro:if>
         <geometry>
@@ -117,11 +117,11 @@
       </xacro:if>
       <xacro:if value="${input == 'RightAngle' and output == 'Inline'}">
-        <origin xyz="${extension} 0 ${edge_to_center}" rpy="${pi/2} ${twist+pi} ${pi/2}"/>
+        <origin xyz="${extension} 0 ${edge_to_center}" rpy="${pi/2} ${twist+pi/2} ${pi/2}"/>
       </xacro:if>
       <xacro:if value="${input == 'Inline' and output =='RightAngle'}">
-        <origin xyz="${edge_to_center * sin(twist+pi/2)} ${edge_to_center * -cos(twist+pi/2)} ${extension}" rpy="${pi/2} ${-pi/2} ${twist+pi/2}"/>
+        <origin xyz="${edge_to_center * sin(twist-pi/2)} ${edge_to_center * -cos(twist-pi/2)} ${extension}" rpy="${pi/2} ${-pi/2} ${twist-pi/2}"/>
       </xacro:if>
       <xacro:if value="${input == 'Inline' and output =='Inline'}">
-        <origin xyz="${0} ${0} ${extension}" rpy="${0} ${0} ${twist-pi/2}"/>
+        <origin xyz="${0} ${0} ${extension}" rpy="${0} ${0} ${twist}"/>
       </xacro:if>
     </joint>

Commit message: Fixed R8 bracket collision bug

File: urdf/components/bracket.xacro (robot description, xacro)
@@ -62,8 +62,8 @@
       <collision>
         <xacro:if value="${bracket_type.endswith('Left')}">
-          <origin xyz="0 0 0" rpy="${pi/2} 0 ${pi/2}"/>
-        </xacro:if>
-        <xacro:if value="${bracket_type.endswith('Right')}">
-          <origin xyz="0 0 0" rpy="${pi/2} 0 ${-pi/2}"/>
+          <origin xyz="0 0 0" rpy="0 0 ${pi}"/>
+        </xacro:if>
+        <xacro:if value="${bracket_type.endswith('Right')}">
+          <origin xyz="0 0 0" rpy="0 0 0"/>
         </xacro:if>
         <geometry>
@@ -209,14 +209,14 @@
       <collision>
         <xacro:if value="${bracket_type.endswith('RightOutside')}">
-          <origin xyz="0 0 0.005" rpy="${pi/2} 0 ${pi/2}"/>
-        </xacro:if>
-        <xacro:if value="${bracket_type.endswith('RightInside')}">
-          <origin xyz="0 0 0.005" rpy="${pi/2} 0 ${-pi/2}"/>
-        </xacro:if>
-        <xacro:if value="${bracket_type.endswith('LeftOutside')}">
-          <origin xyz="0 0 0.005" rpy="${pi/2} 0 ${-pi/2}"/>
-        </xacro:if>
-        <xacro:if value="${bracket_type.endswith('LeftInside')}">
-          <origin xyz="0 0 0.005" rpy="${pi/2} 0 ${pi/2}"/>
+          <origin xyz="0 0 0" rpy="0 0 0"/>
+        </xacro:if>
+        <xacro:if value="${bracket_type.endswith('RightInside')}">
+          <origin xyz="0 0 0" rpy="0 0 ${pi}"/>
+        </xacro:if>
+        <xacro:if value="${bracket_type.endswith('LeftOutside')}">
+          <origin xyz="0 0 0" rpy="0 0 ${pi}"/>
+        </xacro:if>
+        <xacro:if value="${bracket_type.endswith('LeftInside')}">
+          <origin xyz="0 0 0" rpy="0 0 0"/>
         </xacro:if>
         <geometry>

File: urdf/components/end_effector.xacro (robot description, xacro)
@@ -67,5 +67,4 @@
           <mesh filename="file://$(find hebi_description)/meshes/PM-2358-02.stl" scale="0.001 0.001 0.001"/>
         </geometry>
-        <xacro:black_material/>
       </collision>
       <inertial>
