Commit message: Changed limit values in end_effector to double

File: urdf/components/end_effector.xacro (robot description, xacro)
@@ -141,5 +141,5 @@
       <parent link="${name}/INPUT_INTERFACE"/>
       <child link="${name}/${prefix}_finger"/>
-      <limit effort="1000" velocity="1000" lower="0" upper="${0.37*pi}"/>
+      <limit effort="1000.0" velocity="1000.0" lower="0" upper="${0.37*pi}"/>
     </joint>
     <gazebo reference="${name}/input_${prefix}_finger">
@@ -160,5 +160,5 @@
       <child link="${name}/${prefix}_gripper"/>
       <mimic joint="${name}/input_l_finger" multiplier="-1.0" />
-      <limit effort="1000" velocity="1000" lower="${-pi/2}" upper="0"/>
+      <limit effort="1000.0" velocity="1000.0" lower="${-pi/2}" upper="0"/>
     </joint>
   </xacro:macro>
@@ -306,5 +306,5 @@
         <origin xyz="0 0 0" rpy="0 0 0" />
         <axis xyz="0 0 1" />
-        <limit effort="1000" velocity="1000" lower="-1.0" upper="1.0"/>
+        <limit effort="1000.0" velocity="1000.0" lower="-1.0" upper="1.0"/>
         <!-- Don't actually want the pinion to move (only needed fore gazebo)
              so set multiplier very small -->
@@ -336,6 +336,6 @@
               <lower>${-2*pi}</lower>
               <upper>${2*pi}</upper>
-              <effort>1000</effort>
-              <velocity>1000</velocity>
+              <effort>1000.0</effort>
+              <velocity>1000.0</velocity>
             </limit>
           </axis>
@@ -350,6 +350,6 @@
               <lower>${-2*pi}</lower>
               <upper>${2*pi}</upper>
-              <effort>1000</effort>
-              <velocity>1000</velocity>
+              <effort>1000.0</effort>
+              <velocity>1000.0</velocity>
             </limit>
           </axis>

Commit message: New end effector xacro

File: urdf/components/end_effector.xacro (robot description, xacro)
@@ -197,5 +197,5 @@
     </joint>
   </xacro:macro>
-  <xacro:macro name="gripper" params="name type:=Custom mass:=0.0 com_trans:='0 0 0' output_trans:='0 0 0'">
+  <xacro:macro name="gripper" params="name type:=Custom mass:=0.01 com_trans:='0 0 0' com_rot:='0 0 0' output_trans:='0 0 0' output_rot:='0 0 0' ixx='None' iyy='None' izz='None' ixy=0.0 ixz=0.0 iyz=0.0 mesh_path='' mesh_rot='0 0 0' mesh_trans='0 0 0' mesh_scale='1 1 1'">
     <xacro:property name="com_trans_list" value="${list(map(float, com_trans.split(' ')))}" />
     <xacro:if value="${ com_trans_list[0] + com_trans_list[1] + com_trans_list[2] >= 0.01 }">
@@ -205,21 +205,62 @@
       <xacro:property name="gripper_len" value="0.1" />
     </xacro:unless>
+    <xacro:if value="${ixx == 'None'}">
+      <xacro:property name="_ixx" value="${2.0/5.0 * mass * pow(gripper_len, 2)}" />
+    </xacro:if>
+    <xacro:unless value="${ixx == 'None'}">
+      <xacro:property name="_ixx" value="${ixx}" />
+    </xacro:unless>
+    <xacro:if value="${iyy == 'None'}">
+      <xacro:property name="_iyy" value="${2.0/5.0 * mass * pow(gripper_len, 2)}" />
+    </xacro:if>
+    <xacro:unless value="${iyy == 'None'}">
+      <xacro:property name="_iyy" value="${iyy}" />
+    </xacro:unless>
+    <xacro:if value="${izz == 'None'}">
+      <xacro:property name="_izz" value="${2.0/5.0 * mass * pow(gripper_len, 2)}" />
+    </xacro:if>
+    <xacro:unless value="${izz == 'None'}">
+      <xacro:property name="_izz" value="${izz}" />
+    </xacro:unless>
     <xacro:if value="${type == 'Custom'}">
       <link name="${name}/INPUT_INTERFACE">
-        <visual>
-          <origin xyz="0 0 0.0005" rpy="0 0 0" />
-          <geometry>
-            <box size="0.001 0.001 0.001" />
-          </geometry>
-        </visual>
+        <xacro:if value="${mesh_path != ''}">
+          <visual>
+            <origin xyz="${mesh_trans}" rpy="${mesh_rot}"/>
+            <geometry>
+              <mesh filename="${mesh_path}" scale="${mesh_scale}"/>
+            </geometry>
+            <xacro:black_material/>
+          </visual>
+          <collision>
+            <origin xyz="${mesh_trans}" rpy="${mesh_rot}"/>
+            <geometry>
+              <mesh filename="${mesh_path}" scale="${mesh_scale}"/>
+            </geometry>
+          </collision>
+        </xacro:if>
+        <xacro:unless value="${mesh_path != ''}">
+          <visual>
+            <origin xyz="0 0 0.0005" rpy="0 0 0" />
+            <geometry>
+              <box size="0.001 0.001 0.001" />
+            </geometry>
+          </visual>
+        </xacro:unless>
         <inertial>
-          <origin xyz="${com_trans}" rpy="0 0 0" />
+          <origin xyz="${com_trans}" rpy="${com_rot}" />
           <mass value="${mass}" />
           <inertia
-            ixx="${2.0/5.0 * mass * pow(gripper_len, 2)}" ixy="0.0" ixz="0.0"
-            iyy="${2.0/5.0 * mass * pow(gripper_len, 2)}" iyz="0.0"
-            izz="${2.0/5.0 * mass * pow(gripper_len, 2)}" />
+            ixx="${_ixx}" ixy="${ixy}" ixz="${ixz}"
+            iyy="${_iyy}" iyz="${iyz}"
+            izz="${_izz}"/>
         </inertial>
       </link>
+      <link name="${name}/OUTPUT_INTERFACE"/>
+      <joint name="${name}/OUTPUT_JOINT" type="fixed">
+        <origin xyz="${output_trans}" rpy="${output_rot}" />
+        <parent link="${name}/INPUT_INTERFACE"/>
+        <child link="${name}/OUTPUT_INTERFACE"/>
+      </joint>
     </xacro:if>
     <xacro:if value="${type.endswith('Parallel')}">

File: urdf/kits/A-2240-06.urdf.xacro (robot description, xacro)
@@ -21,4 +21,7 @@
   <xacro:bracket type="R8LightRight" name="$(arg prefix)wrist3_bracket" child="$(arg prefix)J6_wrist3"/>
   <xacro:actuator type="R8_3" name="$(arg prefix)J6_wrist3" child="$(arg prefix)end_effector"/>
-  <xacro:gripper type="Custom" name="$(arg prefix)end_effector" mass="0.005"/>
+  <xacro:gripper type="Custom" name="$(arg prefix)end_effector" mass="0.005"
+                               output_trans="0.1 0 0.1" output_rot="0 1.57 0"
+                               mesh_path="file://$(find hebi_description)/meshes/PM-2132-01L.stl"
+                               mesh_trans="0 0 0.1" mesh_rot="1.57 0 1.57" mesh_scale="0.001 0.001 0.001"/>
 </robot>

Commit message: Modified URDF and HRDF

File: urdf/components/end_effector.xacro (robot description, xacro)
@@ -197,5 +197,5 @@
     </joint>
   </xacro:macro>
-  <xacro:macro name="gripper" params="name type:=Custom mass:=0.01 com_trans:='0 0 0' com_rot:='0 0 0' output_trans:='0 0 0' output_rot:='0 0 0' ixx='None' iyy='None' izz='None' ixy=0.0 ixz=0.0 iyz=0.0 mesh_path='' mesh_rot='0 0 0' mesh_trans='0 0 0' mesh_scale='1 1 1'">
+  <xacro:macro name="gripper" params="name type:=Custom mass:=0.01 com_trans:='0 0 0' com_rot:='0 0 0' output_trans:='0 0 0' output_rot:='0 0 0' ixx='None' iyy='None' izz='None' ixy=0.0 ixz=0.0 iyz=0.0 mesh_path='' mesh_rot='0 0 0' mesh_trans='0 0 0'">
     <xacro:property name="com_trans_list" value="${list(map(float, com_trans.split(' ')))}" />
     <xacro:if value="${ com_trans_list[0] + com_trans_list[1] + com_trans_list[2] >= 0.01 }">
@@ -229,5 +229,5 @@
             <origin xyz="${mesh_trans}" rpy="${mesh_rot}"/>
             <geometry>
-              <mesh filename="${mesh_path}" scale="${mesh_scale}"/>
+              <mesh filename="${mesh_path}"/>
             </geometry>
             <xacro:black_material/>
@@ -236,5 +236,5 @@
             <origin xyz="${mesh_trans}" rpy="${mesh_rot}"/>
             <geometry>
-              <mesh filename="${mesh_path}" scale="${mesh_scale}"/>
+              <mesh filename="${mesh_path}"/>
             </geometry>
           </collision>

File: urdf/kits/A-2240-06.urdf.xacro (robot description, xacro)
@@ -23,5 +23,5 @@
   <xacro:gripper type="Custom" name="$(arg prefix)end_effector" mass="0.005"
                                output_trans="0.1 0 0.1" output_rot="0 1.57 0"
-                               mesh_path="file://$(find hebi_description)/meshes/PM-2132-01L.stl"
-                               mesh_trans="0 0 0.1" mesh_rot="1.57 0 1.57" mesh_scale="0.001 0.001 0.001"/>
+                               mesh_path="file://$(find hebi_description)/meshes/A-2038-02.obj"
+                               mesh_trans="0 0 0.1" mesh_rot="1.57 0 1.57" />
 </robot>

Commit message: Updated end effector xacro

File: urdf/components/end_effector.xacro (robot description, xacro)
@@ -197,5 +197,5 @@
     </joint>
   </xacro:macro>
-  <xacro:macro name="gripper" params="name type:=Custom mass:=0.0 com_trans:='0 0 0' output_trans:='0 0 0'">
+  <xacro:macro name="gripper" params="name type:=Custom mass:=0.01 output_trans:='0 0 0' output_rot:='0 0 0' com_trans:='0 0 0' com_rot:='0 0 0' ixx='None' iyy='None' izz='None' ixy=0 ixz=0 iyz=0">
     <xacro:property name="com_trans_list" value="${list(map(float, com_trans.split(' ')))}" />
     <xacro:if value="${ com_trans_list[0] + com_trans_list[1] + com_trans_list[2] >= 0.01 }">
@@ -204,4 +204,22 @@
     <xacro:unless value="${ com_trans_list[0] + com_trans_list[1] + com_trans_list[2] >= 0.01 }">
       <xacro:property name="gripper_len" value="0.1" />
+    </xacro:unless>
+    <xacro:if value="${ixx == 'None'}">
+      <xacro:property name="_ixx" value="${2.0/5.0 * mass * pow(gripper_len, 2)}" />
+    </xacro:if>
+    <xacro:unless value="${ixx == 'None'}">
+      <xacro:property name="_ixx" value="${ixx}" />
+    </xacro:unless>
+    <xacro:if value="${iyy == 'None'}">
+      <xacro:property name="_iyy" value="${2.0/5.0 * mass * pow(gripper_len, 2)}" />
+    </xacro:if>
+    <xacro:unless value="${iyy == 'None'}">
+      <xacro:property name="_iyy" value="${iyy}" />
+    </xacro:unless>
+    <xacro:if value="${izz == 'None'}">
+      <xacro:property name="_izz" value="${2.0/5.0 * mass * pow(gripper_len, 2)}" />
+    </xacro:if>
+    <xacro:unless value="${izz == 'None'}">
+      <xacro:property name="_izz" value="${izz}" />
     </xacro:unless>
     <xacro:if value="${type == 'Custom'}">
@@ -214,12 +232,18 @@
         </visual>
         <inertial>
-          <origin xyz="${com_trans}" rpy="0 0 0" />
+          <origin xyz="${com_trans}" rpy="${com_rot}" />
           <mass value="${mass}" />
           <inertia
-            ixx="${2.0/5.0 * mass * pow(gripper_len, 2)}" ixy="0.0" ixz="0.0"
-            iyy="${2.0/5.0 * mass * pow(gripper_len, 2)}" iyz="0.0"
-            izz="${2.0/5.0 * mass * pow(gripper_len, 2)}" />
+            ixx="${_ixx}" ixy="${ixy}" ixz="${ixz}"
+            iyy="${_iyy}" iyz="${iyz}"
+            izz="${_izz}"/>
         </inertial>
       </link>
+      <link name="${name}/output"/>
+      <joint name="${name}/output_joint" type="fixed">
+        <origin xyz="${output_trans}" rpy="${output_rot}" />
+        <parent link="${name}"/>
+        <child link="${name}/output"/>
+      </joint>
     </xacro:if>
     <xacro:if value="${type.endswith('Parallel')}">
@@ -369,4 +393,10 @@
         </joint>
       </gazebo>
+      <link name="${name}/output"/>
+      <joint name="${name}/output_joint" type="fixed">
+        <origin xyz="0 0 0.05" rpy="0 0 0" />
+        <parent link="${name}"/>
+        <child link="${name}/output"/>
+      </joint>
     </xacro:if>
   </xacro:macro>

Commit message: Modified end effector default mass

File: urdf/components/end_effector.xacro (robot description, xacro)
@@ -197,5 +197,5 @@
     </joint>
   </xacro:macro>
-  <xacro:macro name="gripper" params="name type:=Custom mass:=0.01 output_trans:='0 0 0' output_rot:='0 0 0' com_trans:='0 0 0' com_rot:='0 0 0' ixx='None' iyy='None' izz='None' ixy=0 ixz=0 iyz=0">
+  <xacro:macro name="gripper" params="name type:=Custom mass:=0.001 output_trans:='0 0 0' output_rot:='0 0 0' com_trans:='0 0 0' com_rot:='0 0 0' ixx='None' iyy='None' izz='None' ixy=0 ixz=0 iyz=0">
     <xacro:property name="com_trans_list" value="${list(map(float, com_trans.split(' ')))}" />
     <xacro:if value="${ com_trans_list[0] + com_trans_list[1] + com_trans_list[2] >= 0.01 }">

File: urdf/kits/A-2084-01.urdf.xacro (robot description, xacro)
@@ -18,4 +18,4 @@
   <xacro:link type="X5" extension="0.325" twist="0" name="$(arg prefix)link_2" child="$(arg prefix)J4_wrist/body"/>
   <xacro:actuator type="X5_1" name="$(arg prefix)J4_wrist" child="$(arg prefix)end_effector_1"/>
-  <xacro:gripper mass="0.01" name="$(arg prefix)end_effector_1"/>
+  <xacro:gripper name="$(arg prefix)end_effector_1"/>
 </robot>

File: urdf/kits/A-2085-03.urdf.xacro (robot description, xacro)
@@ -16,4 +16,4 @@
   <xacro:link type="X5" extension="0.325" twist="${pi}" name="$(arg prefix)link_1" child="$(arg prefix)J3_elbow/body"/>
   <xacro:actuator type="X5_4" name="$(arg prefix)J3_elbow" child="$(arg prefix)end_effector_1"/>
-  <xacro:gripper mass="0.01" name="$(arg prefix)end_effector_1"/>
+  <xacro:gripper name="$(arg prefix)end_effector_1"/>
 </robot>

File: urdf/kits/A-2085-04.urdf.xacro (robot description, xacro)
@@ -18,4 +18,4 @@
   <xacro:link type="X5" extension="0.325" twist="${pi}" name="$(arg prefix)link_2" child="$(arg prefix)J4_wrist/body"/>
   <xacro:actuator type="X5_1" name="$(arg prefix)J4_wrist" child="$(arg prefix)end_effector_1"/>
-  <xacro:gripper mass="0.01" name="$(arg prefix)end_effector_1"/>
+  <xacro:gripper name="$(arg prefix)end_effector_1"/>
 </robot>

File: urdf/kits/A-2085-05.urdf.xacro (robot description, xacro)
@@ -21,4 +21,4 @@
   <xacro:output type="X5LightRight" parent="$(arg prefix)bracket_2" child="$(arg prefix)J5_wrist2/body" name="$(arg prefix)bracket_2_J5_wrist2"/>
   <xacro:actuator type="X5_1" name="$(arg prefix)J5_wrist2" child="$(arg prefix)end_effector_1"/>
-  <xacro:gripper mass="0.01" name="$(arg prefix)end_effector_1"/>
+  <xacro:gripper name="$(arg prefix)end_effector_1"/>
 </robot>

File: urdf/kits/A-2085-05G.urdf.xacro (robot description, xacro)
@@ -21,4 +21,4 @@
   <xacro:output type="X5LightRight" parent="$(arg prefix)bracket_2" child="$(arg prefix)J5_wrist2/body" name="$(arg prefix)bracket_2_J5_wrist2"/>
   <xacro:actuator type="X5_1" name="$(arg prefix)J5_wrist2" child="$(arg prefix)end_effector_1"/>
-  <xacro:gripper type="X5Parallel" mass="0.01" name="$(arg prefix)end_effector_1"/>
+  <xacro:gripper type="X5Parallel" name="$(arg prefix)end_effector_1"/>
 </robot>

File: urdf/kits/A-2085-06.urdf.xacro (robot description, xacro)
@@ -24,4 +24,4 @@
   <xacro:output type="X5LightRight" parent="$(arg prefix)bracket_3" child="$(arg prefix)J6_wrist3/body" name="$(arg prefix)bracket_3_J6_wrist3"/>
   <xacro:actuator type="X5_1" name="$(arg prefix)J6_wrist3" child="$(arg prefix)end_effector_1"/>
-  <xacro:gripper mass="0.01" name="$(arg prefix)end_effector_1"/>
+  <xacro:gripper name="$(arg prefix)end_effector_1"/>
 </robot>

File: urdf/kits/A-2085-06G.urdf.xacro (robot description, xacro)
@@ -24,4 +24,4 @@
   <xacro:output type="X5LightRight" parent="$(arg prefix)bracket_3" child="$(arg prefix)J6_wrist3/body" name="$(arg prefix)bracket_3_J6_wrist3"/>
   <xacro:actuator type="X5_1" name="$(arg prefix)J6_wrist3" child="$(arg prefix)end_effector_1"/>
-  <xacro:gripper type="X5Parallel" mass="0.01" name="$(arg prefix)end_effector_1"/>
+  <xacro:gripper type="X5Parallel" name="$(arg prefix)end_effector_1"/>
 </robot>

File: urdf/kits/A-2099-07.urdf.xacro (robot description, xacro)
@@ -27,4 +27,4 @@
   <xacro:output type="X5LightRight" parent="$(arg prefix)bracket_3" child="$(arg prefix)J7_wrist2/body" name="$(arg prefix)bracket_3_J7_wrist2"/>
   <xacro:actuator type="X5_4" name="$(arg prefix)J7_wrist2" child="$(arg prefix)end_effector_1"/>
-  <xacro:gripper mass="0.01" name="$(arg prefix)end_effector_1"/>
+  <xacro:gripper name="$(arg prefix)end_effector_1"/>
 </robot>

File: urdf/kits/A-2099-07G.urdf.xacro (robot description, xacro)
@@ -27,4 +27,4 @@
   <xacro:output type="X5LightRight" parent="$(arg prefix)bracket_3" child="$(arg prefix)J7_wrist2/body" name="$(arg prefix)bracket_3_J7_wrist2"/>
   <xacro:actuator type="X5_4" name="$(arg prefix)J7_wrist2" child="$(arg prefix)end_effector_1"/>
-  <xacro:gripper type="X5Parallel" mass="0.01" name="$(arg prefix)end_effector_1"/>
+  <xacro:gripper type="X5Parallel" name="$(arg prefix)end_effector_1"/>
 </robot>

File: urdf/kits/A-2240-04.urdf.xacro (robot description, xacro)
@@ -18,4 +18,4 @@
   <xacro:link type="R8" extension="0.325" twist="${pi}" name="$(arg prefix)link_2" child="$(arg prefix)J4_wrist/body"/>
   <xacro:actuator type="R8_3" name="$(arg prefix)J4_wrist" child="$(arg prefix)end_effector_1"/>
-  <xacro:gripper mass="0.01" name="$(arg prefix)end_effector_1"/>
+  <xacro:gripper name="$(arg prefix)end_effector_1"/>
 </robot>

File: urdf/kits/A-2240-05.urdf.xacro (robot description, xacro)
@@ -21,4 +21,4 @@
   <xacro:output type="R8LightRight" parent="$(arg prefix)bracket_2" child="$(arg prefix)J5_wrist2/body" name="$(arg prefix)bracket_2_J5_wrist2"/>
   <xacro:actuator type="R8_3" name="$(arg prefix)J5_wrist2" child="$(arg prefix)end_effector_1"/>
-  <xacro:gripper mass="0.01" name="$(arg prefix)end_effector_1"/>
+  <xacro:gripper name="$(arg prefix)end_effector_1"/>
 </robot>

File: urdf/kits/A-2240-05G.urdf.xacro (robot description, xacro)
@@ -21,4 +21,4 @@
   <xacro:output type="R8LightRight" parent="$(arg prefix)bracket_2" child="$(arg prefix)J5_wrist2/body" name="$(arg prefix)bracket_2_J5_wrist2"/>
   <xacro:actuator type="R8_3" name="$(arg prefix)J5_wrist2" child="$(arg prefix)end_effector_1"/>
-  <xacro:gripper type="R8Parallel" mass="0.01" name="$(arg prefix)end_effector_1"/>
+  <xacro:gripper type="R8Parallel" name="$(arg prefix)end_effector_1"/>
 </robot>

File: urdf/kits/A-2240-06.urdf.xacro (robot description, xacro)
@@ -24,4 +24,4 @@
   <xacro:output type="R8LightRight" parent="$(arg prefix)bracket_3" child="$(arg prefix)J6_wrist3/body" name="$(arg prefix)bracket_3_J6_wrist3"/>
   <xacro:actuator type="R8_3" name="$(arg prefix)J6_wrist3" child="$(arg prefix)end_effector_1"/>
-  <xacro:gripper mass="0.01" name="$(arg prefix)end_effector_1"/>
+  <xacro:gripper name="$(arg prefix)end_effector_1"/>
 </robot>

File: urdf/kits/A-2240-06G.urdf.xacro (robot description, xacro)
@@ -24,4 +24,4 @@
   <xacro:output type="R8LightRight" parent="$(arg prefix)bracket_3" child="$(arg prefix)J6_wrist3/body" name="$(arg prefix)bracket_3_J6_wrist3"/>
   <xacro:actuator type="R8_3" name="$(arg prefix)J6_wrist3" child="$(arg prefix)end_effector_1"/>
-  <xacro:gripper type="R8Parallel" mass="0.01" name="$(arg prefix)end_effector_1"/>
+  <xacro:gripper type="R8Parallel" name="$(arg prefix)end_effector_1"/>
 </robot>

File: urdf/kits/A-2302-01.urdf.xacro (robot description, xacro)
@@ -18,4 +18,4 @@
   <xacro:link type="R8" extension="0.325" twist="0" name="$(arg prefix)link_2" child="$(arg prefix)J4_wrist/body"/>
   <xacro:actuator type="R8_3" name="$(arg prefix)J4_wrist" child="$(arg prefix)end_effector_1"/>
-  <xacro:gripper mass="0.01" name="$(arg prefix)end_effector_1"/>
+  <xacro:gripper name="$(arg prefix)end_effector_1"/>
 </robot>

File: urdf/kits/A-2303-01.urdf.xacro (robot description, xacro)
@@ -27,4 +27,4 @@
   <xacro:output type="R8LightRight" parent="$(arg prefix)bracket_3" child="$(arg prefix)J7_wrist2/body" name="$(arg prefix)bracket_3_J7_wrist2"/>
   <xacro:actuator type="R8_3" name="$(arg prefix)J7_wrist2" child="$(arg prefix)end_effector_1"/>
-  <xacro:gripper mass="0.01" name="$(arg prefix)end_effector_1"/>
+  <xacro:gripper name="$(arg prefix)end_effector_1"/>
 </robot>

File: urdf/kits/A-2303-01G.urdf.xacro (robot description, xacro)
@@ -27,4 +27,4 @@
   <xacro:output type="R8LightRight" parent="$(arg prefix)bracket_3" child="$(arg prefix)J7_wrist2/body" name="$(arg prefix)bracket_3_J7_wrist2"/>
   <xacro:actuator type="R8_3" name="$(arg prefix)J7_wrist2" child="$(arg prefix)end_effector_1"/>
-  <xacro:gripper type="R8Parallel" mass="0.01" name="$(arg prefix)end_effector_1"/>
+  <xacro:gripper type="R8Parallel" name="$(arg prefix)end_effector_1"/>
 </robot>

File: urdf/kits/A-2580-04.urdf.xacro (robot description, xacro)
@@ -18,4 +18,4 @@
   <xacro:link type="R8" extension="0.325" twist="${pi}" name="$(arg prefix)link_2" child="$(arg prefix)J4_wrist/body"/>
   <xacro:actuator type="T5_1" name="$(arg prefix)J4_wrist" child="$(arg prefix)end_effector_1"/>
-  <xacro:gripper mass="0.01" name="$(arg prefix)end_effector_1"/>
+  <xacro:gripper name="$(arg prefix)end_effector_1"/>
 </robot>

File: urdf/kits/A-2580-05.urdf.xacro (robot description, xacro)
@@ -21,4 +21,4 @@
   <xacro:output type="R8LightRight" parent="$(arg prefix)bracket_2" child="$(arg prefix)J5_wrist2/body" name="$(arg prefix)bracket_2_J5_wrist2"/>
   <xacro:actuator type="T5_1" name="$(arg prefix)J5_wrist2" child="$(arg prefix)end_effector_1"/>
-  <xacro:gripper mass="0.01" name="$(arg prefix)end_effector_1"/>
+  <xacro:gripper name="$(arg prefix)end_effector_1"/>
 </robot>
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