Commit message: Updated URDF

File: urdf/components/end_effector.xacro (robot description, xacro)
@@ -1,27 +1,27 @@
 <?xml version="1.0"?>
 <robot xmlns:xacro="http://www.ros.org/wiki/xacro">
-  <xacro:macro name="null_end_effector" params="name">
+  <xacro:macro name="null_end_effector" params="name output_trans:='0 0 0' output_rot:='0 0 0'">
     <link name="${name}">
-      <collision>
-        <origin xyz="0 0 0.0005" rpy="0 0 0"/>
+        <visual>
+          <origin xyz="0 0 0.0005" rpy="0 0 0"/>
           <geometry>
             <box size="0.001 0.001 0.001" rpy="0 0 0"/>
           </geometry>
-      </collision>
-      <visual>
-        <origin xyz="0 0 0.0005" rpy="0 0 0"/>
-          <geometry>
-            <box size="0.001 0.001 0.001" rpy="0 0 0"/>
-          </geometry>
-      </visual>
-      <inertial>
-        <origin xyz="0 0 0.0005" rpy="0 0 0"/>
+        </visual>
+        <inertial>
+          <origin xyz="0 0 0.0005" rpy="0 0 0"/>
           <mass value="0.001"/>
-        <inertia
-          ixx="0.001" ixy="0.0" ixz="0.0"
-          iyy="0.001" iyz="0.0"
-          izz="0.001"/>
-      </inertial>
-    </link>
+          <inertia
+            ixx="0.001" ixy="0.0" ixz="0.0"
+            iyy="0.001" iyz="0.0"
+            izz="0.001"/>
+          </inertial>
+      </link>
+      <link name="${name}/output"/>
+      <joint name="${name}/output_joint" type="fixed">
+        <origin xyz="${output_trans}" rpy="${output_rot}" />
+        <parent link="${name}"/>
+        <child link="${name}/output"/>
+      </joint>
   </xacro:macro>
   <xacro:macro name="parallel_gripper_outer_subassembly" params="name prefix">

File: urdf/kits/A-2240-06.urdf.xacro (robot description, xacro)
@@ -23,7 +23,23 @@
   <xacro:bracket type="R8LightRight" name="$(arg prefix)bracket_3"/>
   <xacro:output type="R8LightRight" parent="$(arg prefix)bracket_3" child="$(arg prefix)J6_wrist3/body" name="$(arg prefix)bracket_3_J6_wrist3"/>
-  <xacro:actuator type="R8_3" name="$(arg prefix)J6_wrist3" child="$(arg prefix)rigid_body_1"/>
-  <xacro:rigid-body mass="0.001" mesh_path="file://$(find hebi_description)/meshes/end_effector.obj" mesh_trans="0 0 0" mesh_rot="1.5708 -1.5708 0" mesh_scale="1 1 1" name="$(arg prefix)rigid_body_1"/>
-  <xacro:output trans="0.13 0.005 0.06" rot="-0 1.5708 0" parent="$(arg prefix)rigid_body_1" child="$(arg prefix)end_effector_1" name="$(arg prefix)rigid_body_1_end_effector_1"/>
-  <xacro:gripper name="$(arg prefix)end_effector_1"/>
+  <xacro:actuator type="R8_3" name="$(arg prefix)J6_wrist3" child="$(arg prefix)link_3"/>
+  <link name="$(arg prefix)link_3">
+    <visual>
+      <geometry>
+        <cylinder length="0.0005" radius="0.0075"/>
+      </geometry>
+    </visual>
+    <collision>
+      <geometry>
+        <cylinder length="0.0005" radius="0.0075"/>
+      </geometry>
+    </collision>
+  </link>
+  <joint name="link3_to_ee" type="fixed">
+    <parent link="$(arg prefix)link_3"/>
+    <child link="$(arg prefix)rigid_body_1"/>
+  </joint>
+  <xacro:rigid-body mass="0.001" mesh_path="file://$(find hebi_description)/meshes/end_effector.stl" mesh_trans="-0.1 0.08 0.1725" mesh_rot="0 ${pi} ${pi}" mesh_scale="1 1 1" name="$(arg prefix)rigid_body_1"/>
+  <xacro:output trans="0 0 0" rot="0 0 0" parent="$(arg prefix)rigid_body_1" child="$(arg prefix)end_effector_1" name="$(arg prefix)rigid_body_1_end_effector_1"/>
+  <xacro:null_end_effector name="$(arg prefix)end_effector_1" output_trans="0.005 0 0.13"/>
 </robot>

Commit message: Updated end-effector xacro from ros2/humble

File: urdf/components/end_effector.xacro (robot description, xacro)
@@ -1,27 +1,27 @@
 <?xml version="1.0"?>
 <robot xmlns:xacro="http://www.ros.org/wiki/xacro">
-  <xacro:macro name="null_end_effector" params="name output_trans:='0 0 0' output_rot:='0 0 0'">
+  <xacro:macro name="null_end_effector" params="name">
     <link name="${name}">
-        <visual>
-          <origin xyz="0 0 0.0005" rpy="0 0 0"/>
+      <collision>
+        <origin xyz="0 0 0.0005" rpy="0 0 0"/>
           <geometry>
             <box size="0.001 0.001 0.001" rpy="0 0 0"/>
           </geometry>
-        </visual>
-        <inertial>
-          <origin xyz="0 0 0.0005" rpy="0 0 0"/>
+      </collision>
+      <visual>
+        <origin xyz="0 0 0.0005" rpy="0 0 0"/>
+          <geometry>
+            <box size="0.001 0.001 0.001" rpy="0 0 0"/>
+          </geometry>
+      </visual>
+      <inertial>
+        <origin xyz="0 0 0.0005" rpy="0 0 0"/>
           <mass value="0.001"/>
-          <inertia
-            ixx="0.001" ixy="0.0" ixz="0.0"
-            iyy="0.001" iyz="0.0"
-            izz="0.001"/>
-          </inertial>
-      </link>
-      <link name="${name}/output"/>
-      <joint name="${name}/output_joint" type="fixed">
-        <origin xyz="${output_trans}" rpy="${output_rot}" />
-        <parent link="${name}"/>
-        <child link="${name}/output"/>
-      </joint>
+        <inertia
+          ixx="0.001" ixy="0.0" ixz="0.0"
+          iyy="0.001" iyz="0.0"
+          izz="0.001"/>
+      </inertial>
+    </link>
   </xacro:macro>
   <xacro:macro name="parallel_gripper_outer_subassembly" params="name prefix">

Commit message: Updated end-effector xacro again for null end effector

File: urdf/components/end_effector.xacro (robot description, xacro)
@@ -1,5 +1,5 @@
 <?xml version="1.0"?>
 <robot xmlns:xacro="http://www.ros.org/wiki/xacro">
-  <xacro:macro name="null_end_effector" params="name">
+  <xacro:macro name="null_end_effector" params="name output_trans:='0 0 0' output_rot:='0 0 0'">
     <link name="${name}">
       <collision>
@@ -24,4 +24,10 @@
       </inertial>
     </link>
+    <link name="${name}/output"/>
+    <joint name="${name}/output_joint" type="fixed">
+      <origin xyz="${output_trans}" rpy="${output_rot}" />
+      <parent link="${name}"/>
+      <child link="${name}/output"/>
+    </joint>
   </xacro:macro>
   <xacro:macro name="parallel_gripper_outer_subassembly" params="name prefix">

Commit message: Added collision geometry to end effector xacro

File: urdf/components/end_effector.xacro (robot description, xacro)
@@ -3,16 +3,16 @@
   <xacro:macro name="null_end_effector" params="name mass:=0.001 mass_offset:=0.0">
     <link name="${name}">
-      <collision>
+      <visual>
         <origin xyz="0 0 0.0005" rpy="0 0 0"/>
           <geometry>
             <box size="0.001 0.001 0.001" rpy="0 0 0"/>
           </geometry>
-      </collision>
-      <visual>
+      </visual>
+      <collision>
         <origin xyz="0 0 0.0005" rpy="0 0 0"/>
           <geometry>
             <box size="0.001 0.001 0.001" rpy="0 0 0"/>
           </geometry>
-      </visual>
+      </collision>
       <inertial>
         <origin xyz="0 0 0.0005" rpy="0 0 0"/>
@@ -62,4 +62,11 @@
         <xacro:black_material/>
       </visual>
+      <collision>
+        <origin xyz="-0.0115 0.029 -0.004" rpy="${pi/2} 0 0" />
+        <geometry>
+          <mesh filename="file://$(find hebi_description)/meshes/PM-2358-02.stl" scale="0.001 0.001 0.001"/>
+        </geometry>
+        <xacro:black_material/>
+      </collision>
       <inertial>
         <origin xyz="0 0.015 0.007" rpy="0 0 0"/>
@@ -109,4 +116,11 @@
         <xacro:silver_material/>
       </visual>
+      <collision>
+        <origin xyz="0 0 0" rpy="0 ${0.5*pi} 0"/>
+        <geometry>
+          <cylinder length="0.02" radius=".002" />
+        </geometry>
+        <xacro:silver_material/>
+      </collision>
       <inertial>
         <origin xyz="0 0 0" rpy="0 ${0.5*pi} 0"/>
@@ -172,4 +186,11 @@
         <xacro:black_material/>
       </visual>
+      <collision>
+        <origin xyz="-0.0115 -0.004 -0.004" rpy="0 0 0" />
+        <geometry>
+          <mesh filename="file://$(find hebi_description)/meshes/PM-2359-02.stl" scale="0.001 0.001 0.001"/>
+        </geometry>
+        <xacro:black_material/>
+      </collision>
       <inertial>
         <origin xyz="0 0 0.0215" rpy="${pi/2} 0 0"/>
@@ -231,4 +252,10 @@
           </geometry>
         </visual>
+        <collision>
+          <origin xyz="0 0 0.0005" rpy="0 0 0" />
+          <geometry>
+            <box size="0.001 0.001 0.001" />
+          </geometry>
+        </collision>
         <inertial>
           <origin xyz="${com_trans}" rpy="${com_rot}" />
@@ -257,4 +284,11 @@
           <xacro:black_material/>
         </visual>
+        <collision>
+          <origin xyz="0 0 0.00375" />
+            <geometry>
+            <cylinder length="0.0075" radius=".0225" />
+          </geometry>
+          <xacro:black_material/>
+        </collision>
         <inertial>
           <origin xyz="0 0 0" rpy="0 0 0"/>
@@ -279,4 +313,11 @@
           <xacro:black_material/>
         </visual>
+        <collision>
+          <origin xyz="-0.0225 0.0225 0" rpy="${pi/2} 0 0" />
+          <geometry>
+            <mesh filename="file://$(find hebi_description)/meshes/PM-2357-02.stl" scale="0.001 0.001 0.001"/>
+          </geometry>
+          <xacro:black_material/>
+        </collision>
         <inertial>
           <origin xyz="0 0 0" rpy="0 0 0"/>
