Commit message: Updated HRDF to URDF script with tree support

File: urdf/components/actuator.xacro (robot description, xacro)
@@ -74,5 +74,5 @@
       <xacro:property name="friction" value="0.5"/>
     </xacro:if>
-    <link name="${name}/INPUT_INTERFACE">
+    <link name="${name}">
       <visual>
         <origin xyz="0 0 0" rpy="0 0 0" />
@@ -115,5 +115,5 @@
       </inertial>
     </link>
-    <gazebo reference="${name}/INPUT_INTERFACE">
+    <gazebo reference="${name}">
       <xacro:unless value="${model_name.startswith('R8')}">
         <xacro:gazebo_red_material/>
@@ -124,6 +124,6 @@
     </gazebo>
     <joint name="${name}" type="${urdf_joint_type}">
-      <parent link="${name}/INPUT_INTERFACE"/>
-      <child link="${child}/INPUT_INTERFACE"/>
+      <parent link="${name}"/>
+      <child link="${child}"/>
       <xacro:if value="${model_name.startswith('X5')}">
         <origin xyz="0 0 0.031" rpy="0 0 0"/>
@@ -220,5 +220,5 @@
       <xacro:property name="friction" value="0.5"/>
     </xacro:if>
-    <link name="${name}/INPUT_INTERFACE">
+    <link name="${name}">
       <visual>
         <origin xyz="0 0 0" rpy="0 0 0" />
@@ -261,5 +261,5 @@
       </inertial>
     </link>
-    <gazebo reference="${name}/INPUT_INTERFACE">
+    <gazebo reference="${name}">
       <xacro:unless value="${model_name.startswith('R8')}">
         <xacro:gazebo_red_material/>
@@ -270,6 +270,6 @@
     </gazebo>
     <joint name="${name}" type="${urdf_joint_type}">
-      <parent link="${parent}/INPUT_INTERFACE"/>
-      <child link="${name}/INPUT_INTERFACE"/>
+      <parent link="${parent}"/>
+      <child link="${name}"/>
       <xacro:if value="${model_name.startswith('X5')}">
         <origin xyz="0 0 0.031" rpy="0 ${pi} 0"/>
@@ -293,6 +293,6 @@
     </joint>
     <joint name="${name}_fixed" type="fixed">
-      <parent link="${name}/INPUT_INTERFACE"/>
-      <child link="${child}/INPUT_INTERFACE"/>
+      <parent link="${name}"/>
+      <child link="${child}"/>
       <xacro:if value="${model_name.startswith('X5')}">
         <origin xyz="0 0 0" rpy="0 0 0"/>

File: urdf/components/bracket.xacro (robot description, xacro)
@@ -1,7 +1,7 @@
 <?xml version="1.0"?>
 <robot xmlns:xacro="http://www.ros.org/wiki/xacro">
-  <xacro:macro name="bracket" params="name child type">
+  <xacro:macro name="bracket" params="name type">
   <xacro:property name="bracket_type" value="${type}"/>
-  <link name="${name}/INPUT_INTERFACE">
+  <link name="${name}">
     <!-- Light bracket -->
     <xacro:if value="${bracket_type.startswith('X5Light')}">
@@ -248,5 +248,5 @@
     </xacro:if>
   </link>
-  <gazebo reference="${name}/INPUT_INTERFACE">
+  <gazebo reference="${name}">
     <xacro:if value="${bracket_type.startswith('X5Light')}">
       <xacro:gazebo_beige_material/>
@@ -256,26 +256,4 @@
     </xacro:if>
   </gazebo>
-  <joint name="${name}/OUTPUT_INTERFACE" type="fixed">
-    <parent link="${name}/INPUT_INTERFACE"/>
-    <child link="${child}/INPUT_INTERFACE"/>
-    <xacro:if value="${bracket_type.endswith('RightOutside')}">
-      <origin xyz="0 -.0375 .055" rpy="${pi/2} 0 0"/>
-    </xacro:if>
-    <xacro:if value="${bracket_type.endswith('RightInside')}">
-      <origin xyz="0 .0225 .055" rpy="${pi/2} 0 0"/>
-    </xacro:if>
-    <xacro:if value="${bracket_type.endswith('LeftOutside')}">
-      <origin xyz="0 .0375 .055" rpy="${-pi/2} 0 0"/>
-    </xacro:if>
-    <xacro:if value="${bracket_type.endswith('LeftInside')}">
-      <origin xyz="0 -.0225 .055" rpy="${-pi/2} 0 0"/>
-    </xacro:if>
-    <xacro:if value="${bracket_type.endswith('Left')}">
-      <origin xyz="0 .043 .04" rpy="${-pi/2} 0 0"/>
-    </xacro:if>
-    <xacro:if value="${bracket_type.endswith('Right')}">
-      <origin xyz="0 -.043 .04" rpy="${pi/2} 0 0"/>
-    </xacro:if>
-  </joint>
   </xacro:macro>
 </robot>

File: urdf/components/end_effector.xacro (robot description, xacro)
@@ -2,5 +2,5 @@
 <robot xmlns:xacro="http://www.ros.org/wiki/xacro">
   <xacro:macro name="null_end_effector" params="name">
-    <link name="${name}/INPUT_INTERFACE">
+    <link name="${name}">
       <collision>
         <origin xyz="0 0 0.0005" rpy="0 0 0"/>
@@ -139,5 +139,5 @@
         <mimic joint="${name}/input_l_finger" multiplier="1.0" offset="0" />
       </xacro:if>
-      <parent link="${name}/INPUT_INTERFACE"/>
+      <parent link="${name}"/>
       <child link="${name}/${prefix}_finger"/>
       <limit effort="1000.0" velocity="1000.0" lower="0" upper="${0.37*pi}"/>
@@ -206,5 +206,5 @@
     </xacro:unless>
     <xacro:if value="${type == 'Custom'}">
-      <link name="${name}/INPUT_INTERFACE">
+      <link name="${name}">
         <visual>
           <origin xyz="0 0 0.0005" rpy="0 0 0" />
@@ -225,5 +225,5 @@
     <xacro:if value="${type.endswith('Parallel')}">
       <!-- The base body of the gripper -->
-      <link name="${name}/INPUT_INTERFACE">
+      <link name="${name}">
         <visual>
           <origin xyz="0 0 0.00375" />
@@ -243,5 +243,5 @@
         </inertial>
       </link>
-      <gazebo reference="${name}/INPUT_INTERFACE">
+      <gazebo reference="${name}">
         <xacro:gazebo_black_material/>
       </gazebo>
@@ -270,5 +270,5 @@
       <joint name="${name}/input_center_hub" type="fixed">
         <origin xyz="0 0 0.0045" rpy="0 0 0" />
-        <parent link="${name}/INPUT_INTERFACE"/>
+        <parent link="${name}"/>
         <child link="${name}/center_hub"/>
       </joint>
@@ -359,5 +359,5 @@
           <parent>${name}/r_finger</parent>
           <child>${name}/l_finger</child>
-          <gearbox_reference_body>${name}/INPUT_INTERFACE</gearbox_reference_body>
+          <gearbox_reference_body>${name}</gearbox_reference_body>
           <gearbox_ratio>1</gearbox_ratio>
           <axis>

File: urdf/components/hebi.xacro (robot description, xacro)
@@ -44,4 +44,6 @@
   <xacro:include filename="./bracket.xacro"/>
   <xacro:include filename="./end_effector.xacro"/>
+  <xacro:include filename="./rigid_body.xacro"/>
+  <xacro:include filename="./output.xacro"/>
   <xacro:include filename="./omnibase.xacro"/>
 </robot>

File: urdf/components/link.xacro (robot description, xacro)
@@ -2,8 +2,8 @@
 <robot xmlns:xacro="http://www.ros.org/wiki/xacro">
   <!-- NOTE: joint must match the name of the module -->
-  <xacro:macro name="link" params="name child type:=X5 input:=RightAngle output:=RightAngle extension twist">
+  <xacro:macro name="link" params="name child type:=X5 input:=RightAngle output:=None extension twist">
     <xacro:property name="mass" value="${0.4 * (extension + 0.03) + 0.26}"/>
     <xacro:property name="edge_to_center" value="${.02}"/>
-    <link name="${name}/INPUT_INTERFACE">
+    <link name="${name}">
       <!-- Input Cap -->
       <visual>
@@ -55,49 +55,51 @@
       </collision>
       <!-- Output Cap -->
-      <visual>
-        <xacro:if value="${input == 'RightAngle' and output == 'RightAngle'}">
-          <origin xyz="${extension} ${sin(-twist) * edge_to_center} ${edge_to_center * (1 + cos(-twist))}" rpy="${twist} 0 0"/>
-        </xacro:if>
-        <xacro:if value="${input == 'RightAngle' and output == 'Inline'}">
-          <origin xyz="${extension} 0 ${edge_to_center}" rpy="${pi/2} ${twist+pi} ${pi/2}"/>
-        </xacro:if>
-        <xacro:if value="${input == 'Inline' and output =='RightAngle'}">
-          <origin xyz="${edge_to_center * sin(twist+pi/2)} ${edge_to_center * -cos(twist+pi/2)} ${extension}" rpy="${pi/2} ${-pi/2} ${twist+pi/2}"/>
-        </xacro:if>
-        <xacro:if value="${input == 'Inline' and output =='Inline'}">
-          <origin xyz="${0} ${0} ${extension}" rpy="${0} ${0} ${twist-pi/2}"/>
-        </xacro:if>
-        <geometry>
-          <xacro:if value="${output == 'RightAngle'}">
-            <mesh filename="file://$(find hebi_description)/meshes/A-2039-02.stl"/>
+      <xacro:if value="${output != 'None'}">
+        <visual>
+          <xacro:if value="${input == 'RightAngle' and output == 'RightAngle'}">
+            <origin xyz="${extension} ${sin(-twist) * edge_to_center} ${edge_to_center * (1 + cos(-twist))}" rpy="${twist} 0 0"/>
           </xacro:if>
-          <xacro:if value="${output == 'Inline'}">
-            <mesh filename="file://$(find hebi_description)/meshes/A-2226-01.stl" scale="0.001 0.001 0.001"/>
+          <xacro:if value="${input == 'RightAngle' and output == 'Inline'}">
+            <origin xyz="${extension} 0 ${edge_to_center}" rpy="${pi/2} ${twist+pi} ${pi/2}"/>
           </xacro:if>
-        </geometry>
-        <xacro:black_material/>
-      </visual>
-      <collision>
-        <xacro:if value="${input == 'RightAngle' and output == 'RightAngle'}">
-          <origin xyz="${extension} ${sin(-twist) * edge_to_center} ${edge_to_center * (1 + cos(-twist))}" rpy="${twist} 0 0"/>
-        </xacro:if>
-        <xacro:if value="${input == 'RightAngle' and output == 'Inline'}">
-          <origin xyz="${extension} 0 ${edge_to_center}" rpy="${pi/2} ${twist+pi} ${pi/2}"/>
-        </xacro:if>
-        <xacro:if value="${input == 'Inline' and output =='RightAngle'}">
-          <origin xyz="${edge_to_center * sin(twist+pi/2)} ${edge_to_center * -cos(twist+pi/2)} ${extension}" rpy="${pi/2} ${-pi/2} ${twist+pi/2}"/>
-        </xacro:if>
-        <xacro:if value="${input == 'Inline' and output =='Inline'}">
-          <origin xyz="${0} ${0} ${extension}" rpy="${0} ${0} ${twist-pi/2}"/>
-        </xacro:if>
-        <geometry>
-          <xacro:if value="${input == 'RightAngle'}">
-            <mesh filename="file://$(find hebi_description)/meshes/A-2039-02.stl"/>
+          <xacro:if value="${input == 'Inline' and output =='RightAngle'}">
+            <origin xyz="${edge_to_center * sin(twist+pi/2)} ${edge_to_center * -cos(twist+pi/2)} ${extension}" rpy="${pi/2} ${-pi/2} ${twist+pi/2}"/>
           </xacro:if>
-          <xacro:if value="${input == 'Inline'}">
-            <mesh filename="file://$(find hebi_description)/meshes/A-2226-01.stl" scale="0.001 0.001 0.001"/>
+          <xacro:if value="${input == 'Inline' and output =='Inline'}">
+            <origin xyz="${0} ${0} ${extension}" rpy="${0} ${0} ${twist-pi/2}"/>
           </xacro:if>
-        </geometry>
-      </collision>
+          <geometry>
+            <xacro:if value="${output == 'RightAngle'}">
+              <mesh filename="file://$(find hebi_description)/meshes/A-2039-02.stl"/>
+            </xacro:if>
+            <xacro:if value="${output == 'Inline'}">
+              <mesh filename="file://$(find hebi_description)/meshes/A-2226-01.stl" scale="0.001 0.001 0.001"/>
+            </xacro:if>
+          </geometry>
+          <xacro:black_material/>
+        </visual>
+        <collision>
+          <xacro:if value="${input == 'RightAngle' and output == 'RightAngle'}">
+            <origin xyz="${extension} ${sin(-twist) * edge_to_center} ${edge_to_center * (1 + cos(-twist))}" rpy="${twist} 0 0"/>
+          </xacro:if>
+          <xacro:if value="${input == 'RightAngle' and output == 'Inline'}">
+            <origin xyz="${extension} 0 ${edge_to_center}" rpy="${pi/2} ${twist+pi} ${pi/2}"/>
+          </xacro:if>
+          <xacro:if value="${input == 'Inline' and output =='RightAngle'}">
+            <origin xyz="${edge_to_center * sin(twist+pi/2)} ${edge_to_center * -cos(twist+pi/2)} ${extension}" rpy="${pi/2} ${-pi/2} ${twist+pi/2}"/>
+          </xacro:if>
+          <xacro:if value="${input == 'Inline' and output =='Inline'}">
+            <origin xyz="${0} ${0} ${extension}" rpy="${0} ${0} ${twist-pi/2}"/>
+          </xacro:if>
+          <geometry>
+            <xacro:if value="${input == 'RightAngle'}">
+              <mesh filename="file://$(find hebi_description)/meshes/A-2039-02.stl"/>
+            </xacro:if>
+            <xacro:if value="${input == 'Inline'}">
+              <mesh filename="file://$(find hebi_description)/meshes/A-2226-01.stl" scale="0.001 0.001 0.001"/>
+            </xacro:if>
+          </geometry>
+        </collision>
+      </xacro:if>
       <!-- Approximate inertia as thin rod about x axis -->
       <inertial>
@@ -107,10 +109,10 @@
       </inertial>
     </link>
-    <gazebo reference="${name}/INPUT_INTERFACE">
+    <gazebo reference="${name}">
       <xacro:gazebo_black_material/>
     </gazebo>
     <joint name="${name}/OUTPUT_JOINT" type="fixed">
-      <parent link="${name}/INPUT_INTERFACE"/>
-      <child link="${child}/INPUT_INTERFACE"/>
+      <parent link="${name}"/>
+      <child link="${child}"/>
       <xacro:if value="${input == 'RightAngle' and output == 'RightAngle'}">
         <origin xyz="${extension} ${-sin(twist) * edge_to_center} ${edge_to_center * (1 + cos(twist))}" rpy="${twist} 0 0"/>
@@ -125,4 +127,10 @@
         <origin xyz="${0} ${0} ${extension}" rpy="${0} ${0} ${twist-pi/2}"/>
       </xacro:if>
+      <xacro:if value="${input == 'RightAngle' and output =='None'}">
+        <origin xyz="${extension} 0 ${edge_to_center}" rpy="${pi/2} ${twist+pi} ${pi/2}"/>
+      </xacro:if>
+      <xacro:if value="${input == 'Inline' and output =='None'}">
+        <origin xyz="${0} ${0} ${extension}" rpy="${0} ${0} ${twist-pi/2}"/>
+      </xacro:if>
     </joint>
   </xacro:macro>

File: urdf/components/omnibase.xacro (robot description, xacro)
@@ -39,18 +39,18 @@
       <origin xyz="0.0788 -0.1364 0" rpy="0 ${pi/2} ${-pi/3}" />
       <parent link="omni_base" />
-      <child link="wheel_1/INPUT_INTERFACE"/>
+      <child link="wheel_1"/>
     </joint>
     <joint name="wheel_2_joint" type="fixed">
       <origin xyz="0.0788 0.1364 0" rpy="0 ${pi/2} ${pi/3}" />
       <parent link="omni_base" />
-      <child link="wheel_2/INPUT_INTERFACE"/>
+      <child link="wheel_2"/>
     </joint>
     <joint name="wheel_3_joint" type="fixed">
       <origin xyz="-0.1575 0 0" rpy="0 ${pi/2} ${pi}" />
       <parent link="omni_base" />
-      <child link="wheel_3/INPUT_INTERFACE"/>
+      <child link="wheel_3"/>
     </joint>
     <xacro:actuator type="X5_4" name="wheel_1" child="wheel_1_end"/>
-    <link name="wheel_1_end/INPUT_INTERFACE">
+    <link name="wheel_1_end">
       <visual>
         <origin xyz="0 0 0" rpy="0 0 0" />
@@ -74,5 +74,5 @@
     </link>
     <xacro:actuator type="X5_4" name="wheel_2" child="wheel_2_end"/>
-    <link name="wheel_2_end/INPUT_INTERFACE">
+    <link name="wheel_2_end">
       <visual>
         <origin xyz="0 0 0" rpy="0 0 0" />
@@ -96,5 +96,5 @@
     </link>
     <xacro:actuator type="X5_4" name="wheel_3" child="wheel_3_end"/>
-    <link name="wheel_3_end/INPUT_INTERFACE">
+    <link name="wheel_3_end">
       <visual>
         <origin xyz="0 0 0" rpy="0 0 0" />
