Commit message: Added T-Series

File: urdf/components/actuator.xacro (robot description, xacro)
@@ -58,4 +58,34 @@
       <xacro:property name="velocity_limit" value="1.571"/>
     </xacro:if>
+    <xacro:if value="${model_name == 'T5_1'}">
+      <xacro:property name="actuator_mass" value="0.450"/>
+      <xacro:property name="effort_limit" value="2.5"/>
+      <xacro:property name="velocity_limit" value="9.425"/>
+    </xacro:if>
+    <xacro:if value="${model_name == 'T5_4'}">
+      <xacro:property name="actuator_mass" value="0.450"/>
+      <xacro:property name="effort_limit" value="7.0"/>
+      <xacro:property name="velocity_limit" value="3.351"/>
+    </xacro:if>
+    <xacro:if value="${model_name == 'T5_9'}">
+      <xacro:property name="actuator_mass" value="0.450"/>
+      <xacro:property name="effort_limit" value="13.0"/>
+      <xacro:property name="velocity_limit" value="1.466"/>
+    </xacro:if>
+    <xacro:if value="${model_name == 'T8_3'}">
+      <xacro:property name="actuator_mass" value="0.575"/>
+      <xacro:property name="effort_limit" value="8.0"/>
+      <xacro:property name="velocity_limit" value="11.520"/>
+    </xacro:if>
+    <xacro:if value="${model_name == 'T8_9'}">
+      <xacro:property name="actuator_mass" value="0.575"/>
+      <xacro:property name="effort_limit" value="23.0"/>
+      <xacro:property name="velocity_limit" value="4.084"/>
+    </xacro:if>
+    <xacro:if value="${model_name == 'T8_16'}">
+      <xacro:property name="actuator_mass" value="0.575"/>
+      <xacro:property name="effort_limit" value="44.0"/>
+      <xacro:property name="velocity_limit" value="2.094"/>
+    </xacro:if>
     <!-- Note: the frction/damping probably need to be tuned more for accurate simulation -->
     <xacro:if value="${model_name.startswith('X5')}">
@@ -74,14 +104,32 @@
       <xacro:property name="friction" value="0.5"/>
     </xacro:if>
+    <xacro:if value="${model_name.startswith('T5')}">
+      <xacro:property name="mesh_filename" value="file://$(find hebi_description)/meshes/T5.stl"/>
+      <xacro:property name="damping" value="0.1"/>
+      <xacro:property name="friction" value="0.1"/>
+    </xacro:if>
+    <xacro:if value="${model_name.startswith('T8')}">
+      <xacro:property name="mesh_filename" value="file://$(find hebi_description)/meshes/T8.stl"/>
+      <xacro:property name="damping" value="0.5"/>
+      <xacro:property name="friction" value="0.5"/>
+    </xacro:if>
     <link name="${name}">
       <visual>
         <origin xyz="0 0 0" rpy="0 0 0" />
         <geometry>
-          <mesh filename="${mesh_filename}" scale="0.001 0.001 0.001"/>
+          <xacro:if value="${model_name.startswith('T')}">
+            <mesh filename="${mesh_filename}"/>
+          </xacro:if>
+          <xacro:unless value="${model_name.startswith('T')}">
+            <mesh filename="${mesh_filename}" scale="0.001 0.001 0.001"/>
+          </xacro:unless>
         </geometry>
-        <xacro:unless value="${model_name.startswith('R8')}">
+        <xacro:if value="${model_name.startswith('X')}">
           <xacro:red_material/>
-        </xacro:unless>
-        <xacro:if value="${model_name.startswith('R8')}">
+        </xacro:if>
+        <xacro:if value="${model_name.startswith('T')}">
+          <xacro:tangerine_material/>
+        </xacro:if>
+        <xacro:if value="${model_name.startswith('R')}">
           <xacro:black_material/>
         </xacro:if>
@@ -90,5 +138,10 @@
         <origin xyz="0 0 0" rpy="0 0 0" />
         <geometry>
-          <mesh filename="${mesh_filename}" scale="0.001 0.001 0.001"/>
+          <xacro:if value="${model_name.startswith('T')}">
+            <mesh filename="${mesh_filename}"/>
+          </xacro:if>
+          <xacro:unless value="${model_name.startswith('T')}">
+            <mesh filename="${mesh_filename}" scale="0.001 0.001 0.001"/>
+          </xacro:unless>
         </geometry>
       </collision>
@@ -113,13 +166,28 @@
                    izz="0.001186" />
         </xacro:if>
+        <xacro:if value="${model_name.startswith('T5')}">
+          <origin xyz="-0.0240 -0.00161 0.0165" rpy="0 0 0" />
+          <inertia ixx="0.00015"  ixy="0.0000341"  ixz="0.0000118"
+                   iyy="0.000255" iyz="0.00000229"
+                   izz="0.000350" />
+        </xacro:if>
+        <xacro:if value="${model_name.startswith('T8')}">
+          <origin xyz="-0.0240 -0.00161 0.0256" rpy="0 0 0" />
+          <inertia ixx="0.000246" ixy="0.0000444" ixz="0.0000266"
+                   iyy="0.000380" iyz="0.00000422"
+                   izz="0.000463"/>
+        </xacro:if>
       </inertial>
     </link>
     <gazebo reference="${name}">
-      <xacro:unless value="${model_name.startswith('R8')}">
+      <xacro:if value="${model_name.startswith('X')}">
         <xacro:gazebo_red_material/>
-      </xacro:unless>
-      <xacro:if value="${model_name.startswith('R8')}">
-        <xacro:gazebo_black_material/>
-      </xacro:if>
+        </xacro:if>
+        <xacro:if value="${model_name.startswith('T')}">
+          <xacro:gazebo_tangerine_material/>
+        </xacro:if>
+        <xacro:if value="${model_name.startswith('R')}">
+          <xacro:gazebo_black_material/>
+        </xacro:if>
     </gazebo>
     <joint name="${name}" type="${urdf_joint_type}">
@@ -134,4 +202,10 @@
       <xacro:if value="${model_name.startswith('R8')}">
         <origin xyz="0 0 0.051" rpy="0 0 0"/>
+      </xacro:if>
+      <xacro:if value="${model_name.startswith('T5')}">
+        <origin xyz="0 0 0.034" rpy="0 0 0"/>
+      </xacro:if>
+      <xacro:if value="${model_name.startswith('T8')}">
+        <origin xyz="0 0 0.0475" rpy="0 0 0"/>
       </xacro:if>
       <axis xyz="0 0 1"/>
@@ -204,4 +278,34 @@
       <xacro:property name="velocity_limit" value="1.571"/>
     </xacro:if>
+    <xacro:if value="${model_name == 'T5_1'}">
+      <xacro:property name="actuator_mass" value="0.450"/>
+      <xacro:property name="effort_limit" value="2.5"/>
+      <xacro:property name="velocity_limit" value="9.425"/>
+    </xacro:if>
+    <xacro:if value="${model_name == 'T5_4'}">
+      <xacro:property name="actuator_mass" value="0.450"/>
+      <xacro:property name="effort_limit" value="7.0"/>
+      <xacro:property name="velocity_limit" value="3.351"/>
+    </xacro:if>
+    <xacro:if value="${model_name == 'T5_9'}">
+      <xacro:property name="actuator_mass" value="0.450"/>
+      <xacro:property name="effort_limit" value="13.0"/>
+      <xacro:property name="velocity_limit" value="1.466"/>
+    </xacro:if>
+    <xacro:if value="${model_name == 'T8_3'}">
+      <xacro:property name="actuator_mass" value="0.575"/>
+      <xacro:property name="effort_limit" value="8.0"/>
+      <xacro:property name="velocity_limit" value="11.520"/>
+    </xacro:if>
+    <xacro:if value="${model_name == 'T8_9'}">
+      <xacro:property name="actuator_mass" value="0.575"/>
+      <xacro:property name="effort_limit" value="23.0"/>
+      <xacro:property name="velocity_limit" value="4.084"/>
+    </xacro:if>
+    <xacro:if value="${model_name == 'T8_16'}">
+      <xacro:property name="actuator_mass" value="0.575"/>
+      <xacro:property name="effort_limit" value="44.0"/>
+      <xacro:property name="velocity_limit" value="2.094"/>
+    </xacro:if>
     <!-- Note: the frction/damping probably need to be tuned more for accurate simulation -->
     <xacro:if value="${model_name.startswith('X5')}">
@@ -220,14 +324,32 @@
       <xacro:property name="friction" value="0.5"/>
     </xacro:if>
+    <xacro:if value="${model_name.startswith('T5')}">
+      <xacro:property name="mesh_filename" value="file://$(find hebi_description)/meshes/T5.stl"/>
+      <xacro:property name="damping" value="0.1"/>
+      <xacro:property name="friction" value="0.1"/>
+    </xacro:if>
+    <xacro:if value="${model_name.startswith('T8')}">
+      <xacro:property name="mesh_filename" value="file://$(find hebi_description)/meshes/T8.stl"/>
+      <xacro:property name="damping" value="0.5"/>
+      <xacro:property name="friction" value="0.5"/>
+    </xacro:if>
     <link name="${name}">
       <visual>
         <origin xyz="0 0 0" rpy="0 0 0" />
         <geometry>
-          <mesh filename="${mesh_filename}" scale="0.001 0.001 0.001"/>
+          <xacro:if value="${model_name.startswith('T')}">
+            <mesh filename="${mesh_filename}"/>
+          </xacro:if>
+          <xacro:unless value="${model_name.startswith('T')}">
+            <mesh filename="${mesh_filename}" scale="0.001 0.001 0.001"/>
+          </xacro:unless>
         </geometry>
-        <xacro:unless value="${model_name.startswith('R8')}">
+        <xacro:if value="${model_name.startswith('X')}">
           <xacro:red_material/>
-        </xacro:unless>
-        <xacro:if value="${model_name.startswith('R8')}">
+        </xacro:if>
+        <xacro:if value="${model_name.startswith('T')}">
+          <xacro:tangerine_material/>
+        </xacro:if>
+        <xacro:if value="${model_name.startswith('R')}">
           <xacro:black_material/>
         </xacro:if>
@@ -236,5 +358,10 @@
         <origin xyz="0 0 0" rpy="0 0 0" />
         <geometry>
-          <mesh filename="${mesh_filename}" scale="0.001 0.001 0.001"/>
+          <xacro:if value="${model_name.startswith('T')}">
+            <mesh filename="${mesh_filename}"/>
+          </xacro:if>
+          <xacro:unless value="${model_name.startswith('T')}">
+            <mesh filename="${mesh_filename}" scale="0.001 0.001 0.001"/>
+          </xacro:unless>
         </geometry>
       </collision>
@@ -259,11 +386,26 @@
                    izz="0.001186" />
         </xacro:if>
+        <xacro:if value="${model_name.startswith('T5')}">
+          <origin xyz="-0.0240 -0.00161 0.0165" rpy="0 0 0" />
+          <inertia ixx="0.00015"  ixy="0.0000341"  ixz="0.0000118"
+                   iyy="0.000255" iyz="0.00000229"
+                   izz="0.000350" />
+        </xacro:if>
+        <xacro:if value="${model_name.startswith('T8')}">
+          <origin xyz="-0.0240 -0.00161 0.0256" rpy="0 0 0" />
+          <inertia ixx="0.000246" ixy="0.0000444" ixz="0.0000266"
+                   iyy="0.000380" iyz="0.00000422"
+                   izz="0.000463"/>
+        </xacro:if>
       </inertial>
     </link>
     <gazebo reference="${name}">
-      <xacro:unless value="${model_name.startswith('R8')}">
+      <xacro:if value="${model_name.startswith('X')}">
         <xacro:gazebo_red_material/>
-      </xacro:unless>
-      <xacro:if value="${model_name.startswith('R8')}">
+        </xacro:if>
+        <xacro:if value="${model_name.startswith('T')}">
+          <xacro:gazebo_tangerine_material/>
+        </xacro:if>
+        <xacro:if value="${model_name.startswith('R')}">
         <xacro:gazebo_black_material/>
       </xacro:if>
@@ -280,4 +422,10 @@
       <xacro:if value="${model_name.startswith('R8')}">
         <origin xyz="0 0 0.051" rpy="0 ${pi} 0"/>
+      </xacro:if>
+      <xacro:if value="${model_name.startswith('T5')}">
+        <origin xyz="0 0 0.034" rpy="0 ${pi} 0"/>
+      </xacro:if>
+      <xacro:if value="${model_name.startswith('T8')}">
+        <origin xyz="0 0 0.0475" rpy="0 ${pi} 0"/>
       </xacro:if>
       <axis xyz="0 0 -1"/>
@@ -295,11 +443,11 @@
       <parent link="${name}"/>
       <child link="${child}"/>
-      <xacro:if value="${model_name.startswith('X5')}">
+      <xacro:if value="${model_name.startswith('X')}">
         <origin xyz="0 0 0" rpy="0 0 0"/>
       </xacro:if>
-      <xacro:if value="${model_name.startswith('X8')}">
+      <xacro:if value="${model_name.startswith('T')}">
         <origin xyz="0 0 0" rpy="0 0 0"/>
       </xacro:if>
-      <xacro:if value="${model_name.startswith('R8')}">
+      <xacro:if value="${model_name.startswith('R')}">
         <origin xyz="0 0 0" rpy="0 0 0"/>
       </xacro:if>

File: urdf/components/bracket.xacro (robot description, xacro)
@@ -83,4 +83,40 @@
       </inertial>
     </xacro:if>
+    <xacro:if value="${bracket_type.startswith('T5Light') or bracket_type.startswith('T8Light')}">
+      <visual>
+        <xacro:if value="${bracket_type.endswith('Left')}">
+          <origin xyz="0 0 0" rpy="0 0 ${pi}"/>
+        </xacro:if>
+        <xacro:if value="${bracket_type.endswith('Right')}">
+          <origin xyz="0 0 0" rpy="0 0 0"/>
+        </xacro:if>
+        <geometry>
+          <mesh filename="file://$(find hebi_description)/meshes/A-2220-01.stl" scale="0.001 0.001 0.001"/>
+        </geometry>
+        <xacro:black_material/>
+      </visual>
+      <collision>
+        <xacro:if value="${bracket_type.endswith('Left')}">
+          <origin xyz="0 0 0" rpy="${pi/2} 0 ${pi/2}"/>
+        </xacro:if>
+        <xacro:if value="${bracket_type.endswith('Right')}">
+          <origin xyz="0 0 0" rpy="${pi/2} 0 ${-pi/2}"/>
+        </xacro:if>
+        <geometry>
+          <mesh filename="file://$(find hebi_description)/meshes/A-2220-01.stl" scale="0.001 0.001 0.001"/>
+        </geometry>
+      </collision>
+      <!-- inertia is just modelled as small sphere, and could be improved. -->
+      <inertial>
+        <xacro:if value="${bracket_type.endswith('Left')}">
+          <origin xyz="0 .0215 .02" rpy="0 0 0" />
+        </xacro:if>
+        <xacro:if value="${bracket_type.endswith('Right')}">
+          <origin xyz="0 -.0215 .02" rpy="0 0 0" />
+        </xacro:if>
+        <mass value="0.1"/>
+        <inertia ixx="${0.4 * 0.1 * 0.06 * 0.06}" ixy="0.0" ixz="0.0" iyy="${0.4 * 0.1 * 0.06 * 0.06}" iyz="0.0" izz="${0.4 * 0.1 * 0.06 * 0.06}"/>
+      </inertial>
+    </xacro:if>
     <!-- Heavy bracket -->
     <xacro:if value="${bracket_type.startswith('X5Heavy')}">
@@ -184,4 +220,68 @@
     </xacro:if>
     <xacro:if value="${bracket_type.startswith('R8Heavy')}">
+      <visual>
+        <xacro:if value="${bracket_type.endswith('RightOutside')}">
+          <origin xyz="0 0 0" rpy="0 0 0"/>
+        </xacro:if>
+        <xacro:if value="${bracket_type.endswith('RightInside')}">
+          <origin xyz="0 0 0" rpy="0 0 ${pi}"/>
+        </xacro:if>
+        <xacro:if value="${bracket_type.endswith('LeftOutside')}">
+          <origin xyz="0 0 0" rpy="0 0 ${pi}"/>
+        </xacro:if>
+        <xacro:if value="${bracket_type.endswith('LeftInside')}">
+          <origin xyz="0 0 0" rpy="0 0 0"/>
+        </xacro:if>
+        <geometry>
+          <xacro:if value="${bracket_type.endswith('Outside')}">
+            <mesh filename="file://$(find hebi_description)/meshes/A-2221-01-Outside.stl" scale="0.001 0.001 0.001"/>
+          </xacro:if>
+          <xacro:if value="${bracket_type.endswith('Inside')}">
+            <mesh filename="file://$(find hebi_description)/meshes/A-2221-01-Inside.stl" scale="0.001 0.001 0.001"/>
+          </xacro:if>
+        </geometry>
+        <xacro:black_material/>
+      </visual>
+      <collision>
+        <xacro:if value="${bracket_type.endswith('RightOutside')}">
+          <origin xyz="0 0 0.005" rpy="${pi/2} 0 ${pi/2}"/>
+        </xacro:if>
+        <xacro:if value="${bracket_type.endswith('RightInside')}">
+          <origin xyz="0 0 0.005" rpy="${pi/2} 0 ${-pi/2}"/>
+        </xacro:if>
+        <xacro:if value="${bracket_type.endswith('LeftOutside')}">
+          <origin xyz="0 0 0.005" rpy="${pi/2} 0 ${-pi/2}"/>
+        </xacro:if>
+        <xacro:if value="${bracket_type.endswith('LeftInside')}">
+          <origin xyz="0 0 0.005" rpy="${pi/2} 0 ${pi/2}"/>
+        </xacro:if>
+        <geometry>
+          <xacro:if value="${bracket_type.endswith('Outside')}">
+            <mesh filename="file://$(find hebi_description)/meshes/A-2221-01-Outside.stl" scale="0.001 0.001 0.001"/>
+          </xacro:if>
+          <xacro:if value="${bracket_type.endswith('Inside')}">
+            <mesh filename="file://$(find hebi_description)/meshes/A-2221-01-Inside.stl" scale="0.001 0.001 0.001"/>
+          </xacro:if>
+        </geometry>
+      </collision>
+      <!-- inertia is just modelled as small sphere, and could be improved. -->
+      <inertial>
+        <xacro:if value="${bracket_type.endswith('RightOutside')}">
+          <origin xyz="0 ${0.5 * -.0375} .0275" rpy="0 0 0" />
+        </xacro:if>
+        <xacro:if value="${bracket_type.endswith('RightInside')}">
+          <origin xyz="0 ${0.5 * .0225} .0275" rpy="0 0 0" />
+        </xacro:if>
+        <xacro:if value="${bracket_type.endswith('LeftOutside')}">
+          <origin xyz="0 ${0.5 * .0375} .0275" rpy="0 0 0" />
+        </xacro:if>
+        <xacro:if value="${bracket_type.endswith('LeftInside')}">
+          <origin xyz="0 ${0.5 * -.0225} .0275" rpy="0 0 0" />
+        </xacro:if>
+        <mass value="0.215"/>
+        <inertia ixx="${0.4 * 0.215 * 0.06 * 0.06}" ixy="0.0" ixz="0.0" iyy="${0.4 * 0.215 * 0.06 * 0.06}" iyz="0.0" izz="${0.4 * 0.215 * 0.06 * 0.06}"/>
+      </inertial>
+    </xacro:if>
+    <xacro:if value="${bracket_type.startswith('T5Heavy') or bracket_type.startswith('T8Heavy')}">
       <visual>
         <xacro:if value="${bracket_type.endswith('RightOutside')}">
@@ -252,5 +352,5 @@
       <xacro:gazebo_beige_material/>
     </xacro:if>
-    <xacro:if value="${bracket_type.startswith('X5Heavy') or bracket_type.startswith('R8')}">
+    <xacro:if value="${bracket_type.startswith('X5Heavy') or bracket_type.startswith('R8') or bracket_type.startswith('T')}">
       <xacro:gazebo_black_material/>
     </xacro:if>

File: urdf/components/hebi.xacro (robot description, xacro)
@@ -27,4 +27,17 @@
     <material>Gazebo/Black</material>
   </xacro:macro>
+  <xacro:macro name="tangerine_material">
+    <material name="tangerine">
+      <color rgba="0.91 0.43 0.218 1"/>
+    </material>
+  </xacro:macro>
+  <xacro:macro name="gazebo_tangerine_material">
+    <visual>
+      <material>
+          <ambient>0.91 0.43 0.218 1</ambient>
+          <diffuse>0.91 0.43 0.218 1</diffuse>
+      </material>
+    </visual>
+  </xacro:macro>
   <xacro:macro name="beige_material">
     <material name="beige">
