Commit message: Added T-Series actuators to xacro

File: urdf/components/actuator.xacro (robot description, xacro)
@@ -58,4 +58,34 @@
       <xacro:property name="velocity_limit" value="1.571"/>
     </xacro:if>
+    <xacro:if value="${model_name == 'T5_1'}">
+      <xacro:property name="actuator_mass" value="0.450"/>
+      <xacro:property name="effort_limit" value="2.5"/>
+      <xacro:property name="velocity_limit" value="9.425"/>
+    </xacro:if>
+    <xacro:if value="${model_name == 'T5_4'}">
+      <xacro:property name="actuator_mass" value="0.450"/>
+      <xacro:property name="effort_limit" value="7.0"/>
+      <xacro:property name="velocity_limit" value="3.351"/>
+    </xacro:if>
+    <xacro:if value="${model_name == 'T5_9'}">
+      <xacro:property name="actuator_mass" value="0.450"/>
+      <xacro:property name="effort_limit" value="13.0"/>
+      <xacro:property name="velocity_limit" value="1.466"/>
+    </xacro:if>
+    <xacro:if value="${model_name == 'T8_3'}">
+      <xacro:property name="actuator_mass" value="0.575"/>
+      <xacro:property name="effort_limit" value="8.0"/>
+      <xacro:property name="velocity_limit" value="11.520"/>
+    </xacro:if>
+    <xacro:if value="${model_name == 'T8_9'}">
+      <xacro:property name="actuator_mass" value="0.575"/>
+      <xacro:property name="effort_limit" value="23.0"/>
+      <xacro:property name="velocity_limit" value="4.084"/>
+    </xacro:if>
+    <xacro:if value="${model_name == 'T8_16'}">
+      <xacro:property name="actuator_mass" value="0.575"/>
+      <xacro:property name="effort_limit" value="44.0"/>
+      <xacro:property name="velocity_limit" value="2.094"/>
+    </xacro:if>
     <!-- Note: the frction/damping probably need to be tuned more for accurate simulation -->
     <xacro:if value="${model_name.startswith('X5')}">
@@ -74,14 +104,32 @@
       <xacro:property name="friction" value="0.5"/>
     </xacro:if>
+    <xacro:if value="${model_name.startswith('T5')}">
+      <xacro:property name="mesh_filename" value="file://$(find hebi_description)/meshes/T5.stl"/>
+      <xacro:property name="damping" value="0.1"/>
+      <xacro:property name="friction" value="0.1"/>
+    </xacro:if>
+    <xacro:if value="${model_name.startswith('T8')}">
+      <xacro:property name="mesh_filename" value="file://$(find hebi_description)/meshes/T8.stl"/>
+      <xacro:property name="damping" value="0.5"/>
+      <xacro:property name="friction" value="0.5"/>
+    </xacro:if>
     <link name="${name}/INPUT_INTERFACE">
       <visual>
         <origin xyz="0 0 0" rpy="0 0 0" />
         <geometry>
+          <xacro:if value="${model_name.startswith('T')}">
+            <mesh filename="${mesh_filename}"/>
+          </xacro:if>
+          <xacro:unless value="${model_name.startswith('T')}">
           <mesh filename="${mesh_filename}" scale="0.001 0.001 0.001"/>
+          </xacro:unless>
         </geometry>
-        <xacro:unless value="${model_name.startswith('R8')}">
+        <xacro:if value="${model_name.startswith('X')}">
           <xacro:red_material/>
-        </xacro:unless>
-        <xacro:if value="${model_name.startswith('R8')}">
+        </xacro:if>
+        <xacro:if value="${model_name.startswith('T')}">
+          <xacro:tangerine_material/>
+        </xacro:if>
+        <xacro:if value="${model_name.startswith('R')}">
           <xacro:black_material/>
         </xacro:if>
@@ -90,5 +138,10 @@
         <origin xyz="0 0 0" rpy="0 0 0" />
         <geometry>
+          <xacro:if value="${model_name.startswith('T')}">
+            <mesh filename="${mesh_filename}"/>
+          </xacro:if>
+          <xacro:unless value="${model_name.startswith('T')}">
           <mesh filename="${mesh_filename}" scale="0.001 0.001 0.001"/>
+          </xacro:unless>
         </geometry>
       </collision>
@@ -113,11 +166,26 @@
                    izz="0.001186" />
         </xacro:if>
+        <xacro:if value="${model_name.startswith('T5')}">
+          <origin xyz="-0.0240 -0.00161 0.0165" rpy="0 0 0" />
+          <inertia ixx="0.00015"  ixy="0.0000341"  ixz="0.0000118"
+                   iyy="0.000255" iyz="0.00000229"
+                   izz="0.000350" />
+        </xacro:if>
+        <xacro:if value="${model_name.startswith('T8')}">
+          <origin xyz="-0.0240 -0.00161 0.0256" rpy="0 0 0" />
+          <inertia ixx="0.000246" ixy="0.0000444" ixz="0.0000266"
+                   iyy="0.000380" iyz="0.00000422"
+                   izz="0.000463"/>
+        </xacro:if>
       </inertial>
     </link>
     <gazebo reference="${name}/INPUT_INTERFACE">
-      <xacro:unless value="${model_name.startswith('R8')}">
+      <xacro:if value="${model_name.startswith('X')}">
         <xacro:gazebo_red_material/>
-      </xacro:unless>
-      <xacro:if value="${model_name.startswith('R8')}">
+        </xacro:if>
+        <xacro:if value="${model_name.startswith('T')}">
+          <xacro:gazebo_tangerine_material/>
+        </xacro:if>
+        <xacro:if value="${model_name.startswith('R')}">
         <xacro:gazebo_black_material/>
       </xacro:if>
@@ -134,4 +202,10 @@
       <xacro:if value="${model_name.startswith('R8')}">
         <origin xyz="0 0 0.051" rpy="0 0 0"/>
+      </xacro:if>
+      <xacro:if value="${model_name.startswith('T5')}">
+        <origin xyz="0 0 0.034" rpy="0 0 0"/>
+      </xacro:if>
+      <xacro:if value="${model_name.startswith('T8')}">
+        <origin xyz="0 0 0.0475" rpy="0 0 0"/>
       </xacro:if>
       <axis xyz="0 0 1"/>
@@ -204,4 +278,34 @@
       <xacro:property name="velocity_limit" value="1.571"/>
     </xacro:if>
+    <xacro:if value="${model_name == 'T5_1'}">
+      <xacro:property name="actuator_mass" value="0.450"/>
+      <xacro:property name="effort_limit" value="2.5"/>
+      <xacro:property name="velocity_limit" value="9.425"/>
+    </xacro:if>
+    <xacro:if value="${model_name == 'T5_4'}">
+      <xacro:property name="actuator_mass" value="0.450"/>
+      <xacro:property name="effort_limit" value="7.0"/>
+      <xacro:property name="velocity_limit" value="3.351"/>
+    </xacro:if>
+    <xacro:if value="${model_name == 'T5_9'}">
+      <xacro:property name="actuator_mass" value="0.450"/>
+      <xacro:property name="effort_limit" value="13.0"/>
+      <xacro:property name="velocity_limit" value="1.466"/>
+    </xacro:if>
+    <xacro:if value="${model_name == 'T8_3'}">
+      <xacro:property name="actuator_mass" value="0.575"/>
+      <xacro:property name="effort_limit" value="8.0"/>
+      <xacro:property name="velocity_limit" value="11.520"/>
+    </xacro:if>
+    <xacro:if value="${model_name == 'T8_9'}">
+      <xacro:property name="actuator_mass" value="0.575"/>
+      <xacro:property name="effort_limit" value="23.0"/>
+      <xacro:property name="velocity_limit" value="4.084"/>
+    </xacro:if>
+    <xacro:if value="${model_name == 'T8_16'}">
+      <xacro:property name="actuator_mass" value="0.575"/>
+      <xacro:property name="effort_limit" value="44.0"/>
+      <xacro:property name="velocity_limit" value="2.094"/>
+    </xacro:if>
     <!-- Note: the frction/damping probably need to be tuned more for accurate simulation -->
     <xacro:if value="${model_name.startswith('X5')}">
@@ -220,14 +324,32 @@
       <xacro:property name="friction" value="0.5"/>
     </xacro:if>
+    <xacro:if value="${model_name.startswith('T5')}">
+      <xacro:property name="mesh_filename" value="file://$(find hebi_description)/meshes/T5.stl"/>
+      <xacro:property name="damping" value="0.1"/>
+      <xacro:property name="friction" value="0.1"/>
+    </xacro:if>
+    <xacro:if value="${model_name.startswith('T8')}">
+      <xacro:property name="mesh_filename" value="file://$(find hebi_description)/meshes/T8.stl"/>
+      <xacro:property name="damping" value="0.5"/>
+      <xacro:property name="friction" value="0.5"/>
+    </xacro:if>
     <link name="${name}/INPUT_INTERFACE">
       <visual>
         <origin xyz="0 0 0" rpy="0 0 0" />
         <geometry>
+          <xacro:if value="${model_name.startswith('T')}">
+            <mesh filename="${mesh_filename}"/>
+          </xacro:if>
+          <xacro:unless value="${model_name.startswith('T')}">
           <mesh filename="${mesh_filename}" scale="0.001 0.001 0.001"/>
+          </xacro:unless>
         </geometry>
-        <xacro:unless value="${model_name.startswith('R8')}">
+        <xacro:if value="${model_name.startswith('X')}">
           <xacro:red_material/>
-        </xacro:unless>
-        <xacro:if value="${model_name.startswith('R8')}">
+        </xacro:if>
+        <xacro:if value="${model_name.startswith('T')}">
+          <xacro:tangerine_material/>
+        </xacro:if>
+        <xacro:if value="${model_name.startswith('R')}">
           <xacro:black_material/>
         </xacro:if>
@@ -236,5 +358,10 @@
         <origin xyz="0 0 0" rpy="0 0 0" />
         <geometry>
+          <xacro:if value="${model_name.startswith('T')}">
+            <mesh filename="${mesh_filename}"/>
+          </xacro:if>
+          <xacro:unless value="${model_name.startswith('T')}">
           <mesh filename="${mesh_filename}" scale="0.001 0.001 0.001"/>
+          </xacro:unless>
         </geometry>
       </collision>
@@ -259,11 +386,26 @@
                    izz="0.001186" />
         </xacro:if>
+        <xacro:if value="${model_name.startswith('T5')}">
+          <origin xyz="-0.0240 -0.00161 0.0165" rpy="0 0 0" />
+          <inertia ixx="0.00015"  ixy="0.0000341"  ixz="0.0000118"
+                   iyy="0.000255" iyz="0.00000229"
+                   izz="0.000350" />
+        </xacro:if>
+        <xacro:if value="${model_name.startswith('T8')}">
+          <origin xyz="-0.0240 -0.00161 0.0256" rpy="0 0 0" />
+          <inertia ixx="0.000246" ixy="0.0000444" ixz="0.0000266"
+                   iyy="0.000380" iyz="0.00000422"
+                   izz="0.000463"/>
+        </xacro:if>
       </inertial>
     </link>
     <gazebo reference="${name}/INPUT_INTERFACE">
-      <xacro:unless value="${model_name.startswith('R8')}">
+      <xacro:if value="${model_name.startswith('X')}">
         <xacro:gazebo_red_material/>
-      </xacro:unless>
-      <xacro:if value="${model_name.startswith('R8')}">
+        </xacro:if>
+        <xacro:if value="${model_name.startswith('T')}">
+          <xacro:gazebo_tangerine_material/>
+        </xacro:if>
+        <xacro:if value="${model_name.startswith('R')}">
         <xacro:gazebo_black_material/>
       </xacro:if>
@@ -280,4 +422,10 @@
       <xacro:if value="${model_name.startswith('R8')}">
         <origin xyz="0 0 0.051" rpy="0 ${pi} 0"/>
+      </xacro:if>
+      <xacro:if value="${model_name.startswith('T5')}">
+        <origin xyz="0 0 0.034" rpy="0 ${pi} 0"/>
+      </xacro:if>
+      <xacro:if value="${model_name.startswith('T8')}">
+        <origin xyz="0 0 0.0475" rpy="0 ${pi} 0"/>
       </xacro:if>
       <axis xyz="0 0 -1"/>
@@ -295,13 +443,5 @@
       <parent link="${name}/INPUT_INTERFACE"/>
       <child link="${child}/INPUT_INTERFACE"/>
-      <xacro:if value="${model_name.startswith('X5')}">
         <origin xyz="0 0 0" rpy="0 0 0"/>
-      </xacro:if>
-      <xacro:if value="${model_name.startswith('X8')}">
-        <origin xyz="0 0 0" rpy="0 0 0"/>
-      </xacro:if>
-      <xacro:if value="${model_name.startswith('R8')}">
-        <origin xyz="0 0 0" rpy="0 0 0"/>
-      </xacro:if>
     </joint>
   </xacro:macro>

File: urdf/components/hebi.xacro (robot description, xacro)
@@ -27,4 +27,17 @@
     <material>Gazebo/Black</material>
   </xacro:macro>
+  <xacro:macro name="tangerine_material">
+    <material name="tangerine">
+      <color rgba="0.91 0.43 0.218 1"/>
+    </material>
+  </xacro:macro>
+  <xacro:macro name="gazebo_tangerine_material">
+    <visual>
+      <material>
+          <ambient>0.91 0.43 0.218 1</ambient>
+          <diffuse>0.91 0.43 0.218 1</diffuse>
+      </material>
+    </visual>
+  </xacro:macro>
   <xacro:macro name="beige_material">
     <material name="beige">

Commit message: Resolved missed merge conflicts from 'ros2/humble'

File: urdf/components/actuator.xacro (robot description, xacro)
@@ -443,13 +443,5 @@
       <parent link="${name}"/>
       <child link="${child}"/>
-      <xacro:if value="${model_name.startswith('X')}">
-        <origin xyz="0 0 0" rpy="0 0 0"/>
-      </xacro:if>
-      <xacro:if value="${model_name.startswith('T')}">
-        <origin xyz="0 0 0" rpy="0 0 0"/>
-      </xacro:if>
-      <xacro:if value="${model_name.startswith('R')}">
-        <origin xyz="0 0 0" rpy="0 0 0"/>
-      </xacro:if>
+      <origin xyz="0 0 0" rpy="0 0 0"/>
     </joint>
   </xacro:macro>

File: urdf/components/bracket.xacro (robot description, xacro)
@@ -83,40 +83,4 @@
       </inertial>
     </xacro:if>
-    <xacro:if value="${bracket_type.startswith('T5Light') or bracket_type.startswith('T8Light')}">
-      <visual>
-        <xacro:if value="${bracket_type.endswith('Left')}">
-          <origin xyz="0 0 0" rpy="0 0 ${pi}"/>
-        </xacro:if>
-        <xacro:if value="${bracket_type.endswith('Right')}">
-          <origin xyz="0 0 0" rpy="0 0 0"/>
-        </xacro:if>
-        <geometry>
-          <mesh filename="file://$(find hebi_description)/meshes/A-2220-01.stl" scale="0.001 0.001 0.001"/>
-        </geometry>
-        <xacro:black_material/>
-      </visual>
-      <collision>
-        <xacro:if value="${bracket_type.endswith('Left')}">
-          <origin xyz="0 0 0" rpy="${pi/2} 0 ${pi/2}"/>
-        </xacro:if>
-        <xacro:if value="${bracket_type.endswith('Right')}">
-          <origin xyz="0 0 0" rpy="${pi/2} 0 ${-pi/2}"/>
-        </xacro:if>
-        <geometry>
-          <mesh filename="file://$(find hebi_description)/meshes/A-2220-01.stl" scale="0.001 0.001 0.001"/>
-        </geometry>
-      </collision>
-      <!-- inertia is just modelled as small sphere, and could be improved. -->
-      <inertial>
-        <xacro:if value="${bracket_type.endswith('Left')}">
-          <origin xyz="0 .0215 .02" rpy="0 0 0" />
-        </xacro:if>
-        <xacro:if value="${bracket_type.endswith('Right')}">
-          <origin xyz="0 -.0215 .02" rpy="0 0 0" />
-        </xacro:if>
-        <mass value="0.1"/>
-        <inertia ixx="${0.4 * 0.1 * 0.06 * 0.06}" ixy="0.0" ixz="0.0" iyy="${0.4 * 0.1 * 0.06 * 0.06}" iyz="0.0" izz="${0.4 * 0.1 * 0.06 * 0.06}"/>
-      </inertial>
-    </xacro:if>
     <!-- Heavy bracket -->
     <xacro:if value="${bracket_type.startswith('X5Heavy')}">
@@ -220,68 +184,4 @@
     </xacro:if>
     <xacro:if value="${bracket_type.startswith('R8Heavy')}">
-      <visual>
-        <xacro:if value="${bracket_type.endswith('RightOutside')}">
-          <origin xyz="0 0 0" rpy="0 0 0"/>
-        </xacro:if>
-        <xacro:if value="${bracket_type.endswith('RightInside')}">
-          <origin xyz="0 0 0" rpy="0 0 ${pi}"/>
-        </xacro:if>
-        <xacro:if value="${bracket_type.endswith('LeftOutside')}">
-          <origin xyz="0 0 0" rpy="0 0 ${pi}"/>
-        </xacro:if>
-        <xacro:if value="${bracket_type.endswith('LeftInside')}">
-          <origin xyz="0 0 0" rpy="0 0 0"/>
-        </xacro:if>
-        <geometry>
-          <xacro:if value="${bracket_type.endswith('Outside')}">
-            <mesh filename="file://$(find hebi_description)/meshes/A-2221-01-Outside.stl" scale="0.001 0.001 0.001"/>
-          </xacro:if>
-          <xacro:if value="${bracket_type.endswith('Inside')}">
-            <mesh filename="file://$(find hebi_description)/meshes/A-2221-01-Inside.stl" scale="0.001 0.001 0.001"/>
-          </xacro:if>
-        </geometry>
-        <xacro:black_material/>
-      </visual>
-      <collision>
-        <xacro:if value="${bracket_type.endswith('RightOutside')}">
-          <origin xyz="0 0 0.005" rpy="${pi/2} 0 ${pi/2}"/>
-        </xacro:if>
-        <xacro:if value="${bracket_type.endswith('RightInside')}">
-          <origin xyz="0 0 0.005" rpy="${pi/2} 0 ${-pi/2}"/>
-        </xacro:if>
-        <xacro:if value="${bracket_type.endswith('LeftOutside')}">
-          <origin xyz="0 0 0.005" rpy="${pi/2} 0 ${-pi/2}"/>
-        </xacro:if>
-        <xacro:if value="${bracket_type.endswith('LeftInside')}">
-          <origin xyz="0 0 0.005" rpy="${pi/2} 0 ${pi/2}"/>
-        </xacro:if>
-        <geometry>
-          <xacro:if value="${bracket_type.endswith('Outside')}">
-            <mesh filename="file://$(find hebi_description)/meshes/A-2221-01-Outside.stl" scale="0.001 0.001 0.001"/>
-          </xacro:if>
-          <xacro:if value="${bracket_type.endswith('Inside')}">
-            <mesh filename="file://$(find hebi_description)/meshes/A-2221-01-Inside.stl" scale="0.001 0.001 0.001"/>
-          </xacro:if>
-        </geometry>
-      </collision>
-      <!-- inertia is just modelled as small sphere, and could be improved. -->
-      <inertial>
-        <xacro:if value="${bracket_type.endswith('RightOutside')}">
-          <origin xyz="0 ${0.5 * -.0375} .0275" rpy="0 0 0" />
-        </xacro:if>
-        <xacro:if value="${bracket_type.endswith('RightInside')}">
-          <origin xyz="0 ${0.5 * .0225} .0275" rpy="0 0 0" />
-        </xacro:if>
-        <xacro:if value="${bracket_type.endswith('LeftOutside')}">
-          <origin xyz="0 ${0.5 * .0375} .0275" rpy="0 0 0" />
-        </xacro:if>
-        <xacro:if value="${bracket_type.endswith('LeftInside')}">
-          <origin xyz="0 ${0.5 * -.0225} .0275" rpy="0 0 0" />
-        </xacro:if>
-        <mass value="0.215"/>
-        <inertia ixx="${0.4 * 0.215 * 0.06 * 0.06}" ixy="0.0" ixz="0.0" iyy="${0.4 * 0.215 * 0.06 * 0.06}" iyz="0.0" izz="${0.4 * 0.215 * 0.06 * 0.06}"/>
-      </inertial>
-    </xacro:if>
-    <xacro:if value="${bracket_type.startswith('T5Heavy') or bracket_type.startswith('T8Heavy')}">
       <visual>
         <xacro:if value="${bracket_type.endswith('RightOutside')}">
@@ -352,5 +252,5 @@
       <xacro:gazebo_beige_material/>
     </xacro:if>
-    <xacro:if value="${bracket_type.startswith('X5Heavy') or bracket_type.startswith('R8') or bracket_type.startswith('T')}">
+    <xacro:if value="${bracket_type.startswith('X5Heavy') or bracket_type.startswith('R8')}">
       <xacro:gazebo_black_material/>
     </xacro:if>

File: urdf/kits/ros2_control/A-2085-05_macro.ros2_control.xacro (robot description, xacro)
@@ -21,5 +21,5 @@
         </xacro:if>
         <xacro:if value="${sim_gazebo}">
-          <plugin>gz_ros2_control/GazeboSimSystem</plugin>
+          <plugin>ign_ros2_control/IgnitionSystem</plugin>
         </xacro:if>
         <xacro:unless value="${use_mock_hardware or sim_gazebo_classic or sim_gazebo}">
@@ -91,5 +91,5 @@
     <xacro:if value="${sim_gazebo}">
       <gazebo>
-        <plugin filename="gz_ros2_control-system" name="gz_ros2_control::GazeboSimROS2ControlPlugin">
+        <plugin filename="ign_ros2_control-system" name="ign_ros2_control::IgnitionROS2ControlPlugin">
           <parameters>$(find hebi_bringup)/config/A-2085-05_controllers.yaml</parameters>
         </plugin>

File: urdf/kits/ros2_control/A-2085-06_macro.ros2_control.xacro (robot description, xacro)
@@ -21,5 +21,5 @@
         </xacro:if>
         <xacro:if value="${sim_gazebo}">
-          <plugin>gz_ros2_control/GazeboSimSystem</plugin>
+          <plugin>ign_ros2_control/IgnitionSystem</plugin>
         </xacro:if>
         <xacro:unless value="${use_mock_hardware or sim_gazebo_classic or sim_gazebo}">
@@ -101,5 +101,5 @@
     <xacro:if value="${sim_gazebo}">
       <gazebo>
-        <plugin filename="gz_ros2_control-system" name="gz_ros2_control::GazeboSimROS2ControlPlugin">
+        <plugin filename="ign_ros2_control-system" name="ign_ros2_control::IgnitionROS2ControlPlugin">
           <parameters>$(find hebi_bringup)/config/A-2085-06_controllers.yaml</parameters>
         </plugin>

Commit message: Fixed actuators with joint name as main name

File: urdf/components/actuator.xacro (robot description, xacro)
@@ -114,5 +114,5 @@
       <xacro:property name="friction" value="0.5"/>
     </xacro:if>
-    <link name="${name}">
+    <link name="${name}_body">
       <visual>
         <origin xyz="0 0 0" rpy="0 0 0" />
@@ -180,5 +180,5 @@
       </inertial>
     </link>
-    <gazebo reference="${name}">
+    <gazebo reference="${name}_body">
       <xacro:if value="${model_name.startswith('X')}">
         <xacro:gazebo_red_material/>
@@ -192,5 +192,5 @@
     </gazebo>
     <joint name="${name}" type="${urdf_joint_type}">
-      <parent link="${name}"/>
+      <parent link="${name}_body"/>
       <child link="${child}"/>
       <xacro:if value="${model_name.startswith('X5')}">
@@ -334,5 +334,5 @@
       <xacro:property name="friction" value="0.5"/>
     </xacro:if>
-    <link name="${name}">
+    <link name="${name}_body">
       <visual>
         <origin xyz="0 0 0" rpy="0 0 0" />
@@ -400,5 +400,5 @@
       </inertial>
     </link>
-    <gazebo reference="${name}">
+    <gazebo reference="${name}_body">
       <xacro:if value="${model_name.startswith('X')}">
         <xacro:gazebo_red_material/>
@@ -413,5 +413,5 @@
     <joint name="${name}" type="${urdf_joint_type}">
       <parent link="${parent}"/>
-      <child link="${name}"/>
+      <child link="${name}_body"/>
       <xacro:if value="${model_name.startswith('X5')}">
         <origin xyz="0 0 0.031" rpy="0 ${pi} 0"/>
@@ -441,5 +441,5 @@
     </joint>
     <joint name="${name}_fixed" type="fixed">
-      <parent link="${name}"/>
+      <parent link="${name}_body"/>
       <child link="${child}"/>
       <origin xyz="0 0 0" rpy="0 0 0"/>

File: urdf/components/link.xacro (robot description, xacro)
@@ -2,5 +2,5 @@
 <robot xmlns:xacro="http://www.ros.org/wiki/xacro">
   <!-- NOTE: joint must match the name of the module -->
-  <xacro:macro name="link" params="name child type:=X5 input:=RightAngle output:=None extension twist">
+  <xacro:macro name="link" params="name child type:=X5 input:=RightAngle output:=RightAngle extension twist">
     <xacro:property name="mass" value="${0.4 * (extension + 0.03) + 0.26}"/>
     <xacro:property name="edge_to_center" value="${.02}"/>
@@ -112,5 +112,5 @@
       <xacro:gazebo_black_material/>
     </gazebo>
-    <joint name="${name}/OUTPUT_JOINT" type="fixed">
+    <joint name="${name}_joint" type="fixed">
       <parent link="${name}"/>
       <child link="${child}"/>
