Commit message: Set default scale to 0.001 for meshes

File: urdf/components/actuator.xacro (robot description, xacro)
@@ -118,10 +118,5 @@
         <origin xyz="0 0 0" rpy="0 0 0" />
         <geometry>
-          <xacro:if value="${model_name.startswith('T')}">
-            <mesh filename="${mesh_filename}"/>
-          </xacro:if>
-          <xacro:unless value="${model_name.startswith('T')}">
-            <mesh filename="${mesh_filename}" scale="0.001 0.001 0.001"/>
-          </xacro:unless>
+          <mesh filename="${mesh_filename}" scale="0.001 0.001 0.001"/>
         </geometry>
         <xacro:if value="${model_name.startswith('X')}">
@@ -138,10 +133,5 @@
         <origin xyz="0 0 0" rpy="0 0 0" />
         <geometry>
-          <xacro:if value="${model_name.startswith('T')}">
-            <mesh filename="${mesh_filename}"/>
-          </xacro:if>
-          <xacro:unless value="${model_name.startswith('T')}">
-            <mesh filename="${mesh_filename}" scale="0.001 0.001 0.001"/>
-          </xacro:unless>
+          <mesh filename="${mesh_filename}" scale="0.001 0.001 0.001"/>
         </geometry>
       </collision>
@@ -338,10 +328,5 @@
         <origin xyz="0 0 0" rpy="0 0 0" />
         <geometry>
-          <xacro:if value="${model_name.startswith('T')}">
-            <mesh filename="${mesh_filename}"/>
-          </xacro:if>
-          <xacro:unless value="${model_name.startswith('T')}">
-            <mesh filename="${mesh_filename}" scale="0.001 0.001 0.001"/>
-          </xacro:unless>
+          <mesh filename="${mesh_filename}" scale="0.001 0.001 0.001"/>
         </geometry>
         <xacro:if value="${model_name.startswith('X')}">
@@ -358,10 +343,5 @@
         <origin xyz="0 0 0" rpy="0 0 0" />
         <geometry>
-          <xacro:if value="${model_name.startswith('T')}">
-            <mesh filename="${mesh_filename}"/>
-          </xacro:if>
-          <xacro:unless value="${model_name.startswith('T')}">
-            <mesh filename="${mesh_filename}" scale="0.001 0.001 0.001"/>
-          </xacro:unless>
+          <mesh filename="${mesh_filename}" scale="0.001 0.001 0.001"/>
         </geometry>
       </collision>

File: urdf/components/link.xacro (robot description, xacro)
@@ -11,5 +11,5 @@
         <geometry>
           <xacro:if value="${input == 'RightAngle'}">
-            <mesh filename="file://$(find hebi_description)/meshes/A-2038-02.stl"/>
+            <mesh filename="file://$(find hebi_description)/meshes/A-2038-02.stl" scale="0.001 0.001 0.001"/>
           </xacro:if>
           <xacro:if value="${input == 'Inline'}">
@@ -23,5 +23,5 @@
         <geometry>
           <xacro:if value="${input == 'RightAngle'}">
-            <mesh filename="file://$(find hebi_description)/meshes/A-2038-02.stl"/>
+            <mesh filename="file://$(find hebi_description)/meshes/A-2038-02.stl" scale="0.001 0.001 0.001"/>
           </xacro:if>
           <xacro:if value="${input == 'Inline'}">
@@ -71,5 +71,5 @@
           <geometry>
             <xacro:if value="${output == 'RightAngle'}">
-              <mesh filename="file://$(find hebi_description)/meshes/A-2039-02.stl"/>
+              <mesh filename="file://$(find hebi_description)/meshes/A-2039-02.stl" scale="0.001 0.001 0.001"/>
             </xacro:if>
             <xacro:if value="${output == 'Inline'}">
@@ -94,5 +94,5 @@
           <geometry>
             <xacro:if value="${input == 'RightAngle'}">
-              <mesh filename="file://$(find hebi_description)/meshes/A-2039-02.stl"/>
+              <mesh filename="file://$(find hebi_description)/meshes/A-2039-02.stl" scale="0.001 0.001 0.001"/>
             </xacro:if>
             <xacro:if value="${input == 'Inline'}">

File: urdf/components/rigid_body.xacro (robot description, xacro)
@@ -1,5 +1,5 @@
 <?xml version="1.0"?>
 <robot xmlns:xacro="http://www.ros.org/wiki/xacro">
-  <xacro:macro name="rigid-body" params="name mass com_rot='0 0 0' com_trans='0 0 0' ixx=0.001 iyy=0.001 izz=0.001 ixy=0 ixz=0 iyz=0 mesh_path='' mesh_rot='0 0 0' mesh_trans='0 0 0'">
+  <xacro:macro name="rigid-body" params="name mass com_rot='0 0 0' com_trans='0 0 0' ixx=0.001 iyy=0.001 izz=0.001 ixy=0 ixz=0 iyz=0 mesh_path='' mesh_rot='0 0 0' mesh_trans='0 0 0' mesh_scale='0.001 0.001 0.001'">
     <link name="${name}">
       <xacro:if value="${mesh_path != ''}">
@@ -7,5 +7,5 @@
           <origin xyz="${mesh_trans}" rpy="${mesh_rot}"/>
           <geometry>
-            <mesh filename="${mesh_path}"/>
+            <mesh filename="${mesh_path}" scale="${mesh_scale}"/>
           </geometry>
           <xacro:black_material/>
@@ -14,5 +14,5 @@
           <origin xyz="${mesh_trans}" rpy="${mesh_rot}"/>
           <geometry>
-            <mesh filename="${mesh_path}"/>
+            <mesh filename="${mesh_path}" scale="${mesh_scale}"/>
           </geometry>
         </collision>

Commit message: Added mass_offset to URDF xacros

File: urdf/components/actuator.xacro (robot description, xacro)
@@ -2,5 +2,5 @@
 <robot xmlns:xacro="http://www.ros.org/wiki/xacro">
   <!-- NOTE: joint must match the name of the module -->
-  <xacro:macro name="actuator" params="name child:='' type limits:=${[]}">
+  <xacro:macro name="actuator" params="name child:='' type limits:=${[]} mass_offset:=0.0">
     <xacro:property name="model_name" value="${type}"/>
     <!-- Continuous joints (no position limits) -->
@@ -137,5 +137,5 @@
       </collision>
       <inertial>
-        <mass value="${actuator_mass}"/>
+        <mass value="${actuator_mass + mass_offset}"/>
         <xacro:if value="${model_name.startswith('X5')}">
           <origin xyz="-0.0142 -0.0031 0.0165" rpy="0 0 0" />
@@ -212,5 +212,5 @@
   </xacro:macro>
   <!-- This macro is used when an actuator is "flipped" so parent feeds into input-->
-  <xacro:macro name="reverse_actuator" params="name parent:='' child:='' type limits:=${[]}">
+  <xacro:macro name="reverse_actuator" params="name parent:='' child:='' type limits:=${[]} mass_offset:=0.0">
     <xacro:property name="model_name" value="${type}"/>
     <!-- Continuous joints (no position limits) -->
@@ -347,5 +347,5 @@
       </collision>
       <inertial>
-        <mass value="${actuator_mass}"/>
+        <mass value="${actuator_mass + mass_offset}"/>
         <xacro:if value="${model_name.startswith('X5')}">
           <origin xyz="-0.0142 -0.0031 0.0165" rpy="0 0 0" />

File: urdf/components/bracket.xacro (robot description, xacro)
@@ -1,5 +1,5 @@
 <?xml version="1.0"?>
 <robot xmlns:xacro="http://www.ros.org/wiki/xacro">
-  <xacro:macro name="bracket" params="name type">
+  <xacro:macro name="bracket" params="name type mass_offset:=0.0">
   <xacro:property name="bracket_type" value="${type}"/>
   <link name="${name}">
@@ -43,5 +43,5 @@
           <origin xyz="0 -.0215 .02" rpy="0 0 0" />
         </xacro:if>
-        <mass value="0.1"/>
+        <mass value="${0.1 + mass_offset}"/>
         <inertia ixx="${0.4 * 0.1 * 0.06 * 0.06}" ixy="0.0" ixz="0.0" iyy="${0.4 * 0.1 * 0.06 * 0.06}" iyz="0.0" izz="${0.4 * 0.1 * 0.06 * 0.06}"/>
       </inertial>
@@ -79,5 +79,5 @@
           <origin xyz="0 -.0215 .02" rpy="0 0 0" />
         </xacro:if>
-        <mass value="0.1"/>
+        <mass value="${0.1 + mass_offset}"/>
         <inertia ixx="${0.4 * 0.1 * 0.06 * 0.06}" ixy="0.0" ixz="0.0" iyy="${0.4 * 0.1 * 0.06 * 0.06}" iyz="0.0" izz="${0.4 * 0.1 * 0.06 * 0.06}"/>
       </inertial>
@@ -179,5 +179,5 @@
           <origin xyz="0 ${0.5 * -.0225} .0275" rpy="0 0 0" />
         </xacro:if>
-        <mass value="0.215"/>
+        <mass value="${0.215 + mass_offset}"/>
         <inertia ixx="${0.4 * 0.215 * 0.06 * 0.06}" ixy="0.0" ixz="0.0" iyy="${0.4 * 0.215 * 0.06 * 0.06}" iyz="0.0" izz="${0.4 * 0.215 * 0.06 * 0.06}"/>
       </inertial>
@@ -243,5 +243,5 @@
           <origin xyz="0 ${0.5 * -.0225} .0275" rpy="0 0 0" />
         </xacro:if>
-        <mass value="0.215"/>
+        <mass value="${0.215 + mass_offset}"/>
         <inertia ixx="${0.4 * 0.215 * 0.06 * 0.06}" ixy="0.0" ixz="0.0" iyy="${0.4 * 0.215 * 0.06 * 0.06}" iyz="0.0" izz="${0.4 * 0.215 * 0.06 * 0.06}"/>
       </inertial>

File: urdf/components/end_effector.xacro (robot description, xacro)
@@ -1,5 +1,5 @@
 <?xml version="1.0"?>
 <robot xmlns:xacro="http://www.ros.org/wiki/xacro">
-  <xacro:macro name="null_end_effector" params="name">
+  <xacro:macro name="null_end_effector" params="name mass:=0.001 mass_offset:=0.0">
     <link name="${name}">
       <collision>
@@ -17,5 +17,5 @@
       <inertial>
         <origin xyz="0 0 0.0005" rpy="0 0 0"/>
-          <mass value="0.001"/>
+          <mass value="${mass + mass_offset}"/>
         <inertia
           ixx="0.001" ixy="0.0" ixz="0.0"
@@ -197,5 +197,5 @@
     </joint>
   </xacro:macro>
-  <xacro:macro name="gripper" params="name type:=Custom mass:=0.001 output_trans:='0 0 0' output_rot:='0 0 0' com_trans:='0 0 0' com_rot:='0 0 0' ixx='None' iyy='None' izz='None' ixy=0 ixz=0 iyz=0">
+  <xacro:macro name="gripper" params="name type:=Custom mass:=0.001 mass_offset:=0.0 output_trans:='0 0 0' output_rot:='0 0 0' com_trans:='0 0 0' com_rot:='0 0 0' ixx='None' iyy='None' izz='None' ixy=0 ixz=0 iyz=0">
     <xacro:property name="com_trans_list" value="${list(map(float, com_trans.split(' ')))}" />
     <xacro:if value="${ com_trans_list[0] + com_trans_list[1] + com_trans_list[2] >= 0.01 }">
@@ -206,5 +206,5 @@
     </xacro:unless>
     <xacro:if value="${ixx == 'None'}">
-      <xacro:property name="_ixx" value="${2.0/5.0 * mass * pow(gripper_len, 2)}" />
+      <xacro:property name="_ixx" value="${2.0/5.0 * (mass + mass_offset) * pow(gripper_len, 2)}" />
     </xacro:if>
     <xacro:unless value="${ixx == 'None'}">
@@ -212,5 +212,5 @@
     </xacro:unless>
     <xacro:if value="${iyy == 'None'}">
-      <xacro:property name="_iyy" value="${2.0/5.0 * mass * pow(gripper_len, 2)}" />
+      <xacro:property name="_iyy" value="${2.0/5.0 * (mass + mass_offset) * pow(gripper_len, 2)}" />
     </xacro:if>
     <xacro:unless value="${iyy == 'None'}">
@@ -218,5 +218,5 @@
     </xacro:unless>
     <xacro:if value="${izz == 'None'}">
-      <xacro:property name="_izz" value="${2.0/5.0 * mass * pow(gripper_len, 2)}" />
+      <xacro:property name="_izz" value="${2.0/5.0 * (mass + mass_offset) * pow(gripper_len, 2)}" />
     </xacro:if>
     <xacro:unless value="${izz == 'None'}">
@@ -233,5 +233,5 @@
         <inertial>
           <origin xyz="${com_trans}" rpy="${com_rot}" />
-          <mass value="${mass}" />
+          <mass value="${mass + mass_offset}" />
           <inertia
             ixx="${_ixx}" ixy="${ixy}" ixz="${ixz}"
@@ -259,5 +259,5 @@
         <inertial>
           <origin xyz="0 0 0" rpy="0 0 0"/>
-          <mass value="0.072"/>
+          <mass value="${0.072 + mass_offset}"/>
           <!-- Approximated as solid cylinder -->
           <inertia
@@ -281,5 +281,5 @@
         <inertial>
           <origin xyz="0 0 0" rpy="0 0 0"/>
-          <mass value="0.010"/>
+          <mass value="${0.010 + mass_offset}"/>
           <!-- Approximated as hollow sphere -->
           <inertia
@@ -313,5 +313,5 @@
         <inertial>
           <origin xyz="0 0 0" rpy="0 0 0"/>
-          <mass value="0.010"/>
+          <mass value="${0.010 + mass_offset}"/>
           <!-- Approximated as hollow sphere -->
           <inertia

File: urdf/components/link.xacro (robot description, xacro)
@@ -2,6 +2,6 @@
 <robot xmlns:xacro="http://www.ros.org/wiki/xacro">
   <!-- NOTE: joint must match the name of the module -->
-  <xacro:macro name="link" params="name child type:=X5 input:=RightAngle output:=RightAngle extension twist">
-    <xacro:property name="mass" value="${0.4 * (extension + 0.03) + 0.26}"/>
+  <xacro:macro name="link" params="name child type:=X5 input:=RightAngle output:=RightAngle extension twist mass_offset:=0.0">
+    <xacro:property name="mass" value="${0.4 * (extension + 0.03) + 0.26 + mass_offset}"/>
     <xacro:property name="edge_to_center" value="${.02}"/>
     <link name="${name}">

Commit message: Add R25 and T25 to URDF xacros; fix settings for others and documentation

File: urdf/components/actuator.xacro (robot description, xacro)
@@ -31,31 +31,46 @@
     <xacro:if value="${model_name == 'X8_3'}">
       <xacro:property name="actuator_mass" value="0.460" />
-      <xacro:property name="effort_limit" value="7" />
-      <xacro:property name="velocity_limit" value="8.796" />
+      <xacro:property name="effort_limit" value="8" />
+      <xacro:property name="velocity_limit" value="11.520" />
     </xacro:if>
     <xacro:if value="${model_name == 'X8_9'}">
       <xacro:property name="actuator_mass" value="0.480" />
-      <xacro:property name="effort_limit" value="20" />
-      <xacro:property name="velocity_limit" value="3.142" />
+      <xacro:property name="effort_limit" value="23" />
+      <xacro:property name="velocity_limit" value="4.084" />
     </xacro:if>
     <xacro:if value="${model_name == 'X8_16'}">
       <xacro:property name="actuator_mass" value="0.500" />
-      <xacro:property name="effort_limit" value="38" />
-      <xacro:property name="velocity_limit" value="1.571" />
+      <xacro:property name="effort_limit" value="44" />
+      <xacro:property name="velocity_limit" value="2.094" />
     </xacro:if>
     <xacro:if value="${model_name == 'R8_3'}">
       <xacro:property name="actuator_mass" value="0.670" />
-      <xacro:property name="effort_limit" value="7" />
-      <xacro:property name="velocity_limit" value="8.796" />
+      <xacro:property name="effort_limit" value="8" />
+      <xacro:property name="velocity_limit" value="11.5120" />
     </xacro:if>
     <xacro:if value="${model_name == 'R8_9'}">
       <xacro:property name="actuator_mass" value="0.685" />
-      <xacro:property name="effort_limit" value="20" />
-      <xacro:property name="velocity_limit" value="3.142" />
+      <xacro:property name="effort_limit" value="23" />
+      <xacro:property name="velocity_limit" value="4.084" />
     </xacro:if>
     <xacro:if value="${model_name == 'R8_16'}">
       <xacro:property name="actuator_mass" value="0.715" />
-      <xacro:property name="effort_limit" value="38" />
-      <xacro:property name="velocity_limit" value="1.571" />
+      <xacro:property name="effort_limit" value="44" />
+      <xacro:property name="velocity_limit" value="2.094" />
+    </xacro:if>
+    <xacro:if value="${model_name == 'R25_8'}">
+      <xacro:property name="actuator_mass" value="1.9" />
+      <xacro:property name="effort_limit" value="16.0" />
+      <xacro:property name="velocity_limit" value="12.357" />
+    </xacro:if>
+    <xacro:if value="${model_name == 'R25_20'}">
+      <xacro:property name="actuator_mass" value="1.9" />
+      <xacro:property name="effort_limit" value="40.0" />
+      <xacro:property name="velocity_limit" value="4.922" />
+    </xacro:if>
+    <xacro:if value="${model_name == 'R25_40'}">
+      <xacro:property name="actuator_mass" value="1.9" />
+      <xacro:property name="effort_limit" value="80.0" />
+      <xacro:property name="velocity_limit" value="2.409" />
     </xacro:if>
     <xacro:if value="${model_name == 'T5_1'}">
@@ -88,4 +103,19 @@
       <xacro:property name="effort_limit" value="44.0" />
       <xacro:property name="velocity_limit" value="2.094" />
+    </xacro:if>
+    <xacro:if value="${model_name == 'T25_8'}">
+      <xacro:property name="actuator_mass" value="1.5" />
+      <xacro:property name="effort_limit" value="16.0" />
+      <xacro:property name="velocity_limit" value="12.357" />
+    </xacro:if>
+    <xacro:if value="${model_name == 'T25_20'}">
+      <xacro:property name="actuator_mass" value="1.5" />
+      <xacro:property name="effort_limit" value="40.0" />
+      <xacro:property name="velocity_limit" value="4.922" />
+    </xacro:if>
+    <xacro:if value="${model_name == 'T25_40'}">
+      <xacro:property name="actuator_mass" value="1.5" />
+      <xacro:property name="effort_limit" value="80.0" />
+      <xacro:property name="velocity_limit" value="2.409" />
     </xacro:if>
     <!-- Note: the frction/damping probably need to be tuned more for accurate simulation -->
@@ -105,4 +135,9 @@
       <xacro:property name="friction" value="0.5" />
     </xacro:if>
+    <xacro:if value="${model_name.startswith('R25')}">
+      <xacro:property name="mesh_filename" value="file://$(find hebi_description)/meshes/R25.stl" />
+      <xacro:property name="damping" value="0.5" />
+      <xacro:property name="friction" value="0.5" />
+    </xacro:if>
     <xacro:if value="${model_name.startswith('T5')}">
       <xacro:property name="mesh_filename" value="file://$(find hebi_description)/meshes/T5.stl" />
@@ -115,4 +150,9 @@
       <xacro:property name="friction" value="0.5" />
     </xacro:if>
+    <xacro:if value="${model_name.startswith('T25')}">
+      <xacro:property name="mesh_filename" value="file://$(find hebi_description)/meshes/T25.stl" />
+      <xacro:property name="damping" value="0.5" />
+      <xacro:property name="friction" value="0.5" />
+    </xacro:if>
     <!-- Set joint origin offsets based on actuator type -->
     <xacro:if value="${model_name.startswith('X5')}">
@@ -125,4 +165,7 @@
       <xacro:property name="joint_offset" value="0.051" />
     </xacro:if>
+    <xacro:if value="${model_name.startswith('R25')}">
+      <xacro:property name="joint_offset" value="0.069" />
+    </xacro:if>
     <xacro:if value="${model_name.startswith('T5')}">
       <xacro:property name="joint_offset" value="0.034" />
@@ -130,4 +173,7 @@
     <xacro:if value="${model_name.startswith('T8')}">
       <xacro:property name="joint_offset" value="0.0475" />
+    </xacro:if>
+    <xacro:if value="${model_name.startswith('T25')}">
+      <xacro:property name="joint_offset" value="0.067" />
     </xacro:if>
     <!-- Link definition -->
@@ -174,4 +220,10 @@
             izz="0.001186" />
         </xacro:if>
+        <xacro:if value="${model_name.startswith('R25')}">
+          <origin xyz="-0.0268 -0.000357 0.0349" rpy="0 0 0" />
+          <inertia ixx="0.0026" ixy="-0.0002" ixz="0.0001"
+            iyy="0.0044" iyz="0.000"
+            izz="0.0054" />
+        </xacro:if>
         <xacro:if value="${model_name.startswith('T5')}">
           <origin xyz="-0.0240 -0.00161 0.0165" rpy="0 0 0" />
@@ -185,4 +237,10 @@
             iyy="0.000380" iyz="0.00000422"
             izz="0.000463" />
+        </xacro:if>
+        <xacro:if value="${model_name.startswith('T25')}">
+          <origin xyz="-0.0241 -0.0001 0.0338" rpy="0 0 0" />
+          <inertia ixx="0.0019" ixy="-0.0002" ixz="0.0001"
+            iyy="0.0031" iyz="0.000"
+            izz="0.0038" />
         </xacro:if>
       </inertial>

Commit message: Fixed axis of rotation for reversed modules

File: urdf/components/actuator.xacro (robot description, xacro)
@@ -281,5 +281,5 @@
         <parent link="${parent}" />
         <child link="${name}/body" />
-        <origin xyz="0 0 ${joint_offset}" rpy="0 ${pi} 0" />
+        <origin xyz="0 0 ${joint_offset}" rpy="${pi} 0 0" />
         <axis xyz="0 0 -1" />
         <!-- Continuous joints (no position limits) -->
