Commit message: Removed base_link from hexapod URDF

File: urdf/kits/hexapod/T-daisy.urdf.xacro (robot description, xacro)
@@ -4,10 +4,4 @@
   <!-- HEBI daisy Arm Kit -->
   <xacro:include filename="$(find hebi_description)/urdf/components/hebi.xacro"/>
-  <link name="$(arg prefix)base_link"/>
-  <joint name="$(arg prefix)base_joint" type="fixed">
-    <origin xyz="0 0 0" rpy="0 0 0"/>
-    <parent link="$(arg prefix)base_link"/>
-    <child link="$(arg prefix)RB1"/>
-  </joint>
   <xacro:rigid-body mass="0.01" name="$(arg prefix)RB1"/>
   <xacro:output rot="0 0 0.5236" parent="$(arg prefix)RB1" child="$(arg prefix)RB2" name="$(arg prefix)RB1_RB2"/>

File: urdf/kits/hexapod/X-daisy.urdf.xacro (robot description, xacro)
@@ -4,10 +4,4 @@
   <!-- HEBI daisy Arm Kit -->
   <xacro:include filename="$(find hebi_description)/urdf/components/hebi.xacro"/>
-  <link name="$(arg prefix)base_link"/>
-  <joint name="$(arg prefix)base_joint" type="fixed">
-    <origin xyz="0 0 0" rpy="0 0 0"/>
-    <parent link="$(arg prefix)base_link"/>
-    <child link="$(arg prefix)RB1"/>
-  </joint>
   <xacro:rigid-body mass="0.01" name="$(arg prefix)RB1"/>
   <xacro:output rot="0 0 0.5236" parent="$(arg prefix)RB1" child="$(arg prefix)RB2" name="$(arg prefix)RB1_RB2"/>
@@ -15,6 +9,6 @@
   <xacro:output trans="0.2375 0 0" parent="$(arg prefix)RB2" child="$(arg prefix)J1" name="$(arg prefix)RB2_J1"/>
   <xacro:actuator type="X8_9" name="$(arg prefix)J1" child="$(arg prefix)B1"/>
-  <xacro:bracket type="R8HeavyLeftInside" name="$(arg prefix)B1"/>
-  <xacro:output type="R8HeavyLeftInside" parent="$(arg prefix)B1" child="$(arg prefix)J2" name="$(arg prefix)B1_J2"/>
+  <xacro:bracket type="X5HeavyLeftInside" name="$(arg prefix)B1"/>
+  <xacro:output type="X5HeavyLeftInside" parent="$(arg prefix)B1" child="$(arg prefix)J2" name="$(arg prefix)B1_J2"/>
   <xacro:actuator type="X8_16" name="$(arg prefix)J2" child="$(arg prefix)L1"/>
   <xacro:link type="X8" extension="0.325" twist="${pi}" name="$(arg prefix)L1" child="$(arg prefix)J3" output="RightAngle"/>
@@ -26,6 +20,6 @@
   <xacro:output trans="0.2375 0 0" parent="$(arg prefix)RB3" child="$(arg prefix)J4" name="$(arg prefix)RB3_J4"/>
   <xacro:actuator type="X8_9" name="$(arg prefix)J4" child="$(arg prefix)B2"/>
-  <xacro:bracket type="R8HeavyRightInside" name="$(arg prefix)B2"/>
-  <xacro:output type="R8HeavyRightInside" parent="$(arg prefix)B2" child="$(arg prefix)J5" name="$(arg prefix)B2_J5"/>
+  <xacro:bracket type="X5HeavyRightInside" name="$(arg prefix)B2"/>
+  <xacro:output type="X5HeavyRightInside" parent="$(arg prefix)B2" child="$(arg prefix)J5" name="$(arg prefix)B2_J5"/>
   <xacro:actuator type="X8_16" name="$(arg prefix)J5" child="$(arg prefix)L3"/>
   <xacro:link type="X8" extension="0.325" twist="${pi}" name="$(arg prefix)L3" child="$(arg prefix)J6" output="RightAngle"/>
@@ -37,6 +31,6 @@
   <xacro:output trans="0.1875 0 0" parent="$(arg prefix)RB4" child="$(arg prefix)J7" name="$(arg prefix)RB4_J7"/>
   <xacro:actuator type="X8_9" name="$(arg prefix)J7" child="$(arg prefix)B3"/>
-  <xacro:bracket type="R8HeavyLeftInside" name="$(arg prefix)B3"/>
-  <xacro:output type="R8HeavyLeftInside" parent="$(arg prefix)B3" child="$(arg prefix)J8" name="$(arg prefix)B3_J8"/>
+  <xacro:bracket type="X5HeavyLeftInside" name="$(arg prefix)B3"/>
+  <xacro:output type="X5HeavyLeftInside" parent="$(arg prefix)B3" child="$(arg prefix)J8" name="$(arg prefix)B3_J8"/>
   <xacro:actuator type="X8_16" name="$(arg prefix)J8" child="$(arg prefix)L5"/>
   <xacro:link type="X8" extension="0.325" twist="${pi}" name="$(arg prefix)L5" child="$(arg prefix)J9" output="RightAngle"/>
@@ -48,6 +42,6 @@
   <xacro:output trans="0.1875 0 0" parent="$(arg prefix)RB5" child="$(arg prefix)J10" name="$(arg prefix)RB5_J10"/>
   <xacro:actuator type="X8_9" name="$(arg prefix)J10" child="$(arg prefix)B4"/>
-  <xacro:bracket type="R8HeavyRightInside" name="$(arg prefix)B4"/>
-  <xacro:output type="R8HeavyRightInside" parent="$(arg prefix)B4" child="$(arg prefix)J11" name="$(arg prefix)B4_J11"/>
+  <xacro:bracket type="X5HeavyRightInside" name="$(arg prefix)B4"/>
+  <xacro:output type="X5HeavyRightInside" parent="$(arg prefix)B4" child="$(arg prefix)J11" name="$(arg prefix)B4_J11"/>
   <xacro:actuator type="X8_16" name="$(arg prefix)J11" child="$(arg prefix)L7"/>
   <xacro:link type="X8" extension="0.325" twist="${pi}" name="$(arg prefix)L7" child="$(arg prefix)J12" output="RightAngle"/>
@@ -59,6 +53,6 @@
   <xacro:output trans="0.2375 0 0" parent="$(arg prefix)RB6" child="$(arg prefix)J13" name="$(arg prefix)RB6_J13"/>
   <xacro:actuator type="X8_9" name="$(arg prefix)J13" child="$(arg prefix)B5"/>
-  <xacro:bracket type="R8HeavyLeftInside" name="$(arg prefix)B5"/>
-  <xacro:output type="R8HeavyLeftInside" parent="$(arg prefix)B5" child="$(arg prefix)J14" name="$(arg prefix)B5_J14"/>
+  <xacro:bracket type="X5HeavyLeftInside" name="$(arg prefix)B5"/>
+  <xacro:output type="X5HeavyLeftInside" parent="$(arg prefix)B5" child="$(arg prefix)J14" name="$(arg prefix)B5_J14"/>
   <xacro:actuator type="X8_16" name="$(arg prefix)J14" child="$(arg prefix)L9"/>
   <xacro:link type="X8" extension="0.325" twist="${pi}" name="$(arg prefix)L9" child="$(arg prefix)J15" output="RightAngle"/>
@@ -70,6 +64,6 @@
   <xacro:output trans="0.2375 0 0" parent="$(arg prefix)RB7" child="$(arg prefix)J16" name="$(arg prefix)RB7_J16"/>
   <xacro:actuator type="X8_9" name="$(arg prefix)J16" child="$(arg prefix)B6"/>
-  <xacro:bracket type="R8HeavyRightInside" name="$(arg prefix)B6"/>
-  <xacro:output type="R8HeavyRightInside" parent="$(arg prefix)B6" child="$(arg prefix)J17" name="$(arg prefix)B6_J17"/>
+  <xacro:bracket type="X5HeavyRightInside" name="$(arg prefix)B6"/>
+  <xacro:output type="X5HeavyRightInside" parent="$(arg prefix)B6" child="$(arg prefix)J17" name="$(arg prefix)B6_J17"/>
   <xacro:actuator type="X8_16" name="$(arg prefix)J17" child="$(arg prefix)L11"/>
   <xacro:link type="X8" extension="0.325" twist="${pi}" name="$(arg prefix)L11" child="$(arg prefix)J18" output="RightAngle"/>
@@ -78,5 +72,5 @@
   <xacro:gripper type="Custom" mass="0.060" name="$(arg prefix)EE6"/>
   <xacro:output parent="$(arg prefix)RB1" child="$(arg prefix)RB8" name="$(arg prefix)RB1_RB8"/>
-  <xacro:rigid-body mass="5.00" com_trans="0.050 0.000 0.075" mesh_path="file:///home/hariharan/hebi_ws/src/hebi_description/meshes/A-2051-01.stl" mesh_trans="0 0 -0.019" name="$(arg prefix)RB8"/>
+  <xacro:rigid-body mass="5.00" com_trans="0.050 0.000 0.075" mesh_path="file:///home/hariharan/hebi_ws/src/meshes/A-2051-01.stl" mesh_trans="0 0 -0.019" name="$(arg prefix)RB8"/>
   <xacro:output trans="0.000 0.000 0.075" parent="$(arg prefix)RB8" child="$(arg prefix)EE7" name="$(arg prefix)RB8_EE7"/>
   <xacro:gripper name="$(arg prefix)EE7" type="Custom" mass="0.01"/>
